File: pcb/digital-power-meter/qo-100-digital-power-meter.brd (EAGLE design)
At the start: 60 x 30 mm, 14 parts, among them CON1 2EDG-5P, CON2 4P-SH-SIDE, U1 LTC4151HDD

Commit message: Update 2EDG connector on power meter
Parts:
- CON1: value 2EDG-5P -> 2EDG-5P-5MM; device Generic Connector:2EDG-5P -> Generic Connector:2EDG-5P-5MM
Changed lines of the file:
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@@
 <drawing>
 <settings>
-<setting alwaysvectorfont="yes"/>
+<setting alwaysvectorfont="no"/>
 <setting verticaltext="up"/>
 </settings>
@@
 <attribute name="VALUE" x="4.405" y="10.555" size="0.8" layer="27" font="vector" ratio="10" rot="R180" align="center-left"/>
 </element>
-<element name="CON1" library="Generic Connector" package="2EDG-5P" value="2EDG-5P" x="40" y="15" smashed="yes" rot="R90"/>
+<element name="CON1" library="Generic Connector" package="2EDG-5P-5MM" value="2EDG-5P-5MM" x="40" y="15" smashed="yes" rot="R90"/>
 <element name="LOGO1" library="Silkscreen" package="JS_5MM" value="JS-5MM" x="8" y="26.6" smashed="yes"/>
 <element name="R2" library="Resistor" package="RES2512" value="0.012 Ohms" x="25" y="15" smashed="yes" rot="MR90">
@@
 <via x="29.5" y="15.6" extent="1-16" drill="0.3"/>
 <wire x1="29.5" y1="15.6" x2="29.5" y2="18.1496" width="0.254" layer="16"/>
-<wire x1="19.5" y1="16.425" x2="19.5" y2="17.1" width="0.254" layer="1"/>
-<wire x1="19.5" y1="17.1" x2="22.5" y2="20.1" width="0.254" layer="1" curve="-90"/>
-<wire x1="22.5" y1="20.1" x2="39.98" y2="20.1" width="0.254" layer="1"/>
-<wire x1="39.98" y1="20.1" x2="40" y2="20.08" width="0.254" layer="1"/>
+<wire x1="19.5" y1="16.425" x2="19.5" y2="17" width="0.254" layer="1"/>
+<wire x1="19.5" y1="17" x2="22.5" y2="20" width="0.254" layer="1" curve="-90"/>
+<wire x1="22.5" y1="20" x2="40" y2="20" width="0.254" layer="1"/>
 </signal>
 <signal name="N$2" class="1" airwireshidden="yes">
@@
 <wire x1="29.5" y1="14.4" x2="29.5" y2="11.8504" width="0.254" layer="16"/>
 <contactref element="R5" pad="1"/>
-<wire x1="40" y1="9.92" x2="39.98" y2="9.9" width="0.254" layer="1"/>
-<via x="14" y="9.9" extent="1-16" drill="0.3"/>
-<wire x1="14" y1="9.9" x2="14" y2="22.2" width="0.254" layer="16"/>
+<via x="14" y="10" extent="1-16" drill="0.3"/>
+<wire x1="14" y1="10" x2="14" y2="22.2" width="0.254" layer="16"/>
 <via x="14" y="22.2" extent="1-16" drill="0.3"/>
 <wire x1="14" y1="22.2" x2="14" y2="20.81915" width="0.254" layer="1"/>
 <wire x1="14" y1="20.81915" x2="13.98085" y2="20.8" width="0.254" layer="1"/>
-<wire x1="39.98" y1="9.9" x2="14" y2="9.9" width="0.254" layer="1"/>
+<wire x1="40" y1="10" x2="14" y2="10" width="0.254" layer="1"/>
 </signal>
 <signal name="N$1">
