File: pcb/lnb-controller/qo-100-lnb-controller.brd (EAGLE design)
At the start: 60 x 75 mm, 71 parts, among them CON1 2EDG-2P, Q1 AO3401, U1 LT8636, U2 ADP7142AUJZ-3.3, U3 DSC1201DE3-25M00000, U4 DSB321SDA, U5 MXT573ABC25M0000

Commit message: GPSDO progress Added general filter PCB
Parts:
- C13: value 51pF -> 330pF
- C16: value 160pF -> 330pF
- C19: value 51pF -> 100pF
- L5: value 820nH -> 120nH
- L6: value 270nH -> 120nH
- L8: value 820nH -> 390nH
- moved L5 7.81 mm to (44.0, 21.1), turned to 0 degrees
- moved C13 6.00 mm to (44.0, 22.9), turned to 0 degrees
- moved C16 3.00 mm to (38.0, 22.9)
- moved C19 3.00 mm to (41.0, 22.8)
- moved L6 3.00 mm to (38.0, 21.1)
- moved L8 3.00 mm to (41.0, 26.1)
Connections:
- net GND: no longer L5.1
- net N$16: now also C20.1
- net N$17: no longer C13.1
- net N$18: now also C13.1, L5.1; no longer C20.1
Routing:
- net N$16: track 1.66 -> 5.51 mm
- net N$17: track 12.2 -> 9.21 mm
- net N$18: track 9.80 -> 7.70 mm
- net GND: vias 711 -> 710
Other:
- board text added: "IcyRadio LNB controller v1 Jun 2020"
- board text removed: "IcyRadio LNB controller v1 June 2020"

Commit message: Change some component values
Parts:
- C15, C22: value 51pF -> 100pF
- C18: value 620pF -> 1nF
- C20, C9: value 100nF -> 68pF
- L4, L9: value 820nH -> 470nH
- L7: value 68nH -> 43nH
- L8: value 390nH -> 330nH
Changed lines of the file:
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@@
 <attribute name="VOLTAGE" value="" x="-48.15" y="28.3" size="1.778" layer="27" rot="R270" display="off"/>
 </element>
-<element name="C9" library="Capacitor" package="CAP0603" value="100nF" x="26.8" y="22" smashed="yes">
+<element name="C9" library="Capacitor" package="CAP0603" value="68pF" x="26.8" y="22" smashed="yes">
 <attribute name="NAME" x="27.2536" y="20.616" size="0.8" layer="25" font="vector" ratio="10" rot="SR0" align="center-left"/>
 <attribute name="VALUE" x="23.8536" y="19.968" size="0.8" layer="27" font="vector" ratio="10" rot="SR0" align="center-left"/>
@@
 <attribute name="VOLTAGE" value="" x="65.44" y="-57.25" size="1.778" layer="27" display="off"/>
 </element>
-<element name="C22" library="Capacitor" package="CAP0603" value="51pF" x="34.5" y="36.1" smashed="yes" rot="R90">
+<element name="C22" library="Capacitor" package="CAP0603" value="100pF" x="34.5" y="36.1" smashed="yes" rot="R90">
 <attribute name="NAME" x="32.984" y="34.5536" size="0.8" layer="25" font="vector" ratio="10" rot="SR90" align="center-left"/>
 <attribute name="VALUE" x="36.532" y="33.1536" size="0.8" layer="27" font="vector" ratio="10" rot="SR90" align="center-left"/>
 <attribute name="VOLTAGE" value="" x="117.05" y="81.82" size="1.778" layer="27" rot="R90" display="off"/>
 </element>
-<element name="C18" library="Capacitor" package="CAP0603" value="620pF" x="33.7" y="30.3" smashed="yes" rot="R180">
+<element name="C18" library="Capacitor" package="CAP0603" value="1nF" x="33.7" y="30.3" smashed="yes" rot="R180">
 <attribute name="NAME" x="35.4536" y="30.316" size="0.8" layer="25" font="vector" ratio="10" rot="SR0" align="center-left"/>
 <attribute name="VALUE" x="36.6464" y="32.332" size="0.8" layer="27" font="vector" ratio="10" rot="SR180" align="center-left"/>
 <attribute name="VOLTAGE" value="" x="-17.1" y="112.85" size="1.778" layer="27" rot="R180" display="off"/>
 </element>
-<element name="C15" library="Capacitor" package="CAP0603" value="51pF" x="34.5" y="26.1" smashed="yes" rot="R90">
+<element name="C15" library="Capacitor" package="CAP0603" value="100pF" x="34.5" y="26.1" smashed="yes" rot="R90">
 <attribute name="NAME" x="32.984" y="24.5536" size="0.8" layer="25" font="vector" ratio="10" rot="SR90" align="center-left"/>
 <attribute name="VALUE" x="36.532" y="23.1536" size="0.8" layer="27" font="vector" ratio="10" rot="SR90" align="center-left"/>
@@
 <attribute name="VOLTAGE" value="" x="109.12" y="-59.65" size="1.778" layer="27" display="off"/>
 </element>
-<element name="C20" library="Capacitor" package="CAP0603" value="100nF" x="49.5" y="22" smashed="yes">
+<element name="C20" library="Capacitor" package="CAP0603" value="68pF" x="49.5" y="22" smashed="yes">
 <attribute name="NAME" x="47.8536" y="23.316" size="0.8" layer="25" font="vector" ratio="10" rot="SR0" align="center-left"/>
 <attribute name="VALUE" x="46.5536" y="19.968" size="0.8" layer="27" font="vector" ratio="10" rot="SR0" align="center-left"/>
@@
 <element name="F2" library="PTC Fuses" package="0805" value="" x="24" y="37.9" smashed="yes" rot="R90">
 <attribute name="HOLD" value="750 mA" x="65.91" y="111.56" size="1.778" layer="27" rot="R90" display="off"/>
+<attribute name="NAME" x="27.81" y="35.36" size="0.8" layer="27" font="vector" ratio="10" rot="R90" align="center-left"/>
 <attribute name="NAME" x="22.26" y="35.96" size="0.8" layer="25" font="vector" ratio="10" rot="R90" align="center-left"/>
-<attribute name="NAME" x="27.81" y="35.36" size="0.8" layer="27" font="vector" ratio="10" rot="R90" align="center-left"/>
 <attribute name="TRIP" value="1.5 A" x="65.91" y="111.56" size="1.778" layer="27" rot="R90" display="off"/>
 </element>
@@
 <attribute name="VALUE" x="21.968" y="26.2544" size="0.8" layer="27" font="vector" ratio="10" rot="SR270" align="center-left"/>
 </element>
-<element name="L9" library="Inductor" package="IND0603" value="820nH" x="34.5" y="32.8" smashed="yes" rot="R90">
+<element name="L9" library="Inductor" package="IND0603" value="470nH" x="34.5" y="32.8" smashed="yes" rot="R90">
 <attribute name="CURRENT" value="" x="106.89" y="97.57" size="1.778" layer="27" rot="R90" display="off"/>
 <attribute name="NAME" x="35.984" y="33.2456" size="0.8" layer="25" font="vector" ratio="10" rot="SR90" align="center-left"/>
 <attribute name="VALUE" x="36.532" y="29.3456" size="0.8" layer="27" font="vector" ratio="10" rot="SR90" align="center-left"/>
 </element>
-<element name="L7" library="Inductor" package="IND0603" value="68nH" x="35.3" y="28.6" smashed="yes">
+<element name="L7" library="Inductor" package="IND0603" value="43nH" x="35.3" y="28.6" smashed="yes">
 <attribute name="CURRENT" value="" x="106.42" y="-43.79" size="1.778" layer="27" display="off"/>
 <attribute name="NAME" x="32.3456" y="28.616" size="0.8" layer="25" font="vector" ratio="10" rot="SR0" align="center-left"/>
 <attribute name="VALUE" x="31.8456" y="26.568" size="0.8" layer="27" font="vector" ratio="10" rot="SR0" align="center-left"/>
 </element>
-<element name="L4" library="Inductor" package="IND0603" value="820nH" x="34.5" y="22.8" smashed="yes" rot="R90">
+<element name="L4" library="Inductor" package="IND0603" value="470nH" x="34.5" y="22.8" smashed="yes" rot="R90">
 <attribute name="CURRENT" value="" x="106.89" y="100.27" size="1.778" layer="27" rot="R90" display="off"/>
 <attribute name="NAME" x="34.484" y="19.9456" size="0.8" layer="25" font="vector" ratio="10" rot="SR90" align="center-left"/>
 <attribute name="VALUE" x="36.532" y="19.3456" size="0.8" layer="27" font="vector" ratio="10" rot="SR90" align="center-left"/>
 </element>
-<element name="L8" library="Inductor" package="IND0603" value="390nH" x="41" y="26.1" smashed="yes" rot="R270">
+<element name="L8" library="Inductor" package="IND0603" value="330nH" x="41" y="26.1" smashed="yes" rot="R270">
 <attribute name="CURRENT" value="" x="-36.47" y="10.86" size="1.778" layer="27" rot="R270" display="off"/>
 <attribute name="NAME" x="39.584" y="26.5456" size="0.8" layer="25" font="vector" ratio="10" rot="SR90" align="center-left"/>

Commit message: Change upconverter input attenuation Rename general filter to generic filter Generate generic filter panel Change capacitor value on LNB controller Add PA gain response
Parts:
- C9: value 68pF -> 100nF
Changed lines of the file:
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@@
 <attribute name="VOLTAGE" value="" x="-48.15" y="28.3" size="1.778" layer="27" rot="R270" display="off"/>
 </element>
-<element name="C9" library="Capacitor" package="CAP0603" value="68pF" x="26.8" y="22" smashed="yes">
+<element name="C9" library="Capacitor" package="CAP0603" value="100nF" x="26.8" y="22" smashed="yes">
 <attribute name="NAME" x="27.2536" y="20.616" size="0.8" layer="25" font="vector" ratio="10" rot="SR0" align="center-left"/>
 <attribute name="VALUE" x="23.8536" y="19.968" size="0.8" layer="27" font="vector" ratio="10" rot="SR0" align="center-left"/>
