File: pcb/lnb-controller/qo-100-lnb-controller.brd (EAGLE design)
At the start: 70 x 100 mm, 168 parts, among them CON1 3P-SH-SIDE, CON2 2EDG-2P-5MM, U1 EFM32TG11B120F128GM32, U2 DSB321SDA, U3 SI5351C-B-GM, U4 LT8650S-1, U5 MCP4728-A2, U6 MIC23155, U7 LT8636, U8 ADP7142AUJZ-3.3

Commit message: Work on PCBs
Parts:
- R29, R30: value 2.5K Ohms -> 2.55K Ohms
Changed lines of the file:
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@@
 <drawing>
 <settings>
-<setting alwaysvectorfont="yes"/>
+<setting alwaysvectorfont="no"/>
 <setting verticaltext="up"/>
 </settings>
@@
 <attribute name="VALUE" x="28.2544" y="64.632" size="0.8" layer="27" font="vector" ratio="10" rot="SR180" align="center-left"/>
 </element>
-<element name="R29" library="Resistor" package="RES0603" value="2.5K Ohms" x="22" y="36.6" smashed="yes" rot="R90">
+<element name="R29" library="Resistor" package="RES0603" value="2.55K Ohms" x="22" y="36.6" smashed="yes" rot="R90">
 <attribute name="NAME" x="21.984" y="32.7456" size="0.8" layer="25" font="vector" ratio="10" rot="SR90" align="center-left"/>
 <attribute name="TOLERANCE" value="" x="22" y="36.6" size="1.778" layer="27" rot="R90" display="off"/>
@@
 <attribute name="VALUE" x="18.168" y="39.5464" size="0.8" layer="27" font="vector" ratio="10" rot="SR270" align="center-left"/>
 </element>
-<element name="R30" library="Resistor" package="RES0603" value="2.5K Ohms" x="22" y="63.4" smashed="yes" rot="R270">
+<element name="R30" library="Resistor" package="RES0603" value="2.55K Ohms" x="22" y="63.4" smashed="yes" rot="R270">
 <attribute name="NAME" x="21.984" y="65.2456" size="0.8" layer="25" font="vector" ratio="10" rot="SR90" align="center-left"/>
 <attribute name="TOLERANCE" value="" x="22" y="63.4" size="1.778" layer="27" rot="R270" display="off"/>

Commit message: Update I2C slave resistors to minimize load effect when powered down
Parts:
- R4, R5: value 0 Ohms -> 1K Ohms
- R45, R46: value 1K Ohms -> 47K Ohms
Changed lines of the file:
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@@
 <attribute name="VALUE" x="69.905" y="44.58" size="0.8" layer="27" font="vector" ratio="10" rot="R180" align="center-left"/>
 </element>
-<element name="R4" library="Resistor" package="RES0603" value="0 Ohms" x="61.6" y="38.6" smashed="yes" rot="R180">
+<element name="R4" library="Resistor" package="RES0603" value="1K Ohms" x="61.6" y="38.6" smashed="yes" rot="R180">
 <attribute name="NAME" x="62.6456" y="37.116" size="0.8" layer="25" font="vector" ratio="10" rot="SR0" align="center-left"/>
 <attribute name="TOLERANCE" value="" x="61.6" y="35.3" size="0.8" layer="27" font="vector" ratio="10" rot="R180" display="off"/>
 <attribute name="VALUE" x="65.0544" y="40.632" size="0.8" layer="27" font="vector" ratio="10" rot="SR180" align="center-left"/>
 </element>
-<element name="R5" library="Resistor" package="RES0603" value="0 Ohms" x="61.6" y="40.4" smashed="yes" rot="R180">
+<element name="R5" library="Resistor" package="RES0603" value="1K Ohms" x="61.6" y="40.4" smashed="yes" rot="R180">
 <attribute name="NAME" x="61.9456" y="41.816" size="0.8" layer="25" font="vector" ratio="10" rot="SR0" align="center-left"/>
 <attribute name="TOLERANCE" value="" x="61.6" y="37.1" size="0.8" layer="27" font="vector" ratio="10" rot="R180" display="off"/>
@@
 <attribute name="NAME" x="49.5" y="68.9" size="0.8" layer="25" font="vector" ratio="10" align="center-left"/>
 </element>
-<element name="R45" library="Resistor" package="RES0603" value="1K Ohms" x="57.4" y="58.1" smashed="yes" rot="R270">
+<element name="R45" library="Resistor" package="RES0603" value="47K Ohms" x="57.4" y="58.1" smashed="yes" rot="R270">
 <attribute name="NAME" x="57.384" y="59.8456" size="0.8" layer="25" font="vector" ratio="10" rot="SR90" align="center-left"/>
 <attribute name="TOLERANCE" value="" x="57.4" y="58.1" size="1.778" layer="27" rot="R270" display="off"/>
 <attribute name="VALUE" x="55.368" y="61.5544" size="0.8" layer="27" font="vector" ratio="10" rot="SR270" align="center-left"/>
 </element>
-<element name="R46" library="Resistor" package="RES0603" value="1K Ohms" x="59.1" y="58.1" smashed="yes" rot="R270">
+<element name="R46" library="Resistor" package="RES0603" value="47K Ohms" x="59.1" y="58.1" smashed="yes" rot="R270">
 <attribute name="NAME" x="59.084" y="59.8456" size="0.8" layer="25" font="vector" ratio="10" rot="SR90" align="center-left"/>
 <attribute name="TOLERANCE" value="" x="59.1" y="58.1" size="1.778" layer="27" rot="R270" display="off"/>

Commit message: Assembly LNB Controller changes
Parts:
- C7, C8: value 100pF -> 150pF
Changed lines of the file:
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@@
 <attribute name="VOLTAGE" value="" x="60.36" y="-54.25" size="1.778" layer="27" display="off"/>
 </element>
-<element name="C7" library="Capacitor" package="CAP0603" value="100pF" x="24.8" y="23.3" smashed="yes">
+<element name="C7" library="Capacitor" package="CAP0603" value="150pF" x="24.8" y="23.3" smashed="yes">
 <attribute name="NAME" x="21.8536" y="23.316" size="0.8" layer="25" font="vector" ratio="10" rot="SR0" align="center-left"/>
 <attribute name="VALUE" x="21.8536" y="21.268" size="0.8" layer="27" font="vector" ratio="10" rot="SR0" align="center-left"/>
@@
 <attribute name="VOLTAGE" value="" x="-41.2" y="84.7" size="1.778" layer="27" display="off"/>
 </element>
-<element name="C8" library="Capacitor" package="CAP0603" value="100pF" x="24.8" y="76.7" smashed="yes">
+<element name="C8" library="Capacitor" package="CAP0603" value="150pF" x="24.8" y="76.7" smashed="yes">
 <attribute name="NAME" x="21.8536" y="76.716" size="0.8" layer="25" font="vector" ratio="10" rot="SR0" align="center-left"/>
 <attribute name="VALUE" x="21.8536" y="74.668" size="0.8" layer="27" font="vector" ratio="10" rot="SR0" align="center-left"/>

Commit message: Revert I2C resistor chnges because they do not work
Parts:
- R4, R5: value 1K Ohms -> 100 Ohms
Changed lines of the file:
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@@
 <attribute name="VALUE" x="69.905" y="44.58" size="0.8" layer="27" font="vector" ratio="10" rot="R180" align="center-left"/>
 </element>
-<element name="R4" library="Resistor" package="RES0603" value="1K Ohms" x="61.6" y="38.6" smashed="yes" rot="R180">
+<element name="R4" library="Resistor" package="RES0603" value="100 Ohms" x="61.6" y="38.6" smashed="yes" rot="R180">
 <attribute name="NAME" x="62.6456" y="37.116" size="0.8" layer="25" font="vector" ratio="10" rot="SR0" align="center-left"/>
 <attribute name="TOLERANCE" value="" x="61.6" y="35.3" size="0.8" layer="27" font="vector" ratio="10" rot="R180" display="off"/>
 <attribute name="VALUE" x="65.0544" y="40.632" size="0.8" layer="27" font="vector" ratio="10" rot="SR180" align="center-left"/>
 </element>
-<element name="R5" library="Resistor" package="RES0603" value="1K Ohms" x="61.6" y="40.4" smashed="yes" rot="R180">
+<element name="R5" library="Resistor" package="RES0603" value="100 Ohms" x="61.6" y="40.4" smashed="yes" rot="R180">
 <attribute name="NAME" x="61.9456" y="41.816" size="0.8" layer="25" font="vector" ratio="10" rot="SR0" align="center-left"/>
 <attribute name="TOLERANCE" value="" x="61.6" y="37.1" size="0.8" layer="27" font="vector" ratio="10" rot="R180" display="off"/>
