File: pcb/lnb-controller/qo-100-lnb-controller.sch (EAGLE design)
At the start: 71 parts, among them CON1 2EDG-2P, Q1 AO3401, U1 LT8636, U2 ADP7142AUJZ-3.3, U3 DSC1201DE3-25M00000, U4 DSB321SDA, U5 MXT573ABC25M0000

Commit message: Re-design LNB controller
Parts:
- removed JP3: PINHD-1X2, Pin Header:PINHD-1X2
- removed Q1: AO3401, Alpha Omega:AO3401
- added C23, C24: 100pF, Capacitor:CAPACITOR-0603
- added C35, C48, C49, C53, C59, C60, C61, C62, C70, C71, C72, C84, C85, C90: 100nF, Capacitor:CAPACITOR-0603
- added C36, C37, C75, C76: 4.7uF, Capacitor:CAPACITOR-0603
- added C38, C39, C40, C41, C42, C54, C73, C78, C80, C81, C91: 1uF, Capacitor:CAPACITOR-0603
- added C43, C44: DNP, Capacitor:CAPACITOR-0603
- added C45, C77, C79, C83, C87: 470pF, Capacitor:CAPACITOR-0603
- added C46, C47, C82: 10nF, Capacitor:CAPACITOR-0603
- added C50, C51: 4.7pF, Capacitor:CAPACITOR-0603
- added C52, C69, C92: 10uF, Capacitor:CAPACITOR-0603
- added C55, C56, C57, C58, C63, C64, C65, C66: 22uF, Capacitor:CAPACITOR-1206
- added C86: 10pF, Capacitor:CAPACITOR-0603
- added C88, C89: 100uF, Capacitor:CAPACITOR-1206
- added C93: 10uF, Capacitor:CAPACITOR-1206
- added D5: SMAJ24A, TVS:SMAJ24A
- added F3: 2.6A Hold, PTC Fuses:PTC1206
- added JP1: PINHD-1X3, Pin Header:PINHD-1X3
- added L10, L12: 43nH, Inductor:INDUCTOR-0603
- added L11, L13: 330nH, Inductor:INDUCTOR-0603
- added L14, L16: 470nH, Inductor:INDUCTOR-0603
- added L15, L17: 120nH, Inductor:INDUCTOR-0603
- added L18, L19: 4.7uH, Inductor:INDUCTOR-4X4MM
- added L20: 2.2uH, Inductor:INDUCTOR-2.5X2X1.2MM
- added L21: 4.7uH, Inductor:INDUCTOR-2.5X2X1.2MM
- added R13, R14, R15, R19, R20: 0 Ohms, Resistor:RESISTOR-0603
- added R16: 15K Ohms, Resistor:RESISTOR-0603
- added R17, R18, R24, R25, R34: 100K Ohms, Resistor:RESISTOR-0603
- added R21: 1K Ohms, Resistor:RESISTOR-0603
- added R22, R23, R27, R30: DNP, Resistor:RESISTOR-0603
- added R26, R29, R43: 1M Ohms, Resistor:RESISTOR-0603
- added R28, R31: 40.2K Ohms, Resistor:RESISTOR-0603
- added R32, R33: 2.5K Ohms, Resistor:RESISTOR-0603
- added R35: 10K Ohms, Resistor:RESISTOR-0603
- added R36, R41: 90.9K Ohms, Resistor:RESISTOR-0603
- added R37, R42: 12K Ohms, Resistor:RESISTOR-0603
- added R38: 41.2K Ohms, Resistor:RESISTOR-0603
- added R39: 309K Ohms, Resistor:RESISTOR-0603
- added R40: 71.5K Ohms, Resistor:RESISTOR-0603
- added R44: 226K Ohms, Resistor:RESISTOR-0603
- added R45: 510 Ohms, Resistor:RESISTOR-0603
- added RFCON4: RFCON-SMA-EDGE, RF Connector:RFCON-SMA-EDGE
- added TC1: TC2050-IDC, TagConnect:TC2050-IDC
- added U10: ADP7142AUJZ-3.3, Analog Devices:ADP7142AUJZ-3.3
- added U6, U7: AD5272-100, Analog Devices:AD5272-100
- added U8: MIC23155, Microchip:MIC23155
- added U9: LT8636, Analog Devices:LT8636
- C1: value 4.7uF -> 100nF; VOLTAGE 35V -> (none)
- C10, C17, C9: value 100nF -> 100pF
- C11: value 10pF -> 100nF
- C12, C30: value 22uF -> 100nF; device Capacitor:CAPACITOR-1206 -> Capacitor:CAPACITOR-0603; VOLTAGE 25V -> (none)
- C14: value 22uF -> 330pF; device Capacitor:CAPACITOR-1206 -> Capacitor:CAPACITOR-0603; VOLTAGE 25V -> (none)
- C16: value 330pF -> 100pF
- C18: value 1nF -> 100pF
- C19: value 100pF -> 1nF
- C2, C3: value 1uF -> 100nF; VOLTAGE 50V -> (none)
- C20: value 68pF -> 1nF
- C21: value 1uF -> 330pF
- C22: value 100pF -> 330pF
- C25: value 10uF -> 68pF
- C26: value 100nF -> 68pF
- C29, C31: value DNP -> 100nF
- C32: value DNP -> 15pF
- C33, C34: value 100nF -> 10pF
- C4: value 100nF -> 4.7uF
- C6: value 10uF -> 100nF; device Capacitor:CAPACITOR-1206 -> Capacitor:CAPACITOR-0603; VOLTAGE 50V -> (none)
- C7: value 10nF -> 100nF
- D1: value SMAJ24A -> LED0603; device TVS:SMAJ24A -> LED:LED0603; COLOR (none) -> BLUE
- D2: value LEDTH3MM -> LED0603; device LED:LEDTH3MM -> LED:LED0603; COLOR BLUE -> RED
- D3, D4: value LEDTH3MM -> LED0603; device LED:LEDTH3MM -> LED:LED0603
- F1: value 2.6A Hold -> (none); device PTC Fuses:PTC1206 -> PTC Fuses:PTC0805; HOLD 3A -> 750 mA; OCLCSC C207041 -> (none); TRIP 6A -> 1.5 A
- L1: value 470nH -> 4.7uH; CURRENT 600 mA -> (none); OCLCSC (none) -> C281111
- L3: value 4.7uH -> 470nH; device Inductor:INDUCTOR-6X6MM -> Inductor:INDUCTOR-0603; CURRENT 3A -> 600 mA; OCLCSC C326336 -> (none)
- L4: CURRENT (none) -> 600 mA
- L5: value 120nH -> 470nH; CURRENT (none) -> 600 mA
- L6: value 120nH -> 470nH
- L7: value 43nH -> 470nH
- L8: value 330nH -> 120nH
- L9: value 470nH -> 120nH
- R1: value 41.2K Ohms -> 10K Ohms
- R10: value 10K Ohms -> 100K Ohms
- R12: value 2.5K Ohms -> 0 Ohms
- R2: value 43.2 Ohms -> 10K Ohms
- R3: value 100K Ohms -> 330 Ohms; device Potentiometer:POTENTIOMETER-TH -> Resistor:RESISTOR-0603
- R4: value 1M Ohms -> 43.2 Ohms
- R5: value DNP -> 43.2 Ohms
- R6: value 47K Ohms -> 86.6 Ohms
- R8: value 2.5K Ohms -> 10K Ohms
- R9: value 2.5K Ohms -> 8.4K Ohms
- RFCON2: value RFCON-SMA-EDGE -> RFCON-F-EDGE; device RF Connector:RFCON-SMA-EDGE -> RF Connector:RFCON-F-EDGE
- U1: value LT8636 -> EFM32PG1B200F256GM32; device Analog Devices:LT8636 -> EFM32:EFM32PG1B200F256GM32
- U2: value ADP7142AUJZ-3.3 -> IQXT-210-3; device Analog Devices:ADP7142AUJZ-3.3 -> Crystal:IQXT-210-3
- U3: value DSC1201DE3-25M00000 -> DSB321SDA; device Microchip:DSC1201DE3-25M00000 -> Crystal:DSB321SDA
- U4: value DSB321SDA -> SI5351C-B-GM1; device Crystal:DSB321SDA -> Silicon Labs:SI5351C-B-GM1
- U5: value MXT573ABC25M0000 -> LT8650S-1; device Microchip:MXT573ABC25M0000 -> Analog Devices:LT8650S-1
Connections:
- removed net 12V0: C11.C1, C12.C1, C14.C1, C17.C1, C21.C1, L3.2, Q1.S, R10.2, R4.2, R8.2, R9.2, U1.BIAS, U2.EN, U2.VIN
- removed net 12V0_BST: C10.C2, U1.BST
- removed net 12V0_FB: C11.C2, R3.CW, R4.1, R5.2, U1.FB
- removed net 12V0_INTVCC: C5.C1, U1.INTVCC, U1.SYNC/MODE
- removed net 12V0_RT: R1.2, U1.RT
- removed net 12V0_SS: C7.C1, U1.TR/SS
- removed net 12V0_SW: C10.C1, L3.1, U1.SW
- removed net LNB_BIAS: C30.C1, C34.C1, C4.C1, F2.1, L1.1, R12.2
- removed net LNB_REF: C22.C2, C29.C2, C31.C2, C32.C2, C33.C2
- removed net N$2: D3.C, JP3-1.S, R11.1
- removed net N$5: D3.A, R9.1
- new net !REF_SYNTH_OE: R10.1, U4.!OE
- new net !RESET: R1.1, TC1-10(!RESET!).S, U1.!RESET
- new net 1V8: C4.C1, L1.1, U1.DVDD
- new net 3V1: R10.2
- new net 3V3_FB: R39.1, R40.2, U8.FB
- new net 3V3_REF_CLEAN: C28.C1, C29.C1, C30.C1, C31.C1, C35.C1, C92.C1, R8.2, U10.SENSE/ADJ, U10.VOUT, U2.VDD, U3.VDD, U4.VDDOA, U4.VDDOB, U4.VDDOC, U4.VDDOD
- new net 3V3_SOFTSTART: C79.C1, U8.SS
- new net 3V3_SW: L20.1, U8.SW
- new net 5V0: C76.C1, C86.C1, C89.C1, C90.C1, C91.C1, L21.2, R43.2, R45.2, U10.EN, U10.VIN, U8.EN, U8.VIN@0, U8.VIN@1, U9.BIAS
- new net 5V0_BST: C85.C2, U9.BST
- new net 5V0_FB: C86.C2, R43.1, R44.2, U9.FB
- new net 5V0_INTVCC: C81.C1, U9.INTVCC, U9.SYNC/MODE
- new net 5V0_RT: R38.2, U9.RT
- new net 5V0_SS: C82.C1, U9.TR/SS
- new net 5V0_SW: C85.C1, L21.1, U9.SW
- new net BIAS_REG_TEMP: C45.C1, R21.1
- new net CLK_MNGR_CLK0: R12.2, U4.CLK0
- new net CLK_MNGR_CLK1: R14.2, U4.CLK1
- new net CLK_MNGR_CLK2: R13.2, U4.CLK2
- new net CLK_MNGR_CLK3: R15.2, U4.CLK3
- new net I2C_SCL: U4.SCL, U6.SCL, U7.SCL
- new net I2C_SDA: U4.SDA, U6.SDA, U7.SDA
- new net LED: R3.2, U1.PC10
- new net LNB_BIAS_SEL: C6.C1, JP1-2.S, R2.2, U1.PC11
- new net N$23: D3.A, R33.1
- new net N$24: C12.C1, L5.2, RFCON2.SIGNAL
- new net N$25: D1.A, R3.1
- new net N$26: C12.C2, R5.2
- new net N$27: C10.C1, L3.2, L5.1
- new net N$28: C24.C1, L16.2
- new net N$29: C16.C1, L7.2
- new net N$30: C16.C2, C20.C1, L12.1, L16.1
- new net N$31: C14.C1, L7.1, L9.1, R5.1, R7.2
- new net N$32: C14.C2, C18.C1, C22.C1, L17.1, L9.2
- new net N$33: C26.C2, RFCON4.SIGNAL
- new net N$34: C18.C2, L13.2
- new net N$35: C22.C2, C26.C1, L17.2
- new net N$36: C34.C2, U4.XA
- new net N$37: C32.C1, U2.CLK, U4.CLKIN
- new net N$39: C54.C1, U6.EXT_CAP
- new net N$40: C73.C1, U7.EXT_CAP
- new net REF1: C23.C2, R12.1
- new net REF2: C24.C2, R14.1
- new net REF_XO_VC: R8.1, R9.2, U2.VCONT
- new net SWCLK: TC1-4(TCK/SWCLK).S, U1.PF0
- new net SWDIO: TC1-2(TMS/SWDIO).S, U1.PF1
- new net SWO: TC1-6(TDO/SWO).S, U1.PF2
- new net VBIAS1: C63.C1, C65.C1, C7.C1, C70.C1, F1.1, L2.1, R32.2, R36.2
- new net VBIAS1_BST: C48.C2, U5.2.BST
- new net VBIAS1_EN: R17.2, U5.2.EN/UV
- new net VBIAS1_FB: C50.C2, R26.1, R27.2, U5.2.FB, U6.A
- new net VBIAS1_FB_DIV: R27.1, R28.2, U6.W
- new net VBIAS1_PG: R24.1, U5.2.PG
- new net VBIAS1_SS: C46.C1, U5.2.SS
- new net VBIAS1_SW: C48.C1, L18.1, U5.2.SW
- new net VBIAS1_UNFUSED: C50.C1, C55.C1, C57.C1, C59.C1, C61.C1, F1.2, L18.2, R26.2, U5.CNTRL.BIAS
- new net VBIAS1_VC: R19.1, R22.2, U5.2.VC
- new net VBIAS1_VSENSE: C83.C1, R36.1, R37.2, U1.PB11
- new net VBIAS2: C64.C1, C66.C1, C71.C1, C8.C1, F2.1, L3.1, R33.2, R41.2
- new net VBIAS2_BST: C49.C2, U5.1.BST
- new net VBIAS2_EN: R18.2, U5.1.EN/UV
- new net VBIAS2_FB: C51.C2, R29.1, R30.2, U5.1.FB, U7.A
- new net VBIAS2_FB_DIV: R30.1, R31.2, U7.W
- new net VBIAS2_PG: R25.1, U5.1.PG
- new net VBIAS2_SS: C47.C1, U5.1.SS
- new net VBIAS2_SW: C49.C1, L19.1, U5.1.SW
- new net VBIAS2_UNFUSED: C51.C1, C56.C1, C58.C1, C60.C1, C62.C1, F2.2, L19.2, R29.2
- new net VBIAS2_VC: R20.1, R23.2, U5.1.VC
- new net VBIAS2_VSENSE: C87.C1, R41.1, R42.2, U1.PB12
- new net VBIAS_VCC: C40.C1, R19.2, R20.2, U5.CNTRL.SYNC, U5.CNTRL.VCC
- new net VIN_VSENSE: C77.C1, R34.1, R35.2, U1.PB13
- net 3V3: now also C1.C1, C2.C1, C3.C1, C52.C1, C53.C1, C69.C1, C72.C1, C84.C1, C88.C1, JP1-1.S, L20.2, R1.2, R24.2, R25.2, R39.2, TC1-1(VTARGET).S, U1.AVDD@0, U1.AVDD@1, U1.IOVDD0@0, U1.VREGVDD, U6.!RESET, U6.ADDR, U6.VDD, U7.!RESET, U7.VDD, U8.SNS; no longer C25.C1, C26.C1, C28.C1, U2.SENSE/ADJ, U2.VOUT, U3.!STDBY, U3.VDD, U5.OE, U5.VDD
- net GND: now also C10.C2, C19.C2, C20.C2, C29.C2, C31.C2, C32.C2, C33.C2, C35.C2, C36.C2, C37.C2, C38.C2, C39.C2, C40.C2, C41.C2, C42.C2, C43.C2, C44.C2, C45.C2, C46.C2, C47.C2, C52.C2, C53.C2, C54.C2, C55.C2, C56.C2, C57.C2, C58.C2, C59.C2, C60.C2, C61.C2, C62.C2, C63.C2, C64.C2, C65.C2, C66.C2, C69.C2, C70.C2, C71.C2, C72.C2, C73.C2, C75.C2, C76.C2, C77.C2, C78.C2, C79.C2, C80.C2, C81.C2, C82.C2, C83.C2, C84.C2, C87.C2, C88.C2, C89.C2, C9.C2, C90.C2, C91.C2, C92.C2, C93.C2, D1.C, D3.C, D5.A, JP1-3.S, L10.2, L11.1, L12.2, L13.1, R11.1, R16.1, R17.1, R18.1, R2.1, R28.1, R31.1, R35.1, R37.1, R38.1, R40.1, R42.1, R44.1, R9.1, RFCON4.GND, TC1-3(GND).S, U1.VREGVSS, U1.VSS@0, U10.GND, U5.1.GND, U5.2.GND, U5.CNTRL.GND, U6.GND, U6.VSS, U7.ADDR, U7.GND, U7.VSS, U8.AGND, U8.PGND@0, U8.PGND@1, U9.GND; no longer C12.C2, C14.C2, C17.C2, C18.C2, C21.C2, C25.C2, C26.C2, C34.C2, D1.A, JP3-2.S, L7.2, L8.1, R1.1, U1.GND, U5.GND
- net N$1: now also C43.C1, R22.1; no longer F2.2, Q1.D
- net N$10: now also C11.C2, R4.2; no longer C9.C2, R2.2
- net N$11: now also D2.A, R32.1; no longer D4.A, R12.1
- net N$12: now also C23.C1, L14.2; no longer C22.C1, L9.2
- net N$13: now also C9.C1, L2.2, L4.1; no longer C8.C1, L1.2, L2.1
- net N$14: now also L6.2; no longer L4.2
- net N$149: now also D4.A, R45.1; no longer D2.A, R8.1
- net N$15: now also C19.C1, L10.1, L14.1; no longer C18.C1, L7.1, L9.1
- net N$16: now also C21.C2, C25.C1, L15.2; no longer C13.C2, C20.C1, L5.2
- net N$17: now also C13.C1, L8.1, R4.1, R6.2; no longer C16.C1, L4.1, R2.1, R7.2
- net N$18: now also C13.C2, C17.C1, C21.C1, L15.1, L8.2; no longer C13.C1, C16.C2, C19.C1, L5.1, L6.2
- net N$19: now also F3.2; no longer F1.2
- net N$20: now also C25.C2, RFCON3.SIGNAL; no longer C20.C2, RFCON2.SIGNAL
- net N$21: now also L1.2, U1.VREGSW; no longer R3.WIPER, R5.1, R6.2
- net N$22: now also C17.C2, L11.2; no longer C19.C2, L8.2
- net N$3: now also R16.2, U5.CNTRL.RT; no longer Q1.G, R10.1, R11.2
- net N$4: now also C44.C1, R23.1; no longer C29.C1, RFCON3.SIGNAL
- net N$6: now also C5.C1, U1.DECOUPLE; no longer C31.C1, U3.CLK
- net N$7: now also C33.C1, C34.C1, R11.2, U3.CLK; no longer C32.C1, U4.CLK
- net N$8: now also R21.2, U5.CNTRL.TEMP; no longer C33.C1, U5.CLK
- net N$9: now also C11.C1, L4.2; no longer C9.C1, L2.2
- net VIN: now also C36.C1, C37.C1, C38.C1, C39.C1, C41.C1, C42.C1, C75.C1, C78.C1, C80.C1, C93.C1, D5.C, F3.1, R34.2, U5.1.VIN, U5.2.VIN, U9.EN/UV, U9.VIN; no longer C1.C1, C2.C1, C3.C1, C6.C1, D1.C, F1.1, U1.EN/UV, U1.VIN
Other:
- note added: "FCM w/ Spread Spectrum"
- note added: "I2C Address 0x2C"
- note added: "I2C Address 0x2F"
- note added: "I2C Address 0x60"
- note added: "LNB Bias selector 0 = TODO (default) 1 = TODO"
- note added: "Vout = ((R24/R25) + 1) * 0.97"
- note added: "Vout = ((R4/(R3+R6)) + 1) * 0.8"
- note added: "f = 2 MHz DS. Table 1"
- note removed: "VGSon = -6.5V at 13V VGSon = -9.0V at 18V"
- note removed: "Vout = ((R4/(R3+R6)) + 1) * 0.97"

Commit message: LNB controller v2 work
Parts:
- removed C26: 68pF, Capacitor:CAPACITOR-0603
- removed C85, C90: 100nF, Capacitor:CAPACITOR-0603
- removed C86: 10pF, Capacitor:CAPACITOR-0603
- removed C87: 470pF, Capacitor:CAPACITOR-0603
- removed C88, C89: 100uF, Capacitor:CAPACITOR-1206
- removed C91: 1uF, Capacitor:CAPACITOR-0603
- removed C92: 10uF, Capacitor:CAPACITOR-0603
- removed C93: 10uF, Capacitor:CAPACITOR-1206
- removed R43: 1M Ohms, Resistor:RESISTOR-0603
- removed R44: 226K Ohms, Resistor:RESISTOR-0603
- removed R45: 510 Ohms, Resistor:RESISTOR-0603
- added C67, C68: 470pF, Capacitor:CAPACITOR-0603
- added RFCON5: RFCON-U.FL, RF Connector:RFCON-U.FL
- C10: value 100pF -> 100nF
- C12: value 100nF -> 330pF
- C14, C22: value 330pF -> 100pF
- C18: value 100pF -> 1nF
- C20: value 1nF -> 330pF
- C24: value 100pF -> 68pF
- C3: value 100nF -> 4.7uF
- C31: value 100nF -> 15pF
- C32: value 15pF -> 10pF
- C34: value 10pF -> 100nF
- C35, C71: value 100nF -> 1uF
- C36, C37: value 4.7uF -> 10nF; VOLTAGE 35V -> (none)
- C38, C73: value 1uF -> 470pF; VOLTAGE 50V -> (none)
- C39, C54, C80: value 1uF -> 100nF; VOLTAGE 50V -> (none)
- C4: value 4.7uF -> 1uF
- C40, C5: value 1uF -> 100nF
- C41: value 1uF -> 4.7uF; VOLTAGE 50V -> 35V
- C42: value 1uF -> 4.7pF; VOLTAGE 50V -> (none)
- C43: value DNP -> 4.7pF
- C44: value DNP -> 1uF; VOLTAGE (none) -> 50V
- C45: value 470pF -> 22uF; device Capacitor:CAPACITOR-0603 -> Capacitor:CAPACITOR-1206; VOLTAGE (none) -> 25V
- C46, C47: value 10nF -> 22uF; device Capacitor:CAPACITOR-0603 -> Capacitor:CAPACITOR-1206; VOLTAGE (none) -> 25V
- C48, C59: value 100nF -> 22uF; device Capacitor:CAPACITOR-0603 -> Capacitor:CAPACITOR-1206; VOLTAGE (none) -> 25V
- C50, C51: value 4.7pF -> 100nF
- C55, C64: value 22uF -> 1uF; device Capacitor:CAPACITOR-1206 -> Capacitor:CAPACITOR-0603; VOLTAGE 25V -> 50V
- C62: value 100nF -> 10uF
- C63: value 22uF -> 100nF; device Capacitor:CAPACITOR-1206 -> Capacitor:CAPACITOR-0603; VOLTAGE 25V -> (none)
- C65: value 22uF -> 4.7uF; device Capacitor:CAPACITOR-1206 -> Capacitor:CAPACITOR-0603; VOLTAGE 25V -> 35V
- C66: value 22uF -> 4.7uF; device Capacitor:CAPACITOR-1206 -> Capacitor:CAPACITOR-0603; VOLTAGE 25V -> (none)
- C69: value 10uF -> 1uF; VOLTAGE (none) -> 50V
- C70: value 100nF -> 1uF; VOLTAGE (none) -> 50V
- C72: value 100nF -> 10nF
- C75: value 4.7uF -> 100nF; VOLTAGE 35V -> (none)
- C76: value 4.7uF -> 10pF
- C78: value 1uF -> 100uF; device Capacitor:CAPACITOR-0603 -> Capacitor:CAPACITOR-1206; VOLTAGE 50V -> (none)
- C79: value 470pF -> 100uF; device Capacitor:CAPACITOR-0603 -> Capacitor:CAPACITOR-1206
- C8: value 100nF -> 100pF
- C82: value 10nF -> 10uF
- C83: value 470pF -> 10uF; device Capacitor:CAPACITOR-0603 -> Capacitor:CAPACITOR-1206; VOLTAGE (none) -> 50V
- R10: value 100K Ohms -> 10K Ohms
- R11: value 10K Ohms -> 8.4K Ohms
- R12, R20: value 0 Ohms -> 100K Ohms
- R13: value 0 Ohms -> 10K Ohms
- R16: value 15K Ohms -> 0 Ohms
- R19: value 0 Ohms -> 15K Ohms
- R2: value 10K Ohms -> 1K Ohms
- R21: value 1K Ohms -> 100K Ohms
- R22: value DNP -> 1K Ohms
- R23: value DNP -> 1M Ohms
- R24: value 100K Ohms -> DNP
- R25: value 100K Ohms -> 40.2K Ohms
- R29: value 1M Ohms -> 2.5K Ohms
- R3: value 330 Ohms -> 1K Ohms
- R30: value DNP -> 2.5K Ohms
- R31: value 40.2K Ohms -> 100K Ohms
- R32: value 2.5K Ohms -> 10K Ohms
- R33: value 2.5K Ohms -> 90.9K Ohms
- R34: value 100K Ohms -> 12K Ohms
- R35: value 10K Ohms -> 41.2K Ohms
- R36: value 90.9K Ohms -> 309K Ohms
- R37: value 12K Ohms -> 71.5K Ohms
- R38: value 41.2K Ohms -> 90.9K Ohms
- R39: value 309K Ohms -> 12K Ohms
- R4: value 43.2 Ohms -> 10K Ohms
- R40: value 71.5K Ohms -> 1M Ohms
- R41: value 90.9K Ohms -> 226K Ohms
- R42: value 12K Ohms -> 510 Ohms
- R5: value 43.2 Ohms -> 330 Ohms
- R6, R7: value 86.6 Ohms -> 43.2 Ohms
- R8: value 10K Ohms -> 86.6 Ohms
- R9: value 8.4K Ohms -> 86.6 Ohms
- renumbered C84 to C74
Connections:
- removed net 3V1: R10.2
- removed net CLK_MNGR_CLK0: R12.2, U4.CLK0
- removed net CLK_MNGR_CLK1: R14.2, U4.CLK1
- removed net CLK_MNGR_CLK2: R13.2, U4.CLK2
- removed net CLK_MNGR_CLK3: R15.2, U4.CLK3
- removed net N$4: C44.C1, R23.1
- removed net VBIAS1_VC: R19.1, R22.2, U5.2.VC
- removed net VBIAS2_VC: R20.1, R23.2, U5.1.VC
- new net N$2: R15.2, U4.CLK2
- new net N$41: R16.1, RFCON5.SIGNAL
- new net N$5: R14.2, U4.CLK0
- net !REF_SYNTH_OE: now also R12.1, U1.PD9; no longer R10.1
- net 1V8: now also C3.C1; no longer C4.C1
- net 3V3: now also C54.C1, C62.C1, C63.C1, C78.C1, R12.2, R2.2, R20.2, R21.2, R3.2, R36.2; no longer C27.C1, C3.C1, C53.C1, C69.C1, C72.C1, C88.C1, R24.2, R25.2, R39.2, U4.VDD
- net 3V3_FB: now also R36.1, R37.2; no longer R39.1, R40.2
- net 3V3_REF_CLEAN: now also C27.C1, C34.C1, C82.C1, R10.2, U4.VDD; no longer C31.C1, C35.C1, C92.C1, R8.2
- net 3V3_SOFTSTART: now also C68.C1; no longer C79.C1
- net 5V0: now also C66.C1, C79.C1, C80.C1, C81.C1, R40.2, R42.2; no longer C86.C1, C89.C1, C90.C1, C91.C1, R43.2, R45.2
- net 5V0_BST: now also C75.C2; no longer C85.C2
- net 5V0_FB: now also C76.C2, R40.1, R41.2; no longer C86.C2, R43.1, R44.2
- net 5V0_INTVCC: now also C71.C1; no longer C81.C1
- net 5V0_RT: now also R35.2; no longer R38.2
- net 5V0_SS: now also C72.C1; no longer C82.C1
- net 5V0_SW: now also C75.C1; no longer C85.C1
- net BIAS_REG_TEMP: now also C38.C1, R22.1, U1.PB11; no longer C45.C1, R21.1
- net GND: now also C18.C2, C34.C2, C48.C2, C49.C2, C50.C2, C51.C2, C67.C2, C68.C2, R13.1, R19.1, R25.1, R32.1, R34.1, R39.1, R4.1, R41.1, R8.1, RFCON5.GND; no longer C10.C2, C20.C2, C33.C2, C39.C2, C40.C2, C42.C2, C43.C2, C75.C2, C76.C2, C87.C2, C88.C2, C89.C2, C90.C2, C91.C2, C92.C2, C93.C2, R16.1, R2.1, R31.1, R38.1, R40.1, R42.1, R44.1, R6.1, R7.1
- net I2C_SCL: now also R3.1, U1.PC11
- net I2C_SDA: now also R2.1, U1.PC10
- net LED: now also R5.2, U1.PF3; no longer R3.2, U1.PC10
- net LNB_BIAS_SEL: now also C5.C1, R4.2, U1.PD10; no longer C6.C1, R2.2, U1.PC11
- net N$1: now also R16.2, U4.CLK3; no longer C43.C1, R22.1
- net N$10: now also C10.C2, R6.2; no longer C11.C2, R4.2
- net N$11: now also R29.1; no longer R32.1
- net N$12: now also C22.C1; no longer C23.C1
- net N$13: now also C8.C1; no longer C9.C1
- net N$14: now also C14.C1; no longer C15.C1
- net N$149: now also R42.1; no longer R45.1
- net N$15: now also C14.C2, C18.C1; no longer C15.C2, C19.C1
- net N$16: now also C20.C2, C24.C1; no longer C21.C2, C25.C1
- net N$17: now also C12.C1, R6.1, R8.2; no longer C13.C1, R4.1, R6.2
- net N$18: now also C12.C2, C16.C1, C20.C1; no longer C13.C2, C17.C1, C21.C1
- net N$20: now also C24.C2; no longer C25.C2
- net N$22: now also C16.C2; no longer C17.C2
- net N$23: now also R30.1; no longer R33.1
- net N$24: now also C11.C1; no longer C12.C1
- net N$25: now also R5.1; no longer R3.1
- net N$26: now also C11.C2, R7.2; no longer C12.C2, R5.2
- net N$27: now also C9.C1; no longer C10.C1
- net N$28: now also C23.C1; no longer C24.C1
- net N$29: now also C15.C1; no longer C16.C1
- net N$3: now also R19.2; no longer R16.2
- net N$30: now also C15.C2, C19.C1; no longer C16.C2, C20.C1
- net N$31: now also C13.C1, R7.1, R9.2; no longer C14.C1, R5.1, R7.2
- net N$32: now also C13.C2, C17.C1, C21.C1; no longer C14.C2, C18.C1, C22.C1
- net N$33: now also C25.C2; no longer C26.C2
- net N$34: now also C17.C2; no longer C18.C2
- net N$35: now also C21.C2, C25.C1; no longer C22.C2, C26.C1
- net N$36: now also C33.C2; no longer C34.C2
- net N$37: now also C31.C1; no longer C32.C1
- net N$39: now also C55.C1; no longer C54.C1
- net N$40: now also C64.C1; no longer C73.C1
- net N$6: now also C4.C1; no longer C5.C1
- net N$7: now also C32.C1, R13.2; no longer C34.C1, R11.2
- net N$8: now also R22.2; no longer R21.2
- net N$9: now also C10.C1; no longer C11.C1
- net REF1: now also C22.C2, R14.1; no longer C23.C2, R12.1
- net REF2: now also C23.C2, R15.1; no longer C24.C2, R14.1
- net REF_XO_VC: now also R10.1, R11.2; no longer R8.1, R9.2
- net VBIAS1: now also C56.C1, C58.C1, C6.C1, C60.C1, R29.2, R33.2; no longer C63.C1, C65.C1, C7.C1, C70.C1, R32.2, R36.2
- net VBIAS1_BST: now also C39.C2; no longer C48.C2
- net VBIAS1_EN: now also U1.PD15
- net VBIAS1_FB: now also C42.C2, R23.1, R24.2; no longer C50.C2, R26.1, R27.2
- net VBIAS1_FB_DIV: now also R24.1, R25.2; no longer R27.1, R28.2
- net VBIAS1_PG: now also R20.1, U1.PA1; no longer R24.1
- net VBIAS1_SS: now also C36.C1; no longer C46.C1
- net VBIAS1_SW: now also C39.C1; no longer C48.C1
- net VBIAS1_UNFUSED: now also C42.C1, C45.C1, C47.C1, C49.C1, C51.C1, R23.2; no longer C50.C1, C55.C1, C57.C1, C59.C1, C61.C1, R26.2
- net VBIAS1_VSENSE: now also C73.C1, R33.1, R34.2, U1.PB12; no longer C83.C1, R36.1, R37.2, U1.PB11
- net VBIAS2: now also C57.C1, C59.C1, C61.C1, C7.C1, R30.2, R38.2; no longer C64.C1, C66.C1, C71.C1, C8.C1, R33.2, R41.2
- net VBIAS2_BST: now also C40.C2; no longer C49.C2
- net VBIAS2_EN: now also U1.PD14
- net VBIAS2_FB: now also C43.C2, R26.1, R27.2; no longer C51.C2, R29.1, R30.2
- net VBIAS2_FB_DIV: now also R27.1, R28.2; no longer R30.1, R31.2
- net VBIAS2_PG: now also R21.1, U1.PA0; no longer R25.1
- net VBIAS2_SS: now also C37.C1; no longer C47.C1
- net VBIAS2_SW: now also C40.C1; no longer C49.C1
- net VBIAS2_UNFUSED: now also C43.C1, C46.C1, C48.C1, C50.C1, C53.C1, R26.2; no longer C51.C1, C56.C1, C58.C1, C60.C1, C62.C1, R29.2
- net VBIAS2_VSENSE: now also C77.C1, R38.1, R39.2, U1.PB13; no longer C87.C1, R41.1, R42.2, U1.PB12
- net VBIAS_VCC: now also C35.C1, U5.1.VC, U5.2.VC; no longer C40.C1, R19.2, R20.2
- net VIN: now also C44.C1, C65.C1, C69.C1, C70.C1, C83.C1, R31.2; no longer C36.C1, C37.C1, C38.C1, C39.C1, C42.C1, C75.C1, C78.C1, C80.C1, C93.C1, R34.2
- net VIN_VSENSE: now also C67.C1, R31.1, R32.2, U1.PB14; no longer C77.C1, R34.1, R35.2, U1.PB13
Other:
- moved on the sheet: C10, C11, C12, C13, C14, C15, C16, C17, C18, C19, C20, C21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

Commit message: LNB converter work
Connections:
- net 5V0: now also U5.CNTRL.BIAS
- net VBIAS1_UNFUSED: no longer U5.CNTRL.BIAS
Changed lines of the file:
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@@
 <part name="R3" library="Resistor" deviceset="RESISTOR" device="-0603" value="1K Ohms"/>
 <part name="3V22" library="Supply Symbol" deviceset="3V3" device=""/>
+<part name="5V00003" library="Supply Symbol" deviceset="5V0" device=""/>
 </parts>
 <sheets>
@@
 </instance>
 <instance part="F1" gate="G$1" x="256.54" y="340.36" smashed="yes">
-<attribute name="HOLD" x="256.54" y="336.296" size="1.778" layer="97" align="top-left"/>
-<attribute name="TRIP" x="256.54" y="333.756" size="1.778" layer="97" align="top-left"/>
+<attribute name="HOLD" x="256.54" y="336.296" size="1.778" layer="97" align="top-left" display="both"/>
+<attribute name="TRIP" x="256.54" y="333.756" size="1.778" layer="97" align="top-left" display="both"/>
 <attribute name="NAME" x="256.54" y="345.1606" size="1.778" layer="95" ratio="10" rot="SR0"/>
 </instance>
@@
 </instance>
 <instance part="F2" gate="G$1" x="256.54" y="101.6" smashed="yes">
-<attribute name="HOLD" x="256.54" y="97.536" size="1.778" layer="97" align="top-left"/>
-<attribute name="TRIP" x="256.54" y="94.996" size="1.778" layer="97" align="top-left"/>
+<attribute name="HOLD" x="256.54" y="97.536" size="1.778" layer="97" align="top-left" display="both"/>
+<attribute name="TRIP" x="256.54" y="94.996" size="1.778" layer="97" align="top-left" display="both"/>
 <attribute name="NAME" x="256.54" y="106.4006" size="1.778" layer="95" ratio="10" rot="SR0"/>
 </instance>
@@
 <instance part="VIN7" gate="G$1" x="180.34" y="185.42" smashed="yes">
 <attribute name="VALUE" x="177.8" y="182.88" size="1.778" layer="96" rot="R90"/>
+</instance>
+<instance part="5V00003" gate="G$1" x="76.2" y="226.06" smashed="yes">
+<attribute name="VALUE" x="73.66" y="223.52" size="1.778" layer="96" rot="R90"/>
 </instance>
 </instances>
@@
 <label x="256.54" y="353.06" size="1.778" layer="95" xref="yes"/>
 </segment>
-<segment>
-<wire x1="81.28" y1="215.9" x2="71.12" y2="215.9" width="0.1524" layer="91"/>
-<label x="71.12" y="215.9" size="1.778" layer="95" rot="R180" xref="yes"/>
-<pinref part="U5" gate=".CNTRL" pin="BIAS"/>
-</segment>
 </net>
 <net name="VBIAS2_SW" class="0">
@@
 </segment>
 </net>
+<net name="5V0" class="0">
+<segment>
+<pinref part="5V00003" gate="G$1" pin="5V0"/>
+<pinref part="U5" gate=".CNTRL" pin="BIAS"/>
+<wire x1="76.2" y1="226.06" x2="76.2" y2="215.9" width="0.1524" layer="91"/>
+<wire x1="76.2" y1="215.9" x2="81.28" y2="215.9" width="0.1524" layer="91"/>
+</segment>
+</net>

Commit message: Work on LNB Controller
Parts:
- removed C83: 10uF, Capacitor:CAPACITOR-1206
- removed JP1: PINHD-1X3, Pin Header:PINHD-1X3
- removed L21: 4.7uH, Inductor:INDUCTOR-2.5X2X1.2MM
- removed R42: 510 Ohms, Resistor:RESISTOR-0603
- added C26: 100nF, Capacitor:CAPACITOR-0603
- added CON2: 2EDG-2P-5MM, Generic Connector:2EDG-2P-5MM
- C11: value 100nF -> 330pF
- C13, C21: value 330pF -> 100pF
- C17: value 100pF -> 1nF
- C19: value 1nF -> 330pF
- C23: value 100pF -> 68pF
- C25: value 68pF -> 100nF
- C27: value 100nF -> 33nF
- C28: value 100nF -> 15pF
- C3: value 4.7uF -> 100nF
- C30, C75: value 100nF -> 10pF
- C31: value 15pF -> 100nF
- C33: value 10pF -> 100nF
- C34, C80: value 100nF -> 1uF
- C35, C71: value 1uF -> 10nF
- C37, C72: value 10nF -> 470pF
- C38, C73: value 470pF -> 100nF
- C40: value 100nF -> 4.7uF; VOLTAGE (none) -> 35V
- C41: value 4.7uF -> 4.7pF; VOLTAGE 35V -> (none)
- C43: value 4.7pF -> 1uF; VOLTAGE (none) -> 50V
- C44, C55: value 1uF -> 22uF; device Capacitor:CAPACITOR-0603 -> Capacitor:CAPACITOR-1206; VOLTAGE 50V -> 25V
- C48, C59: value 22uF -> 100nF; device Capacitor:CAPACITOR-1206 -> Capacitor:CAPACITOR-0603; VOLTAGE 25V -> (none)
- C51, C61: value 100nF -> 10uF
- C52, C62: value 10uF -> 100nF
- C54, C63: value 100nF -> 1uF; VOLTAGE (none) -> 50V
- C64: value 1uF -> 4.7uF; VOLTAGE 50V -> 35V
- C65: VOLTAGE 35V -> (none)
- C66: value 4.7uF -> 470pF
- C68: value 470pF -> 1uF; VOLTAGE (none) -> 50V
- C7: value 100nF -> 100pF
- C70: VOLTAGE 50V -> (none)
- C76: value 10pF -> 470pF
- C77: value 470pF -> 100uF; device Capacitor:CAPACITOR-0603 -> Capacitor:CAPACITOR-1206
- C79: value 100uF -> 100nF; device Capacitor:CAPACITOR-1206 -> Capacitor:CAPACITOR-0603
- C81: value 1uF -> 10uF
- C82: device Capacitor:CAPACITOR-0603 -> Capacitor:CAPACITOR-1206; VOLTAGE (none) -> 50V
- C9: value 100pF -> 100nF
- CON1: value 2EDG-2P -> 3P-SH-SIDE; device Generic Connector:2EDG-2P -> JST:3P-SH-SIDE
- L1: value 4.7uH -> 470nH; CURRENT (none) -> 600 mA; OCLCSC C281111 -> (none)
- L10, L12: value 43nH -> 330nH
- L11: value 330nH -> 43nH
- L13: value 330nH -> 470nH
- L14, L16, L7: value 470nH -> 120nH
- L15: value 120nH -> 470nH
- L17: value 120nH -> 4.7uH; device Inductor:INDUCTOR-0603 -> Inductor:INDUCTOR-4X4MM; CURRENT (none) -> 4A
- L19: value 4.7uH -> 2.2uH; device Inductor:INDUCTOR-4X4MM -> Inductor:INDUCTOR-2.5X2X1.2MM; CURRENT 4A -> 2.2A; OCLCSC (none) -> C375952
- L20: value 2.2uH -> 4.7uH; CURRENT 2.2A -> 1.4A; OCLCSC C375952 -> C443497
- L5: CURRENT 600 mA -> (none)
- L9: value 120nH -> 43nH
- R10: value 10K Ohms -> 86.6 Ohms
- R11: value 8.4K Ohms -> 100K Ohms
- R12, R31: value 100K Ohms -> 10K Ohms
- R13: value 10K Ohms -> 0 Ohms
- R16: value 0 Ohms -> 100K Ohms
- R18: value 100K Ohms -> 15K Ohms
- R19: value 15K Ohms -> 100K Ohms
- R21: value 100K Ohms -> 1K Ohms
- R22: value 1K Ohms -> 1M Ohms
- R23, R26: value 1M Ohms -> DNP
- R24, R27: value DNP -> 40.2K Ohms
- R25: value 40.2K Ohms -> 1M Ohms
- R28: value 40.2K Ohms -> 2.5K Ohms
- R30: value 2.5K Ohms -> 100K Ohms
- R32: value 10K Ohms -> 90.9K Ohms
- R33, R38: value 90.9K Ohms -> 12K Ohms
- R34: value 12K Ohms -> 41.2K Ohms
- R35: value 41.2K Ohms -> 309K Ohms
- R36: value 309K Ohms -> 71.5K Ohms
- R37: value 71.5K Ohms -> 90.9K Ohms
- R39: value 12K Ohms -> 1M Ohms
- R4: value 10K Ohms -> 100 Ohms
- R40: value 1M Ohms -> 226K Ohms
- R41: value 226K Ohms -> 510 Ohms
- R5: value 330 Ohms -> 100 Ohms
- R6: value 43.2 Ohms -> 330 Ohms
- R8: value 86.6 Ohms -> 43.2 Ohms
- U1: value EFM32PG1B200F256GM32 -> EFM32PG1B100F256GM32; device EFM32:EFM32PG1B200F256GM32 -> EFM32:EFM32PG1B100F256GM32
- U2: value IQXT-210-3 -> TX-8010-EAW-1070-25M0000000; device Crystal:IQXT-210-3 -> Microchip:TX-8010-EAW-1070-25M0000000
- U4: value SI5351C-B-GM1 -> SI5351C-B-GM; device Silicon Labs:SI5351C-B-GM1 -> Silicon Labs:SI5351C-B-GM
Connections:
- removed net 1V8: C3.C1, L1.1, U1.DVDD
- removed net LNB_BIAS_SEL: C5.C1, JP1-2.S, R4.2, U1.PD10
- removed net N$27 (its old number): C9.C1, L3.2, L5.1
- removed net N$29 (its old number): C15.C1, L7.2
- removed net REF_XO_VC: R10.1, R11.2, U2.VCONT
- new net N$13: C7.C1, L1.2, L3.1
- new net N$14: C13.C1, L5.2
- new net N$38: CON1-1.S, R4.1
- new net N$4: CON1-2.S, R5.1
- new net UART_RX: R4.2, U1.PF3
- new net UART_TX: R5.2, U1.PF4
- net !REF_SYNTH_OE: now also R11.1, U1.PC11; no longer R12.1, U1.PD9
- net 3V3: now also C3.C1, C51.C1, C53.C1, C61.C1, C73.C1, C77.C1, L19.2, R11.2, R19.2, R35.2, U1.DVDD; no longer C52.C1, C54.C1, C63.C1, C74.C1, C78.C1, JP1-1.S, L20.2, R12.2, R21.2, R36.2, U1.VREGVDD
- net 3V3_FB: now also R35.1, R36.2; no longer R36.1, R37.2
- net 3V3_REF_CLEAN: now also C25.C1, C26.C1, C31.C1, C33.C1, C81.C1, U2.OE; no longer C27.C1, C28.C1, C30.C1, C34.C1, C82.C1, R10.2
- net 3V3_SOFTSTART: now also C67.C1; no longer C68.C1
- net 3V3_SW: now also L19.1; no longer L20.1
- net 5V0: now also C65.C1, C75.C1, C78.C1, L20.2, R39.2, R41.2; no longer C66.C1, C76.C1, C81.C1, L21.2, R40.2, R42.2
- net 5V0_BST: now also C74.C2; no longer C75.C2
- net 5V0_FB: now also C75.C2, R39.1, R40.2; no longer C76.C2, R40.1, R41.2
- net 5V0_INTVCC: now also C70.C1; no longer C71.C1
- net 5V0_RT: now also R34.2; no longer R35.2
- net 5V0_SS: now also C71.C1; no longer C72.C1
- net 5V0_SW: now also C74.C1, L20.1; no longer C75.C1, L21.1
- net BIAS_REG_TEMP: now also C37.C1, R21.1; no longer C38.C1, R22.1
- net GND: now also C17.C2, C25.C2, C26.C2, C33.C2, C40.C2, C43.C2, C76.C2, CON1-3.S, CON2-1.S, L10.1, L11.2, L12.1, L9.2, R10.1, R12.1, R16.1, R24.1, R27.1, R31.1, R33.1, R36.1, R38.1, R40.1; no longer C19.C2, C32.C2, C38.C2, C41.C2, C74.C2, C83.C2, C9.C2, CON1-1.S, JP1-3.S, L10.2, L11.1, L12.2, L13.1, R11.1, R13.1, R19.1, R25.1, R28.1, R32.1, R35.1, R37.1, R39.1, R4.1, R41.1, R8.1, U1.VREGVSS
- net I2C_SCL: now also U1.PC10; no longer U1.PC11
- net I2C_SDA: now also U1.PC9; no longer U1.PC10
- net LED: now also R6.2, U1.PC8; no longer R5.2, U1.PF3
- net N$1: now also R15.2, U4.CLK7; no longer R16.2, U4.CLK3
- net N$10: now also C9.C2, R7.2; no longer C10.C2, R6.2
- net N$11: now also R28.1; no longer R29.1
- net N$12: now also C21.C1, L13.2; no longer C22.C1, L14.2
- net N$149: now also R41.1; no longer R42.1
- net N$15: now also C13.C2, C17.C1, L13.1, L9.1; no longer C14.C2, C18.C1, L10.1, L14.1
- net N$16: now also C19.C2, C23.C1, L14.2; no longer C20.C2, C24.C1, L15.2
- net N$17: now also C11.C1, L5.1, L7.1, R7.1, R9.2; no longer C12.C1, L6.1, L8.1, R6.1, R8.2
- net N$18: now also C11.C2, C15.C1, C19.C1, L14.1, L7.2; no longer C12.C2, C16.C1, C20.C1, L15.1, L8.2
- net N$19: now also CON2-2.S; no longer CON1-2.S
- net N$2: now also R14.2, U4.CLK5; no longer R15.2, U4.CLK2
- net N$20: now also C23.C2; no longer C24.C2
- net N$21: now also C27.C1, U2.FLT; no longer L1.2, U1.VREGSW
- net N$22: now also C15.C2, L10.2; no longer C16.C2, L11.2
- net N$23: now also R29.1; no longer R30.1
- net N$24: now also C10.C1, L4.2; no longer C11.C1, L5.2
- net N$25: now also R6.1; no longer R5.1
- net N$26: now also C10.C2, R8.2; no longer C11.C2, R7.2
- net N$28: now also C22.C1, L15.2; no longer C23.C1, L16.2
- net N$3: now also R18.2; no longer R19.2
- net N$30: now also C14.C2, C18.C1, L11.1, L15.1; no longer C15.C2, C19.C1, L12.1, L16.1
- net N$31: now also C12.C1, L6.1, L8.1, R10.2, R8.1; no longer C13.C1, L7.1, L9.1, R7.1, R9.2
- net N$32: now also C12.C2, C16.C1, C20.C1, L16.1, L8.2; no longer C13.C2, C17.C1, C21.C1, L17.1, L9.2
- net N$33: now also C24.C2; no longer C25.C2
- net N$34: now also C16.C2, L12.2; no longer C17.C2, L13.2
- net N$35: now also C20.C2, C24.C1, L16.2; no longer C21.C2, C25.C1, L17.2
- net N$36: now also C32.C2; no longer C33.C2
- net N$37: now also C28.C1; no longer C31.C1
- net N$39: now also C54.C1; no longer C55.C1
- net N$40: now also C63.C1; no longer C64.C1
- net N$41: now also R15.1; no longer R16.1
- net N$5: now also R13.2, U4.CLK1; no longer R14.2, U4.CLK0
- net N$7: now also C30.C1, R12.2; no longer C33.C1, R13.2
- net N$8: now also R21.2; no longer R22.2
- net N$9: now also C9.C1, L3.2; no longer C10.C1, L4.2
- net REF1: now also C21.C2, R13.1; no longer C22.C2, R14.1
- net REF2: now also C22.C2, R14.1; no longer C23.C2, R15.1
- net VBIAS1: now also C5.C1, C55.C1, C57.C1, C59.C1, L1.1, R28.2, R32.2; no longer C56.C1, C58.C1, C6.C1, C60.C1, L2.1, R29.2, R33.2
- net VBIAS1_BST: now also C38.C2; no longer C39.C2
- net VBIAS1_EN: now also R16.2; no longer R17.2
- net VBIAS1_FB: now also C41.C2, R22.1, R23.2; no longer C42.C2, R23.1, R24.2
- net VBIAS1_FB_DIV: now also R23.1, R24.2; no longer R24.1, R25.2
- net VBIAS1_PG: now also R19.1; no longer R20.1
- net VBIAS1_SS: now also C35.C1; no longer C36.C1
- net VBIAS1_SW: now also C38.C1, L17.1; no longer C39.C1, L18.1
- net VBIAS1_UNFUSED: now also C41.C1, C44.C1, C46.C1, C48.C1, C50.C1, L17.2, R22.2; no longer C42.C1, C45.C1, C47.C1, C49.C1, C51.C1, L18.2, R23.2
- net VBIAS1_VSENSE: now also C72.C1, R32.1, R33.2; no longer C73.C1, R33.1, R34.2
- net VBIAS2: now also C56.C1, C58.C1, C6.C1, C60.C1, L2.1, R29.2, R37.2; no longer C57.C1, C59.C1, C61.C1, C7.C1, L3.1, R30.2, R38.2
- net VBIAS2_BST: now also C39.C2; no longer C40.C2
- net VBIAS2_EN: now also R17.2; no longer R18.2
- net VBIAS2_FB: now also C42.C2, R25.1, R26.2; no longer C43.C2, R26.1, R27.2
- net VBIAS2_FB_DIV: now also R26.1, R27.2; no longer R27.1, R28.2
- net VBIAS2_PG: now also R20.1; no longer R21.1
- net VBIAS2_SS: now also C36.C1; no longer C37.C1
- net VBIAS2_SW: now also C39.C1, L18.1; no longer C40.C1, L19.1
- net VBIAS2_UNFUSED: now also C42.C1, C45.C1, C47.C1, C49.C1, C52.C1, L18.2, R25.2; no longer C43.C1, C46.C1, C48.C1, C50.C1, C53.C1, L19.2, R26.2
- net VBIAS2_VSENSE: now also C76.C1, R37.1, R38.2; no longer C77.C1, R38.1, R39.2
- net VBIAS_VCC: now also C34.C1; no longer C35.C1
- net VIN: now also C40.C1, C43.C1, C64.C1, C68.C1, C82.C1, R30.2; no longer C41.C1, C44.C1, C65.C1, C70.C1, C83.C1, R31.2
- net VIN_VSENSE: now also C66.C1, R30.1, R31.2; no longer C67.C1, R31.1, R32.2
Other:
- note removed: "LNB Bias selector 0 = TODO (default) 1 = TODO"
- moved on the sheet: C10, C11, C12, C13, C14, C15, C16, C17, C18, C19, C20, C21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
