File: pcb/lnb-controller/qo-100-lnb-controller.sch (EAGLE design)
At the start: 168 parts, among them CON1 3P-SH-SIDE, CON2 2EDG-2P-5MM, U1 EFM32PG1B100F256GM32, U10 ADP7142AUJZ-3.3, U3 DSB321SDA, U4 SI5351C-B-GM, U5 LT8650S-1, U6 AD5272-100, U7 AD5272-100, U8 MIC23155, U9 LT8636

Commit message: Finish routing LNB Controller PCB
Parts:
- removed C77, C78: 100uF, Capacitor:CAPACITOR-1206
- removed C79: 100nF, Capacitor:CAPACITOR-0603
- removed C80: 1uF, Capacitor:CAPACITOR-0603
- removed C81: 10uF, Capacitor:CAPACITOR-0603
- removed C82: 10uF, Capacitor:CAPACITOR-1206
- removed U10: ADP7142AUJZ-3.3, Analog Devices:ADP7142AUJZ-3.3
- removed U9: LT8636, Analog Devices:LT8636
- added C25: 100nF, Capacitor:CAPACITOR-0603
- added C27, C28: 10pF, Capacitor:CAPACITOR-0603
- added R43: 75K Ohms, Resistor:RESISTOR-0603
- added R44: 100K Ohms, Resistor:RESISTOR-0603
- added R45, R46: 1K Ohms, Resistor:RESISTOR-0603
- added U2: DSB321SDA, Crystal:DSB321SDA
- C30: value 10pF -> 100nF
- C31, C73: value 100nF -> 1uF
- C32: value 10pF -> 10nF
- C33: value 100nF -> 10nF
- C34: value 1uF -> 470pF
- C35, C36: value 10nF -> 100nF
- C37: value 470pF -> 4.7uF; VOLTAGE (none) -> 35V
- C38, C39: value 100nF -> 4.7pF
- C40: value 4.7uF -> 1uF; VOLTAGE 35V -> 50V
- C41, C42: value 4.7pF -> 22uF; device Capacitor:CAPACITOR-0603 -> Capacitor:CAPACITOR-1206; VOLTAGE (none) -> 25V
- C43, C54: value 1uF -> 22uF; device Capacitor:CAPACITOR-0603 -> Capacitor:CAPACITOR-1206; VOLTAGE 50V -> 25V
- C45, C46, C47, C55, C56: value 22uF -> 100nF; device Capacitor:CAPACITOR-1206 -> Capacitor:CAPACITOR-0603; VOLTAGE 25V -> (none)
- C48, C74: value 100nF -> 10uF
- C51: value 10uF -> 22uF; device Capacitor:CAPACITOR-0603 -> Capacitor:CAPACITOR-1206; VOLTAGE (none) -> 25V
- C52, C53: value 100nF -> 22uF; device Capacitor:CAPACITOR-0603 -> Capacitor:CAPACITOR-1206; VOLTAGE (none) -> 25V
- C57: value 22uF -> 4.7uF; device Capacitor:CAPACITOR-1206 -> Capacitor:CAPACITOR-0603; VOLTAGE 25V -> 35V
- C58: value 22uF -> 4.7uF; device Capacitor:CAPACITOR-1206 -> Capacitor:CAPACITOR-0603; VOLTAGE 25V -> (none)
- C59, C60: value 100nF -> 470pF
- C61: value 10uF -> 1uF; VOLTAGE (none) -> 50V
- C62: value 100nF -> 1uF; VOLTAGE (none) -> 50V
- C63: VOLTAGE 50V -> (none)
- C64: value 4.7uF -> 10nF; VOLTAGE 35V -> (none)
- C65: value 4.7uF -> 470pF
- C66, C67, C72: value 470pF -> 100nF
- C68: value 1uF -> 10pF; VOLTAGE 50V -> (none)
- C69: value 1uF -> 470pF; VOLTAGE 50V -> (none)
- C70: value 1uF -> 100uF; device Capacitor:CAPACITOR-0603 -> Capacitor:CAPACITOR-1206
- C71: value 10nF -> 100uF; device Capacitor:CAPACITOR-0603 -> Capacitor:CAPACITOR-1206
- C75: value 10pF -> 10uF; device Capacitor:CAPACITOR-0603 -> Capacitor:CAPACITOR-1206; VOLTAGE (none) -> 50V
- R16: value 100K Ohms -> 0 Ohms
- R18: value 15K Ohms -> 100K Ohms
- R19: value 100K Ohms -> 15K Ohms
- R21: value 1K Ohms -> 100K Ohms
- R22: value 1M Ohms -> 1K Ohms
- R23: value DNP -> 191K Ohms
- R24: value 40.2K Ohms -> 191K Ohms
- R26: value DNP -> 51K Ohms
- R27: value 40.2K Ohms -> 1M Ohms
- R28: value 2.5K Ohms -> 51K Ohms
- R30: value 100K Ohms -> 2.5K Ohms
- R31: value 10K Ohms -> 100K Ohms
- R32: value 90.9K Ohms -> 10K Ohms
- R33, R38: value 12K Ohms -> 90.9K Ohms
- R34: value 41.2K Ohms -> 12K Ohms
- R35: value 309K Ohms -> 41.2K Ohms
- R36: value 71.5K Ohms -> 309K Ohms
- R37: value 90.9K Ohms -> 71.5K Ohms
- R39: value 1M Ohms -> 12K Ohms
- R4, R5: value 100 Ohms -> 0 Ohms
- R40: value 226K Ohms -> 1M Ohms
- R41: value 510 Ohms -> 226K Ohms
- R42: value 0 Ohms -> 510 Ohms
- U1: value EFM32PG1B100F256GM32 -> EFM32TG11B120F128GM32; device EFM32:EFM32PG1B100F256GM32 -> EFM32:EFM32TG11B120F128GM32
- U3: value DSB321SDA -> SI5351C-B-GM; device Crystal:DSB321SDA -> Silicon Labs:SI5351C-B-GM
- U4: value SI5351C-B-GM -> LT8650S-1; device Silicon Labs:SI5351C-B-GM -> Analog Devices:LT8650S-1
- U5: value LT8650S-1 -> MCP4728-A2; device Analog Devices:LT8650S-1 -> Microchip:MCP4728-A2
- U6: value AD5272-100 -> MIC23155; device Analog Devices:AD5272-100 -> Microchip:MIC23155
- U7: value AD5272-100 -> LT8636; device Analog Devices:AD5272-100 -> Analog Devices:LT8636
- U8: value MIC23155 -> ADP7142AUJZ-3.3; device Microchip:MIC23155 -> Analog Devices:ADP7142AUJZ-3.3
Connections:
- removed net I2C_SCL: R3.1, U1.PC10, U4.SCL, U6.SCL, U7.SCL
- removed net I2C_SDA: R2.1, U1.PC9, U4.SDA, U6.SDA, U7.SDA
- removed net N$39: C54.C1, U6.EXT_CAP
- removed net N$40: C63.C1, U7.EXT_CAP
- removed net UART_RX: R4.2, U1.PF3
- removed net UART_TX: R5.2, U1.PF4
- removed net VBIAS1_FB_DIV: R23.1, R24.2, U6.W
- removed net VBIAS2_FB_DIV: R26.1, R27.2, U7.W
- new net 5V0_VSENSE: C76.C1, R43.2, R44.1, U1.PB13
- new net I2C0_SCL: R46.1, R5.2, U1.PD7
- new net I2C0_SDA: R4.2, R45.1, U1.PD6
- new net I2C1_SCL: R3.1, U1.PD5, U3.SCL, U5.SCL
- new net I2C1_SDA: R2.1, U1.PD4, U3.SDA, U5.SDA
- new net VBIAS1_VADJ: R23.2, U5.VOUTA
- new net VBIAS2_VADJ: R24.2, U5.VOUTB
- net !REF_SYNTH_OE: now also U1.PC14, U3.!OE; no longer U1.PC11, U4.!OE
- net 3V3: now also C48.C1, C50.C1, C66.C1, C70.C1, R21.2, R36.2, R45.2, R46.2, U1.IOVDD0@1, U1.IOVDD0@2, U5.!LDAC, U5.VDD, U6.SNS; no longer C73.C1, C77.C1, R19.2, R35.2, U8.SNS
- net 3V3_FB: now also R36.1, R37.2, U6.FB; no longer R35.1, R36.2, U8.FB
- net 3V3_REF_CLEAN: now also C25.C1, C30.C1, C74.C1, U2.VDD, U3.VDDOA, U3.VDDOB, U3.VDDOC, U3.VDDOD, U8.SENSE/ADJ, U8.VOUT; no longer C31.C1, C33.C1, C81.C1, U10.SENSE/ADJ, U10.VOUT, U4.VDD, U4.VDDOA, U4.VDDOB, U4.VDDOC, U4.VDDOD
- net 3V3_SOFTSTART: now also C60.C1, U6.SS; no longer C67.C1, U8.SS
- net 3V3_SW: now also U6.SW; no longer U8.SW
- net 5V0: now also C58.C1, C68.C1, C71.C1, C72.C1, C73.C1, R40.2, R42.2, R44.2, U4.CNTRL.BIAS, U6.EN, U6.VIN@0, U6.VIN@1, U7.BIAS, U8.VIN; no longer C51.C1, C53.C1, C61.C1, C62.C1, C65.C1, C75.C1, C78.C1, C79.C1, C80.C1, R39.2, R41.2, U10.EN, U10.VIN, U5.CNTRL.BIAS, U6.!RESET, U6.ADDR, U6.VDD, U7.!RESET, U7.VDD, U8.VIN@0, U8.VIN@1, U9.BIAS
- net 5V0_BST: now also C67.C2, U7.BST; no longer C74.C2, U9.BST
- net 5V0_FB: now also C68.C2, R40.1, R41.2, U7.FB; no longer C75.C2, R39.1, R40.2, U9.FB
- net 5V0_INTVCC: now also C63.C1, U7.INTVCC, U7.SYNC/MODE; no longer C70.C1, U9.INTVCC, U9.SYNC/MODE
- net 5V0_RT: now also R35.2, U7.RT; no longer R34.2, U9.RT
- net 5V0_SS: now also C64.C1, U7.TR/SS; no longer C71.C1, U9.TR/SS
- net 5V0_SW: now also C67.C1, U7.SW; no longer C74.C1, U9.SW
- net BIAS_REG_TEMP: now also C34.C1, R22.1, U1.PA0; no longer C37.C1, R21.1, U1.PB11
- net EXT_REF_IN: now also R13.2, RFCON5.SIGNAL; no longer R42.2, RFCON6.SIGNAL
- net EXT_REF_OUT: now also R16.1, RFCON6.SIGNAL; no longer R15.1, RFCON5.SIGNAL
- net GND: now also C25.C2, C27.C2, C32.C2, C41.C2, C42.C2, C74.C2, C75.C2, R19.1, R26.1, R28.1, R32.1, R35.1, R37.1, R39.1, R41.1, R43.1, U2.GND, U4.1.GND, U4.2.GND, U4.CNTRL.GND, U5.VSS, U6.AGND, U6.PGND@0, U6.PGND@1, U8.GND; no longer C35.C2, C36.C2, C67.C2, C68.C2, C77.C2, C78.C2, C79.C2, C80.C2, C81.C2, C82.C2, R16.1, R24.1, R27.1, R31.1, R33.1, R36.1, R38.1, R40.1, U10.GND, U4.GND, U5.1.GND, U5.2.GND, U5.CNTRL.GND, U6.GND, U6.VSS, U7.ADDR, U7.VSS, U8.AGND, U8.PGND@0, U8.PGND@1, U9.GND
- net LED: now also U1.PC1; no longer U1.PC8
- net N$1: now also R16.2, U3.CLK7; no longer R15.2, U4.CLK7
- net N$11: now also R29.1; no longer R28.1
- net N$149: now also R42.1; no longer R41.1
- net N$2: now also R15.2, U3.CLK5; no longer R14.2, U4.CLK5
- net N$23: now also R30.1; no longer R29.1
- net N$3: now also R19.2, U4.CNTRL.RT; no longer R18.2, U5.CNTRL.RT
- net N$36: now also C28.C2, U3.XA; no longer C32.C2, U4.XA
- net N$37: now also R13.1, U3.CLKIN; no longer R42.1, U4.CLKIN
- net N$5: now also R14.2, U3.CLK1; no longer R13.2, U4.CLK1
- net N$7: now also C27.C1, C28.C1, U2.CLK; no longer C30.C1, C32.C1, U3.CLK
- net N$8: now also R22.2, U4.CNTRL.TEMP; no longer R21.2, U5.CNTRL.TEMP
- net REF1: now also R14.1; no longer R13.1
- net REF2: now also R15.1; no longer R14.1
- net VBIAS1: now also C51.C1, C53.C1, R29.2, R33.2; no longer C57.C1, C59.C1, R28.2, R32.2
- net VBIAS1_BST: now also C35.C2, U4.2.BST; no longer C38.C2, U5.2.BST
- net VBIAS1_EN: now also R17.2, U1.PE12, U4.2.EN/UV; no longer R16.2, U1.PD15, U5.2.EN/UV
- net VBIAS1_FB: now also C38.C2, R23.1, R25.1, R26.2, U4.2.FB; no longer C41.C2, R22.1, R23.2, U5.2.FB, U6.A
- net VBIAS1_PG: now also R20.1, U1.PE10, U4.2.PG; no longer R19.1, U1.PA1, U5.2.PG
- net VBIAS1_SS: now also C32.C1, U4.2.SS; no longer C35.C1, U5.2.SS
- net VBIAS1_SW: now also C35.C1, U4.2.SW; no longer C38.C1, U5.2.SW
- net VBIAS1_UNFUSED: now also C38.C1, C43.C1, C45.C1, C47.C1, R25.2; no longer C44.C1, C46.C1, C48.C1, C50.C1, R22.2
- net VBIAS1_VSENSE: now also C65.C1, R33.1, R34.2, U1.PA1; no longer C72.C1, R32.1, R33.2, U1.PB12
- net VBIAS2: now also C52.C1, C54.C1, R30.2, R38.2; no longer C58.C1, C60.C1, R29.2, R37.2
- net VBIAS2_BST: now also C36.C2, U4.1.BST; no longer C39.C2, U5.1.BST
- net VBIAS2_EN: now also R18.2, U1.PE13, U4.1.EN/UV; no longer R17.2, U1.PD14, U5.1.EN/UV
- net VBIAS2_FB: now also C39.C2, R24.1, R27.1, R28.2, U4.1.FB; no longer C42.C2, R25.1, R26.2, U5.1.FB, U7.A
- net VBIAS2_PG: now also R21.1, U1.PE11, U4.1.PG; no longer R20.1, U1.PA0, U5.1.PG
- net VBIAS2_SS: now also C33.C1, U4.1.SS; no longer C36.C1, U5.1.SS
- net VBIAS2_SW: now also C36.C1, U4.1.SW; no longer C39.C1, U5.1.SW
- net VBIAS2_UNFUSED: now also C39.C1, C44.C1, C46.C1, R27.2; no longer C45.C1, C47.C1, C52.C1, R25.2
- net VBIAS2_VSENSE: now also C69.C1, R38.1, R39.2, U1.PA2; no longer C76.C1, R37.1, R38.2, U1.PB13
- net VBIAS_VCC: now also C31.C1, U4.1.VC, U4.2.VC, U4.CNTRL.SYNC, U4.CNTRL.VCC; no longer C34.C1, U5.1.VC, U5.2.VC, U5.CNTRL.SYNC, U5.CNTRL.VCC
- net VIN: now also C37.C1, C57.C1, C61.C1, C62.C1, C75.C1, R31.2, U4.1.VIN, U4.2.VIN, U7.EN/UV, U7.VIN; no longer C43.C1, C64.C1, C68.C1, C69.C1, C82.C1, R30.2, U5.1.VIN, U5.2.VIN, U9.EN/UV, U9.VIN
- net VIN_VSENSE: now also C59.C1, R31.1, R32.2; no longer C66.C1, R30.1, R31.2
Other:
- note added: "I2C Address 0x62"
- note added: "Vadj = -0.191 * Vout + 3.94887 Vout = -5.2356 * Vadj + 20.67475"
- note removed: "I2C Address 0x2C"
- note removed: "I2C Address 0x2F"
- note removed: "Vout = ((R4/(R3+R6)) + 1) * 0.8"
- moved on the sheet: C26, C29, C30, C34, C35, C36, C37, C38, C39, C40, C41, C42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

Commit message: Work on PCBs
Parts:
- R29, R30: value 2.5K Ohms -> 2.55K Ohms
Changed lines of the file:
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@@
 <part name="R39" library="Resistor" deviceset="RESISTOR" device="-0603" value="12K Ohms"/>
 <part name="R38" library="Resistor" deviceset="RESISTOR" device="-0603" value="90.9K Ohms"/>
-<part name="R29" library="Resistor" deviceset="RESISTOR" device="-0603" value="2.5K Ohms"/>
+<part name="R29" library="Resistor" deviceset="RESISTOR" device="-0603" value="2.55K Ohms"/>
 <part name="D2" library="LED" deviceset="LED" device="0603">
 <attribute name="COLOR" value="RED"/>
 </part>
 <part name="GND53" library="Supply Symbol" deviceset="GND" device=""/>
-<part name="R30" library="Resistor" deviceset="RESISTOR" device="-0603" value="2.5K Ohms"/>
+<part name="R30" library="Resistor" deviceset="RESISTOR" device="-0603" value="2.55K Ohms"/>
 <part name="D3" library="LED" deviceset="LED" device="0603">
 <attribute name="COLOR" value="RED"/>
