File: pcb/upconverter/qo-100-upconverter.sch (EAGLE design)
At the start: 171 parts, among them CON1 3P-SH-SIDE, CON2 2EDG-2P-5MM, U1 EFM32PG1B100F256GM32, U10 MIC23155, U11 LT8636, U12 MCP3421-A0, U13 MCP6C02-020, U14 ADP7142AUJZ-3.3, U15 ADP7142AUJZ-3.3, U16 ADP3334, U17 ADM7171ACPZ-5.0, U2 DSB321SDA, U3 ADF4351, U4 F1951NBGI, U5 MAX2671, U6 2450BP15E0100, U7 F1478NLGA, U8 F1951NBGI, U9 ADL5606

Commit message: Finish routing Upconverter PCB
Parts:
- added C7: 15pF, Capacitor:CAPACITOR-0603
- C39: value 100nF -> 10pF
- C56: value 3.3F -> 3.3pF
- R17, R23: value 100K Ohms -> 1K Ohms
- R28: value 100K Ohms -> 75K Ohms
- R33: value 226K Ohms -> 221K Ohms
- R4, R5: value 100 Ohms -> 0 Ohms
- U1: value EFM32PG1B100F256GM32 -> EFM32TG11B120F128GM32; device EFM32:EFM32PG1B100F256GM32 -> EFM32:EFM32TG11B120F128GM32
Connections:
- removed net !IF_ATT_RST: R17.2, U1.PF4, U4.!RST
- removed net !RF_ATT_RST: R23.2, U1.PA1, U8.!RST
- removed net 3V3_MIXER_CLEAN: C26.C1, C28.C1, C29.C1, C31.C1, C32.C1, C82.C1, L5.2, U14.SENSE/ADJ, U14.VOUT, U4.VDD, U5.VCC
- removed net I2C_SCL: R2.1, U1.PC7, U12.SCL
- removed net I2C_SDA: R3.1, U1.PC8, U12.SDA
- removed net UART_RX: R4.2, U1.PC10
- removed net UART_TX: R5.2, U1.PC11
- new net 3V3_ATT_MIXER_CLEAN: C26.C1, C28.C1, C29.C1, C31.C1, C32.C1, C45.C1, C7.C1, C82.C1, L5.2, U14.SENSE/ADJ, U14.VOUT, U4.VDD, U5.VCC, U8.VDD
- new net I2C0_SCL: R17.1, R5.2, U1.PD7
- new net I2C0_SDA: R23.1, R4.2, U1.PD6
- new net I2C1_SCL: R2.1, U1.PD5, U12.SCL
- new net I2C1_SDA: R3.1, U1.PD4, U12.SDA
- net !IF_ATT_CS: now also U1.PC13; no longer U1.PF3
- net !MIXER_SHDN: now also U1.PC14; no longer U1.PD9
- net !PA_STG1_BIAS_EN: now also U1.PA2; no longer U1.PB12
- net !PLL_MUTE: now also U1.PE13; no longer U1.PD15
- net !RF_ATT_CS: now also U1.PA1; no longer U1.PA0
- net 3V3: now also R17.2, R23.2, U1.IOVDD0@1, U1.IOVDD0@2
- net 5V0_PA_STG1_CLEAN: no longer C45.C1, U8.VDD
- net 5V0_VSENSE: now also U1.PB13; no longer U1.PB14
- net GND: now also C7.C2; no longer R17.1, R23.1
- net LED: now also U1.PB7; no longer U1.PC9
- net PA_STG2_BIAS_EN: now also U1.PC0; no longer U1.PB13
- net PLL_EN: now also U1.PC15; no longer U1.PD10
- net PLL_LE: now also U1.PA0; no longer U1.PD11
- net PLL_MUXOUT: now also U1.PE11; no longer U1.PD14
- net SPI_MOSI: now also U1.PE10; no longer U1.PD12
- net SPI_SCK: now also U1.PE12; no longer U1.PD13
- net VIN_VSENSE: now also U1.PB14; no longer U1.PB15
Other:
- note added: "Kelvin connection to R36"
- note removed: "Kelvin connection to R33"
- moved on the sheet: C45, R2, R3, U1
