File: pcb/upconverter/qo-100-upconverter.sch (EAGLE design)
At the start: 227 parts, among them CON1 3P-SH-SIDE, CON2 2EDG-2P-5MM, U1 EFM32TG11B120F128GM32, U10 LTC5597, U11 2450BP15E0100, U12 MCP6V31, U13 DC2337J5010AHF, U14 ADL5606, U15 F1958NBGK, U16 MCP1700-330, U17 LT8636, U18 MCP3421-A0, U19 MCP6C02-020, U2 DSB321SDA, U20 ADP7142AUJZ-3.3, U21 ADP7142AUJZ-3.3, U22 ADP7142AUJZ-3.3, U23 ADM7171ACPZ-5.0, U24 ADM7171ACPZ-5.0, U3 ADF4351, U4 F1958NBGK, U5 MAX2671, U6 2450BP15E0100, U7 F1958NBGK, U8 ADL5601, U9 F1490NLGA

Commit message: Add upconverter power tree
Other:
- note added: "ADM7171 5.0V @ 1A"
- note added: "ADP150/ADP7142 3.3V @ 150mA"
- note added: "Analog Rail 1st and 2nd RF Amplifiers"
- note added: "Analog Rail Final RF Amplifier"
- note added: "Analog Rail IF Attenuator, Mixer"
- note added: "Analog Rail LO Synthesizer"
- note added: "Analog Rail RF Attenuators, Power detector"
- note added: "Current sensing"
- note added: "Digital Rail MCU, ADC, ..."
- note added: "LT8636 5.2V @ 3A"
- note added: "MCP1700 3.3V @ 200mA"
- note added: "VIN 7 to 24V"
Changed lines of the file:
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@@
 <?xml version="1.0" encoding="utf-8"?>
 <!DOCTYPE eagle SYSTEM "eagle.dtd">
-<eagle version="9.6.1">
+<eagle version="9.6.2">
 <drawing>
 <settings>
@@
 <layer number="155" name="FabDoc3" color="7" fill="15" visible="no" active="no"/>
 <layer number="160" name="O_Dim" color="7" fill="1" visible="yes" active="yes"/>
+<layer number="166" name="AntennaArea" color="7" fill="1" visible="yes" active="yes"/>
+<layer number="168" name="4mmHeightArea" color="7" fill="1" visible="yes" active="yes"/>
 <layer number="191" name="mNets" color="7" fill="1" visible="yes" active="yes"/>
 <layer number="192" name="mBusses" color="7" fill="1" visible="yes" active="yes"/>
@@
 <part name="GND8" library="Supply Symbol" deviceset="GND" device=""/>
 <part name="GND1" library="Supply Symbol" deviceset="GND" device=""/>
+<part name="FRAME7" library="Frame" deviceset="A2-LANDSCAPE" device=""/>
 </parts>
 <sheets>
@@
 </nets>
 </sheet>
+<sheet>
+<description>Power tree</description>
+<plain>
+<wire x1="271.78" y1="200.66" x2="297.18" y2="200.66" width="0.1524" layer="97"/>
+<wire x1="271.78" y1="210.82" x2="271.78" y2="200.66" width="0.1524" layer="97"/>
+<text x="284.48" y="205.74" size="1.778" layer="97" align="center">ADP150/ADP7142
+3.3V @ 150mA</text>
+<wire x1="271.78" y1="210.82" x2="297.18" y2="210.82" width="0.1524" layer="97"/>
+<wire x1="297.18" y1="210.82" x2="297.18" y2="200.66" width="0.1524" layer="97"/>
+<wire x1="259.08" y1="205.74" x2="271.78" y2="205.74" width="0.1524" layer="97"/>
+<wire x1="264.16" y1="203.2" x2="266.7" y2="205.74" width="0.1524" layer="97"/>
+<wire x1="266.7" y1="205.74" x2="264.16" y2="208.28" width="0.1524" layer="97"/>
+<wire x1="297.18" y1="205.74" x2="309.88" y2="205.74" width="0.1524" layer="97"/>
+<wire x1="302.26" y1="203.2" x2="304.8" y2="205.74" width="0.1524" layer="97"/>
+<wire x1="304.8" y1="205.74" x2="302.26" y2="208.28" width="0.1524" layer="97"/>
+<wire x1="259.08" y1="231.14" x2="271.78" y2="231.14" width="0.1524" layer="97"/>
+<wire x1="264.16" y1="228.6" x2="266.7" y2="231.14" width="0.1524" layer="97"/>
+<wire x1="266.7" y1="231.14" x2="264.16" y2="233.68" width="0.1524" layer="97"/>
+<wire x1="180.34" y1="226.06" x2="205.74" y2="226.06" width="0.1524" layer="97"/>
+<wire x1="205.74" y1="226.06" x2="205.74" y2="231.14" width="0.1524" layer="97"/>
+<wire x1="205.74" y1="231.14" x2="205.74" y2="236.22" width="0.1524" layer="97"/>
+<wire x1="205.74" y1="236.22" x2="180.34" y2="236.22" width="0.1524" layer="97"/>
+<wire x1="180.34" y1="236.22" x2="180.34" y2="226.06" width="0.1524" layer="97"/>
+<text x="193.04" y="231.14" size="1.778" layer="97" align="center">VIN
+7 to 24V</text>
+<wire x1="205.74" y1="231.14" x2="213.36" y2="231.14" width="0.1524" layer="97"/>
+<wire x1="210.82" y1="228.6" x2="213.36" y2="231.14" width="0.1524" layer="97"/>
+<wire x1="213.36" y1="231.14" x2="210.82" y2="233.68" width="0.1524" layer="97"/>
+<wire x1="218.44" y1="231.14" x2="213.36" y2="231.14" width="0.1524" layer="97"/>
+<wire x1="218.44" y1="226.06" x2="243.84" y2="226.06" width="0.1524" layer="97"/>
+<wire x1="243.84" y1="226.06" x2="243.84" y2="236.22" width="0.1524" layer="97"/>
+<wire x1="243.84" y1="236.22" x2="218.44" y2="236.22" width="0.1524" layer="97"/>
+<wire x1="218.44" y1="236.22" x2="218.44" y2="226.06" width="0.1524" layer="97"/>
+<text x="231.14" y="231.14" size="1.778" layer="97" align="center">LT8636
+5.2V @ 3A</text>
+<wire x1="243.84" y1="231.14" x2="251.46" y2="231.14" width="0.1524" layer="97"/>
+<wire x1="248.92" y1="228.6" x2="251.46" y2="231.14" width="0.1524" layer="97"/>
+<wire x1="251.46" y1="231.14" x2="248.92" y2="233.68" width="0.1524" layer="97"/>
+<wire x1="271.78" y1="226.06" x2="297.18" y2="226.06" width="0.1524" layer="97"/>
+<wire x1="271.78" y1="236.22" x2="271.78" y2="226.06" width="0.1524" layer="97"/>
+<text x="284.48" y="231.14" size="1.778" layer="97" align="center">MCP1700
+3.3V @ 200mA</text>
+<wire x1="271.78" y1="236.22" x2="297.18" y2="236.22" width="0.1524" layer="97"/>
+<wire x1="297.18" y1="236.22" x2="297.18" y2="226.06" width="0.1524" layer="97"/>
+<wire x1="297.18" y1="231.14" x2="309.88" y2="231.14" width="0.1524" layer="97"/>
+<wire x1="302.26" y1="228.6" x2="304.8" y2="231.14" width="0.1524" layer="97"/>
+<wire x1="304.8" y1="231.14" x2="302.26" y2="233.68" width="0.1524" layer="97"/>
+<text x="312.42" y="231.14" size="1.778" layer="97" align="center-left">Digital Rail
+MCU, ADC, ...</text>
+<text x="312.42" y="205.74" size="1.778" layer="97" align="center-left">Analog Rail
+LO Synthesizer</text>
+<wire x1="271.78" y1="185.42" x2="297.18" y2="185.42" width="0.1524" layer="97"/>
+<wire x1="271.78" y1="195.58" x2="271.78" y2="185.42" width="0.1524" layer="97"/>
+<text x="284.48" y="190.5" size="1.778" layer="97" align="center">ADP150/ADP7142
+3.3V @ 150mA</text>
+<wire x1="271.78" y1="195.58" x2="297.18" y2="195.58" width="0.1524" layer="97"/>
+<wire x1="297.18" y1="195.58" x2="297.18" y2="185.42" width="0.1524" layer="97"/>
+<wire x1="259.08" y1="190.5" x2="271.78" y2="190.5" width="0.1524" layer="97"/>
+<wire x1="264.16" y1="187.96" x2="266.7" y2="190.5" width="0.1524" layer="97"/>
+<wire x1="266.7" y1="190.5" x2="264.16" y2="193.04" width="0.1524" layer="97"/>
+<wire x1="297.18" y1="190.5" x2="309.88" y2="190.5" width="0.1524" layer="97"/>
+<wire x1="302.26" y1="187.96" x2="304.8" y2="190.5" width="0.1524" layer="97"/>
+<wire x1="304.8" y1="190.5" x2="302.26" y2="193.04" width="0.1524" layer="97"/>
+<text x="312.42" y="190.5" size="1.778" layer="97" align="center-left">Analog Rail
+RF Attenuators, Power detector</text>
+<wire x1="259.08" y1="175.26" x2="271.78" y2="175.26" width="0.1524" layer="97"/>
+<wire x1="264.16" y1="172.72" x2="266.7" y2="175.26" width="0.1524" layer="97"/>
+<wire x1="266.7" y1="175.26" x2="264.16" y2="177.8" width="0.1524" layer="97"/>
+<wire x1="271.78" y1="170.18" x2="297.18" y2="170.18" width="0.1524" layer="97"/>
+<wire x1="271.78" y1="180.34" x2="271.78" y2="170.18" width="0.1524" layer="97"/>
+<text x="284.48" y="175.26" size="1.778" layer="97" align="center">ADP150/ADP7142
+3.3V @ 150mA</text>
+<wire x1="271.78" y1="180.34" x2="297.18" y2="180.34" width="0.1524" layer="97"/>
+<wire x1="297.18" y1="180.34" x2="297.18" y2="170.18" width="0.1524" layer="97"/>
+<wire x1="297.18" y1="175.26" x2="309.88" y2="175.26" width="0.1524" layer="97"/>
+<wire x1="302.26" y1="172.72" x2="304.8" y2="175.26" width="0.1524" layer="97"/>
+<wire x1="304.8" y1="175.26" x2="302.26" y2="177.8" width="0.1524" layer="97"/>
+<text x="312.42" y="175.26" size="1.778" layer="97" align="center-left">Analog Rail
+IF Attenuator, Mixer</text>
+<wire x1="259.08" y1="160.02" x2="271.78" y2="160.02" width="0.1524" layer="97"/>
+<wire x1="264.16" y1="157.48" x2="266.7" y2="160.02" width="0.1524" layer="97"/>
+<wire x1="266.7" y1="160.02" x2="264.16" y2="162.56" width="0.1524" layer="97"/>
+<wire x1="271.78" y1="154.94" x2="297.18" y2="154.94" width="0.1524" layer="97"/>
+<wire x1="271.78" y1="165.1" x2="271.78" y2="154.94" width="0.1524" layer="97"/>
+<text x="284.48" y="160.02" size="1.778" layer="97" align="center">ADM7171
+5.0V @ 1A</text>
+<wire x1="271.78" y1="165.1" x2="297.18" y2="165.1" width="0.1524" layer="97"/>
+<wire x1="297.18" y1="165.1" x2="297.18" y2="154.94" width="0.1524" layer="97"/>
+<wire x1="297.18" y1="160.02" x2="309.88" y2="160.02" width="0.1524" layer="97"/>
+<wire x1="302.26" y1="157.48" x2="304.8" y2="160.02" width="0.1524" layer="97"/>
+<wire x1="304.8" y1="160.02" x2="302.26" y2="162.56" width="0.1524" layer="97"/>
+<text x="312.42" y="160.02" size="1.778" layer="97" align="center-left">Analog Rail
+1st and 2nd RF Amplifiers</text>
+<wire x1="259.08" y1="144.78" x2="271.78" y2="144.78" width="0.1524" layer="97"/>
+<wire x1="264.16" y1="142.24" x2="266.7" y2="144.78" width="0.1524" layer="97"/>
+<wire x1="266.7" y1="144.78" x2="264.16" y2="147.32" width="0.1524" layer="97"/>
+<wire x1="271.78" y1="139.7" x2="297.18" y2="139.7" width="0.1524" layer="97"/>
+<wire x1="271.78" y1="149.86" x2="271.78" y2="139.7" width="0.1524" layer="97"/>
+<text x="284.48" y="144.78" size="1.778" layer="97" align="center">ADM7171
+5.0V @ 1A</text>
+<wire x1="271.78" y1="149.86" x2="297.18" y2="149.86" width="0.1524" layer="97"/>
+<wire x1="297.18" y1="149.86" x2="297.18" y2="139.7" width="0.1524" layer="97"/>
+<wire x1="297.18" y1="144.78" x2="309.88" y2="144.78" width="0.1524" layer="97"/>
+<wire x1="302.26" y1="142.24" x2="304.8" y2="144.78" width="0.1524" layer="97"/>
+<wire x1="304.8" y1="144.78" x2="302.26" y2="147.32" width="0.1524" layer="97"/>
+<text x="312.42" y="144.78" size="1.778" layer="97" align="center-left">Analog Rail
+Final RF Amplifier</text>
+<wire x1="259.08" y1="231.14" x2="259.08" y2="144.78" width="0.1524" layer="97"/>
+<wire x1="251.46" y1="231.14" x2="259.08" y2="231.14" width="0.1524" layer="97"/>
+<circle x="259.08" y="218.44" radius="2.54" width="0.1524" layer="97"/>
+<wire x1="256.54" y1="218.44" x2="246.38" y2="218.44" width="0.1524" layer="97"/>
+<text x="238.76" y="218.44" size="1.778" layer="97" align="center">Current
+sensing</text>
+</plain>
+<instances>
+<instance part="FRAME7" gate="G$1" x="0" y="0" smashed="yes">
+<attribute name="DRAWING_NAME" x="447.04" y="20.574" size="2.54" layer="94" font="vector"/>
+<attribute name="LAST_DATE_TIME" x="458.47" y="5.334" size="2.286" layer="94" font="vector"/>
+<attribute name="SHEET" x="458.47" y="10.414" size="2.54" layer="94" font="vector"/>
+<attribute name="CNAME" x="447.04" y="25.654" size="2.54" layer="94" font="vector"/>
+<attribute name="DESIGNER" x="447.04" y="15.494" size="2.54" layer="94" font="vector"/>
+<attribute name="CREVISION" x="500.35" y="5.234" size="2.54" layer="94" font="vector"/>
+<attribute name="SHEET_HEADLINE" x="491.69" y="10.414" size="2.54" layer="94" font="vector"/>
+</instance>
+</instances>
+<busses>
+</busses>
+<nets>
+</nets>
+</sheet>

Commit message: Change wrong resistor name in upconverter schematic
Signed-off-by: João Silva <jgc3silva@gmail.com>
Other:
- note added: "Kelvin connection to R50"
- note removed: "Kelvin connection to R36"
Changed lines of the file:
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@@
 <text x="203.962" y="300.482" size="1.27" layer="98" rot="R180">Vout = ((R24/R25) + 1) * 0.97</text>
 <text x="173.482" y="186.182" size="1.27" layer="98" rot="R180">Kelvin connection
-to R36</text>
+to R50</text>
 </plain>
 <instances>

Commit message: Upconverter: Changed final amplifier to SKY66292-11 Upconverter: Added Pi attenuator before final amplifier Upconverter: Removed GND exposed pads below PLL VTUNE Upconverter: Added temperature sensor near final amplifier Upconverter: Exposed bottom layer copper for heat sinking
Signed-off-by: João Silva <jgc3silva@gmail.com>
Parts:
- removed C100, C101: 10uF, Capacitor:CAPACITOR-0603
- removed C102, C103: 1nF, Capacitor:CAPACITOR-0603
- removed C104: 10uF, Capacitor:CAPACITOR-1206
- removed L20: 4.7uH, Inductor:INDUCTOR-6X6MM
- removed TP1, TP2, TP3, TP4, TP5, TP6: TESTPOINT-1.27MM, PADs:TESTPOINT-1.27MM
- added R54: 10K Ohms, Resistor:RESISTOR-0603
- added R55: 0.03 Ohms, Resistor:RESISTOR-1206
- added R56, R57: 100K Ohms, Resistor:RESISTOR-0603
- added R58: 1K Ohms, Resistor:RESISTOR-0603
- added SJ1: SJCS, Solder Jumper:SJCS
- added U25: ADM7172ACPZ-5.0, Analog Devices:ADM7172ACPZ-5.0
- C59, C84: value 10uF -> 100uF; device Capacitor:CAPACITOR-0603 -> Capacitor:CAPACITOR-1206
- C60: value 10nF -> 10uF
- C61: value 15pF -> 10uF
- C63, C90: value 100uF -> 1uF; device Capacitor:CAPACITOR-1206 -> Capacitor:CAPACITOR-0603
- C64: value 100pF -> 10nF
- C65: value 2pF -> 10nF
- C66, C81: value 1uF -> 100nF
- C67: value 10nF -> 15pF
- C68: value 100pF -> 4.7uF; VOLTAGE (none) -> 35V
- C69: value 15pF -> 100nF
- C70: value 3.3pF -> 470pF
- C71: value 15pF -> 470pF
- C72: value 100nF -> 4.7uF
- C73: value 15pF -> 1uF; VOLTAGE (none) -> 50V
- C74: value 4.7uF -> 1uF; VOLTAGE 35V -> 50V
- C75, C83, C91, C92: value 100nF -> 1uF
- C76: value 470pF -> 10nF
- C77: value 470pF -> 100nF
- C78: value 4.7uF -> 10uF
- C79: value 1uF -> 10uF; VOLTAGE 50V -> (none)
- C80: value 1uF -> 100nF; VOLTAGE 50V -> (none)
- C82: value 10nF -> 10pF
- C85, C99: value 10uF -> 100nF
- C87: value 100nF -> 22uF; device Capacitor:CAPACITOR-0603 -> Capacitor:CAPACITOR-1206
- C88: value 10pF -> 1uF
- C93: value 22uF -> 10uF; device Capacitor:CAPACITOR-1206 -> Capacitor:CAPACITOR-0603
- C94, C95: value 1uF -> 10uF
- C96, C97: value 1uF -> 1nF
- C98: value 1uF -> 10uF; device Capacitor:CAPACITOR-0603 -> Capacitor:CAPACITOR-1206; VOLTAGE (none) -> 50V
- CON2: value 2EDG-2P-5MM -> 2EDG-2P-5MM-H; device Generic Connector:2EDG-2P-5MM -> Generic Connector:2EDG-2P-5MM-H
- L18: value 62nH -> 0 Ohms
- L19: value 0 Ohms -> 4.7uH; device Inductor:INDUCTOR-0603 -> Inductor:INDUCTOR-6X6MM; CURRENT (none) -> 3A; OCLCSC (none) -> C326336
- R29: value 0 Ohms -> DNP
- R38: value 100 Ohms -> 49.9 Ohms
- R39: value 49.9 Ohms -> 100 Ohms
- R40: value 510 Ohms -> 96.1 Ohms
- R41: value 100K Ohms -> 71.5 Ohms
- R42: value 10K Ohms -> 96.1 Ohms
- R43: value 100K Ohms -> 10K Ohms
- R44: value 75K Ohms -> 7.5K Ohms
- R45: value 41.2K Ohms -> 510 Ohms
- R46: value 1M Ohms -> 100K Ohms
- R47: value 221K Ohms -> 10K Ohms
- R48: value 10K Ohms -> 100K Ohms
- R49: value 10K Ohms -> 75K Ohms
- R50: value 0.03 Ohms -> 41.2K Ohms; device Resistor:RESISTOR-1206 -> Resistor:RESISTOR-0603; TOLERANCE 1% -> (none)
- R51: value 100K Ohms -> 1M Ohms
- R52: value 100K Ohms -> 221K Ohms
- R53: value 1K Ohms -> 10K Ohms
- U12: value MCP6V31 -> DC2337J5010AHF; device Microchip:MCP6V31 -> Anaren:DC2337J5010AHF; OCLCSC (none) -> C509396
- U13: value DC2337J5010AHF -> MCP6V31; device Anaren:DC2337J5010AHF -> Microchip:MCP6V31; OCLCSC C509396 -> (none)
- U14: value ADL5606 -> SKY66292-11; device Analog Devices:ADL5606 -> Skyworks:SKY66292-11
- U16: value MCP1700-330 -> MCP9802-A0; device Microchip:MCP1700-330 -> Microchip:MCP9802-A0
- U17: value LT8636 -> MCP1700-330; device Analog Devices:LT8636 -> Microchip:MCP1700-330
- U18: value MCP3421-A0 -> LT8636; device Microchip:MCP3421-A0 -> Analog Devices:LT8636
- U19: value MCP6C02-020 -> MCP3421-A0; device Microchip:MCP6C02-020 -> Microchip:MCP3421-A0
- U20: value ADP7142AUJZ-3.3 -> MCP6C02-020; device Analog Devices:ADP7142AUJZ-3.3 -> Microchip:MCP6C02-020
- U23: value ADM7171ACPZ-5.0 -> ADP7142AUJZ-3.3; device Analog Devices:ADM7171ACPZ-5.0 -> Analog Devices:ADP7142AUJZ-3.3
Connections:
- removed net N$5: C61.C2, C65.C1, U14.RFIN
- removed net RF_FINAL_DCC: C70.C1, C71.C1, L18.1, U14.RFOUT
- new net PA3_EN: R43.1, R44.2, SJ1.1, U14.PAEN
- new net PA_TEMP_ALERT: SJ1.2, U16.ALERT
- new net RF_PRE2_ATT_FLT_THRU_ACC_ATT: R41.1, R42.2, U14.RFIN
- net 3V3: now also C77.C1, C78.C1, C79.C1, C80.C1, C99.C1, U16.VDD, U17.VOUT, U19.VDD; no longer C83.C1, C84.C1, C85.C1, C86.C1, U16.VOUT, U18.VDD
- net 3V3_IF_ATT_MIXER_CLEAN: now also C93.C1, U21.SENSE/ADJ, U21.VOUT; no longer C99.C1, U20.SENSE/ADJ, U20.VOUT
- net 3V3_PLL_CLEAN: now also C95.C1, U23.SENSE/ADJ, U23.VOUT; no longer C101.C1, U22.SENSE/ADJ, U22.VOUT
- net 3V3_RF_ATT_PDET_CLEAN: now also C66.C1, C94.C1, U13.PWR.V+, U22.SENSE/ADJ, U22.VOUT; no longer C100.C1, C72.C1, U12.PWR.V+, U21.SENSE/ADJ, U21.VOUT
- net 5V0: now also C69.C1, C72.C1, C82.C1, C83.C1, C84.C1, C86.C1, L19.2, R48.2, R51.2, R55.2, R58.2, U17.VIN, U18.BIAS, U20.VDD, U20.VIP; no longer C75.C1, C78.C1, C88.C1, C89.C1, C90.C1, C92.C1, L20.2, R43.2, R46.2, R50.2, R53.2, U16.VIN, U17.BIAS, U19.VDD, U19.VIP
- net 5V0_BST: now also C81.C2, U18.BST; no longer C87.C2, U17.BST
- net 5V0_FB: now also C82.C2, R51.1, R52.2, U18.FB; no longer C88.C2, R46.1, R47.2, U17.FB
- net 5V0_INTVCC: now also C75.C1, U18.INTVCC, U18.SYNC/MODE; no longer C81.C1, U17.INTVCC, U17.SYNC/MODE
- net 5V0_ISENSE: now also C87.C1, C88.C1, C89.C1, C90.C1, C91.C1, C92.C1, R55.1, U20.VIM, U23.EN, U25.VIN; no longer C93.C1, C94.C1, C95.C1, C96.C1, C97.C1, C98.C1, R50.1, U19.VIM, U20.EN, U20.VIN
- net 5V0_ISENSE_VN: now also C85.C2, R54.1, U19.VIN-; no longer C91.C2, R49.1, U18.VIN-
- net 5V0_ISENSE_VP: now also C85.C1, R53.1, U19.VIN+; no longer C91.C1, R48.1, U18.VIN+
- net 5V0_PA_STG1_2_CLEAN: now also U24.SENSE, U24.VOUT; no longer U23.SENSE, U23.VOUT
- net 5V0_PA_STG3_CLEAN: now also C61.C1, C65.C1, R43.2, R45.2, U25.SENSE, U25.VOUT; no longer C66.C1, C67.C1, C68.C1, C69.C1, L18.2, R40.2, U24.SENSE, U24.VOUT
- net 5V0_RT: now also R50.2, U18.RT; no longer R45.2, U17.RT
- net 5V0_SS: now also C76.C1, U18.TR/SS; no longer C82.C1, U17.TR/SS
- net 5V0_SW: now also C81.C1, L19.1, U18.SW; no longer C87.C1, L20.1, U17.SW
- net 5V0_VSENSE: now also C71.C1, R48.1, R49.2; no longer C77.C1, R43.1, R44.2
- net GND: now also C61.C2, C71.C2, C73.C2, C87.C2, C88.C2, C91.C2, R38.1, R40.1, R49.1, R50.1, R54.2, R56.1, R57.1, U12.GND, U13.PWR.V-, U18.GND, U20.VREF, U20.VSS, U25.GND, U3.RFOUTB+, U3.RFOUTB-; no longer C100.C2, C101.C2, C102.C2, C103.C2, C104.C2, C67.C2, C81.C2, C82.C2, C85.C2, R39.1, R45.1, R49.2, R51.1, TP1.TP, TP2.TP, TP3.TP, TP4.TP, TP5.TP, TP6.TP, U12.PWR.V-, U13.GND, U14.DISABLE, U18.VSS, U19.VREF, U20.GND
- net I2C1_SCL: now also U16.SCL, U19.SCL; no longer U18.SCL
- net I2C1_SDA: now also U16.SDA, U19.SDA; no longer U18.SDA
- net N$10: now also R53.2, U20.VOUT; no longer R48.2, U19.VOUT
- net N$149: now also R58.1; no longer R53.1
- net N$2: now also C97.C1, U25.SS; no longer C103.C1, U24.SS
- net N$20: now also C96.C1, U24.SS; no longer C102.C1, U23.SS
- net N$3: now also R45.1; no longer R40.1
- net N$39: now also L18.2; no longer L19.2
- net N$42: now also R38.2, U12.ISOLATED; no longer R39.2, U13.ISOLATED
- net N$7: now also U13.1.-IN; no longer U12.1.-IN
- net PA_STG1_2_BIAS_EN: now also R56.2, U24.EN; no longer R51.2, U23.EN
- net PA_STG3_BIAS_EN: now also R57.2, U25.EN; no longer R52.2, U24.EN
- net RF_FINAL_ACC: now also U14.RFOUT; no longer C71.C2
- net RF_PRE2_ACC: now also L18.1; no longer L19.1
- net RF_PRE2_ATT_ACC: now also C67.C2; no longer C73.C2
- net RF_PRE2_ATT_DCC: now also C67.C1; no longer C73.C1
- net RF_PRE2_ATT_FLT_ACC: now also U12.IN; no longer U13.IN
- net RF_PRE2_ATT_FLT_CPL_ACC: now also U12.COUPLED; no longer U13.COUPLED
- net RF_PRE2_ATT_FLT_THRU_ACC: now also R40.2, R41.2, U12.OUT; no longer C61.C1, U13.OUT
- net VIN: now also C68.C1, C73.C1, C98.C1, R46.2, U18.EN/UV, U18.VIN; no longer C104.C1, C79.C1, C80.C1, R41.2, U17.EN/UV, U17.VIN
- net VIN_VSENSE: now also C70.C1, R46.1, R47.2; no longer C76.C1, R41.1, R42.2
- net VPDET_AMP: now also R39.2, U13.1.OUT; no longer R38.2, U12.1.OUT
- net VPDET_FLT: now also U13.1.+IN; no longer U12.1.+IN
- net VPDET_SENSE: now also R39.1; no longer R38.1
Other:
- note added: "+34 dB"
- note added: "-10 dB"
- note added: "Kelvin connection to R52"
- note added: "Vout = ((R48/R49) + 1) * 0.97"
- note removed: "+20 dB"
- note removed: "Kelvin connection to R50"
- note removed: "Vout = ((R24/R25) + 1) * 0.97"
- moved on the sheet: C59, C60, C61, C63, C64, C65, C66, C67, C74, C75, C76, C77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
