File: pcb/upconverter/qo-100-upconverter.sch (EAGLE design)
At the start: 215 parts, among them CON1 3P-SH-SIDE, CON2 2EDG-2P-5MM-H, U1 EFM32TG11B120F128GM32, U10 ADL5601, U11 F1490NLGA, U12 LTC5597, U13 2450BP15E0100, U14 DC2337J5010AHF, U15 MCP6V31, U16 MCP9802-A0, U17 SKY66292-11, U18 F1958NBGK, U19 MCP1700-330, U2 DSB321SDA, U20 LT8636, U22 MCP6C02-020, U23 ADP7142AUJZ-3.3, U24 ADP7142AUJZ-3.3, U25 ADP7142AUJZ-3.3, U26 ADM7171ACPZ-5.0, U27 ADM7172ACPZ-5.0, U3 ADF4351, U4 JSW2-63DR+, U5 2450BP15E0100, U6 F1958NBGK, U7 MAX2671, U8 2450BP15E0100, U9 F1958NBGK

Commit message: Update PLL Loop filter
Signed-off-by: João Silva <jgc3silva@gmail.com>
Parts:
- removed R53: 0.03 Ohms, Resistor:RESISTOR-1206
- removed R54, R55: 100K Ohms, Resistor:RESISTOR-0603
- removed R57, R58: 330 Ohms, Resistor:RESISTOR-0603
- added C100: 1nF, Capacitor:CAPACITOR-0603
- added C101: 10uF, Capacitor:CAPACITOR-1206
- added C81: 100nF, Capacitor:CAPACITOR-0603
- added R10: 100K Ohms, Resistor:RESISTOR-0603
- added SJ2: SJCS, Solder Jumper:SJCS
- added U21: LT8636, Analog Devices:LT8636
- C10, C12, C14, C16, C18, C44: value 10pF -> 100nF
- C13, C15, C17: value 100nF -> 10pF
- C19: value 0.7pF -> 10pF
- C20: value 0.7pF -> 100nF
- C21, C47: value 15pF -> 10pF
- C22: value 20nF -> 0.7pF
- C23: value 1nF -> 0.7pF
- C24, C71: value 470pF -> 15pF
- C25: value 100nF -> 20nF
- C26: value 15pF -> 1nF
- C27: value 15pF -> 470pF
- C28, C46, C58, C84, C89: value 1uF -> 100nF
- C29, C30, C7, C8: value 100nF -> 15pF
- C31: value 100pF -> 1uF
- C32: value 47pF -> 100nF
- C33, C51, C68: value 15pF -> 100nF
- C35: value 220pF -> 47pF
- C36, C59: value 100uF -> 15pF; device Capacitor:CAPACITOR-1206 -> Capacitor:CAPACITOR-0603
- C37: value 1uF -> 100pF
- C38: value 100nF -> 220pF
- C39: value 1uF -> 100uF; device Capacitor:CAPACITOR-0603 -> Capacitor:CAPACITOR-1206
- C40, C49: value 33pF -> 1uF
- C42: value 0.8pF -> 1uF
- C43: value 100nF -> 33pF
- C45: value 47pF -> 0.8pF
- C48: value 100nF -> 47pF
- C52: value 22pF -> 33pF
- C53: value 0.7pF -> 15pF
- C54: value 4.7uF -> 15pF
- C55: value 100nF -> 22pF
- C56: value 15pF -> 0.7pF
- C57: value 10nF -> 4.7uF
- C60, C80: value 10uF -> 10nF
- C61, C79, C94, C95: value 10uF -> 1uF
- C62: value 10nF -> 100uF; device Capacitor:CAPACITOR-0603 -> Capacitor:CAPACITOR-1206
- C63: value 1uF -> 10uF
- C64: value 10nF -> 10uF
- C65, C67: value 100nF -> 10nF
- C66: value 10nF -> 1uF
- C69: value 4.7uF -> 10nF; VOLTAGE 35V -> (none)
- C72: value 470pF -> 4.7uF; VOLTAGE (none) -> 35V
- C73: value 4.7uF -> 100nF
- C74, C75: value 1uF -> 470pF; VOLTAGE 50V -> (none)
- C76: value 1uF -> 4.7uF
- C77: value 10nF -> 1uF; VOLTAGE (none) -> 50V
- C78: value 100nF -> 1uF; VOLTAGE (none) -> 50V
- C82: value 100nF -> 10uF
- C83: value 10pF -> 10uF
- C85: value 100uF -> 10pF; device Capacitor:CAPACITOR-1206 -> Capacitor:CAPACITOR-0603
- C86: value 100nF -> 1uF
- C87: value 100nF -> 100uF; device Capacitor:CAPACITOR-0603 -> Capacitor:CAPACITOR-1206
- C88: value 22uF -> 100nF; device Capacitor:CAPACITOR-1206 -> Capacitor:CAPACITOR-0603
- C90: value 1uF -> 22uF; device Capacitor:CAPACITOR-0603 -> Capacitor:CAPACITOR-1206
- C97, C98: value 1nF -> 10uF
- C99: value 10uF -> 1nF; device Capacitor:CAPACITOR-1206 -> Capacitor:CAPACITOR-0603; VOLTAGE 50V -> (none)
- D3, D4: COLOR RED -> BLUE
- D5: value SMAJ24A -> LED0603; device TVS:SMAJ24A -> LED:LED0603; COLOR (none) -> RED
- D6: COLOR GREEN -> RED
- D7: value LED0603 -> SMAJ24A; device LED:LED0603 -> TVS:SMAJ24A; COLOR BLUE -> (none)
- D8: COLOR BLUE -> GREEN
- R16: value 105 Ohms -> 4.7K Ohms
- R17: value 330 Ohms -> 1K Ohms
- R18: value 61.9 Ohms -> 330 Ohms
- R19: value 1K Ohms -> 330 Ohms
- R20: value 105 Ohms -> 10K Ohms
- R21: value 10K Ohms -> DNP
- R24, R31: value 0 Ohms -> 1K Ohms
- R27: value 1K Ohms -> 1.5K Ohms
- R28: value DNP -> 0 Ohms
- R29: value DNP -> 510 Ohms
- R30: value 1.5K Ohms -> 0 Ohms
- R32: value 510 Ohms -> 2K Ohms
- R33: value 0 Ohms -> 49.9 Ohms
- R34: value 1K Ohms -> 100 Ohms
- R35: value 2K Ohms -> 96.1 Ohms
- R36: value 49.9 Ohms -> 71.5 Ohms
- R37: value 100 Ohms -> 96.1 Ohms
- R38: value 96.1 Ohms -> 10K Ohms
- R39: value 71.5 Ohms -> 7.5K Ohms
- R40: value 96.1 Ohms -> 510 Ohms
- R41: value 10K Ohms -> 100K Ohms
- R42: value 7.5K Ohms -> 10K Ohms
- R43: value 510 Ohms -> 100K Ohms
- R44: value 100K Ohms -> 75K Ohms
- R45: value 10K Ohms -> 41.2K Ohms
- R46: value 100K Ohms -> 1M Ohms
- R47: value 75K Ohms -> 220K Ohms
- R48: value 41.2K Ohms -> 1K Ohms
- R49: value 1M Ohms -> 0.03 Ohms; device Resistor:RESISTOR-0603 -> Resistor:RESISTOR-1206; TOLERANCE (none) -> 1%
- R50: value 220K Ohms -> 100K Ohms
- R51: value 1K Ohms -> 100K Ohms
- R9: value 100K Ohms -> 10K Ohms
- RFCON2: value RFCON-SMA-EDGE -> RFCON-U.FL; device RF Connector:RFCON-SMA-EDGE -> RF Connector:RFCON-U.FL
- RFCON4: value RFCON-U.FL -> RFCON-SMA-EDGE; device RF Connector:RFCON-U.FL -> RF Connector:RFCON-SMA-EDGE
- SJ1: value SJCS -> (none); device Solder Jumper:SJCS -> Solder Jumper:SJ2S
- U10: value ADL5601 -> F1958NBGK; device Analog Devices:ADL5601 -> Renesas:F1958NBGK
- U11: value F1490NLGA -> ADL5601; device Renesas:F1490NLGA -> Analog Devices:ADL5601
- U12: value LTC5597 -> F1490NLGA; device Analog Devices:LTC5597 -> Renesas:F1490NLGA
- U13: value 2450BP15E0100 -> LTC5597; device Generic Filter:2450BP15E0100 -> Analog Devices:LTC5597
- U14: value DC2337J5010AHF -> 2450BP15E0100; device Anaren:DC2337J5010AHF -> Generic Filter:2450BP15E0100; OCLCSC C509396 -> (none)
- U15: value MCP6V31 -> DC2337J5010AHF; device Microchip:MCP6V31 -> Anaren:DC2337J5010AHF; OCLCSC (none) -> C509396
- U16: value MCP9802-A0 -> MCP6V31; device Microchip:MCP9802-A0 -> Microchip:MCP6V31
- U17: value SKY66292-11 -> MCP9802-A0; device Skyworks:SKY66292-11 -> Microchip:MCP9802-A0
- U18: value F1958NBGK -> SKY66292-11; device Renesas:F1958NBGK -> Skyworks:SKY66292-11
- U19: value MCP1700-330 -> F1958NBGK; device Microchip:MCP1700-330 -> Renesas:F1958NBGK
- U2: value DSB321SDA -> JSW2-63DR+; device Crystal:DSB321SDA -> Mini Circuits:JSW2-63DR+
- U20: value LT8636 -> MCP1700-330; device Analog Devices:LT8636 -> Microchip:MCP1700-330
- U3: value ADF4351 -> DSB321SDA; device Analog Devices:ADF4351 -> Crystal:DSB321SDA
- U4: value JSW2-63DR+ -> ADF4351; device Mini Circuits:JSW2-63DR+ -> Analog Devices:ADF4351
- U5: value 2450BP15E0100 -> JSW2-63DR+; device Generic Filter:2450BP15E0100 -> Mini Circuits:JSW2-63DR+
- U6, U9: value F1958NBGK -> 2450BP15E0100; device Renesas:F1958NBGK -> Generic Filter:2450BP15E0100
- U7: value MAX2671 -> F1958NBGK; device Maxim Integrated:MAX2671 -> Renesas:F1958NBGK
- U8: value 2450BP15E0100 -> MAX2671; device Generic Filter:2450BP15E0100 -> Maxim Integrated:MAX2671
- renumbered R56 to R52
Connections:
- removed net N$29: C21.C2, R16.2, R18.2
- removed net N$45: R22.2, U7.LO
- removed net N$47: R25.1, RFCON5.SIGNAL
- new net LO_OUT: C8.C1, RFCON1.SIGNAL
- new net LO_SW_CTL: R9.2, SJ1.2, U2.CONTROL
- new net N$10: C7.C1, U2.RF2
- new net N$14: C8.C2, U2.RF1
- new net SYNTH_OUT: C24.C2, U2.RFCOM
- net !MIXER_SHDN: now also R19.2, R20.2, U8.!SHDN; no longer R21.2, R57.2, U7.!SHDN
- net 3V3: now also C68.C1, C81.C1, C82.C1, C83.C1, SJ1.3, U17.VDD, U20.VOUT; no longer C65.C1, C78.C1, C79.C1, C80.C1, U16.VDD, U19.VOUT
- net 3V3_IF_ATT_MIXER_SW_CLEAN: now also C31.C1, C33.C1, C35.C1, C96.C1, U5.ENABLE, U5.VDD, U7.VDD, U7.VMODE, U8.VCC; no longer C25.C1, C29.C1, C30.C1, C94.C1, U4.ENABLE, U4.VDD, U6.VDD, U6.VMODE, U7.VCC
- net 3V3_PLL_CLEAN: now also C10.C1, C11.C1, C12.C1, C98.C1, U2.ENABLE, U3.VDD, U4.AVDD, U4.SDVDD, U4.VP, U4.VVCO@0, U4.VVCO@1; no longer C7.C1, C8.C1, C96.C1, U3.AVDD, U3.SDVDD, U3.VP, U3.VVCO@0, U3.VVCO@1
- net 3V3_RF_ATT_PDET_CLEAN: now also C44.C1, C57.C1, C58.C1, C70.C1, C97.C1, U10.VDD, U10.VMODE, U13.EN, U13.VCC, U16.PWR.V+, U19.VDD, U19.VMODE; no longer C41.C1, C54.C1, C55.C1, C67.C1, C95.C1, U12.EN, U12.VCC, U15.PWR.V+, U18.VDD, U18.VMODE, U9.VDD, U9.VMODE
- net 5V0: now also C76.C1, C86.C1, C88.C1, R43.2, U20.VIN, U21.BIAS; no longer C70.C1, C83.C1, C84.C1, R53.2, U19.VIN, U20.BIAS
- net 5V0_BST: now also C84.C2, U21.BST; no longer C82.C2, U20.BST
- net 5V0_FB: now also C85.C2, R46.1, R47.2, U21.FB; no longer C83.C2, R49.1, R50.2, U20.FB
- net 5V0_INTVCC: now also C79.C1, U21.INTVCC, U21.SYNC/MODE; no longer C76.C1, U20.INTVCC, U20.SYNC/MODE
- net 5V0_ISENSE: now also C94.C1, C95.C1, R49.1; no longer C88.C1, C89.C1, R53.1
- net 5V0_PA_STG1_2_CLEAN: now also C41.C1, C42.C1, C50.C1, C51.C1, C52.C1, R24.2, R25.2, R29.2; no longer C36.C1, C37.C1, C38.C1, C45.C1, C47.C1, R28.2, R30.2, R32.2
- net 5V0_PA_STG3_CLEAN: now also C62.C1, C67.C1, C69.C1, R38.2, R40.2, U18.VBIAS, U18.VCC; no longer C59.C1, C60.C1, C61.C1, R41.2, R43.2, U17.VBIAS, U17.VCC
- net 5V0_RT: now also R45.2, U21.RT; no longer R48.2, U20.RT
- net 5V0_SS: now also C80.C1, U21.TR/SS; no longer C77.C1, U20.TR/SS
- net 5V0_SW: now also C84.C1, U21.SW; no longer C82.C1, U20.SW
- net 5V0_VSENSE: now also C75.C1, R43.1, R44.2; no longer C72.C1, R46.1, R47.2
- net GND: now also C100.C2, C101.C2, C12.C2, C19.C2, C21.C2, C26.C2, C27.C2, C31.C2, C33.C2, C35.C2, C44.C2, C50.C2, C51.C2, C52.C2, C56.C2, C57.C2, C68.C2, C81.C2, C82.C2, C83.C2, D5.C, D7.A, R10.1, R31.1, R33.1, R35.1, R37.1, R39.1, R44.1, R51.1, U10.D0, U10.D1, U10.D2, U10.D3, U10.D4, U10.D5, U10.D6, U10.GND, U11.GND@0, U11.GND@1, U12.GND, U13.GND@0, U13.GND@1, U13.GND@2, U13.GND@3, U15.GND, U16.PWR.V-, U19.D0, U19.D1, U19.D2, U19.D3, U19.D4, U19.D5, U19.D6, U21.GND, U4.AGND, U4.AGNDVCO@0, U4.AGNDVCO@1, U4.AGNDVCO@2, U4.CPGND, U4.DGND, U4.RFOUTB+, U4.RFOUTB-, U4.SDGND, U7.D0, U7.D1, U7.D2, U7.D3, U7.D4, U7.D5, U7.D6; no longer C15.C2, C24.C2, C25.C2, C29.C2, C30.C2, C36.C2, C37.C2, C38.C2, C47.C2, C53.C2, C54.C2, C55.C2, C59.C2, C60.C2, C7.C2, C71.C2, C8.C2, C84.C2, C85.C2, D5.A, D7.C, R17.1, R21.1, R34.1, R36.1, R38.1, R40.1, R48.1, R54.1, R55.1, U10.GND@0, U10.GND@1, U11.GND, U12.GND@0, U12.GND@1, U12.GND@2, U12.GND@3, U13.GND, U15.PWR.V-, U16.GND, U18.D0, U18.D1, U18.D2, U18.D3, U18.D4, U18.D5, U18.D6, U3.AGND, U3.AGNDVCO@0, U3.AGNDVCO@1, U3.AGNDVCO@2, U3.CPGND, U3.DGND, U3.RFOUTB+, U3.RFOUTB-, U3.SDGND, U6.D0, U6.D1, U6.D2, U6.D3, U6.D4, U6.D5, U6.D6, U9.D0, U9.D1, U9.D2, U9.D3, U9.D4, U9.D5, U9.D6
- net I2C1_SCL: now also U17.SCL; no longer U16.SCL
- net I2C1_SDA: now also U17.SDA; no longer U16.SDA
- net IF_ATT_ACC: now also R22.1; no longer R24.1
- net IF_ATT_ACC_PROBE: now also C37.C2, R21.1, R22.2; no longer C34.C2, R23.1, R24.2
- net IF_ATT_DCC: now also C37.C1, U7.RF1; no longer C34.C1, U6.RF1
- net IF_ATT_LE: now also U7.LE; no longer U6.LE
- net IF_IN_ACC: now also C34.C2, U7.RF2; no longer C31.C2, U6.RF2
- net IF_IN_DCC: now also C34.C1, RFCON3.SIGNAL; no longer C31.C1, RFCON2.SIGNAL
- net MIXER_IN_DCC: now also U8.IFIN; no longer U7.IFIN
- net MIXER_LO: now also C7.C2, U8.LO; no longer R18.1, R20.2, R22.1, R25.2
- net MIXER_OUT_ACC: now also C38.C2, R23.1, U5.RF2; no longer C35.C2, R26.1, U4.RF2
- net MIXER_OUT_DCC: now also U8.RFOUT; no longer U7.RFOUT
- net N$1: now also C22.C2, C24.C1; no longer C19.C2, C21.C1
- net N$12: now also U12.VDD; no longer U11.VDD
- net N$149: now also D8.A; no longer D6.A
- net N$15: now also R24.1, U12.BIAS1; no longer R27.1, U11.BIAS1
- net N$16: now also R27.1, U12.BIAS2; no longer R30.1, U11.BIAS2
- net N$2: now also C100.C1; no longer C98.C1
- net N$20: now also C99.C1; no longer C97.C1
- net N$21: now also RFCON2.SIGNAL; no longer RFCON1.SIGNAL
- net N$23: now also D5.A, R29.1; no longer D3.A, R32.1
- net N$24: now also R21.2, RFCON5.SIGNAL; no longer R23.2, RFCON4.SIGNAL
- net N$28: now also R23.2; no longer R26.2
- net N$3: now also D6.A, R40.1; no longer D4.A, R43.1
- net N$30: now also C47.C2, U12.RFIN; no longer C44.C2, U11.RFIN
- net N$35: now also R26.2; no longer R29.2
- net N$39: now also U19.RF2; no longer U18.RF2
- net N$4: now also R25.1, U12.GAIN_SEL; no longer R28.1, U11.GAIN_SEL
- net N$42: now also R33.2, U15.ISOLATED; no longer R36.2, U14.ISOLATED
- net N$43: now also C59.C1, U13.RFIN; no longer C56.C1, U12.RFIN
- net N$44: now also C60.C2, U13.FLTR; no longer C57.C2, U12.FLTR
- net N$5: now also D4.A, R19.1; no longer D7.A, R57.1
- net N$6: now also C38.C1; no longer C35.C1
- net N$67: now also C23.C1, U4.RFOUTA-; no longer C20.C1, U3.RFOUTA-
- net N$69: now also C22.C1, U4.RFOUTA+; no longer C19.C1, U3.RFOUTA+
- net N$7: now also R31.2, R32.2, U16.1.-IN; no longer R34.2, R35.2, U15.1.-IN
- net N$8: now also C14.C1, U4.!PDRF, U4.DVDD; no longer C11.C1, U3.!PDRF, U3.DVDD
- net N$84: now also C25.C2, R16.2; no longer C22.C2, R17.2
- net N$88: now also U4.RSET; no longer U3.RSET
- net N$9: now also D3.A, R18.1; no longer D8.A, R58.1
- net PA3_EN: now also R38.1, R39.2, SJ2.1, U18.PAEN; no longer R41.1, R42.2, SJ1.1, U17.PAEN
- net PA_STG1_2_BIAS_EN: now also R50.2; no longer R54.2
- net PA_STG3_BIAS_EN: now also R51.2; no longer R55.2
- net PA_TEMP_ALERT: now also SJ2.2, U17.ALERT; no longer SJ1.2, U16.ALERT
- net PLL_CP_VOUT: now also C25.C1, C26.C1, R17.2, U4.CPOUT; no longer C22.C1, C23.C1, R19.2, U3.CPOUT
- net PLL_EN: now also R10.2, U4.CE; no longer R9.2, U3.CE
- net PLL_FASTLOCK_SW: now also U4.SW; no longer U3.SW
- net PLL_LE: now also U4.LE; no longer U3.LE
- net PLL_LOCK: now also U4.LD; no longer U3.LD
- net PLL_MUXOUT: now also U4.MUXOUT; no longer U3.MUXOUT
- net PLL_REF_ACC: now also C15.C2, U4.REFIN; no longer C12.C2, U3.REFIN
- net PLL_REF_DCC: now also C13.C1, C15.C1, U3.CLK; no longer C10.C1, C12.C1, U2.CLK
- net PLL_TEMP: now also C20.C1, C21.C1, U4.TEMP; no longer C17.C1, C18.C1, U3.TEMP
- net PLL_VCOM: now also C18.C1, C19.C1, U4.VCOM; no longer C15.C1, C16.C1, U3.VCOM
- net PLL_VREF: now also C16.C1, C17.C1, U4.VREF; no longer C13.C1, C14.C1, U3.VREF
- net PLL_VTUNE: now also C27.C1, R17.1, U4.VTUNE; no longer C24.C1, R19.1, U3.VTUNE
- net RF_ATT1_LE: now also U10.LE; no longer U9.LE
- net RF_ATT2_LE: now also U19.LE; no longer U18.LE
- net RF_FINAL_ACC: now also U18.RFOUT; no longer U17.RFOUT
- net RF_FLT_ACC: now also C36.C2, U11.RFIN; no longer C33.C2, U10.RFIN
- net RF_IN_ACC: now also C30.C2, U5.RF1; no longer C27.C2, U4.RF1
- net RF_IN_DCC: now also C30.C1, RFCON4.SIGNAL; no longer C27.C1, RFCON3.SIGNAL
- net RF_PRE1_ACC: now also C54.C2, U10.RF2; no longer C51.C2, U9.RF2
- net RF_PRE1_ATT_ACC: now also R28.1, U9.RFIN; no longer R31.1, U8.RFIN
- net RF_PRE1_ATT_ACC_PROBE: now also C53.C2, R26.1, R28.2; no longer C50.C2, R29.1, R31.2
- net RF_PRE1_ATT_DCC: now also C53.C1, U10.RF1; no longer C50.C1, U9.RF1
- net RF_PRE1_ATT_FLT_ACC: now also C45.C1, C47.C1, U9.RFOUT; no longer C42.C1, C44.C1, U8.RFOUT
- net RF_PRE1_DCC: now also C54.C1, U11.RFOUT; no longer C51.C1, U10.RFOUT
- net RF_PRE2_ACC: now also C55.C2, C56.C1; no longer C52.C2, C53.C1
- net RF_PRE2_ATT_ACC: now also C71.C2, U14.RFIN; no longer C68.C2, U13.RFIN
- net RF_PRE2_ATT_DCC: now also C71.C1, U19.RF1; no longer C68.C1, U18.RF1
- net RF_PRE2_ATT_FLT_ACC: now also U14.RFOUT, U15.IN; no longer U13.RFOUT, U14.IN
- net RF_PRE2_ATT_FLT_CPL_ACC: now also C59.C2, U15.COUPLED; no longer C56.C2, U14.COUPLED
- net RF_PRE2_ATT_FLT_THRU_ACC: now also R35.2, R36.2, U15.OUT; no longer R38.2, R39.2, U14.OUT
- net RF_PRE2_ATT_FLT_THRU_ACC_ATT: now also R36.1, R37.2, U18.RFIN; no longer R39.1, R40.2, U17.RFIN
- net RF_PRE2_DCC: now also C55.C1, U12.RFOUT; no longer C52.C1, U11.RFOUT
- net RF_SEL_ACC: now also C29.C2, U6.RFIN; no longer C26.C2, U5.RFIN
- net RF_SEL_DCC: now also C29.C1, U5.RFCOM; no longer C26.C1, U4.RFCOM
- net RF_SEL_FILT_DCC: now also C36.C1, U6.RFOUT; no longer C33.C1, U5.RFOUT
- net RF_SW_CTL: now also R18.2, SJ1.1, U5.CONTROL; no longer R58.2, U4.CONTROL
- net SPI_MOSI: now also U10.DATA, U19.DATA, U4.DATA, U7.DATA; no longer U18.DATA, U3.DATA, U6.DATA, U9.DATA
- net SPI_SCK: now also U10.CLK, U19.CLK, U4.CLK, U7.CLK; no longer U18.CLK, U3.CLK, U6.CLK, U9.CLK
- net V5V0_ISENSE: now also C89.C1, R48.1; no longer C86.C1, R51.1
- net V5V0_ISENSE-AMP: now also R48.2; no longer R51.2
- net VIN: now also C101.C1, C72.C1, C77.C1, C78.C1, D7.C, R41.2, U21.EN/UV, U21.VIN; no longer C69.C1, C74.C1, C75.C1, C99.C1, D5.C, R44.2, U20.EN/UV, U20.VIN
- net VIN_VSENSE: now also C74.C1, R41.1, R42.2; no longer C71.C1, R44.1, R45.2
- net VPDET_AMP: now also R32.1, R34.2, U16.1.OUT; no longer R35.1, R37.2, U15.1.OUT
- net VPDET_FLT: now also C61.C1, R30.1, U16.1.+IN; no longer C58.C1, R33.1, U15.1.+IN
- net VPDET_RAW: now also C60.C1, R30.2, U13.OUT; no longer C57.C1, R33.2, U12.OUT
- net VPDET_SENSE: now also C65.C1, R34.1; no longer C62.C1, R37.1
Other:
- note added: "27.4kHz Loop Bandwidth at Icp = 5 mA"
- note removed: "-9 dB Pi Attenuator"
- note removed: "100kHz Loop Bandwidth at 2.5 mA"
- moved on the sheet: C10, C11, C12, C13, C14, C15, C16, C17, C18, C19, C20, C21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
