File: pcb/upconverter/qo-100-upconverter.brd (EAGLE design)
At the start: 100 x 70 mm, 227 parts, among them CON1 3P-SH-SIDE, CON2 2EDG-2P-5MM, U1 EFM32TG11B120F128GM32, U10 LTC5597, U11 2450BP15E0100, U12 MCP6V31, U13 DC2337J5010AHF, U14 ADL5606, U15 F1958NBGK, U16 MCP1700-330, U17 LT8636, U18 MCP3421-A0, U19 MCP6C02-020, U2 DSB321SDA, U20 ADP7142AUJZ-3.3, U21 ADP7142AUJZ-3.3, U22 ADP7142AUJZ-3.3, U23 ADM7171ACPZ-5.0, U24 ADM7171ACPZ-5.0, U3 ADF4351, U4 F1958NBGK, U5 MAX2671, U6 2450BP15E0100, U7 F1958NBGK, U8 ADL5601, U9 F1490NLGA

Commit message: Upconverter v3 software Upconverter assembly and tuning schematic changes Upconverter test documentation added
Parts:
- C22: value 1uF -> 20nF
- C23: value 220nF -> 1nF
- C24: value 2.7nF -> 470pF
- C29, C34: value 150pF -> 100pF
- C31: value 1.8pF -> DNP
- C32: value 1.5pF -> DNP
- C33: value 1.5pF -> 12pF
- L10: value 3.9nH -> 1.8pF
- L11: value 5.6nH -> 0 Ohms
- L12: value 3.3nH -> 2.2pF
- L5: value 4.7nH -> 5.1nH
- L6: value 12nH -> 5.1nH
- L8: value 3.9nH -> 0 Ohms
- R17: value 150 Ohms -> 330 Ohms
Changed lines of the file:
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@@
 <setting verticaltext="up"/>
 </settings>
-<grid distance="0.1" unitdist="mm" unit="mm" style="lines" multiple="1" display="yes" altdistance="0.05" altunitdist="mm" altunit="mm"/>
+<grid distance="1" unitdist="mm" unit="mm" style="lines" multiple="1" display="yes" altdistance="0.05" altunitdist="mm" altunit="mm"/>
 <layers>
 <layer number="1" name="Top" color="4" fill="1" visible="yes" active="yes"/>
@@
 </autorouter>
 <elements>
-<element name="C29" library="Capacitor" package="CAP0603" value="150pF" x="88.3" y="9.8" smashed="yes" rot="R90">
+<element name="C29" library="Capacitor" package="CAP0603" value="100pF" x="88.3" y="9.8" smashed="yes" rot="R90">
 <attribute name="NAME" x="86.884" y="8.2536" size="0.8" layer="25" font="vector" ratio="10" rot="SR90" align="center-left"/>
 <attribute name="VALUE" x="90.332" y="6.8536" size="0.8" layer="27" font="vector" ratio="10" rot="SR90" align="center-left"/>
@@
 <attribute name="VOLTAGE" value="" x="156.53" y="76.14" size="1.778" layer="27" rot="R90" display="off"/>
 </element>
-<element name="C22" library="Capacitor" package="CAP0603" value="1uF" x="61.6" y="27.2" smashed="yes" rot="R270">
+<element name="C22" library="Capacitor" package="CAP0603" value="20nF" x="61.6" y="27.2" smashed="yes" rot="R270">
 <attribute name="NAME" x="60.4536" y="29.316" size="0.8" layer="25" font="vector" ratio="10" rot="SR0" align="center-left"/>
 <attribute name="VALUE" x="59.568" y="30.1464" size="0.8" layer="27" font="vector" ratio="10" rot="SR270" align="center-left"/>
 <attribute name="VOLTAGE" value="" x="-26.03" y="-18.52" size="1.778" layer="27" rot="R270" display="off"/>
 </element>
-<element name="C23" library="Capacitor" package="CAP0603" value="220nF" x="63.3" y="27.2" smashed="yes" rot="R270">
+<element name="C23" library="Capacitor" package="CAP0603" value="1nF" x="63.3" y="27.2" smashed="yes" rot="R270">
 <attribute name="NAME" x="62.4536" y="29.316" size="0.8" layer="25" font="vector" ratio="10" rot="SR0" align="center-left"/>
 <attribute name="VALUE" x="61.268" y="30.1464" size="0.8" layer="27" font="vector" ratio="10" rot="SR270" align="center-left"/>
 <attribute name="VOLTAGE" value="" x="-24.33" y="-23.6" size="1.778" layer="27" rot="R270" display="off"/>
 </element>
-<element name="C24" library="Capacitor" package="CAP0603" value="2.7nF" x="66.7" y="27.2" smashed="yes" rot="R90">
+<element name="C24" library="Capacitor" package="CAP0603" value="470pF" x="66.7" y="27.2" smashed="yes" rot="R90">
 <attribute name="NAME" x="68.084" y="25.6536" size="0.8" layer="25" font="vector" ratio="10" rot="SR90" align="center-left"/>
 <attribute name="VALUE" x="68.732" y="24.2536" size="0.8" layer="27" font="vector" ratio="10" rot="SR90" align="center-left"/>
@@
 <attribute name="VALUE" x="60.232" y="23.7456" size="0.8" layer="27" font="vector" ratio="10" rot="SR90" align="center-left"/>
 </element>
-<element name="R17" library="Resistor" package="RES0603" value="150 Ohms" x="59.9" y="27.2" smashed="yes" rot="R270">
+<element name="R17" library="Resistor" package="RES0603" value="330 Ohms" x="59.9" y="27.2" smashed="yes" rot="R270">
 <attribute name="NAME" x="58.3456" y="29.316" size="0.8" layer="25" font="vector" ratio="10" rot="SR0" align="center-left"/>
 <attribute name="TOLERANCE" value="" x="7.83" y="-46.46" size="1.778" layer="27" rot="R270" display="off"/>
@@
 <attribute name="VOLTAGE" value="" x="91.9" y="19.2" size="1.778" layer="27" display="off"/>
 </element>
-<element name="C34" library="Capacitor" package="CAP0603" value="150pF" x="88.3" y="20.5" smashed="yes" rot="R90">
+<element name="C34" library="Capacitor" package="CAP0603" value="100pF" x="88.3" y="20.5" smashed="yes" rot="R90">
 <attribute name="NAME" x="86.884" y="18.9536" size="0.8" layer="25" font="vector" ratio="10" rot="SR90" align="center-left"/>
 <attribute name="VALUE" x="90.332" y="17.5536" size="0.8" layer="27" font="vector" ratio="10" rot="SR90" align="center-left"/>
@@
 <attribute name="VALUE" x="85.7456" y="40.568" size="0.8" layer="27" font="vector" ratio="10" rot="SR0" align="center-left"/>
 </element>
-<element name="L5" library="Inductor" package="IND0603" value="4.7nH" x="88.1" y="48.9" smashed="yes" rot="R225">
+<element name="L5" library="Inductor" package="IND0603" value="5.1nH" x="88.1" y="48.9" smashed="yes" rot="R225">
 <attribute name="CURRENT" value="" x="88.1" y="48.9" size="1.778" layer="27" rot="R225" display="off"/>
 <attribute name="NAME" x="89.43895" y="50.17579375" size="0.8" layer="25" font="vector" ratio="10" rot="SR45" align="center-left"/>
@@
 <attribute name="VOLTAGE" value="" x="85.8" y="50.1" size="1.778" layer="27" rot="R135" display="off"/>
 </element>
-<element name="C31" library="Capacitor" package="CAP0603" value="1.8pF" x="83.5" y="52.4" smashed="yes" rot="R135">
+<element name="C31" library="Capacitor" package="CAP0603" value="DNP" x="83.5" y="52.4" smashed="yes" rot="R135">
 <attribute name="NAME" x="82.864996875" y="49.698159375" size="0.8" layer="25" font="vector" ratio="10" rot="SR135" align="center-left"/>
 <attribute name="VALUE" x="87.020259375" y="51.75341875" size="0.8" layer="27" font="vector" ratio="10" rot="SR135" align="center-left"/>
 <attribute name="VOLTAGE" value="" x="83.5" y="52.4" size="1.778" layer="27" rot="R135" display="off"/>
 </element>
-<element name="C32" library="Capacitor" package="CAP0603" value="1.5pF" x="81.2" y="54.7" smashed="yes" rot="R135">
+<element name="C32" library="Capacitor" package="CAP0603" value="DNP" x="81.2" y="54.7" smashed="yes" rot="R135">
 <attribute name="NAME" x="80.564996875" y="51.898159375" size="0.8" layer="25" font="vector" ratio="10" rot="SR135" align="center-left"/>
 <attribute name="VALUE" x="84.720259375" y="54.05341875" size="0.8" layer="27" font="vector" ratio="10" rot="SR135" align="center-left"/>
 <attribute name="VOLTAGE" value="" x="81.2" y="54.7" size="1.778" layer="27" rot="R135" display="off"/>
 </element>
-<element name="C33" library="Capacitor" package="CAP0603" value="1.5pF" x="77.6" y="55.3" smashed="yes" rot="R180">
+<element name="C33" library="Capacitor" package="CAP0603" value="12pF" x="77.6" y="55.3" smashed="yes" rot="R180">
 <attribute name="NAME" x="76.0536" y="56.716" size="0.8" layer="25" font="vector" ratio="10" rot="SR0" align="center-left"/>
 <attribute name="VALUE" x="80.5464" y="57.332" size="0.8" layer="27" font="vector" ratio="10" rot="SR180" align="center-left"/>
 <attribute name="VOLTAGE" value="" x="77.6" y="55.3" size="1.778" layer="27" rot="R180" display="off"/>
 </element>
-<element name="L10" library="Inductor" package="IND0603" value="3.9nH" x="85.9" y="55.9" smashed="yes" rot="R225">
+<element name="L10" library="Inductor" package="IND0603" value="1.8pF" x="85.9" y="55.9" smashed="yes" rot="R225">
 <attribute name="CURRENT" value="" x="85.9" y="55.9" size="1.778" layer="27" rot="R225" display="off"/>
 <attribute name="NAME" x="87.23895" y="57.17579375" size="0.8" layer="25" font="vector" ratio="10" rot="SR45" align="center-left"/>
 <attribute name="VALUE" x="86.9057875" y="59.77946875" size="0.8" layer="27" font="vector" ratio="10" rot="SR225" align="center-left"/>
 </element>
-<element name="L12" library="Inductor" package="IND0603" value="3.3nH" x="83.6" y="58.2" smashed="yes" rot="R225">
+<element name="L12" library="Inductor" package="IND0603" value="2.2pF" x="83.6" y="58.2" smashed="yes" rot="R225">
 <attribute name="CURRENT" value="" x="83.6" y="58.2" size="1.778" layer="27" rot="R225" display="off"/>
 <attribute name="NAME" x="84.93895" y="59.57579375" size="0.8" layer="25" font="vector" ratio="10" rot="SR45" align="center-left"/>
@@
 <attribute name="VALUE" x="58.032" y="52.7456" size="0.8" layer="27" font="vector" ratio="10" rot="SR90" align="center-left"/>
 </element>
-<element name="L6" library="Inductor" package="IND0603" value="12nH" x="87" y="51.3" smashed="yes" rot="R135">
+<element name="L6" library="Inductor" package="IND0603" value="5.1nH" x="87" y="51.3" smashed="yes" rot="R135">
 <attribute name="CURRENT" value="" x="87" y="51.3" size="1.778" layer="27" rot="R135" display="off"/>
 <attribute name="NAME" x="85.82420625" y="48.038946875" size="0.8" layer="25" font="vector" ratio="10" rot="SR135" align="center-left"/>
 <attribute name="VALUE" x="90.87946875" y="50.294209375" size="0.8" layer="27" font="vector" ratio="10" rot="SR135" align="center-left"/>
 </element>
-<element name="L8" library="Inductor" package="IND0603" value="3.9nH" x="84.7" y="53.6" smashed="yes" rot="R135">
+<element name="L8" library="Inductor" package="IND0603" value="0 Ohms" x="84.7" y="53.6" smashed="yes" rot="R135">
 <attribute name="CURRENT" value="" x="84.7" y="53.6" size="1.778" layer="27" rot="R135" display="off"/>
 <attribute name="NAME" x="83.52420625" y="50.438946875" size="0.8" layer="25" font="vector" ratio="10" rot="SR135" align="center-left"/>
 <attribute name="VALUE" x="88.57946875" y="52.594209375" size="0.8" layer="27" font="vector" ratio="10" rot="SR135" align="center-left"/>
 </element>
-<element name="L11" library="Inductor" package="IND0603" value="5.6nH" x="82.4" y="55.9" smashed="yes" rot="R135">
+<element name="L11" library="Inductor" package="IND0603" value="0 Ohms" x="82.4" y="55.9" smashed="yes" rot="R135">
 <attribute name="CURRENT" value="" x="82.4" y="55.9" size="1.778" layer="27" rot="R135" display="off"/>
 <attribute name="NAME" x="81.22420625" y="52.638946875" size="0.8" layer="25" font="vector" ratio="10" rot="SR135" align="center-left"/>

Commit message: Upconverter: Changed final amplifier to SKY66292-11 Upconverter: Added Pi attenuator before final amplifier Upconverter: Removed GND exposed pads below PLL VTUNE Upconverter: Added temperature sensor near final amplifier Upconverter: Exposed bottom layer copper for heat sinking
Signed-off-by: João Silva <jgc3silva@gmail.com>
Parts:
- removed C100, C101: 10uF, Capacitor:CAP0603
- removed C102, C103: 1nF, Capacitor:CAP0603
- removed C104: 10uF, Capacitor:CAP1206
- removed L20: 4.7uH, Inductor:IND0606
- removed TP1, TP2, TP3, TP4, TP5, TP6: TESTPOINT-1.27MM, PADs:PAD1.27MM
- added R54: 10K Ohms, Resistor:RES0603
- added R55: 0.03 Ohms, Resistor:RES1206
- added R56, R57: 100K Ohms, Resistor:RES0603
- added R58: 1K Ohms, Resistor:RES0603
- added SJ1: SJCS, Solder Jumper:SJC_S
- added U25: ADM7172ACPZ-5.0, Analog Devices:LFCSP8_3X3
- C59, C84: value 10uF -> 100uF; device Capacitor:CAP0603 -> Capacitor:CAP1206
- C60: value 10nF -> 10uF
- C61: value 15pF -> 10uF
- C63, C90: value 100uF -> 1uF; device Capacitor:CAP1206 -> Capacitor:CAP0603
- C64: value 100pF -> 10nF
- C65: value 2pF -> 10nF
- C66, C80, C81: value 1uF -> 100nF
- C67: value 10nF -> 15pF
- C68: value 100pF -> 4.7uF
- C69: value 15pF -> 100nF
- C70: value 3.3pF -> 470pF
- C71: value 15pF -> 470pF
- C72: value 100nF -> 4.7uF
- C73: value 15pF -> 1uF
- C74: value 4.7uF -> 1uF
- C75, C83, C91, C92: value 100nF -> 1uF
- C76: value 470pF -> 10nF
- C77: value 470pF -> 100nF
- C78: value 4.7uF -> 10uF
- C79, C94, C95: value 1uF -> 10uF
- C82: value 10nF -> 10pF
- C85, C99: value 10uF -> 100nF
- C87: value 100nF -> 22uF; device Capacitor:CAP0603 -> Capacitor:CAP1206
- C88: value 10pF -> 1uF
- C93: value 22uF -> 10uF; device Capacitor:CAP1206 -> Capacitor:CAP0603
- C96, C97: value 1uF -> 1nF
- C98: value 1uF -> 10uF; device Capacitor:CAP0603 -> Capacitor:CAP1206
- CON2: value 2EDG-2P-5MM -> 2EDG-2P-5MM-H; device Generic Connector:2EDG-2P-5MM -> Generic Connector:2EDG-2P-5MM-H
- L18: value 62nH -> 0 Ohms
- L19: value 0 Ohms -> 4.7uH; device Inductor:IND0603 -> Inductor:IND0606
- R29: value 0 Ohms -> DNP
- R38: value 100 Ohms -> 49.9 Ohms
- R39: value 49.9 Ohms -> 100 Ohms
- R40: value 510 Ohms -> 96.1 Ohms
- R41: value 100K Ohms -> 71.5 Ohms
- R42: value 10K Ohms -> 96.1 Ohms
- R43: value 100K Ohms -> 10K Ohms
- R44: value 75K Ohms -> 7.5K Ohms
- R45: value 41.2K Ohms -> 510 Ohms
- R46: value 1M Ohms -> 100K Ohms
- R47: value 221K Ohms -> 10K Ohms
- R48: value 10K Ohms -> 100K Ohms
- R49: value 10K Ohms -> 75K Ohms
- R50: value 0.03 Ohms -> 41.2K Ohms; device Resistor:RES1206 -> Resistor:RES0603
- R51: value 100K Ohms -> 1M Ohms
- R52: value 100K Ohms -> 221K Ohms
- R53: value 1K Ohms -> 10K Ohms
- U12: value MCP6V31 -> DC2337J5010AHF; device Microchip:SOT23-5 -> Anaren:DC2337J5010AHF
- U13: value DC2337J5010AHF -> MCP6V31; device Anaren:DC2337J5010AHF -> Microchip:SOT23-5
- U14: value ADL5606 -> SKY66292-11; device Analog Devices:LFCSP16_4X4 -> Skyworks:SKY66292-11
- U16: value MCP1700-330 -> MCP9802-A0; device Microchip:SOT23 -> Microchip:SOT23-5
- U17: value LT8636 -> MCP1700-330; device Analog Devices:QFN20_ASYM_CORNER -> Microchip:SOT23
- U18: value MCP3421-A0 -> LT8636; device Microchip:SOT23-6 -> Analog Devices:QFN20_ASYM_3X4_CORNER
- U19: value MCP6C02-020 -> MCP3421-A0
- U20: value ADP7142AUJZ-3.3 -> MCP6C02-020; device Analog Devices:SOT23-5 -> Microchip:SOT23-6
- U23: value ADM7171ACPZ-5.0 -> ADP7142AUJZ-3.3; device Analog Devices:LFCSP8_3X3 -> Analog Devices:SOT23-5
- moved C99 79.4 mm to (2.10, 44.8), turned to 90 degrees
- moved C70 59.0 mm to (56.4, 3.60), turned to 270 degrees
- moved R38 57.3 mm to (8.50, 53.2), turned to 0 degrees
- moved R39 57.3 mm to (50.8, 14.6), turned to 180 degrees
- moved C94 56.8 mm to (21.2, 50.1), turned to 90 degrees
- moved U21 56.7 mm to (73.8, 20.7), turned to 0 degrees
- moved R44 56.3 mm to (3.55, 48.9), turned to 270 degrees
- moved C71 55.4 mm to (54.7, 3.60)
- moved C73 54.0 mm to (30.0, 2.60), turned to 0 degrees
- moved R43 52.7 mm to (5.25, 48.9), turned to 270 degrees
- moved C88 51.6 mm to (69.8, 20.7), turned to 270 degrees
- moved U16 47.4 mm to (5.60, 43.2)
- moved C72 45.7 mm to (39.3, 17.5)
- moved L19 45.1 mm to (34.2, 10.7), turned to 90 degrees
- moved U20 44.6 mm to (29.5, 26.2), turned to 90 degrees
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Connections:
- removed net N$5: C61.2, C65.1, U14.1
- removed net RF_FINAL_DCC: C70.1, C71.1, L18.1, U14.10, U14.11, U14.12, U14.9
- new net PA3_EN: R43.1, R44.2, SJ1.1, U14.6
- new net PA_TEMP_ALERT: SJ1.2, U16.3
- new net RF_PRE2_ATT_FLT_THRU_ACC_ATT: R41.1, R42.2, U14.2
- net 3V3: now also C77.1, C78.1, C79.1, C80.1, C99.1, U16.1, U17.2, U19.5; no longer C83.1, C84.1, C85.1, C86.1, U16.2, U18.5
- net 3V3_IF_ATT_MIXER_CLEAN: now also C93.1, U21.4, U21.5; no longer C99.1, U20.4, U20.5
- net 3V3_PLL_CLEAN: now also C95.1, U23.4, U23.5; no longer C101.1, U22.4, U22.5
- net 3V3_RF_ATT_PDET_CLEAN: now also C66.1, C94.1, U13.5, U22.4, U22.5; no longer C100.1, C72.1, U12.5, U21.4, U21.5
- net 5V0: now also C69.1, C72.1, C82.1, C83.1, C84.1, C86.1, L19.2, R48.2, R51.2, R55.2, R58.2, U17.3, U18.2, U20.3, U20.6; no longer C75.1, C78.1, C88.1, C89.1, C90.1, C92.1, L20.2, R43.2, R46.2, R50.2, R53.2, U16.3, U17.2, U19.3, U19.6
- net 5V0_BST: now also C81.2, U18.7; no longer C87.2, U17.7
- net 5V0_FB: now also C82.2, R51.1, R52.2, U18.19, U18.20; no longer C88.2, R46.1, R47.2, U17.19, U17.20
- net 5V0_INTVCC: now also C75.1, U18.15, U18.3; no longer C81.1, U17.15, U17.3
- net 5V0_ISENSE: now also C87.1, C88.1, C89.1, C90.1, C91.1, C92.1, R55.1, U20.4, U23.1, U23.3, U25.7, U25.8; no longer C93.1, C94.1, C95.1, C96.1, C97.1, C98.1, R50.1, U19.4, U20.1, U20.3, U23.7, U23.8
- net 5V0_ISENSE_VN: now also C85.2, R54.1, U19.6; no longer C91.2, R49.1, U18.6
- net 5V0_ISENSE_VP: now also C85.1, R53.1, U19.1; no longer C91.1, R48.1, U18.1
- net 5V0_PA_STG1_2_CLEAN: now also U24.1, U24.2, U24.3; no longer U23.1, U23.2, U23.3
- net 5V0_PA_STG3_CLEAN: now also C61.1, C65.1, R43.2, R45.2, U14.12, U14.14, U14.16, U14.5, U25.1, U25.2, U25.3; no longer C66.1, C67.1, C68.1, C69.1, L18.2, R40.2, U14.3, U14.4, U24.1, U24.2, U24.3
- net 5V0_RT: now also R50.2, U18.17; no longer R45.2, U17.17
- net 5V0_SS: now also C76.1, U18.18; no longer C82.1, U17.18
- net 5V0_SW: now also C81.1, L19.1, U18.10, U18.8, U18.9; no longer C87.1, L20.1, U17.10, U17.8, U17.9
- net 5V0_VSENSE: now also C71.1, R48.1, R49.2; no longer C77.1, R43.1, R44.2
- net GND: now also C61.2, C71.2, C73.2, C87.2, C88.2, C91.2, R38.1, R40.1, R49.1, R50.1, R54.2, R56.1, R57.1, U12.3, U12.4, U13.2, U14.1, U14.10, U14.11, U14.3, U14.4, U16.2, U17.1, U18.12, U18.13, U18.21, U18.4, U18.5, U18.M1, U18.M2, U18.M3, U18.M4, U20.5, U23.2, U25.6, U25.9, U3.14, U3.15; no longer C100.2, C101.2, C102.2, C103.2, C104.2, C67.2, C81.2, C82.2, C85.2, R39.1, R45.1, R49.2, R51.1, TP1.TP, TP2.TP, TP3.TP, TP4.TP, TP5.TP, TP6.TP, U12.2, U13.3, U13.4, U14.14, U14.16, U14.2, U14.5, U14.6, U16.1, U17.12, U17.13, U17.21, U17.4, U17.5, U17.M1, U17.M2, U17.M3, U17.M4, U18.2, U19.5, U23.6, U23.9
- net I2C1_SCL: now also U16.4, U19.3; no longer U18.3
- net I2C1_SDA: now also U16.5, U19.4; no longer U18.4
- net N$10: now also R53.2, U20.1; no longer R48.2, U19.1
- net N$149: now also R58.1; no longer R53.1
- net N$2: now also C97.1, U25.4; no longer C103.1, U24.4
- net N$20: now also C96.1, U24.4; no longer C102.1, U23.4
- net N$3: now also R45.1; no longer R40.1
- net N$39: now also L18.2; no longer L19.2
- net N$42: now also R38.2, U12.5; no longer R39.2, U13.5
- net N$7: now also U13.4; no longer U12.4
- net PA_STG1_2_BIAS_EN: now also R56.2, U24.5; no longer R51.2, U23.5
- net PA_STG3_BIAS_EN: now also R57.2, U25.5; no longer R52.2, U24.5
- net RF_FINAL_ACC: now also U14.9; no longer C71.2
- net RF_PRE2_ACC: now also L18.1; no longer L19.1
- net RF_PRE2_ATT_ACC: now also C67.2; no longer C73.2
- net RF_PRE2_ATT_DCC: now also C67.1; no longer C73.1
- net RF_PRE2_ATT_FLT_ACC: now also U12.1; no longer U13.1
- net RF_PRE2_ATT_FLT_CPL_ACC: now also U12.2; no longer U13.2
- net RF_PRE2_ATT_FLT_THRU_ACC: now also R40.2, R41.2, U12.6; no longer C61.1, U13.6
- net VIN: now also C68.1, C73.1, C98.1, R46.2, U18.11, U18.14, U18.6; no longer C104.1, C79.1, C80.1, R41.2, U17.11, U17.14, U17.6
- net VIN_VSENSE: now also C70.1, R46.1, R47.2; no longer C76.1, R41.1, R42.2
- net VPDET_AMP: now also R39.2, U13.1; no longer R38.2, U12.1
- net VPDET_FLT: now also U13.3; no longer U12.3
- net VPDET_SENSE: now also R39.1; no longer R38.1
Routing:
- net I2C1_SCL: track 74.2 -> 116.9 mm, vias 2 -> 3
- net I2C1_SDA: track 74.8 -> 112.9 mm, vias 2 -> 3
- net 3V3: track 59.4 -> 96.8 mm, vias 32 -> 33
- net 5V0_PA_STG3_CLEAN: track 7.51 -> 19.2 mm, vias 38 -> 2
- net PA3_EN: track 0.00 -> 11.5 mm
- net PA_TEMP_ALERT: track 0.00 -> 9.65 mm, vias 0 -> 2
- net RF_FINAL_ACC: track 10.9 -> 16.9 mm
- net RF_FINAL_DCC: track 5.22 -> 0.00 mm
- net N$5: track 4.86 -> 0.00 mm
- net RF_PRE2_ATT_FLT_THRU_ACC_ATT: track 0.00 -> 3.18 mm
- net GND: track 152.2 -> 155.3 mm, vias 1519 -> 1688
- net RF_PRE2_ATT_FLT_THRU_ACC: track 2.01 -> 3.61 mm
- removed copper zone on layer 15, net 5V0_PA_STG3_CLEAN
- removed copper zone on layer 1, net RF_FINAL_DCC
Other:
- board text added: "IcyRadio Upconverter v4 Mar 2022"
- board text removed: "IcyRadio Upconverter v3 Mar 2021"
