File: pcb/opi-dock/qo-100-opi-dock.sch (EAGLE design)
At the start: 70 parts, among them CON1 2P-PH-TOP, CON10 6P-SH-TOP, CON2 4P-SH-TOP, CON3 4P-SH-TOP, CON4 4P-SH-TOP, CON5 3P-SH-TOP, CON6 3P-SH-TOP, CON7 3P-SH-TOP, CON8 3P-SH-TOP, CON9 6P-SH-TOP, U1 ORANGEPIZERO, U10 LTC4313-2, U11 ADUM1250, U2 LTC4313-1, U3 MIC23155, U4 MCP1703-330, U5 MCP23008, U6 LTC4313-2, U7 ADUM1250, U8 MCP1703-330, U9 MCP23008

Commit message: Renamed Orange Pi hat to Orange Pi dock Finished OPi dock routing
Parts:
- removed U11: ADUM1250, Analog Devices:ADUM1250
- added C19, C22, C30, C32, C36: 100nF, Capacitor:CAPACITOR-0603
- added C20, C21, C23, C28: 4.7uF, Capacitor:CAPACITOR-0603
- added C24, C26, C27: 1uF, Capacitor:CAPACITOR-0603
- added C25, C37: 470pF, Capacitor:CAPACITOR-0603
- added C29: 10nF, Capacitor:CAPACITOR-0603
- added C31: 10pF, Capacitor:CAPACITOR-0603
- added C33, C34, C35: 100uF, Capacitor:CAPACITOR-1206
- added C38: 10uF, Capacitor:CAPACITOR-1206
- added CON11, CON12, CON13: 3P-SH-TOP, JST:3P-SH-TOP
- added CON14, CON15, CON16, CON17: 3P-SH-SIDE, JST:3P-SH-SIDE
- added CON18: 2P-PH-TOP, JST:2P-PH-TOP
- added CON19: 2EDG-2P, Generic Connector:2EDG-2P
- added D10, D5, D6, D7, D8: LED0603, LED:LED0603
- added D11: SMAJ12A, TVS:SMAJ12A
- added D2, D3, D4, D9: B0530W, Generic Diode:B0530W
- added L2: 3.3uH, Inductor:INDUCTOR-6X6MM
- added Q1: AO3400, Alpha Omega:AO3400
- added R28, R29, R32, R33, R34, R35, R41, R42: 1K Ohms, Resistor:RESISTOR-0603
- added R30, R31, R40, R53: 10K Ohms, Resistor:RESISTOR-0603
- added R36, R37, R38, R39: 330 Ohms, Resistor:RESISTOR-0603
- added R43, R44, R45, R46: DNP, Resistor:RESISTOR-0603
- added R47: 41.2K Ohms, Resistor:RESISTOR-0603
- added R48: 309K Ohms, Resistor:RESISTOR-0603
- added R49: 71.5K Ohms, Resistor:RESISTOR-0603
- added R50: 1M Ohms, Resistor:RESISTOR-0603
- added R51: 226K Ohms, Resistor:RESISTOR-0603
- added R52: 22 Ohms, Resistor:RESISTOR-0603
- added R54: 510 Ohms, Resistor:RESISTOR-0603
- added R55: 147K Ohms, Resistor:RESISTOR-0603
- added R56: 21K Ohms, Resistor:RESISTOR-0603
- added T1, T2, T3, T4: BC817, Generic BJT:BC817
- added U12: DS2484, Maxim Integrated:DS2484
- added U13: LTC4313-1, Analog Devices:LTC4313-1
- added U14: MCP1525, Microchip:MCP1525
- added U15: MIC23155, Microchip:MIC23155
- added U16: LT8640S, Analog Devices:LT8640S
- added U17: MCP3221-A0, Microchip:MCP3221-A0
- C14, C16: value 1uF -> 100nF
- C2: value 100uF -> 1uF; device Capacitor:CAPACITOR-1206 -> Capacitor:CAPACITOR-0603
- C4: value 470pF -> 1uF
- C6: value 100uF -> 100nF; device Capacitor:CAPACITOR-1206 -> Capacitor:CAPACITOR-0603
- CON1: value 2P-PH-TOP -> 6P-SH-SIDE; device JST:2P-PH-TOP -> JST:6P-SH-SIDE
- CON10, CON9: value 6P-SH-TOP -> 3P-SH-TOP; device JST:6P-SH-TOP -> JST:3P-SH-TOP
- CON2: value 4P-SH-TOP -> 6P-SH-SIDE; device JST:4P-SH-TOP -> JST:6P-SH-SIDE
- CON3, CON4: value 4P-SH-TOP -> 4P-SH-SIDE; device JST:4P-SH-TOP -> JST:4P-SH-SIDE
- CON5, CON6, CON7: value 3P-SH-TOP -> 4P-SH-SIDE; device JST:3P-SH-TOP -> JST:4P-SH-SIDE
- D1: value SMAJ5.0A -> B0530W; device TVS:SMAJ5.0A -> Generic Diode:B0530W
- F1: value (none) -> 2.6A Hold; device Fuses:PTC1206 -> PTC Fuses:PTC1206; HOLD 2A -> 3A; OCLCSC (none) -> C207041; TRIP 3.5A -> 6A
- R1, R10, R11, R19, R20: value 10K Ohms -> 4.7K Ohms
- R12, R13, R21, R22: value 510 Ohms -> 1K Ohms
- R14, R23: value 1K Ohms -> 10K Ohms
- R15, R24, R25, R5, R6: value 4.7K Ohms -> 10K Ohms
- R16, R7: value 4.7K Ohms -> 510 Ohms
- R17: value 1K Ohms -> 510 Ohms
- R2, R3: value 1K Ohms -> 4.7K Ohms
- R8: value 309K Ohms -> 510 Ohms
- R9: value 71.5K Ohms -> 1K Ohms
- U10: value LTC4313-2 -> CP2108; device Analog Devices:LTC4313-2 -> Silicon Labs:CP2108
- U2: value LTC4313-1 -> MCP1703-330; device Analog Devices:LTC4313-1 -> Microchip:MCP1703-330
- U3: value MIC23155 -> MCP23008; device Microchip:MIC23155 -> Microchip:MCP23008
- U4, U8: value MCP1703-330 -> LTC4313-2; device Microchip:MCP1703-330 -> Analog Devices:LTC4313-2
- U5, U9: value MCP23008 -> ADUM1250; device Microchip:MCP23008 -> Analog Devices:ADUM1250
- U6: value LTC4313-2 -> MCP1703-330; device Analog Devices:LTC4313-2 -> Microchip:MCP1703-330
- U7: value ADUM1250 -> MCP23008; device Analog Devices:ADUM1250 -> Microchip:MCP23008
Connections:
- removed net N$12: CON1-1.S, F1.1
- new net !UART0_ACTIVE: D8.C, U10.P0.DTR
- new net !UART1_ACTIVE: D7.C, U10.P1.DTR
- new net !UART2_ACTIVE: D6.C, U10.P2.DTR
- new net !UART3_ACTIVE: D5.C, U10.P3(HD).DTR
- new net 2V5_ADC_CLEAN: C28.C1, C30.C1, U14.VOUT, U17.VDD
- new net 5V0_FB: C31.C2, R50.1, R51.2, U16.FB
- new net 5V0_INTVCC: C27.C1, U16.INTVCC, U16.SYNC/MODE
- new net 5V0_RT: R47.2, U16.RT
- new net 5V0_SS: C29.C1, U16.TR/SS
- new net 5V0_SW: L2.1, U16.SW
- new net FAN_PWM: R52.2, U1.DEBUG.(UART0_RX)PA5
- new net N$11: R23.1, U10.CTL.!RST
- new net N$149: D10.A, R54.1
- new net N$15: D8.A, R39.1
- new net N$18: D7.A, R38.1
- new net N$19: CON19-2.S, F1.2
- new net N$22: D6.A, R37.1
- new net N$25: D5.A, R36.1
- new net N$26: R24.1, T1.B
- new net N$27: R25.1, T2.B
- new net N$28: R30.1, T3.B
- new net N$29: R31.1, T4.B
- new net N$30: CON14-1.S, R43.1
- new net N$31: CON17-1.S, R46.1
- new net N$32: CON16-1.S, R45.1
- new net N$33: CON15-1.S, R44.1
- new net N$34: CON18-2.S, D9.A, Q1.D
- new net N$35: Q1.G, R52.1, R53.2
- new net SBC_USB_DM2: U1.AUX.USB_DM2, U10.CTL.D-
- new net SBC_USB_DP2: U1.AUX.USB_DP2, U10.CTL.D+
- new net UART0_RX: R26.1, T1.C, U10.P0.RX
- new net UART0_TRX: CON14-2.S, D1.A, R28.1, T1.E
- new net UART0_TX: D1.C, R24.2, U10.P0.TX
- new net UART1_RX: R27.1, T2.C, U10.P1.RX
- new net UART1_TRX: CON15-2.S, D2.A, R29.1, T2.E
- new net UART1_TX: D2.C, R25.2, U10.P1.TX
- new net UART2_RX: R32.1, T3.C, U10.P2.RX
- new net UART2_TRX: CON16-2.S, D3.A, R34.1, T3.E
- new net UART2_TX: D3.C, R30.2, U10.P2.TX
- new net UART3_RX: R33.1, T4.C, U10.P3(HD).RX
- new net UART3_TRX: CON17-2.S, D4.A, R35.1, T4.E
- new net UART3_TX: D4.C, R31.2, U10.P3(HD).TX
- new net VBUS: C17.C1, U1.AUX.5V0, U10.CTL.VBUS
- new net VIN: C20.C1, C24.C1, C26.C1, C38.C1, CON18-1.S, D11.C, D9.C, F1.1, R55.2, U16.EN/UV, U16.VIN
- new net VIN_VSENSE: C37.C1, R55.1, R56.2, U17.AIN
- net !ENABLE_PSU1: now also CON1-3.S, R8.1; no longer CON9-3.S, R13.1
- net !ENABLE_PSU2: now also CON2-3.S, R17.1; no longer CON10-3.S, R22.1
- net !PRESENT_PSU1: now also CON1-2.S, R7.1, R9.1; no longer CON9-2.S, R12.1, R14.1
- net !PRESENT_PSU2: now also CON2-2.S, R16.1, R18.1; no longer CON10-2.S, R21.1, R23.1
- net 12V0SB_PSU1: now also C2.C1, CON1-1.S, U2.VIN; no longer C8.C1, CON9-1.S, U4.VIN
- net 12V0SB_PSU2: now also C8.C1, CON2-1.S, U6.VIN; no longer C14.C1, CON10-1.S, U8.VIN
- net 3V3: now also C13.C1, C14.C1, C16.C1, C18.C1, C19.C1, C21.C1, C3.C1, C32.C1, C33.C1, CON10-1.S, CON11-1.S, CON12-1.S, CON13-1.S, CON9-1.S, R10.2, R11.2, R19.2, R20.2, R23.2, R26.2, R27.2, R28.2, R29.2, R32.2, R33.2, R34.2, R35.2, R36.2, R37.2, R38.2, R39.2, R40.2, R41.2, R42.2, R43.2, R44.2, R45.2, R46.2, R48.2, U10.CTL.VDD, U10.CTL.VIO@0, U10.CTL.VIO@1, U10.CTL.VIOHD, U10.CTL.VREGIN, U12.SLPZ, U12.VCC, U13.VCC, U14.VDD, U15.SNS, U4.VCC, U5.VDD@0, U8.VCC, U9.VDD@0; no longer C1.C1, C17.C1, C6.C1, CON2-1.S, R15.2, R16.2, R24.2, R25.2, R5.2, R6.2, R7.2, R8.2, U10.VCC, U11.VDD@0, U2.VCC, U3.SNS, U6.VCC, U7.VDD@0
- net 3V3SB_PSU1: now also C1.C1, C4.C1, C6.C1, R12.2, R13.2, R6.2, R9.2, U2.VOUT, U3.VDD, U5.VDD@1; no longer C10.C1, C12.C1, C7.C1, R11.2, R14.2, R17.2, R18.2, U4.VOUT, U5.VDD, U7.VDD@1
- net 3V3SB_PSU2: now also C10.C1, C12.C1, C7.C1, R15.2, R18.2, R21.2, R22.2, U6.VOUT, U7.VDD, U9.VDD@1; no longer C13.C1, C16.C1, C18.C1, R20.2, R23.2, R26.2, R27.2, U11.VDD@1, U8.VOUT, U9.VDD
- net 3V3_FB: now also R48.1, R49.2, U15.FB; no longer R8.1, R9.2, U3.FB
- net 3V3_SOFTSTART: now also C25.C1, U15.SS; no longer C4.C1, U3.SS
- net 3V3_SW: now also U15.SW; no longer U3.SW
- net 5V0: now also C22.C1, C23.C1, C31.C1, C34.C1, C35.C1, C36.C1, L2.2, R50.2, R54.2, U15.EN, U15.VIN@0, U15.VIN@1, U16.BIAS; no longer C2.C1, C3.C1, D1.C, F1.2, U1.AUX.5V0, U3.EN, U3.VIN@0, U3.VIN@1
- net GND: now also C13.C2, C14.C2, C16.C2, C18.C2, C19.C2, C20.C2, C21.C2, C22.C2, C23.C2, C24.C2, C25.C2, C26.C2, C27.C2, C28.C2, C29.C2, C30.C2, C32.C2, C33.C2, C34.C2, C35.C2, C36.C2, C37.C2, C38.C2, CON10-3.S, CON11-3.S, CON12-3.S, CON13-3.S, CON14-3.S, CON15-3.S, CON16-3.S, CON17-3.S, CON19-1.S, CON5-4.S, CON6-4.S, CON7-4.S, CON9-3.S, D10.C, D11.A, Q1.S, R14.1, R47.1, R49.1, R5.1, R51.1, R53.1, R56.1, U10.CTL.VSS@0, U10.CTL.VSS@1, U10.CTL.VSS@2, U10.CTL.VSSHD, U12.GND, U13.GND, U14.GND, U15.AGND, U15.PGND@0, U15.PGND@1, U16.GND, U17.VSS, U4.GND, U5.GND@0, U8.GND, U9.GND@0; no longer C1.C2, C2.C2, C4.C2, C6.C2, CON1-2.S, CON2-4.S, CON5-3.S, CON6-3.S, CON7-3.S, D1.A, R10.1, R19.1, R9.1, U10.GND, U11.GND@0, U2.GND, U3.AGND, U3.PGND@0, U3.PGND@1, U6.GND, U7.GND@0
- net GND_PSU1: now also C1.C2, C2.C2, C4.C2, C6.C2, CON1-6.S, U2.GND, U3.A0, U3.A1, U3.A2, U3.VSS, U5.GND@1; no longer C10.C2, C12.C2, C7.C2, C8.C2, CON9-6.S, U4.GND, U5.A0, U5.A1, U5.A2, U5.VSS, U7.GND@1
- net GND_PSU2: now also C10.C2, C12.C2, C7.C2, C8.C2, CON2-6.S, U6.GND, U7.A0, U7.A1, U7.A2, U7.VSS, U9.GND@1; no longer C13.C2, C14.C2, C16.C2, C18.C2, CON10-6.S, U11.GND@1, U8.GND, U9.A0, U9.A1, U9.A2, U9.VSS
- net I2C0_SCL: now also R1.1, U12.SCL, U13.SCLIN, U17.SCL; no longer R4.1, U10.SCLIN, U6.SCLIN
- net I2C0_SDA: now also R2.1, U12.SDA, U13.SDAIN, U17.SDA; no longer R5.1, U10.SDAIN, U6.SDAIN
- net I2C1_SCL: now also R3.1, U4.SCLIN, U8.SCLIN; no longer R6.1, U2.SCLIN
- net I2C1_SDA: now also R4.1, U4.SDAIN, U8.SDAIN; no longer R7.1, U2.SDAIN
- net I2C_SCL_EXT: now also CON5-3.S, CON6-3.S, CON7-3.S, R42.1, U13.SCLOUT; no longer CON2-3.S, R3.1, U2.SCLOUT
- net I2C_SCL_PSU1: now also CON1-4.S, R13.1, U3.SCL, U5.SCL@1; no longer CON9-4.S, R18.1, U5.SCL, U7.SCL@1
- net I2C_SCL_PSU2: now also CON2-4.S, R22.1, U7.SCL, U9.SCL@1; no longer CON10-4.S, R27.1, U11.SCL@1, U9.SCL
- net I2C_SDA_EXT: now also CON5-2.S, CON6-2.S, CON7-2.S, R41.1, U13.SDAOUT; no longer CON2-2.S, R2.1, U2.SDAOUT
- net I2C_SDA_PSU1: now also CON1-5.S, R12.1, U3.SDA, U5.SDA@1; no longer CON9-5.S, R17.1, U5.SDA, U7.SDA@1
- net I2C_SDA_PSU2: now also CON2-5.S, R21.1, U7.SDA, U9.SDA@1; no longer CON10-5.S, R26.1, U11.SDA@1, U9.SDA
- net N$1: now also R11.1, U4.SCLOUT, U5.SCL@0; no longer R16.1, U6.SCLOUT, U7.SCL@0
- net N$10: now also R16.2, U7.GP0; no longer R21.2, U9.GP0
- net N$13: now also R40.1, U13.ENABLE; no longer R1.1, U2.ENABLE
- net N$2: now also R10.1, U4.SDAOUT, U5.SDA@0; no longer R15.1, U6.SDAOUT, U7.SDA@0
- net N$3: now also R6.1, U3.!RESET; no longer R11.1, U5.!RESET
- net N$4: now also R8.2, U3.GP4; no longer R13.2, U5.GP4
- net N$5: now also R7.2, U3.GP0; no longer R12.2, U5.GP0
- net N$6: now also R20.1, U8.SCLOUT, U9.SCL@0; no longer R25.1, U10.SCLOUT, U11.SCL@0
- net N$7: now also R19.1, U8.SDAOUT, U9.SDA@0; no longer R24.1, U10.SDAOUT, U11.SDA@0
- net N$8: now also R15.1, U7.!RESET; no longer R20.1, U9.!RESET
- net N$9: now also R17.2, U7.GP4; no longer R22.2, U9.GP4
- net OW_BUS: now also CON10-2.S, CON11-2.S, CON12-2.S, CON13-2.S, CON9-2.S, U12.IO; no longer CON5-2.S, CON6-2.S, CON7-2.S
- net PSU1_I2C_EN: now also R5.2, U4.ENABLE; no longer R10.2, U6.ENABLE
- net PSU2_I2C_EN: now also R14.2, U8.ENABLE; no longer R19.2, U10.ENABLE
Other:
- note added: "I2C1 Addresses: IO EXP - 0x20 (EXP) PSU - 0x58 (EXP) PSU EEPROM - 0x50 I2C0 Addresses: DS2484 - 0x18 MCP3221-A0 - 0x48 (EXP) BME280 - 0x76 (EXP) ENS210 - 0x43 (EXP) MCP3421-A0 - 0x68 (EXP) LTC4151 - 0x6F (EXP) MCP23008 - 0x20 to 0x27 (EXP) MCP23017 - 0x20 to 0x27"
- note added: "Vout = ((R24/R25) + 1) * 0.97"
- note added: "f = 1 MHz DS. Eq. 3 & Table 1"

Commit message: Work on OPi dock
Parts:
- removed D1, D2, D3, D4: B0530W, Generic Diode:B0530W
- removed R32, R33, R34, R35: 1K Ohms, Resistor:RESISTOR-0603
- removed R43, R44, R45, R46: DNP, Resistor:RESISTOR-0603
- removed T1, T2, T3, T4: BC817, Generic BJT:BC817
- CON19: value 2EDG-2P -> 2EDG-2P-5MM; device Generic Connector:2EDG-2P -> Generic Connector:2EDG-2P-5MM
- LOGO1: value JS-5MM -> JS-10MM; device Silkscreen:JS-5MM -> Silkscreen:JS-10MM
- R24, R25, R30, R31: value 10K Ohms -> 100 Ohms
- R26, R27, R28, R29: value 1K Ohms -> 100 Ohms
Connections:
- removed net N$26: R24.1, T1.B
- removed net N$27: R25.1, T2.B
- removed net N$28: R30.1, T3.B
- removed net N$29: R31.1, T4.B
- removed net N$30: CON14-1.S, R43.1
- removed net N$31: CON17-1.S, R46.1
- removed net N$32: CON16-1.S, R45.1
- removed net N$33: CON15-1.S, R44.1
- removed net UART0_TRX: CON14-2.S, D1.A, R28.1, T1.E
- removed net UART1_TRX: CON15-2.S, D2.A, R29.1, T2.E
- removed net UART2_TRX: CON16-2.S, D3.A, R34.1, T3.E
- removed net UART3_TRX: CON17-2.S, D4.A, R35.1, T4.E
- new net N$12: CON14-2.S, R25.1
- new net N$14: CON14-1.S, R24.1
- new net N$16: CON15-2.S, R27.1
- new net N$17: CON15-1.S, R26.1
- new net N$20: CON16-2.S, R29.1
- new net N$21: CON16-1.S, R28.1
- new net N$23: CON17-2.S, R31.1
- new net N$24: CON17-1.S, R30.1
- net 3V3: no longer R26.2, R27.2, R28.2, R29.2, R32.2, R33.2, R34.2, R35.2, R43.2, R44.2, R45.2, R46.2
- net GND: now also U1.MAIN.GND@6, U1.MAIN.GND@7, U1.MAIN.GND@8, U1.MAIN.GND@9
- net UART0_RX: now also R25.2; no longer R26.1, T1.C
- net UART0_TX: no longer D1.C
- net UART1_RX: now also R27.2; no longer R27.1, T2.C
- net UART1_TX: now also R26.2; no longer D2.C, R25.2
- net UART2_RX: now also R29.2; no longer R32.1, T3.C
- net UART2_TX: now also R28.2; no longer D3.C, R30.2
- net UART3_RX: now also R31.2; no longer R33.1, T4.C
- net UART3_TX: now also R30.2; no longer D4.C, R31.2
Other:
- moved on the sheet: CON10-1, CON10-2, CON10-3, CON11-1, CON11-2, CON11-3, CON12-1, CON12-2, CON12-3, CON13-1, CON13-2, CON13-3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

Commit message: Work on OPi dock Added connector for reed switches for intrusion detection
Parts:
- removed D10: LED0603, LED:LED0603
- removed D11: SMAJ12A, TVS:SMAJ12A
- removed D9: B0530W, Generic Diode:B0530W
- removed R53: 10K Ohms, Resistor:RESISTOR-0603
- removed R54: 510 Ohms, Resistor:RESISTOR-0603
- removed R55: 147K Ohms, Resistor:RESISTOR-0603
- removed R56: 21K Ohms, Resistor:RESISTOR-0603
- removed U17: MCP3221-A0, Microchip:MCP3221-A0
- added CON20: 2EDG-2P-5MM, Generic Connector:2EDG-2P-5MM
- added D1, D2, D3: LED0603, LED:LED0603
- added R32, R35: 100 Ohms, Resistor:RESISTOR-0603
- added R33, R34: 1K Ohms, Resistor:RESISTOR-0603
- added R43: 41.2K Ohms, Resistor:RESISTOR-0603
- added R44: 309K Ohms, Resistor:RESISTOR-0603
- added R45: 71.5K Ohms, Resistor:RESISTOR-0603
- added R46: 1M Ohms, Resistor:RESISTOR-0603
- added U11: DS2484, Maxim Integrated:DS2484
- CON14: value 3P-SH-SIDE -> 3P-SH-TOP; device JST:3P-SH-SIDE -> JST:3P-SH-TOP
- CON18: value 2P-PH-TOP -> 3P-SH-SIDE; device JST:2P-PH-TOP -> JST:3P-SH-SIDE
- CON19: value 2EDG-2P-5MM -> 2P-PH-TOP; device Generic Connector:2EDG-2P-5MM -> JST:2P-PH-TOP
- CON3: value 4P-SH-SIDE -> 3P-SH-SIDE; device JST:4P-SH-SIDE -> JST:3P-SH-SIDE
- CON8: value 3P-SH-TOP -> 4P-SH-SIDE; device JST:3P-SH-TOP -> JST:4P-SH-SIDE
- D5: value LED0603 -> B0530W; device LED:LED0603 -> Generic Diode:B0530W; COLOR WHITE -> (none)
- D6: COLOR WHITE -> GREEN
- D7: value LED0603 -> SMAJ12A; device LED:LED0603 -> TVS:SMAJ12A; COLOR WHITE -> (none)
- LOGO1: value JS-10MM -> JS-5MM; device Silkscreen:JS-10MM -> Silkscreen:JS-5MM
- R24, R25, R26, R27: value 100 Ohms -> 330 Ohms
- R28, R29, R30: value 100 Ohms -> 10K Ohms
- R36, R37, R38, R39: value 330 Ohms -> 100 Ohms
- R40: value 10K Ohms -> 100 Ohms
- R41, R42: value 1K Ohms -> 100 Ohms
- R47: value 41.2K Ohms -> 226K Ohms
- R48: value 309K Ohms -> 22 Ohms
- R49: value 71.5K Ohms -> 10K Ohms
- R50: value 1M Ohms -> 510 Ohms
- R51: value 226K Ohms -> 147K Ohms
- R52: value 22 Ohms -> 21K Ohms
- U12: value DS2484 -> LTC4313-1; device Maxim Integrated:DS2484 -> Analog Devices:LTC4313-1
- U13: value LTC4313-1 -> MCP1525; device Analog Devices:LTC4313-1 -> Microchip:MCP1525
- U14: value MCP1525 -> MIC23155; device Microchip:MCP1525 -> Microchip:MIC23155
- U15: value MIC23155 -> LT8640S; device Microchip:MIC23155 -> Analog Devices:LT8640S
- U16: value LT8640S -> MCP3221-A0; device Analog Devices:LT8640S -> Microchip:MCP3221-A0
- U2, U6: value MCP1703-330 -> MCP1703-500; device Microchip:MCP1703-330 -> Microchip:MCP1703-500
- renumbered D8 to D4
Connections:
- net 3V3SB_PSU1 renamed 5V0SB_PSU1
- net 3V3SB_PSU2 renamed 5V0SB_PSU2
- new net LOWER_OPEN: R29.1, R32.2, U1.MAIN.(UART2_RX)PA1
- new net N$26: CON3-2.S, R32.1
- new net N$27: CON3-1.S, R31.1
- new net UPPER_OPEN: R30.1, R31.2, U1.MAIN.(UART2_TX)PA0
- net !UART1_ACTIVE: now also D3.C; no longer D7.C
- net !UART2_ACTIVE: now also D2.C; no longer D6.C
- net !UART3_ACTIVE: now also D1.C; no longer D5.C
- net 2V5_ADC_CLEAN: now also U13.VOUT, U16.VDD; no longer U14.VOUT, U17.VDD
- net 3V3: now also CON14-1.S, R24.2, R25.2, R26.2, R27.2, R28.2, R29.2, R30.2, R33.2, R34.2, R44.2, U11.SLPZ, U11.VCC, U13.VDD, U14.SNS; no longer CON3-1.S, R36.2, R37.2, R38.2, R39.2, R40.2, R41.2, R42.2, R48.2, U12.SLPZ, U13.VCC, U14.VDD, U15.SNS
- net 3V3_FB: now also R44.1, R45.2, U14.FB; no longer R48.1, R49.2, U15.FB
- net 3V3_SOFTSTART: now also U14.SS; no longer U15.SS
- net 3V3_SW: now also U14.SW; no longer U15.SW
- net 5V0: now also R46.2, U14.EN, U14.VIN@0, U14.VIN@1, U15.BIAS; no longer R54.2, U15.EN, U15.VIN@0, U15.VIN@1, U16.BIAS
- net 5V0_FB: now also R46.1, R47.2, U15.FB; no longer R50.1, R51.2, U16.FB
- net 5V0_INTVCC: now also U15.INTVCC, U15.SYNC/MODE; no longer U16.INTVCC, U16.SYNC/MODE
- net 5V0_RT: now also R43.2, U15.RT; no longer R47.2, U16.RT
- net 5V0_SS: now also U15.TR/SS; no longer U16.TR/SS
- net 5V0_SW: now also U15.SW; no longer U16.SW
- net FAN_PWM: now also R48.2; no longer R52.2
- net GND: now also CON18-3.S, CON20-1.S, CON3-3.S, CON8-4.S, D6.C, D7.A, R43.1, R45.1, R52.1, U11.GND, U14.AGND, U14.PGND@0, U14.PGND@1, U15.GND, U16.VSS; no longer CON19-1.S, CON3-4.S, CON8-3.S, D10.C, D11.A, R51.1, R53.1, R56.1, U14.GND, U15.AGND, U15.PGND@0, U15.PGND@1, U16.GND, U17.VSS
- net I2C0_SCL: now also U11.SCL, U12.SCLIN, U16.SCL; no longer U12.SCL, U13.SCLIN, U17.SCL
- net I2C0_SDA: now also U11.SDA, U12.SDAIN, U16.SDA; no longer U12.SDA, U13.SDAIN, U17.SDA
- net I2C_SCL_EXT: now also CON8-3.S, R34.1, U12.SCLOUT; no longer CON3-3.S, R42.1, U13.SCLOUT
- net I2C_SDA_EXT: now also CON8-2.S, R33.1, U12.SDAOUT; no longer CON3-2.S, R41.1, U13.SDAOUT
- net N$12: now also CON15-2.S, R36.1; no longer CON14-2.S, R25.1
- net N$13: now also R28.1, U12.ENABLE; no longer R40.1, U13.ENABLE
- net N$14: now also CON15-1.S, R35.1; no longer CON14-1.S, R24.1
- net N$149: now also D6.A, R50.1; no longer D10.A, R54.1
- net N$15: now also R27.1; no longer R39.1
- net N$16: now also CON16-2.S, R38.1; no longer CON15-2.S, R27.1
- net N$17: now also CON16-1.S, R37.1; no longer CON15-1.S, R26.1
- net N$18: now also D3.A, R26.1; no longer D7.A, R38.1
- net N$19: now also CON20-2.S; no longer CON19-2.S
- net N$20: now also CON17-2.S, R40.1; no longer CON16-2.S, R29.1
- net N$21: now also CON17-1.S, R39.1; no longer CON16-1.S, R28.1
- net N$22: now also D2.A, R25.1; no longer D6.A, R37.1
- net N$23: now also CON18-2.S, R42.1; no longer CON17-2.S, R31.1
- net N$24: now also CON18-1.S, R41.1; no longer CON17-1.S, R30.1
- net N$25: now also D1.A, R24.1; no longer D5.A, R36.1
- net N$34: now also CON19-2.S, D5.A; no longer CON18-2.S, D9.A
- net N$35: now also R48.1, R49.2; no longer R52.1, R53.2
- net OW_BUS: now also CON14-2.S, U11.IO; no longer CON8-2.S, U12.IO
- net UART0_RX: now also R36.2; no longer R25.2
- net UART0_TX: now also R35.2; no longer R24.2
- net UART1_RX: now also R38.2; no longer R27.2
- net UART1_TX: now also R37.2; no longer R26.2
- net UART2_RX: now also R40.2; no longer R29.2
- net UART2_TX: now also R39.2; no longer R28.2
- net UART3_RX: now also R42.2; no longer R31.2
- net UART3_TX: now also R41.2; no longer R30.2
- net VIN: now also CON19-1.S, D5.C, D7.C, R51.2, U15.EN/UV, U15.VIN; no longer CON18-1.S, D11.C, D9.C, R55.2, U16.EN/UV, U16.VIN
- net VIN_VSENSE: now also R51.1, R52.2, U16.AIN; no longer R55.1, R56.2, U17.AIN
Other:
- note added: "Vout = ((R46/R47) + 1) * 0.97"
- note removed: "Vout = ((R24/R25) + 1) * 0.97"
- moved on the sheet: CON10-1, CON10-2, CON10-3, CON11-1, CON11-2, CON11-3, CON12-1, CON12-2, CON12-3, CON13-1, CON13-2, CON13-3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

Commit message: Finish routing OPi dock PCB
Parts:
- removed C13, C14, C15, C16, C17: 100nF, Capacitor:CAPACITOR-0603
- removed CON14: 3P-SH-TOP, JST:3P-SH-TOP
- removed CON15, CON16, CON17, CON18: 3P-SH-SIDE, JST:3P-SH-SIDE
- removed D1, D2, D3, D4: LED0603, LED:LED0603
- removed R23: 10K Ohms, Resistor:RESISTOR-0603
- removed R24, R25, R26, R27: 330 Ohms, Resistor:RESISTOR-0603
- removed R38, R39, R40, R41, R42: 100 Ohms, Resistor:RESISTOR-0603
- removed U10: CP2108, Silicon Labs:CP2108
- added C39: 100nF, Capacitor:CAPACITOR-0603
- added U17: LTC4313-1, Analog Devices:LTC4313-1
- CON10, CON13, CON9: value 3P-SH-TOP -> 4P-SH-SIDE; device JST:3P-SH-TOP -> JST:4P-SH-SIDE
- CON11, CON12: value 3P-SH-TOP -> 3P-SH-SIDE; device JST:3P-SH-TOP -> JST:3P-SH-SIDE
- R35: value 100 Ohms -> 10K Ohms
- R36, R37: value 100 Ohms -> 1K Ohms
Connections:
- net I2C_SCL_EXT renamed I2C_SCL_EXT0
- net I2C_SDA_EXT renamed I2C_SDA_EXT0
- removed net !UART0_ACTIVE: D4.C, U10.P0.DTR
- removed net !UART1_ACTIVE: D3.C, U10.P1.DTR
- removed net !UART2_ACTIVE: D2.C, U10.P2.DTR
- removed net !UART3_ACTIVE: D1.C, U10.P3(HD).DTR
- removed net N$11: R23.1, U10.CTL.!RST
- removed net N$12: CON15-2.S, R36.1
- removed net N$13: R28.1, U12.ENABLE
- removed net N$14: CON15-1.S, R35.1
- removed net N$15: D4.A, R27.1
- removed net N$16: CON16-2.S, R38.1
- removed net N$17: CON16-1.S, R37.1
- removed net N$18: D3.A, R26.1
- removed net N$20: CON17-2.S, R40.1
- removed net N$21: CON17-1.S, R39.1
- removed net N$22: D2.A, R25.1
- removed net N$23: CON18-2.S, R42.1
- removed net N$24: CON18-1.S, R41.1
- removed net N$25: D1.A, R24.1
- removed net SBC_USB_DM2: U1.AUX.USB_DM2, U10.CTL.D-
- removed net SBC_USB_DP2: U1.AUX.USB_DP2, U10.CTL.D+
- removed net UART0_RX: R36.2, U10.P0.RX
- removed net UART0_TX: R35.2, U10.P0.TX
- removed net UART1_RX: R38.2, U10.P1.RX
- removed net UART1_TX: R37.2, U10.P1.TX
- removed net UART2_RX: R40.2, U10.P2.RX
- removed net UART2_TX: R39.2, U10.P2.TX
- removed net UART3_RX: R42.2, U10.P3(HD).RX
- removed net UART3_TX: R41.2, U10.P3(HD).TX
- removed net VBUS: C17.C1, U1.AUX.5V0, U10.CTL.VBUS
- new net EXT_I2C_EN0: R28.2, U1.MAIN.PA6, U12.ENABLE
- new net EXT_I2C_EN1: R35.2, U1.MAIN.(UART2_RTS)PA2, U17.ENABLE
- new net I2C_SCL_EXT1: CON10-3.S, CON13-3.S, CON9-3.S, R37.1, U17.SCLOUT
- new net I2C_SDA_EXT1: CON10-2.S, CON13-2.S, CON9-2.S, R36.1, U17.SDAOUT
- net 3V3: now also C39.C1, R36.2, R37.2, U17.VCC; no longer C13.C1, C14.C1, C15.C1, C16.C1, CON14-1.S, R23.2, R24.2, R25.2, R26.2, R27.2, R28.2, U10.CTL.VDD, U10.CTL.VIO@0, U10.CTL.VIO@1, U10.CTL.VIOHD, U10.CTL.VREGIN
- net GND: now also C39.C2, CON10-4.S, CON13-4.S, CON9-4.S, R28.1, R35.1, U17.GND; no longer C13.C2, C14.C2, C15.C2, C16.C2, C17.C2, CON10-3.S, CON13-3.S, CON14-3.S, CON15-3.S, CON16-3.S, CON17-3.S, CON18-3.S, CON9-3.S, U10.CTL.VSS@0, U10.CTL.VSS@1, U10.CTL.VSS@2, U10.CTL.VSSHD
- net I2C0_SCL: now also U17.SCLIN
- net I2C0_SDA: now also U17.SDAIN
- net OW_BUS: no longer CON10-2.S, CON13-2.S, CON14-2.S, CON9-2.S

Commit message: Work on PCBs
Parts:
- U13: value MCP1525 -> REF3030AIDBZ; device Microchip:MCP1525 -> Texas Instruments:REF3030AIDBZ
Connections:
- net 2V5_ADC_CLEAN renamed 3V0_ADC_CLEAN
Changed lines of the file:
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@@
 <part name="U11" library="Maxim Integrated" deviceset="DS2484" device=""/>
 <part name="U16" library="Microchip" deviceset="MCP3221-A*" device="" technology="0"/>
-<part name="U13" library="Microchip" deviceset="MCP1525" device=""/>
+<part name="U13" library="Texas Instruments" deviceset="REF30*AIDBZ" device="" technology="30"/>
 <part name="3V64" library="Supply Symbol" deviceset="3V3" device=""/>
 <part name="GND45" library="Supply Symbol" deviceset="GND" device=""/>
@@
 </segment>
 </net>
-<net name="2V5_ADC_CLEAN" class="0">
+<net name="3V0_ADC_CLEAN" class="0">
 <segment>
 <pinref part="U16" gate="G$1" pin="VDD"/>
