File: pcb/pa-tec-controller/qo-100-pa-tec-controller.brd (EAGLE design)
At the start: 70 x 80 mm, 91 parts, among them CON1 2EDG-2P-5MM, CON2 2EDG-2P-5MM, CON3 2EDG-2P-5MM, CON4 2EDG-2P-5MM, CON5 2EDG-2P-5MM, U1 LT8640S, U2 LT8640S, U3 LT8640S, U4 LT8640S, U5 MCP4728-A2

Commit message: PA TEC Controller assembly BOM changes
Parts:
- C15, C25, C31, C6: value 10nF -> 68nF
Changed lines of the file:
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@@
 <attribute name="VOLTAGE" value="35V" x="11.2" y="26.4" size="1.778" layer="27" rot="R90" display="off"/>
 </element>
-<element name="C6" library="Capacitor" package="CAP0603" value="10nF" x="48.2" y="27.9" smashed="yes" rot="R270">
+<element name="C6" library="Capacitor" package="CAP0603" value="68nF" x="48.2" y="27.9" smashed="yes" rot="R270">
 <attribute name="NAME" x="49.684" y="26.4536" size="0.8" layer="25" font="vector" ratio="10" rot="SR90" align="center-left"/>
 <attribute name="VALUE" x="46.168" y="30.8464" size="0.8" layer="27" font="vector" ratio="10" rot="SR270" align="center-left"/>
@@
 <attribute name="VOLTAGE" value="35V" x="11.3" y="3.4" size="1.778" layer="27" rot="R90" display="off"/>
 </element>
-<element name="C15" library="Capacitor" package="CAP0603" value="10nF" x="48.2" y="4.9" smashed="yes" rot="R270">
+<element name="C15" library="Capacitor" package="CAP0603" value="68nF" x="48.2" y="4.9" smashed="yes" rot="R270">
 <attribute name="NAME" x="49.584" y="3.3536" size="0.8" layer="25" font="vector" ratio="10" rot="SR90" align="center-left"/>
 <attribute name="VALUE" x="46.168" y="7.8464" size="0.8" layer="27" font="vector" ratio="10" rot="SR270" align="center-left"/>
@@
 <attribute name="VOLTAGE" value="35V" x="39.1" y="52.9" size="1.778" layer="27" rot="R270" display="off"/>
 </element>
-<element name="C25" library="Capacitor" package="CAP0603" value="10nF" x="4.3" y="51.4" smashed="yes" rot="R90">
+<element name="C25" library="Capacitor" package="CAP0603" value="68nF" x="4.3" y="51.4" smashed="yes" rot="R90">
 <attribute name="NAME" x="3.1536" y="53.516" size="0.8" layer="25" font="vector" ratio="10" rot="SR0" align="center-left"/>
 <attribute name="VALUE" x="6.332" y="48.4536" size="0.8" layer="27" font="vector" ratio="10" rot="SR90" align="center-left"/>
@@
 <attribute name="VOLTAGE" value="35V" x="7.2" y="32.6" locked="yes" size="1.778" layer="27" rot="R90" display="off"/>
 </element>
-<element name="C31" library="Capacitor" package="CAP0603" value="10nF" x="48.2" y="50.9" locked="yes" smashed="yes" rot="R270">
+<element name="C31" library="Capacitor" package="CAP0603" value="68nF" x="48.2" y="50.9" locked="yes" smashed="yes" rot="R270">
 <attribute name="NAME" x="49.684" y="49.3536" size="0.8" layer="25" font="vector" ratio="10" rot="SR90" align="center-left"/>
 <attribute name="VALUE" x="46.168" y="53.8464" size="0.8" layer="27" font="vector" ratio="10" rot="SR270" align="center-left"/>
