File: pcb/pa-bias-controller/qo-100-pa-bias-controller.brd (EAGLE design)
At the start: 70 x 80 mm, 115 parts, among them CON1 3P-SH-SIDE, CON2 2EDG-5P-5MM, CON3 2EDG-5P-5MM, CON4 2EDG-2P-5MM, CON5 2P-SH-SIDE, CON6 2P-SH-SIDE, U1 EFM32TG11B120F128GM32, U2 MCP1501-25, U3 MAX11300, U4 MAX44285TAUA+, U5 MIC23155, U6 LT8636

Commit message: PA Bias Controller assembly BOM changes
Parts:
- C15, C16: value DNP -> 100nF
- C40, C44: value 10uF -> 22uF
- C45: value DNP -> 10nF
- C46: value DNP -> 10pF
- R10: value 10K Ohms -> 1\K Ohms
- R11, R12, R19, R20: value 0 Ohms -> 1K Ohms
- R13, R15: value 0.012 Ohms -> DNP
- R14: value 0.012 Ohms -> 0.1 Ohms
- R2, R3: value 0 Ohms -> 100 Ohms
- R21, R22: value 250 Ohms -> 255 Ohms
- R7, R9: value 130K Ohms -> 15K Ohms
- R8: value 10K Ohms -> 1K Ohms

Commit message: Update I2C slave resistors to minimize load effect when powered down
Parts:
- R2, R3: value 100 Ohms -> 1K Ohms
- R39, R40: value 1K Ohms -> 47K Ohms
Changed lines of the file:
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@@
 <attribute name="VALUE" x="0.095" y="42.92" size="0.8" layer="27" font="vector" ratio="10" align="center-left"/>
 </element>
-<element name="R2" library="Resistor" package="RES0603" value="100 Ohms" x="8.5" y="49.7" smashed="yes">
+<element name="R2" library="Resistor" package="RES0603" value="1K Ohms" x="8.5" y="49.7" smashed="yes">
 <attribute name="NAME" x="10.2456" y="49.716" size="0.8" layer="25" font="vector" ratio="10" rot="SR0" align="center-left"/>
 <attribute name="TOLERANCE" value="" x="-15.8" y="16.1" size="1.778" layer="27" display="off"/>
 <attribute name="VALUE" x="5.0456" y="47.668" size="0.8" layer="27" font="vector" ratio="10" rot="SR0" align="center-left"/>
 </element>
-<element name="R3" library="Resistor" package="RES0603" value="100 Ohms" x="8.5" y="48" smashed="yes">
+<element name="R3" library="Resistor" package="RES0603" value="1K Ohms" x="8.5" y="48" smashed="yes">
 <attribute name="NAME" x="10.2456" y="48.016" size="0.8" layer="25" font="vector" ratio="10" rot="SR0" align="center-left"/>
 <attribute name="TOLERANCE" value="" x="-23.4" y="9.3" size="1.778" layer="27" display="off"/>
@@
 <attribute name="NAME" x="13.4" y="49.7" size="0.8" layer="25" font="vector" ratio="10" align="center-left"/>
 </element>
-<element name="R39" library="Resistor" package="RES0603" value="1K Ohms" x="8.5" y="42.9" smashed="yes">
+<element name="R39" library="Resistor" package="RES0603" value="47K Ohms" x="8.5" y="42.9" smashed="yes">
 <attribute name="NAME" x="4.8456" y="42.916" size="0.8" layer="25" font="vector" ratio="10" rot="SR0" align="center-left"/>
 <attribute name="TOLERANCE" value="" x="8.5" y="42.9" size="1.778" layer="27" display="off"/>
 <attribute name="VALUE" x="5.0456" y="40.868" size="0.8" layer="27" font="vector" ratio="10" rot="SR0" align="center-left"/>
 </element>
-<element name="R40" library="Resistor" package="RES0603" value="1K Ohms" x="8.5" y="44.6" smashed="yes">
+<element name="R40" library="Resistor" package="RES0603" value="47K Ohms" x="8.5" y="44.6" smashed="yes">
 <attribute name="NAME" x="4.8456" y="44.616" size="0.8" layer="25" font="vector" ratio="10" rot="SR0" align="center-left"/>
 <attribute name="TOLERANCE" value="" x="8.5" y="44.6" size="1.778" layer="27" display="off"/>

Commit message: Revert I2C resistor chnges because they do not work
Parts:
- R2, R3: value 1K Ohms -> 100 Ohms
- R39, R40: value 47K Ohms -> 1K Ohms
Changed lines of the file:
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@@
 <attribute name="VALUE" x="0.095" y="42.92" size="0.8" layer="27" font="vector" ratio="10" align="center-left"/>
 </element>
-<element name="R2" library="Resistor" package="RES0603" value="1K Ohms" x="8.5" y="49.7" smashed="yes">
+<element name="R2" library="Resistor" package="RES0603" value="100 Ohms" x="8.5" y="49.7" smashed="yes">
 <attribute name="NAME" x="10.2456" y="49.716" size="0.8" layer="25" font="vector" ratio="10" rot="SR0" align="center-left"/>
 <attribute name="TOLERANCE" value="" x="-15.8" y="16.1" size="1.778" layer="27" display="off"/>
 <attribute name="VALUE" x="5.0456" y="47.668" size="0.8" layer="27" font="vector" ratio="10" rot="SR0" align="center-left"/>
 </element>
-<element name="R3" library="Resistor" package="RES0603" value="1K Ohms" x="8.5" y="48" smashed="yes">
+<element name="R3" library="Resistor" package="RES0603" value="100 Ohms" x="8.5" y="48" smashed="yes">
 <attribute name="NAME" x="10.2456" y="48.016" size="0.8" layer="25" font="vector" ratio="10" rot="SR0" align="center-left"/>
 <attribute name="TOLERANCE" value="" x="-23.4" y="9.3" size="1.778" layer="27" display="off"/>
@@
 <attribute name="NAME" x="13.4" y="49.7" size="0.8" layer="25" font="vector" ratio="10" align="center-left"/>
 </element>
-<element name="R39" library="Resistor" package="RES0603" value="47K Ohms" x="8.5" y="42.9" smashed="yes">
+<element name="R39" library="Resistor" package="RES0603" value="1K Ohms" x="8.5" y="42.9" smashed="yes">
 <attribute name="NAME" x="4.8456" y="42.916" size="0.8" layer="25" font="vector" ratio="10" rot="SR0" align="center-left"/>
 <attribute name="TOLERANCE" value="" x="8.5" y="42.9" size="1.778" layer="27" display="off"/>
 <attribute name="VALUE" x="5.0456" y="40.868" size="0.8" layer="27" font="vector" ratio="10" rot="SR0" align="center-left"/>
 </element>
-<element name="R40" library="Resistor" package="RES0603" value="47K Ohms" x="8.5" y="44.6" smashed="yes">
+<element name="R40" library="Resistor" package="RES0603" value="1K Ohms" x="8.5" y="44.6" smashed="yes">
 <attribute name="NAME" x="4.8456" y="44.616" size="0.8" layer="25" font="vector" ratio="10" rot="SR0" align="center-left"/>
 <attribute name="TOLERANCE" value="" x="8.5" y="44.6" size="1.778" layer="27" display="off"/>
