File: pcb/gpsdo/qo-100-gpsdo.sch (EAGLE design)
At the start: 220 parts, among them J1 DCJACK, U1 ICE40HX8K-SG32, U10 74LVC1G17, U11 74LVC1G17, U12 74LVC1G17, U13 74LVC1G17, U14 74LVC1G17, U15 74LVC1G17, U16 74LVC1G17, U17 74LVC1G17, U18 74LVC1G17, U19 MIC23159, U2 MCP1700-330, U20 ADP150UJZ-3.3, U21 ADP3334, U22 LT8636, U23 EFM32GG12B810F1024GM64, U3 NEO-7M, U4 MCP1501-25, U5 AD5541A, U6 MCP6V32, U7 OSC5A2B02, U8 74LVC1G17, U9 SI5351C

Commit message: GPSDO progress Added general filter PCB
Parts:
- added CON1: 3P-SH-TOP, JST:3P-SH-TOP
- D2: COLOR (none) -> GREEN
Connections:
- new net GPS_PROG_RXD: CON1-2.S, U3.RXD2
- new net GPS_PROG_TXD: CON1-1.S, U3.TXD2
- net GND: now also CON1-3.S
- net GPS_RXD: now also U3.RXD1; no longer U3.RXD
- net GPS_TXD: now also U3.TXD1; no longer U3.TXD
Other:
- note added: "Can be replaced with ATGM332D-5N"
- note added: "DNP if GPS module is ATGM332D-5N"
- note added: "DNP if GPS module is NEO-XX"
- moved on the sheet: C3, C4, C5, D1, D2, R1, R2, R3, R4, R5, R7, U2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

Commit message: Change some leaded packages to DFN
Parts:
- U5: value AD5541A -> AD5541ACPZ; device Analog Devices:AD5541A -> Analog Devices:AD5541ACPZ
- U6: value MCP6V32 -> MCP6V32-E/MNY; device Microchip:MCP6V32 -> Microchip:MCP6V32-E/MNY
Other:
- moved on the sheet: U5, U6.PWR
Changed lines of the file:
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@@
 <part name="FRAME1" library="Frame" deviceset="A2-LANDSCAPE" device=""/>
 <part name="LOGO1" library="Silkscreen" deviceset="JS" device="-5MM"/>
-<part name="U5" library="Analog Devices" deviceset="AD5541A" device=""/>
-<part name="U6" library="Microchip" deviceset="MCP6V32" device=""/>
+<part name="U5" library="Analog Devices" deviceset="AD5541A?" device="CPZ"/>
+<part name="U6" library="Microchip" deviceset="MCP6V32" device="-E/MNY"/>
 <part name="U4" library="Microchip" deviceset="MCP1501-*" device="" technology="25"/>
 <part name="U14" library="Logic" deviceset="74LVC1G17" device=""/>

Commit message: Update SI5351 library on GPSDO
Parts:
- U9: value SI5351C -> SI5351C-B-GM; device Silicon Labs:SI5351C -> Silicon Labs:SI5351C-B-GM
Changed lines of the file:
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@@
 <part name="GND6" library="Supply Symbol" deviceset="GND" device=""/>
 <part name="R12" library="Resistor" deviceset="RESISTOR" device="-0603" value="10K Ohms"/>
-<part name="U9" library="Silicon Labs" deviceset="SI5351C" device=""/>
+<part name="U9" library="Silicon Labs" deviceset="SI5351C-B-GM" device=""/>
 <part name="U3" library="U-Blox" deviceset="NEO-7*" device="" technology="M"/>
 <part name="3V1" library="Supply Symbol" deviceset="3V3" device=""/>

Commit message: Work on GPSDO schematic
Parts:
- added R44: 10K Ohms, Resistor:RESISTOR-0603
- U4: value MCP1501-25 -> MCP1501-40; device Microchip:MCP1501-25 -> Microchip:MCP1501-40
Connections:
- new net N$32: R44.1, U6.2.+IN
- net N$8: now also R44.2; no longer U6.2.+IN
Other:
- moved on the sheet: C19, R11, R12, U6.2
Changed lines of the file:
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@@
 <part name="U5" library="Analog Devices" deviceset="AD5541A?" device="CPZ"/>
 <part name="U6" library="Microchip" deviceset="MCP6V32" device="-E/MNY"/>
-<part name="U4" library="Microchip" deviceset="MCP1501-*" device="" technology="25"/>
+<part name="U4" library="Microchip" deviceset="MCP1501-*" device="" technology="40" value="MCP1501-40"/>
 <part name="U14" library="Logic" deviceset="74LVC1G17" device=""/>
 <part name="R25" library="Resistor" deviceset="RESISTOR" device="-0603" value="100 Ohms"/>
@@
 <part name="CON1" library="JST" deviceset="3P" device="-SH-TOP"/>
 <part name="GND103" library="Supply Symbol" deviceset="GND" device=""/>
+<part name="R44" library="Resistor" deviceset="RESISTOR" device="-0603" value="10K Ohms"/>
 </parts>
 <sheets>
@@
 <attribute name="VALUE" x="320.04" y="168.91" size="1.27" layer="96"/>
 </instance>
-<instance part="U6" gate=".2" x="381" y="162.56" smashed="yes">
-<attribute name="NAME" x="383.54" y="168.656" size="1.27" layer="95"/>
-<attribute name="VALUE" x="383.54" y="166.37" size="1.27" layer="96"/>
+<instance part="U6" gate=".2" x="391.16" y="162.56" smashed="yes">
+<attribute name="NAME" x="393.7" y="168.656" size="1.27" layer="95"/>
+<attribute name="VALUE" x="393.7" y="166.37" size="1.27" layer="96"/>
 </instance>
 <instance part="U6" gate=".PWR" x="40.64" y="312.42" smashed="yes">
@@
 <attribute name="VALUE" x="165.1" y="163.83" size="1.27" layer="96"/>
 </instance>
-<instance part="R11" gate="G$1" x="363.22" y="142.24" smashed="yes" rot="R270">
-<attribute name="VALUE" x="360.4514" y="142.24" size="1.778" layer="96" ratio="10" rot="SR270" align="top-left"/>
-<attribute name="NAME" x="365.9886" y="142.24" size="1.778" layer="95" ratio="10" rot="SR270"/>
-<attribute name="TOLERANCE" x="357.9114" y="142.24" size="1.778" layer="97" ratio="10" rot="SR270" align="top-left"/>
-</instance>
-<instance part="GND6" gate="G$1" x="363.22" y="121.92" smashed="yes">
-<attribute name="VALUE" x="363.22" y="116.84" size="1.778" layer="96" align="bottom-center"/>
-</instance>
-<instance part="R12" gate="G$1" x="373.38" y="149.86" smashed="yes">
-<attribute name="VALUE" x="373.38" y="147.0914" size="1.778" layer="96" ratio="10" rot="SR0" align="top-left"/>
-<attribute name="NAME" x="373.38" y="152.6286" size="1.778" layer="95" ratio="10" rot="SR0"/>
-<attribute name="TOLERANCE" x="373.38" y="144.5514" size="1.778" layer="97" ratio="10" rot="SR0" align="top-left"/>
+<instance part="R11" gate="G$1" x="373.38" y="142.24" smashed="yes" rot="R270">
+<attribute name="VALUE" x="370.6114" y="142.24" size="1.778" layer="96" ratio="10" rot="SR270" align="top-left"/>
+<attribute name="NAME" x="376.1486" y="142.24" size="1.778" layer="95" ratio="10" rot="SR270"/>
+<attribute name="TOLERANCE" x="368.0714" y="142.24" size="1.778" layer="97" ratio="10" rot="SR270" align="top-left"/>
+</instance>
+<instance part="GND6" gate="G$1" x="373.38" y="121.92" smashed="yes">
+<attribute name="VALUE" x="373.38" y="116.84" size="1.778" layer="96" align="bottom-center"/>
+</instance>
+<instance part="R12" gate="G$1" x="383.54" y="149.86" smashed="yes">
+<attribute name="VALUE" x="383.54" y="147.0914" size="1.778" layer="96" ratio="10" rot="SR0" align="top-left"/>
+<attribute name="NAME" x="383.54" y="152.6286" size="1.778" layer="95" ratio="10" rot="SR0"/>
+<attribute name="TOLERANCE" x="383.54" y="144.5514" size="1.778" layer="97" ratio="10" rot="SR0" align="top-left"/>
 </instance>
 <instance part="GND17" gate="G$1" x="238.76" y="121.92" smashed="yes">
@@
 <attribute name="VALUE" x="137.16" y="116.84" size="1.778" layer="96" align="bottom-center"/>
 </instance>
-<instance part="C19" gate="G$1" x="411.48" y="149.86" smashed="yes" rot="R270">
-<attribute name="VALUE" x="408.7114" y="149.86" size="1.778" layer="96" ratio="10" rot="SR270" align="top-left"/>
-<attribute name="NAME" x="414.2486" y="149.86" size="1.778" layer="95" ratio="10" rot="SR270"/>
-<attribute name="VOLTAGE" x="406.1714" y="149.86" size="1.778" layer="97" ratio="10" rot="SR270" align="top-left"/>
-</instance>
-<instance part="GND31" gate="G$1" x="411.48" y="121.92" smashed="yes">
-<attribute name="VALUE" x="411.48" y="116.84" size="1.778" layer="96" align="bottom-center"/>
+<instance part="C19" gate="G$1" x="421.64" y="149.86" smashed="yes" rot="R270">
+<attribute name="VALUE" x="418.8714" y="149.86" size="1.778" layer="96" ratio="10" rot="SR270" align="top-left"/>
+<attribute name="NAME" x="424.4086" y="149.86" size="1.778" layer="95" ratio="10" rot="SR270"/>
+<attribute name="VOLTAGE" x="416.3314" y="149.86" size="1.778" layer="97" ratio="10" rot="SR270" align="top-left"/>
+</instance>
+<instance part="GND31" gate="G$1" x="421.64" y="121.92" smashed="yes">
+<attribute name="VALUE" x="421.64" y="116.84" size="1.778" layer="96" align="bottom-center"/>
 </instance>
 <instance part="GND32" gate="G$1" x="411.48" y="281.94" smashed="yes">
@@
 <instance part="GND95" gate="G$1" x="396.24" y="322.58" smashed="yes">
 <attribute name="VALUE" x="396.24" y="317.5" size="1.778" layer="96" align="bottom-center"/>
+</instance>
+<instance part="R44" gate="G$1" x="358.14" y="165.1" smashed="yes">
+<attribute name="VALUE" x="358.14" y="162.3314" size="1.778" layer="96" ratio="10" rot="SR0" align="top-left"/>
+<attribute name="NAME" x="358.14" y="167.8686" size="1.778" layer="95" ratio="10" rot="SR0"/>
+<attribute name="TOLERANCE" x="358.14" y="159.7914" size="1.778" layer="97" ratio="10" rot="SR0" align="top-left"/>
 </instance>
 </instances>
@@
 <pinref part="GND6" gate="G$1" pin="GND"/>
 <pinref part="R11" gate="G$1" pin="1"/>
-<wire x1="363.22" y1="121.92" x2="363.22" y2="129.54" width="0.1524" layer="91"/>
+<wire x1="373.38" y1="121.92" x2="373.38" y2="129.54" width="0.1524" layer="91"/>
 </segment>
 <segment>
@@
 <pinref part="GND31" gate="G$1" pin="GND"/>
 <pinref part="C19" gate="G$1" pin="C2"/>
-<wire x1="411.48" y1="121.92" x2="411.48" y2="142.24" width="0.1524" layer="91"/>
+<wire x1="421.64" y1="121.92" x2="421.64" y2="142.24" width="0.1524" layer="91"/>
 </segment>
 <segment>
@@
 <pinref part="U6" gate=".1" pin="OUT"/>
 <wire x1="335.28" y1="165.1" x2="327.66" y2="165.1" width="0.1524" layer="91"/>
-<pinref part="U6" gate=".2" pin="+IN"/>
-<wire x1="370.84" y1="165.1" x2="347.98" y2="165.1" width="0.1524" layer="91"/>
 <junction x="335.28" y="165.1"/>
 <pinref part="C15" gate="G$1" pin="C1"/>
@@
 <wire x1="347.98" y1="149.86" x2="347.98" y2="165.1" width="0.1524" layer="91"/>
 <junction x="347.98" y="165.1"/>
+<wire x1="358.14" y1="165.1" x2="347.98" y2="165.1" width="0.1524" layer="91"/>
+<pinref part="R44" gate="G$1" pin="2"/>
 </segment>
 </net>
@@
 <segment>
 <pinref part="U6" gate=".2" pin="-IN"/>
-<wire x1="370.84" y1="160.02" x2="363.22" y2="160.02" width="0.1524" layer="91"/>
+<wire x1="381" y1="160.02" x2="373.38" y2="160.02" width="0.1524" layer="91"/>
 <pinref part="R11" gate="G$1" pin="2"/>
-<wire x1="363.22" y1="160.02" x2="363.22" y2="149.86" width="0.1524" layer="91"/>
+<wire x1="373.38" y1="160.02" x2="373.38" y2="149.86" width="0.1524" layer="91"/>
 <pinref part="R12" gate="G$1" pin="2"/>
-<wire x1="363.22" y1="149.86" x2="363.22" y2="142.24" width="0.1524" layer="91"/>
-<wire x1="373.38" y1="149.86" x2="363.22" y2="149.86" width="0.1524" layer="91"/>
-<junction x="363.22" y="149.86"/>
+<wire x1="373.38" y1="149.86" x2="373.38" y2="142.24" width="0.1524" layer="91"/>
+<wire x1="383.54" y1="149.86" x2="373.38" y2="149.86" width="0.1524" layer="91"/>
+<junction x="373.38" y="149.86"/>
 </segment>
 </net>
@@
 <segment>
 <pinref part="R12" gate="G$1" pin="1"/>
-<wire x1="386.08" y1="149.86" x2="398.78" y2="149.86" width="0.1524" layer="91"/>
-<wire x1="398.78" y1="149.86" x2="398.78" y2="162.56" width="0.1524" layer="91"/>
+<wire x1="396.24" y1="149.86" x2="408.94" y2="149.86" width="0.1524" layer="91"/>
+<wire x1="408.94" y1="149.86" x2="408.94" y2="162.56" width="0.1524" layer="91"/>
 <pinref part="U6" gate=".2" pin="OUT"/>
-<wire x1="398.78" y1="162.56" x2="391.16" y2="162.56" width="0.1524" layer="91"/>
+<wire x1="408.94" y1="162.56" x2="401.32" y2="162.56" width="0.1524" layer="91"/>
 <pinref part="C19" gate="G$1" pin="C1"/>
-<wire x1="398.78" y1="162.56" x2="411.48" y2="162.56" width="0.1524" layer="91"/>
-<wire x1="411.48" y1="162.56" x2="411.48" y2="149.86" width="0.1524" layer="91"/>
-<junction x="398.78" y="162.56"/>
-<wire x1="411.48" y1="162.56" x2="424.18" y2="162.56" width="0.1524" layer="91"/>
-<junction x="411.48" y="162.56"/>
-<label x="424.18" y="162.56" size="1.778" layer="95" xref="yes"/>
+<wire x1="408.94" y1="162.56" x2="421.64" y2="162.56" width="0.1524" layer="91"/>
+<wire x1="421.64" y1="162.56" x2="421.64" y2="149.86" width="0.1524" layer="91"/>
+<junction x="408.94" y="162.56"/>
+<wire x1="421.64" y1="162.56" x2="434.34" y2="162.56" width="0.1524" layer="91"/>
+<junction x="421.64" y="162.56"/>
+<label x="434.34" y="162.56" size="1.778" layer="95" xref="yes"/>
 </segment>
 <segment>
@@
 </segment>
 </net>
+<net name="N$32" class="0">
+<segment>
+<pinref part="U6" gate=".2" pin="+IN"/>
+<wire x1="381" y1="165.1" x2="370.84" y2="165.1" width="0.1524" layer="91"/>
+<pinref part="R44" gate="G$1" pin="1"/>
+</segment>
+</net>

Commit message: Work on GPSDO
Signed-off-by: João Silva <jgc3silva@gmail.com>
Parts:
- removed D5: SMAJ24A, TVS:SMAJ24A
- removed D6: LED0603, LED:LED0603
- removed U14, U15, U16, U17, U18: 74LVC1G17, Logic:74LVC1G17
- removed U19: MIC23159, Microchip:MIC23159
- removed U20: ADP150UJZ-3.3, Analog Devices:ADP150UJZ-3.3
- removed U21: ADP3334, Analog Devices:ADP3334
- removed U22: LT8636, Analog Devices:LT8636
- removed U23: EFM32GG12B810F1024GM64, EFM32:EFM32GG12B810F1024GM64
- removed USB1: USB-C-16P-SMD-FLAT-SIDE-TYPE-2, USB Connector:USB-C-16P-SMD-FLAT-SIDE-TYPE-2
- added C103, C114: 10uF, Capacitor:CAPACITOR-0603
- added C104, C105, C106, C107, C115, C116: 100nF, Capacitor:CAPACITOR-0603
- added C108: 10pF, Capacitor:CAPACITOR-0603
- added C109, C111, C112, C113: 100uF, Capacitor:CAPACITOR-1206
- added C110: 10nF, Capacitor:CAPACITOR-0603
- added C117, C118: 470pF, Capacitor:CAPACITOR-0603
- added C119: 10uF, Capacitor:CAPACITOR-1206
- added CON2: 2EDG-2P-5MM, Generic Connector:2EDG-2P-5MM
- added FB1, FB2, FB3, FB4, FB5, FB6: 1uH, Inductor:FERRITE-0805
- added L32, L33: 560nH, Inductor:INDUCTOR-0603
- added L34, L35, L36, L37: 68nH, Inductor:INDUCTOR-0603
- added L38, L39, L40, L41: 1uH, Inductor:INDUCTOR-0603
- added L42, L43, L44, L45: 330nH, Inductor:INDUCTOR-0603
- added L46, L47, L48, L49: 820nH, Inductor:INDUCTOR-0603
- added L50, L51, L52, L53: 220nH, Inductor:INDUCTOR-0603
- added L54, L55, L56, L57: 470nH, Inductor:INDUCTOR-0603
- added L58: 2.2uH, Inductor:INDUCTOR-3.2X3.5X1.5MM
- added L59: 4.7uH, Inductor:INDUCTOR-4X4MM
- added R45: 41.2K Ohms, Resistor:RESISTOR-0603
- added R46: 309K Ohms, Resistor:RESISTOR-0603
- added R47: 71.5K Ohms, Resistor:RESISTOR-0603
- added R48: 1M Ohms, Resistor:RESISTOR-0603
- added R49: 226K Ohms, Resistor:RESISTOR-0603
- added R50: 510 Ohms, Resistor:RESISTOR-0603
- added R51, R53: 100K Ohms, Resistor:RESISTOR-0603
- added R52: 10K Ohms, Resistor:RESISTOR-0603
- added R54: 75K Ohms, Resistor:RESISTOR-0603
- added RFCON11, RFCON12, RFCON13, RFCON14, RFCON15, RFCON16: RFCON-U.FL, RF Connector:RFCON-U.FL
- added TC1: TC2050-IDC, TagConnect:TC2050-IDC
- C1, C87: value 100uF -> 100nF; device Capacitor:CAPACITOR-1206 -> Capacitor:CAPACITOR-0603
- C100: value 1uF -> 10uF; VOLTAGE 50V -> (none)
- C101: value 100nF -> 10nF
- C102: value 10uF -> 100nF; device Capacitor:CAPACITOR-1206 -> Capacitor:CAPACITOR-0603; VOLTAGE 50V -> (none)
- C11, C3, C4, C85, C90, C91: value 1uF -> 100nF
- C12: value 10uF -> 47pF
- C16: value 100uF -> 10uF; device Capacitor:CAPACITOR-1206 -> Capacitor:CAPACITOR-0603
- C17, C18, C21, C23, C37, C42, C47, C48, C51, C55, C7: value 100nF -> 1uF
- C19: value 100nF -> 10uF
- C25, C8: value 100nF -> 100uF; device Capacitor:CAPACITOR-0603 -> Capacitor:CAPACITOR-1206
- C28, C30, C31: value 470pF -> 100nF
- C29: value 470pF -> 6pF
- C33: value 560pF -> 10uF
- C34, C35, C36, C54: value 560pF -> 1uF
- C38, C40, C56: value 510pF -> 1uF
- C39: value 510pF -> 10uF
- C41: value 510pF -> 6pF
- C43: value 200pF -> 10pF
- C44: value 200pF -> 10uF
- C45, C46, C71, C72: value 200pF -> 100nF
- C52: value 470pF -> 1uF
- C57, C73, C74: value 200pF -> 270pF
- C58, C75, C76: value 100nF -> 270pF
- C59, C60: value 470pF -> 270pF
- C61, C62, C83, C84: value 470pF -> 220pF
- C63, C64, C65, C66: value 560pF -> 220pF
- C67, C68: value 510pF -> 220pF
- C69, C70: value 510pF -> 100nF
- C77, C78, C79, C81: value 100nF -> 220pF
- C80: value 4.7uF -> 220pF
- C82: value 100uF -> 220pF; device Capacitor:CAPACITOR-1206 -> Capacitor:CAPACITOR-0603
- C89: value 4.7uF -> 100nF
- C92: value 470pF -> 4.7uF
- C93: value 1uF -> 4.7uF; VOLTAGE 50V -> 35V
- C94: value 4.7uF -> 10nF; VOLTAGE 35V -> (none)
- C95: value 10nF -> 1uF; VOLTAGE (none) -> 50V
- C96: VOLTAGE (none) -> 50V
- C97: value 100uF -> 10nF; device Capacitor:CAPACITOR-1206 -> Capacitor:CAPACITOR-0603
- C98: value 100nF -> 470pF
- C99: value 10pF -> 1uF
- D1: value SP0503BAHT -> LED0603; device TVS:SP0503BAHT -> LED:LED0603; COLOR (none) -> BLUE
- D2: value LED0603 -> B0530W; device LED:LED0603 -> Generic Diode:B0530W; COLOR GREEN -> (none)
- D3: value B0530W -> LED0603; device Generic Diode:B0530W -> LED:LED0603; COLOR (none) -> GREEN
- D4: value LED0603 -> SMAJ24A; device LED:LED0603 -> TVS:SMAJ24A; COLOR GREEN -> (none)
- L1: value (none) -> 27nH
- L10, L11, L12, L13: value 1.1uH -> 1uH
- L14, L15, L17: value 1.3uH -> 330nH
- L16: value 1.1uH -> 330nH
- L18, L19, L20, L21: value 1.3uH -> 820nH
- L2, L3, L4, L5: value 1.3uH -> 560nH
- L22, L23, L24: value 1.3uH -> 220nH
- L25: value 1.1uH -> 220nH
- L26, L27, L28: value 1.1uH -> 470nH
- L29: value 2.2uH -> 470nH; device Inductor:INDUCTOR-0805 -> Inductor:INDUCTOR-0603; CURRENT 1.2A -> (none); OCLCSC C281115 -> (none)
- L30: value 2.2uH -> 560nH; device Inductor:INDUCTOR-2.5X2X1.2MM -> Inductor:INDUCTOR-0603; CURRENT 2.2A -> (none); OCLCSC C375952 -> (none)
- L31: value 4.7uH -> 560nH; device Inductor:INDUCTOR-6X6MM -> Inductor:INDUCTOR-0603; CURRENT 3A -> (none); OCLCSC C326336 -> (none)
- L6, L7, L8, L9: value 1.3uH -> 68nH
- R1: value 5.1K Ohms -> 330 Ohms
- R11, R12: value 10K Ohms -> 2K Ohms
- R13: value 0 Ohms -> 470 Ohms
- R14: value 0 Ohms -> 49.9 Ohms
- R15: value 0 Ohms -> 267 Ohms
- R16: value 0 Ohms -> 865 Ohms
- R17, R18, R19, R20: value 0 Ohms -> 10K Ohms
- R2: value 5.1K Ohms -> 4.7K Ohms
- R21: value 100 Ohms -> 10K Ohms
- R22: value 100 Ohms -> 470 Ohms
- R23: value 100 Ohms -> 865 Ohms
- R24, R25, R26, R27, R28, R29: value 100 Ohms -> 28 Ohms
- R3: value 27 Ohms -> 4.7K Ohms
- R30: value 274K Ohms -> 28 Ohms
- R31: value 294K Ohms -> 28 Ohms
- R32, R33, R37: value 100K Ohms -> 28 Ohms
- R34: value 309K Ohms -> 28 Ohms
- R35: value 71.5K Ohms -> 28 Ohms
- R36: value 330 Ohms -> 28 Ohms
- R38: value 210K Ohms -> 28 Ohms
- R39: value 64.9K Ohms -> 28 Ohms
- R4: value 27 Ohms -> 10K Ohms
- R40: value 41.2K Ohms -> 75K Ohms
- R41: value 1M Ohms -> 10K Ohms
- R42: value 226K Ohms -> 10K Ohms
- R43, R5: value 510 Ohms -> 10K Ohms
- R6: value 10K Ohms -> 49.9 Ohms; device Resistor:RESISTOR-0603 -> Resistor:RESISTOR-1206
- R7: value 1K Ohms -> DNP; device Resistor:RESISTOR-0603 -> Resistor:RESISTOR-1206
- R8: value DNP -> 100 Ohms
- R9: value 100 Ohms -> 1K Ohms; device Resistor:RESISTOR-1206 -> Resistor:RESISTOR-0603
- U1: value ICE40HX8K-SG32 -> EFM32GG11B120F2048GM64; device Lattice:ICE40HX8K-SG32 -> EFM32:EFM32GG11B120F2048GM64
- U10: value 74LVC1G17 -> ADM7171ACPZ-5.0; device Logic:74LVC1G17 -> Analog Devices:ADM7171ACPZ-5.0
- U11: value 74LVC1G17 -> MIC23155; device Logic:74LVC1G17 -> Microchip:MIC23155
- U12: value 74LVC1G17 -> LT8636; device Logic:74LVC1G17 -> Analog Devices:LT8636
- U13: value 74LVC1G17 -> ADM7171ACPZ-3.3; device Logic:74LVC1G17 -> Analog Devices:ADM7171ACPZ-3.3
- U2: value MCP1700-330 -> MAX-M8Q; device Microchip:MCP1700-330 -> U-Blox:MAX-M8Q
- U3: value NEO-7M -> MCP1501-40; device U-Blox:NEO-7M -> Microchip:MCP1501-40
- U4: value MCP1501-40 -> AD5541ACPZ; device Microchip:MCP1501-40 -> Analog Devices:AD5541ACPZ
- U5: value AD5541ACPZ -> MCP6V32-E/MNY; device Analog Devices:AD5541ACPZ -> Microchip:MCP6V32-E/MNY
- U6: value MCP6V32-E/MNY -> OSC5A2B02; device Microchip:MCP6V32-E/MNY -> Crystal:OSC5A2B02
- U7: value OSC5A2B02 -> DSB321SDA; device Crystal:OSC5A2B02 -> Crystal:DSB321SDA
- U8: value 74LVC1G17 -> SI5347A; device Logic:74LVC1G17 -> Silicon Labs:SI5347A
- U9: value SI5351C-B-GM -> ADM7171ACPZ-1.8; device Silicon Labs:SI5351C-B-GM -> Analog Devices:ADM7171ACPZ-1.8
Connections:
- removed net !5V0_PA_BIAS_EN: R37.1, U21.SD
- removed net 1V2: C81.C1, C82.C1, L29.1, R30.2, U19.SNS@0
- removed net 1V2_FB: R30.1, R31.2, U19.FB@0
- removed net 1V2_PGOOD: R32.1, U19.PG@0
- removed net 1V2_SOFTSTART: C83.C1, U19.SS@0
- removed net 3V3_ANA_SYNTH_CLEAN: C21.C1, C22.C1, C23.C1, C24.C1, U8.PWR.VCC, U9.VDDOA, U9.VDDOB, U9.VDDOC, U9.VDDOD
- removed net 3V3_ANA_TXPLL_CLEAN: C90.C1, U20.OUT
- removed net 3V3_FB: R34.1, R35.2, U19.FB@1
- removed net 3V3_SOFTSTART: C84.C1, U19.SS@1
- removed net 3V6_ANA: C85.C1, U20.EN, U20.VIN
- removed net 5V0_ANA_COMP_CLEAN: C10.C1, C11.C1, C13.C1, U4.!SHDN, U4.VDD, U5.VDD, U6.PWR.V+
- removed net 5V0_ANA_OUT_CLEAN: C25.C1, C26.C1, C27.C1, C32.C1, C37.C1, C42.C1, C47.C1, C53.C1, C55.C1, U10.PWR.VCC, U11.PWR.VCC, U12.PWR.VCC, U13.PWR.VCC, U14.PWR.VCC, U15.PWR.VCC, U16.PWR.VCC, U17.PWR.VCC, U18.PWR.VCC
- removed net 5V0_ANA_PA_CLEAN: C92.C1, R38.2, U21.OUT
- removed net GPS_PROG_RXD: CON1-2.S, U3.RXD2
- removed net GPS_PROG_TXD: CON1-1.S, U3.TXD2
- removed net GPS_TXD: U3.TXD1
- removed net GPS_USB_D+: R3.1, U3.USB_DP
- removed net GPS_USB_D-: R4.1, U3.USB_DM
- removed net GPS_VDD_USB: C4.C1, R7.2, U2.VOUT, U3.VDD_USB
- removed net I2S_BRG_VBUS: C3.C1, D1.C1, R5.2, U2.VIN, USB1.VBUS
- removed net N$147: D2.A, R5.1
- removed net N$148: D4.A, R36.1
- removed net OCXO_CLK_SQ_UNBUF: U14.1.A, U7.CLK, U8.1.A
- removed net SYNTH_CLK0: R13.1, U10.1.A
- removed net SYNTH_CLK1: R17.1, U11.1.A
- removed net SYNTH_CLK2: R14.1, U12.1.A
- removed net SYNTH_CLK3: R18.1, U13.1.A
- removed net SYNTH_CLK4: R15.1, U15.1.A
- removed net SYNTH_CLK5: R19.1, U16.1.A
- removed net SYNTH_CLK6: R16.1, U17.1.A
- removed net SYNTH_CLK7: R20.1, U18.1.A
- new net !DAC_CS: U4.!CS
- new net !MCU_RESET: R4.1, TC1-10(!RESET!).S, U1.!RESET
- new net !PLL_IRQ: R18.1, U8.!INTR
- new net !PLL_LOLA: U8.!LOL_A
- new net !PLL_LOLB: U8.!LOL_B
- new net !PLL_LOLC: U8.!LOL_C
- new net !PLL_LOLD: U8.!LOL_D
- new net !PLL_OE0: R19.1, U8.!OE0
- new net !PLL_OE1: R20.1, U8.!OE1
- new net !PLL_OUT0: R32.1, RFCON10.SIGNAL
- new net !PLL_OUT1: R33.1, RFCON13.SIGNAL
- new net !PLL_OUT2: R34.1, RFCON15.SIGNAL
- new net !PLL_OUT3: R35.1, RFCON11.SIGNAL
- new net !PLL_OUT4: R36.1, RFCON14.SIGNAL
- new net !PLL_OUT5: R37.1, RFCON16.SIGNAL
- new net !PLL_OUT6: R38.1, RFCON12.SIGNAL
- new net !PLL_OUT7: R39.1
- new net !PLL_RESET: R17.1, U8.!RST
- new net !PLL_XTAL_LOS: U8.!LOS_XAXB
- new net 1V8_PLL_CLEAN: C100.C1, C102.C1, C39.C1, FB5.1, U9.SENSE, U9.VOUT
- new net 2V5_FB1: R46.1, R47.2, U11.FB
- new net 2V5_SS1: C98.C1, U11.SS
- new net 2V5_SW1: L58.1, U11.SW
- new net 3V3_ANA_MPLL_FILT: C34.C1, C36.C1, C37.C1, C38.C1, C40.C1, C42.C1, C48.C1, C52.C1, C55.C1, FB3.2, U8.VDDA, U8.VDDO0, U8.VDDO1, U8.VDDO2, U8.VDDO3, U8.VDDO4, U8.VDDO5, U8.VDDO6, U8.VDDO7
- new net 3V3_ANA_MPLL_FILT1: C47.C1, C51.C1, C54.C1, FB5.2, U8.VDD
- new net 3V3_ANA_PLL_CLEAN: C114.C1, C116.C1, C33.C1, FB3.1, FB4.1, U13.SENSE, U13.VOUT
- new net 5V0_EN: R40.1, R41.2, U12.EN/UV
- new net 5V0_PGOOD: R44.1, U11.EN, U12.PG
- new net 5V0_VSENSE: C118.C1, R53.1, R54.2
- new net DAC_DIN: U4.DIN
- new net DAC_SCLK: U4.SCLK
- new net GPS_TXD/TXREADY: CON1-1.S, U2.TXD
- new net I2C0_SCL: R3.1, U2.SCL, U8.SCLK
- new net I2C0_SDA: R2.1, U2.SDA, U8.SDA/SDIO
- new net MCU_LED: R1.2
- new net MCU_SWCLK: TC1-4(TCK/SWCLK).S, U1.PF0
- new net MCU_SWDIO: TC1-2(TMS/SWDIO).S, U1.PF1
- new net MCU_SWO: TC1-6(TDO/SWO).S, U1.PF2
- new net N$100: R37.2, U8.!OUT5
- new net N$101: R38.2, U8.!OUT6
- new net N$102: R39.2, U8.!OUT7
- new net N$103: C35.C1, FB4.2, U7.VDD
- new net N$104: C56.C1, FB6.2, U8.VDDS
- new net N$105: C94.C1, U9.SS
- new net N$144: D1.A, R1.1
- new net N$33: L19.2, L23.1, L27.1
- new net N$34: C58.C1, L7.2
- new net N$35: C62.C1, L15.2
- new net N$36: C66.C1, L23.2
- new net N$85: C88.C2, RFCON9.SIGNAL
- new net N$86: L49.2, L53.1, L57.1
- new net N$87: C76.C1, L37.2
- new net N$88: C80.C1, L45.2
- new net N$89: C84.C1, L53.2
- new net N$90: C88.C1, L57.2
- new net N$91: C46.C2, U8.XA
- new net N$92: R6.1, U2.TIMEPULSE
- new net N$93: C41.C2, C49.C1, R22.1, R23.2
- new net N$94: C30.C1, R16.1
- new net N$95: C45.C1, R23.1
- new net N$96: R33.2, U8.!OUT1
- new net N$97: R34.2, U8.!OUT2
- new net N$98: R35.2, U8.!OUT3
- new net N$99: R36.2, U8.!OUT4
- new net OCXO_CLK: C41.C1, R14.1, R22.2
- new net OCXO_EN: R42.2, U10.EN
- new net PLL_FDEC: U8.FDEC
- new net PLL_FINC: U8.FINC
- new net PLL_IN0_N: C32.C1, U8.!IN0
- new net PLL_IN0_P: C31.C2, U8.IN0
- new net PLL_IN1_N: C53.C1, U8.!IN1
- new net PLL_IN1_P: C49.C2, U8.IN1
- new net PLL_OUT0: L2.1, R24.1
- new net PLL_OUT1: L3.1, R25.1
- new net PLL_OUT2: L4.1, R26.1
- new net PLL_OUT3: L5.1, R27.1
- new net PLL_OUT4: L30.1, R28.1
- new net PLL_OUT5: L31.1, R29.1
- new net PLL_OUT6: L32.1, R30.1
- new net PLL_OUT7: L33.1, R31.1
- new net PLL_SEL0: U8.DSPLL_SEL0
- new net PLL_SEL1: U8.DSPLL_SEL1
- new net SMC_VCORE: C7.C1, U1.DECOUPLE
- new net VIN_VSENSE: C117.C1, R51.1, R52.2
- net !GPS_RESET: now also R5.1, U2.!RESET; no longer R6.1, U3.!RESET
- net 3V3: now also C10.C1, C106.C1, C109.C1, C111.C1, C13.C1, C15.C1, C18.C1, C3.C1, C4.C1, C44.C1, C5.C1, C6.C1, C8.C1, C90.C1, D2.A, FB2.1, FB6.1, L58.2, R17.2, R18.2, R19.2, R2.2, R20.2, R3.2, R4.2, R43.2, R46.2, R5.2, TC1-1(VTARGET).S, U1.AVDD@0, U1.AVDD@1, U1.DVDD, U1.IOVDD0@0, U1.IOVDD0@1, U1.IOVDD0@2, U11.SNS, U2.VCC, U2.VCC_IO, U8.A0/!CS, U8.A1/SDO, U9.VIN; no longer C20.C1, C7.C1, C86.C1, C87.C1, D3.A, L30.2, R32.2, R33.2, R34.2, R36.2, R37.2, R6.2, U19.SNS@1, U3.VCC, U5.VLOGIC, U9.VDD
- net 3V3_PGOOD: now also R43.1, U11.PG, U13.EN, U9.EN; no longer R33.1, U19.PG@1
- net 5V0: now also C105.C1, C108.C1, C112.C1, C113.C1, C115.C1, C92.C1, L59.2, R44.2, R48.2, R50.2, R53.2, U10.VIN, U11.VIN@0, U11.VIN@1, U12.BIAS, U13.VIN; no longer C101.C1, C79.C1, C80.C1, C88.C1, C97.C1, C99.C1, L31.2, R41.2, R43.2, U19.AVIN@0, U19.AVIN@1, U19.EN@0, U19.EN@1, U19.VIN@0, U19.VIN@1, U21.IN, U22.BIAS
- net 5V0_ANA_OCXO_CLEAN: now also C103.C1, C104.C1, C21.C1, C23.C1, C25.C1, C26.C1, FB1.1, FB1.2, U10.SENSE, U10.VOUT, U3.!SHDN, U3.VDD, U4.VDD, U5.PWR.V+, U6.VDD; no longer U7.VDD
- net 5V0_BST: now also C107.C2, U12.BST; no longer C98.C2, U22.BST
- net 5V0_FB: now also C108.C2, R48.1, R49.2, U12.FB; no longer C99.C2, R41.1, R42.2, U22.FB
- net 5V0_INTVCC: now also C99.C1, U12.INTVCC, U12.SYNC/MODE; no longer C96.C1, U22.INTVCC, U22.SYNC/MODE
- net 5V0_RT: now also R45.2, U12.RT; no longer R40.2, U22.RT
- net 5V0_SS: now also C101.C1, U12.TR/SS; no longer C95.C1, U22.TR/SS
- net 5V0_SW: now also C107.C1, L59.1, U12.SW; no longer C98.C1, L31.1, U22.SW
- net GND: now also C103.C2, C104.C2, C105.C2, C106.C2, C109.C2, C110.C2, C111.C2, C112.C2, C113.C2, C114.C2, C115.C2, C116.C2, C117.C2, C118.C2, C119.C2, C48.C2, C50.C2, C51.C2, C58.C2, C6.C2, C75.C2, C76.C2, C77.C2, C78.C2, C92.C2, C98.C2, C99.C2, CON2-1.S, D1.C, D3.C, D4.A, R13.1, R21.1, R41.1, R45.1, R47.1, R49.1, R52.1, R54.1, RFCON11.GND, RFCON12.GND, RFCON13.GND, RFCON14.GND, RFCON15.GND, RFCON16.GND, TC1-3(GND).S, U1.VSS@0, U10.GND, U11.AGND, U11.PGND@0, U11.PGND@1, U12.GND, U13.GND, U2.GND@0, U2.GND@1, U2.GND@2, U4.!LDAC, U4.AGND, U4.DGND, U5.PWR.V-, U6.GND, U8.GND; no longer C12.C2, C29.C2, C31.C2, C41.C2, C46.C2, C69.C2, C70.C2, C71.C2, C72.C2, C85.C2, C86.C2, C87.C2, C88.C2, D1.A, D2.C, D4.C, D5.A, D6.C, R1.1, R2.1, R31.1, R35.1, R39.1, R40.1, R7.1, U10.PWR.GND, U11.PWR.GND, U12.PWR.GND, U13.PWR.GND, U14.PWR.GND, U15.PWR.GND, U16.PWR.GND, U17.PWR.GND, U18.PWR.GND, U19.AGND@0, U19.AGND@1, U19.PGND@0, U19.PGND@1, U19.PGND@2, U2.GND, U20.GND, U21.GND, U22.GND, U3.GND@3, U4.GND@0, U4.GND@1, U4.GND@2, U5.AGND, U5.DGND, U6.PWR.V-, U8.PWR.GND, USB1.GND
- net GPS_BIAS_EXT: now also R8.1; no longer R9.1
- net GPS_BIAS_INT: now also C11.C1, R7.2, U2.VCC_RF; no longer C5.C1, R8.2, U3.VCC_RF
- net GPS_RXD: now also CON1-2.S, U2.RXD; no longer U3.RXD1
- net GPS_TIMEPULSE: now also C29.C1, R15.2, R6.2; no longer U3.TIMEPULSE
- net GPS_VBKP: now also C14.C1, R9.1, U2.V_BKP; no longer C8.C1, R10.1, U3.V_BKP
- net N$1: now also C57.C1, L6.2; no longer R25.2, U14.1.Y
- net N$10: now also C70.C2, RFCON3.SIGNAL; no longer R21.2, U10.1.Y
- net N$11: now also D2.C, R9.2; no longer D3.C, R10.2
- net N$12: now also C12.C1, U2.RF_IN; no longer C6.C1, U3.RF_IN
- net N$13: now also C12.C2; no longer C6.C2
- net N$14: now also R7.1, R8.2; no longer R8.1, R9.2
- net N$149: now also D3.A, R50.1; no longer D6.A, R43.1
- net N$15: now also R32.2, U8.!OUT0; no longer D1.C3, R4.2, USB1.D-
- net N$16: now also C29.C2, C31.C1, R15.1, R16.2; no longer D1.C2, R3.2, USB1.D+
- net N$17: now also C43.C1, C46.C1, R21.2, U7.CLK; no longer U8.1.Y, U9.CLKIN
- net N$18: now also R30.2, U8.OUT6; no longer R16.2, U9.CLK6
- net N$19: now also R31.2, U8.OUT7; no longer R20.2, U9.CLK7
- net N$2: now also C61.C1, L14.2; no longer C52.C1, L14.1, R25.1
- net N$20: now also R29.2, U8.OUT5; no longer R19.2, U9.CLK5
- net N$21: now also R28.2, U8.OUT4; no longer R15.2, U9.CLK4
- net N$22: now also R27.2, U8.OUT3; no longer R18.2, U9.CLK3
- net N$23: now also R26.2, U8.OUT2; no longer R14.2, U9.CLK2
- net N$24: now also R25.2, U8.OUT1; no longer R17.2, U9.CLK1
- net N$25: now also R24.2, U8.OUT0; no longer R13.2, U9.CLK0
- net N$26: now also C110.C1, U13.SS; no longer L30.1, U19.SW@1
- net N$27: now also C20.C1, FB2.2, U4.VLOGIC; no longer L29.2, U19.SW@0
- net N$28: now also C97.C1, U10.SS; no longer C92.C2, R38.1, R39.2, U21.FB
- net N$29: now also R14.2, U6.CLK; no longer R1.2, USB1.CC2
- net N$3: now also C65.C1, L22.2; no longer C54.C1, L14.2, L15.1
- net N$30: now also C50.C1, U8.XB; no longer R2.2, USB1.CC1
- net N$31: now also CON2-2.S
- net N$32: now also R10.1, U5.2.+IN; no longer R44.1, U6.2.+IN
- net N$37: now also C19.C1, U3.VOUT, U4.REF; no longer C12.C1, U4.VOUT, U5.REF
- net N$38: now also C70.C1, L27.2; no longer C28.C1, L2.1, R21.1
- net N$39: now also L10.1; no longer C33.C1
- net N$4: now also C69.C1, L26.2; no longer C56.C1, L15.2, L16.1
- net N$40: now also L10.2, L14.1, L18.1; no longer C38.C1, L10.1, L6.2
- net N$41: now also C69.C2; no longer C48.C2
- net N$42: now also L18.2, L22.1, L26.1; no longer C43.C1, C48.C1, L10.2
- net N$43: now also L12.1, L4.2, L8.1; no longer R22.2, U11.1.Y
- net N$44: now also L12.2, L16.1, L20.1; no longer C29.C1, L3.1, R22.1
- net N$45: now also C71.C2, RFCON4.SIGNAL; no longer C34.C1, L3.2, L7.1
- net N$46: now also L20.2, L24.1, L28.1; no longer C39.C1, L11.1, L7.2
- net N$47: now also C59.C1, L8.2; no longer C49.C2, RFCON3.SIGNAL
- net N$48: now also C63.C1, L16.2; no longer C44.C1, C49.C1, L11.2
- net N$49: now also C67.C1, L24.2; no longer R23.2, U12.1.Y
- net N$5: now also L11.1, L3.2, L7.1; no longer C58.C2, RFCON6.SIGNAL
- net N$50: now also C71.C1, L28.2; no longer C30.C1, L4.1, R23.1
- net N$51: now also L13.1, L5.2, L9.1; no longer C35.C1, L4.2, L8.1
- net N$52: now also L13.2, L17.1, L21.1; no longer C40.C1, L12.1, L8.2
- net N$53: now also C72.C2, RFCON5.SIGNAL; no longer C50.C2, RFCON4.SIGNAL
- net N$54: now also L21.2, L25.1, L29.1; no longer C45.C1, C50.C1, L12.2
- net N$55: now also C60.C1, L9.2; no longer R24.2, U13.1.Y
- net N$56: now also C64.C1, L17.2; no longer C31.C1, L5.1, R24.1
- net N$57: now also C68.C1, L25.2; no longer C36.C1, L5.2, L9.1
- net N$58: now also C72.C1, L29.2; no longer C41.C1, L13.1, L9.2
- net N$59: now also L30.2, L34.1, L38.1; no longer C51.C2, RFCON5.SIGNAL
- net N$6: now also L11.2, L15.1, L19.1; no longer C57.C1, C58.C1, L16.2
- net N$60: now also L38.2, L42.1, L46.1; no longer C46.C1, C51.C1, L13.2
- net N$61: now also C85.C2, RFCON6.SIGNAL; no longer R26.2, U15.1.Y
- net N$62: now also L46.2, L50.1, L54.1; no longer C59.C1, L17.1, R26.1
- net N$63: now also C73.C1, L34.2; no longer C63.C1, L17.2, L21.1
- net N$64: now also C77.C1, L42.2; no longer C67.C1, L21.2, L25.1
- net N$65: now also C81.C1, L50.2; no longer C75.C2, RFCON7.SIGNAL
- net N$66: now also C85.C1, L54.2; no longer C71.C1, C75.C1, L25.2
- net N$67: now also L31.2, L35.1, L39.1; no longer R27.2, U16.1.Y
- net N$68: now also L39.2, L43.1, L47.1; no longer C60.C1, L18.1, R27.1
- net N$69: now also C86.C2, RFCON7.SIGNAL; no longer C64.C1, L18.2, L22.1
- net N$7: now also C22.C1, U4.VOUT, U5.1.+IN; no longer C14.C1, U5.VOUT, U6.1.+IN
- net N$70: now also L47.2, L51.1, L55.1; no longer C68.C1, L22.2, L26.1
- net N$71: now also C74.C1, L35.2; no longer C76.C2, RFCON8.SIGNAL
- net N$72: now also C78.C1, L43.2; no longer C72.C1, C76.C1, L26.2
- net N$73: now also C82.C1, L51.2; no longer R28.2, U17.1.Y
- net N$74: now also C86.C1, L55.2; no longer C61.C1, L19.1, R28.1
- net N$75: now also L32.2, L36.1, L40.1; no longer C65.C1, L19.2, L23.1
- net N$76: now also L40.2, L44.1, L48.1; no longer C69.C1, L23.2, L27.1
- net N$77: now also C87.C2, RFCON8.SIGNAL; no longer C77.C2, RFCON9.SIGNAL
- net N$78: now also L48.2, L52.1, L56.1; no longer C73.C1, C77.C1, L27.2
- net N$79: now also C75.C1, L36.2; no longer R29.2, U18.1.Y
- net N$8: now also C24.C1, R10.2, U5.1.-IN, U5.1.OUT; no longer C15.C1, R44.2, U6.1.-IN, U6.1.OUT
- net N$80: now also C79.C1, L44.2; no longer C62.C1, L20.1, R29.1
- net N$81: now also C83.C1, L52.2; no longer C66.C1, L20.2, L24.1
- net N$82: now also C87.C1, L56.2; no longer C70.C1, L24.2, L28.1
- net N$83: now also L33.2, L37.1, L41.1; no longer C78.C2, RFCON10.SIGNAL
- net N$84: now also L41.2, L45.1, L49.1; no longer C74.C1, C78.C1, L28.2
- net N$9: now also U5.2.-IN; no longer U6.2.-IN
- net OCXO_VCONT: now also C27.C1, C28.C1, R13.2, U5.2.OUT, U6.VCONT; no longer C18.C1, C19.C1, U6.2.OUT, U7.VCONT
- net VIN: now also C119.C1, C95.C1, C96.C1, D4.C, R40.2, R51.2, U12.VIN; no longer C100.C1, C102.C1, C94.C1, D5.C, U22.EN/UV, U22.VIN
Other:
- note added: "5th order Eliptic LPF Fc = 13 MHz"
- note added: "ADM7171 1.8V @ 1A"
- note added: "ADM7171 3.3V @ 1A"
- note added: "ADM7171 5V @ 1A"
- note added: "Analog Rail OCXO and comp. network"
- note added: "Analog Rail PLL core"
- note added: "Analog Rail PLL, Clock outputs"
- note added: "Digital Rail MCU"
- note added: "Enable"
- note added: "LT8636 5.2V @ 5A"
- note added: "MIC23155 3.3V @ 2A"
- note added: "VIN 9 to 24V"
- note added: "Ven = ((RTop/RBottom) + 1) * 1"
- note added: "Vout = ((RTop/RBottom) + 1) * 0.97"
- note removed: "7th order Chebyshev LPF Fc = 10 MHz Zi = 100 Ohms Zo = 50 Ohms"
- note removed: "Can be replaced with ATGM332D-5N"
- note removed: "DNP if GPS module is ATGM332D-5N"
- note removed: "DNP if GPS module is NEO-XX"
- note removed: "Vout = ((R24/R25) + 1) * 0.97"
