File: pcb/gpsdo/qo-100-gpsdo.sch (EAGLE design)
At the start: 278 parts, among them CON1 3P-SH-TOP, CON2 2EDG-2P-5MM, J1 DCJACK, U1 EFM32GG11B120F2048GM64, U10 ADM7171ACPZ-5.0, U11 MIC23155, U12 LT8636, U13 ADM7171ACPZ-3.3, U2 MAX-M8Q, U3 MCP1501-40, U4 AD5541ACPZ, U5 MCP6V32-E/MNY, U6 OSC5A2B02, U7 DSB321SDA, U8 SI5347A, U9 ADM7171ACPZ-1.8

Commit message: Work on GPSDO
Signed-off-by: João Silva <jgc3silva@gmail.com>
Parts:
- removed C10, C106, C11, C115, C116, C13, C14, C15, C20, C22, C24, C26, C27, C28, C30, C31, C32, C4, C45, C46, C49, C5, C50, C53, C6, C69, C70, C71, C72, C85, C86, C87, C88, C89, C9, C90, C91: 100nF, Capacitor:CAPACITOR-0603
- removed C108, C43: 10pF, Capacitor:CAPACITOR-0603
- removed C110, C94, C97: 10nF, Capacitor:CAPACITOR-0603
- removed C111: 100uF, Capacitor:CAPACITOR-1206
- removed C117, C118, C98: 470pF, Capacitor:CAPACITOR-0603
- removed C12: 47pF, Capacitor:CAPACITOR-0603
- removed C16, C19, C33: 10uF, Capacitor:CAPACITOR-0603
- removed C17, C18, C21, C23, C34, C35, C36, C37, C38, C40, C42, C47, C48, C51, C52, C54, C55, C56, C7, C99: 1uF, Capacitor:CAPACITOR-0603
- removed C29, C41: 6pF, Capacitor:CAPACITOR-0603
- removed C57, C58, C59, C60, C73, C74, C75, C76: 270pF, Capacitor:CAPACITOR-0603
- removed C61, C62, C63, C64, C65, C66, C67, C68, C77, C78, C79, C80, C81, C82, C83, C84: 220pF, Capacitor:CAPACITOR-0603
- removed D3: LED0603, LED:LED0603
- removed FB1, FB2, FB3, FB4, FB5, FB6: 1uH, Inductor:FERRITE-0805
- removed L10, L11, L12, L13, L38, L39, L40, L41: 1uH, Inductor:INDUCTOR-0603
- removed L14, L15, L16, L17, L42, L43, L44, L45: 330nH, Inductor:INDUCTOR-0603
- removed L18, L19, L20, L21, L46, L47, L48, L49: 820nH, Inductor:INDUCTOR-0603
- removed L2, L3, L30, L31, L32, L33, L4, L5: 560nH, Inductor:INDUCTOR-0603
- removed L22, L23, L24, L25, L50, L51, L52, L53: 220nH, Inductor:INDUCTOR-0603
- removed L26, L27, L28, L29, L54, L55, L56, L57: 470nH, Inductor:INDUCTOR-0603
- removed L34, L35, L36, L37, L6, L7, L8, L9: 68nH, Inductor:INDUCTOR-0603
- removed R1: 330 Ohms, Resistor:RESISTOR-0603
- removed R10, R9: 1K Ohms, Resistor:RESISTOR-0603
- removed R11, R12: 2K Ohms, Resistor:RESISTOR-0603
- removed R13, R22: 470 Ohms, Resistor:RESISTOR-0603
- removed R14: 49.9 Ohms, Resistor:RESISTOR-0603
- removed R15: 267 Ohms, Resistor:RESISTOR-0603
- removed R16, R23: 865 Ohms, Resistor:RESISTOR-0603
- removed R17, R18, R19, R20, R21, R4, R41, R42, R43, R44, R5, R52: 10K Ohms, Resistor:RESISTOR-0603
- removed R2, R3: 4.7K Ohms, Resistor:RESISTOR-0603
- removed R24, R25, R26, R27, R28, R29, R30, R31, R32, R33, R34, R35, R36, R37, R38, R39: 28 Ohms, Resistor:RESISTOR-0603
- removed R40, R54: 75K Ohms, Resistor:RESISTOR-0603
- removed R45: 41.2K Ohms, Resistor:RESISTOR-0603
- removed R46: 309K Ohms, Resistor:RESISTOR-0603
- removed R47: 71.5K Ohms, Resistor:RESISTOR-0603
- removed R48: 1M Ohms, Resistor:RESISTOR-0603
- removed R49: 226K Ohms, Resistor:RESISTOR-0603
- removed R50: 510 Ohms, Resistor:RESISTOR-0603
- removed R51, R53: 100K Ohms, Resistor:RESISTOR-0603
- removed R6: 49.9 Ohms, Resistor:RESISTOR-1206
- removed R7: DNP, Resistor:RESISTOR-1206
- removed R8: 100 Ohms, Resistor:RESISTOR-1206
- removed RFCON1, RFCON9: RFCON-U.FL, RF Connector:RFCON-U.FL
- removed TC1: TC2050-IDC, TagConnect:TC2050-IDC
- removed U3: MCP1501-40, Microchip:MCP1501-40
- removed U5: MCP6V32-E/MNY, Microchip:MCP6V32-E/MNY
- added C202, C203, C204, C206, C207, C306, C307, C309, C311, C313, C314, C402, C403, C404, C417, C418, C421, C422, C425, C513, C514, C515, C516, C529, C530, C531, C601, C602, C603, C614, C616, C617, C619, C620, C626, C628: 100nF, Capacitor:CAPACITOR-0402
- added C205: 47pF, Capacitor:CAPACITOR-0402
- added C302, C305, C615: 10uF, Capacitor:CAPACITOR-0603
- added C303, C304, C308, C310, C406, C407, C408, C409, C410, C412, C414, C419, C420, C423, C424, C426, C427, C428, C611: 1uF, Capacitor:CAPACITOR-0402
- added C401, C413: 6pF, Capacitor:CAPACITOR-0402
- added C415, C618: 10pF, Capacitor:CAPACITOR-0402
- added C501, C502, C503, C504, C517, C518, C519: 270pF, Capacitor:CAPACITOR-0402
- added C505, C506, C507, C508, C509, C510, C511, C512, C521, C522, C523, C525, C526, C527: 220pF, Capacitor:CAPACITOR-0402
- added C606, C609, C612, C622: 10nF, Capacitor:CAPACITOR-0402
- added C610, C629, C630: 470pF, Capacitor:CAPACITOR-0402
- added D101, D601: LED0603, LED:LED0603
- added D201: B0530W, Generic Diode:B0530W
- added FB301, FB302, FB402, FB403, FB404: 1uH, Inductor:FERRITE-0603
- added L501, L502, L503, L504, L529, L530, L531: 560nH, Inductor:INDUCTOR-0402
- added L505, L506, L507, L508, L533, L534, L535: 68nH, Inductor:INDUCTOR-0402
- added L509, L510, L511, L512, L537, L538, L539: 1uH, Inductor:INDUCTOR-0402
- added L513, L514, L515, L516, L541, L542, L543: 330nH, Inductor:INDUCTOR-0402
- added L517, L518, L519, L520, L545, L546, L547: 820nH, Inductor:INDUCTOR-0402
- added L521, L522, L523, L524, L549, L550, L551: 220nH, Inductor:INDUCTOR-0402
- added L525, L526, L527, L528, L553, L554, L555: 470nH, Inductor:INDUCTOR-0402
- added R101: 330 Ohms, Resistor:RESISTOR-0402
- added R102, R103: 4.7K Ohms, Resistor:RESISTOR-0402
- added R104, R201, R403, R404, R405, R406, R407, R602, R603, R604, R605, R613: 10K Ohms, Resistor:RESISTOR-0402
- added R202, R302: 49.9 Ohms, Resistor:RESISTOR-0603
- added R203: 10 Ohms, Resistor:RESISTOR-0603
- added R204: DNP, Resistor:RESISTOR-0603
- added R205: 1K Ohms, Resistor:RESISTOR-0402
- added R301, R408: 470 Ohms, Resistor:RESISTOR-0402
- added R401: 267 Ohms, Resistor:RESISTOR-0402
- added R402, R409: 865 Ohms, Resistor:RESISTOR-0402
- added R410, R411, R412, R413, R414, R415, R416, R418, R419, R420, R421, R422, R423, R424: 28 Ohms, Resistor:RESISTOR-0402
- added R601, R615: 75K Ohms, Resistor:RESISTOR-0402
- added R606: 41.2K Ohms, Resistor:RESISTOR-0402
- added R607: 309K Ohms, Resistor:RESISTOR-0402
- added R608: 71.5K Ohms, Resistor:RESISTOR-0402
- added R609: 1M Ohms, Resistor:RESISTOR-0402
- added R610: 226K Ohms, Resistor:RESISTOR-0402
- added R611: 510 Ohms, Resistor:RESISTOR-0402
- added R612, R614: 100K Ohms, Resistor:RESISTOR-0402
- added RFCON201: RFCON-SMA-EDGE, RF Connector:RFCON-SMA-EDGE
- added TC101: TC2050-IDC, TagConnect:TC2050-IDC
- added U101: EFM32GG11B120F2048GM64, EFM32:EFM32GG11B120F2048GM64
- added U201: MAX-M8Q, U-Blox:MAX-M8Q
- added U301: MCP1501-40, Microchip:MCP1501-40
- added U303: MCP6V31, Microchip:MCP6V31
- C1: value 100nF -> 10uF
- C101: value 10nF -> 100nF; device Capacitor:CAPACITOR-0603 -> Capacitor:CAPACITOR-0402
- C102, C104, C105, C2, C3: device Capacitor:CAPACITOR-0603 -> Capacitor:CAPACITOR-0402
- C103: value 10uF -> 100nF; device Capacitor:CAPACITOR-0603 -> Capacitor:CAPACITOR-0402
- C107: value 100nF -> 1uF; device Capacitor:CAPACITOR-0603 -> Capacitor:CAPACITOR-0402
- D1: value LED0603 -> LEDTH3MM; device LED:LED0603 -> LED:LEDTH3MM; COLOR BLUE -> GREEN
- D2: value B0530W -> LEDTH3MM; device Generic Diode:B0530W -> LED:LEDTH3MM; COLOR (none) -> BLUE
- U1: value EFM32GG11B120F2048GM64 -> 74LVC1G17; device EFM32:EFM32GG11B120F2048GM64 -> Logic:74LVC1G17
- U2: value MAX-M8Q -> 74LVC1G17; device U-Blox:MAX-M8Q -> Logic:74LVC1G17
- renumbered BAT1 to BAT201, C100 to C613, C109 to C621, C112 to C624, C113 to C625, C114 to C627, C119 to C631, C25 to C312, C39 to C411, C44 to C416, C8 to C201, C92 to C604, C93 to C605, C95 to C607, C96 to C608, CON1 to CON201, CON2 to CON601, D4 to D602, F1 to F601, J1 to J601, L1 to L201, L58 to L601, L59 to L602, LOGO1 to LOGO101, RFCON10 to RFCON509, RFCON11 to RFCON510, RFCON12 to RFCON511, RFCON13 to RFCON512, RFCON14 to RFCON513, RFCON15 to RFCON514, RFCON16 to RFCON515, RFCON2 to RFCON501, RFCON3 to RFCON502, RFCON4 to RFCON503, RFCON5 to RFCON504, RFCON6 to RFCON505, RFCON7 to RFCON506, RFCON8 to RFCON507, U10 to U602, U11 to U603, U12 to U604, U13 to U605, U4 to U302, U6 to U304, U7 to U401, U8 to U402, U9 to U601
Connections:
- net 2V5_SW1 renamed 3V3_SW
- removed net !PLL_OUT7: R39.1
- removed net 2V5_FB1: R46.1, R47.2, U603.FB
- removed net 2V5_SS1: C98.C1, U603.SS
- removed net 3V3_ANA_MPLL_FILT: C34.C1, C36.C1, C37.C1, C38.C1, C40.C1, C42.C1, C48.C1, C52.C1, C55.C1, FB3.2, U402.VDDA, U402.VDDO0, U402.VDDO1, U402.VDDO2, U402.VDDO3, U402.VDDO4, U402.VDDO5, U402.VDDO6, U402.VDDO7
- removed net 3V3_ANA_MPLL_FILT1: C47.C1, C51.C1, C54.C1, FB5.2, U402.VDD
- removed net N$102: R39.2, U402.!OUT7
- removed net N$19: R31.2, U402.OUT7
- removed net N$29: R14.2, U304.CLK
- removed net N$32: R10.1, U5.2.+IN
- removed net N$8: C24.C1, R10.2, U5.1.-IN, U5.1.OUT
- removed net N$83: L33.2, L37.1, L41.1
- removed net N$84: L41.2, L45.1, L49.1
- removed net N$85: C88.C2, RFCON9.SIGNAL
- removed net N$86: L49.2, L53.1, L57.1
- removed net N$87: C76.C1, L37.2
- removed net N$88: C80.C1, L45.2
- removed net N$89: C84.C1, L53.2
- removed net N$9: R11.2, R12.2, U5.2.-IN
- removed net N$90: C88.C1, L57.2
- removed net N$92: R6.1, U2.TIMEPULSE
- removed net PLL_OUT7: L33.1, R31.1
- removed net SMC_VCORE: C7.C1, U1.DECOUPLE
- new net 1V8_PLL_CLEAN_FILT: C419.C1, C423.C1, C426.C1, FB403.2, U402.VDD
- new net 3V3_FB: R607.1, R608.2, U603.FB
- new net 3V3_SS: C610.C1, U603.SS
- new net 5V0_ANA_OCXO_FILT: C303.C1, C308.C1, C310.C1, FB301.2, U301.!SHDN, U301.VDD, U302.VDD, U303.PWR.V+
- new net GPS_TIMEPULSE_BUF: U1.1.Y
- new net GPS_TIMEPULSE_KZ: C401.C1, R202.1, R401.2
- new net MCU_VCORE: C107.C1, U101.DECOUPLE
- new net OCXO_CLK_BUF: U2.1.Y
- new net OCXO_CLK_KZ: C413.C1, R302.1, R408.2
- net !GPS_RESET: now also R201.1, U201.!RESET; no longer R5.1, U2.!RESET
- net !MCU_RESET: now also R104.1, TC101-10(!RESET!).S, U101.!RESET; no longer R4.1, TC1-10(!RESET!).S, U1.!RESET
- net !PLL_IRQ: now also R404.1; no longer R18.1
- net !PLL_OE0: now also R405.1; no longer R19.1
- net !PLL_OE1: now also R406.1; no longer R20.1
- net !PLL_OUT0: now also R418.1; no longer R32.1
- net !PLL_OUT1: now also R419.1; no longer R33.1
- net !PLL_OUT2: now also R420.1; no longer R34.1
- net !PLL_OUT3: now also R421.1; no longer R35.1
- net !PLL_OUT4: now also R422.1; no longer R36.1
- net !PLL_OUT5: now also R423.1; no longer R37.1
- net !PLL_OUT6: now also R424.1; no longer R38.1
- net !PLL_RESET: now also R403.1; no longer R17.1
- net 1V8_PLL_CLEAN: now also C614.C1, FB403.1; no longer C102.C1, FB5.1
- net 3V3: now also C101.C1, C102.C1, C103.C1, C104.C1, C105.C1, C202.C1, C203.C1, C206.C1, C304.C1, C602.C1, C620.C1, D201.A, FB302.1, FB404.1, R102.2, R103.2, R104.2, R201.2, R403.2, R404.2, R405.2, R406.2, R604.2, R607.2, TC101-1(VTARGET).S, U1.PWR.VCC, U101.AVDD@0, U101.AVDD@1, U101.DVDD, U101.IOVDD0@0, U101.IOVDD0@1, U101.IOVDD0@2, U2.PWR.VCC, U201.VCC, U201.VCC_IO; no longer C1.C1, C10.C1, C106.C1, C111.C1, C13.C1, C15.C1, C18.C1, C4.C1, C5.C1, C6.C1, C9.C1, C90.C1, D2.A, FB2.1, FB6.1, R17.2, R18.2, R19.2, R2.2, R20.2, R3.2, R4.2, R43.2, R46.2, R5.2, TC1-1(VTARGET).S, U1.AVDD@0, U1.AVDD@1, U1.DVDD, U1.IOVDD0@0, U1.IOVDD0@1, U1.IOVDD0@2, U2.VCC, U2.VCC_IO
- net 3V3_ANA_PLL_CLEAN: now also C406.C1, C408.C1, C409.C1, C410.C1, C412.C1, C414.C1, C420.C1, C424.C1, C427.C1, C628.C1, FB402.1, U402.VDDA, U402.VDDO0, U402.VDDO1, U402.VDDO2, U402.VDDO3, U402.VDDO4, U402.VDDO5, U402.VDDO6, U402.VDDO7; no longer C116.C1, C33.C1, FB3.1, FB4.1
- net 3V3_PGOOD: now also R604.1; no longer R43.1
- net 5V0: now also C601.C1, C603.C1, C618.C1, C619.C1, C626.C1, R605.2, R609.2, R611.2, R614.2; no longer C105.C1, C108.C1, C115.C1, C89.C1, C91.C1, R44.2, R48.2, R50.2, R53.2
- net 5V0_ANA_OCXO_CLEAN: now also C302.C1, C313.C1, C615.C1, C616.C1, FB301.1; no longer C103.C1, C104.C1, C16.C1, C17.C1, C21.C1, C23.C1, C26.C1, FB1.1, FB1.2, U3.!SHDN, U3.VDD, U302.VDD, U5.PWR.V+
- net 5V0_BST: now also C617.C2; no longer C107.C2
- net 5V0_EN: now also R601.1, R602.2; no longer R40.1, R41.2
- net 5V0_FB: now also C618.C2, R609.1, R610.2; no longer C108.C2, R48.1, R49.2
- net 5V0_INTVCC: now also C611.C1; no longer C99.C1
- net 5V0_PGOOD: now also R605.1; no longer R44.1
- net 5V0_RT: now also R606.2; no longer R45.2
- net 5V0_SS: now also C612.C1; no longer C101.C1
- net 5V0_SW: now also C617.C1; no longer C107.C1
- net 5V0_VSENSE: now also C630.C1, R614.1, R615.2; no longer C118.C1, R53.1, R54.2
- net GND: now also C107.C2, C202.C2, C203.C2, C204.C2, C206.C2, C207.C2, C302.C2, C303.C2, C304.C2, C305.C2, C306.C2, C307.C2, C308.C2, C309.C2, C310.C2, C311.C2, C313.C2, C314.C2, C402.C2, C404.C2, C406.C2, C407.C2, C408.C2, C409.C2, C410.C2, C412.C2, C414.C2, C415.C2, C417.C2, C419.C2, C420.C2, C422.C2, C423.C2, C424.C2, C425.C2, C426.C2, C427.C2, C428.C2, C501.C2, C502.C2, C503.C2, C504.C2, C505.C2, C506.C2, C507.C2, C508.C2, C509.C2, C510.C2, C511.C2, C512.C2, C517.C2, C518.C2, C519.C2, C521.C2, C522.C2, C523.C2, C525.C2, C526.C2, C527.C2, C601.C2, C602.C2, C603.C2, C606.C2, C609.C2, C610.C2, C611.C2, C612.C2, C614.C2, C615.C2, C616.C2, C619.C2, C620.C2, C622.C2, C626.C2, C628.C2, C629.C2, C630.C2, D101.C, D2.C, D601.C, R301.1, R407.1, R602.1, R603.1, R606.1, R608.1, R610.1, R613.1, R615.1, RFCON201.GND, TC101-3(GND).S, U1.PWR.GND, U101.VSS@0, U2.PWR.GND, U201.GND@0, U201.GND@1, U201.GND@2, U301.GND@0, U301.GND@1, U301.GND@2, U303.PWR.V-; no longer C10.C2, C106.C2, C11.C2, C110.C2, C111.C2, C115.C2, C116.C2, C117.C2, C118.C2, C13.C2, C14.C2, C15.C2, C16.C2, C17.C2, C18.C2, C19.C2, C20.C2, C21.C2, C22.C2, C23.C2, C24.C2, C26.C2, C27.C2, C28.C2, C30.C2, C32.C2, C33.C2, C34.C2, C35.C2, C36.C2, C37.C2, C38.C2, C4.C2, C40.C2, C42.C2, C43.C2, C45.C2, C47.C2, C48.C2, C5.C2, C50.C2, C51.C2, C52.C2, C53.C2, C54.C2, C55.C2, C56.C2, C57.C2, C58.C2, C59.C2, C6.C2, C60.C2, C61.C2, C62.C2, C63.C2, C64.C2, C65.C2, C66.C2, C67.C2, C68.C2, C7.C2, C73.C2, C74.C2, C75.C2, C76.C2, C77.C2, C78.C2, C79.C2, C80.C2, C81.C2, C82.C2, C83.C2, C84.C2, C89.C2, C9.C2, C90.C2, C91.C2, C94.C2, C97.C2, C98.C2, C99.C2, D3.C, R11.1, R13.1, R21.1, R41.1, R42.1, R45.1, R47.1, R49.1, R52.1, R54.1, RFCON1.GND, RFCON9.GND, TC1-3(GND).S, U1.VSS@0, U2.GND@0, U2.GND@1, U2.GND@2, U3.GND@0, U3.GND@1, U3.GND@2, U5.PWR.V-
- net GPS_BIAS_EXT: now also R204.1; no longer R8.1
- net GPS_BIAS_INT: now also C204.C1, R203.2, U201.VCC_RF; no longer C11.C1, R7.2, U2.VCC_RF
- net GPS_RXD: now also U201.RXD; no longer U2.RXD
- net GPS_TIMEPULSE: now also R202.2, U1.1.A, U201.TIMEPULSE; no longer C29.C1, R15.2, R6.2
- net GPS_TXD/TXREADY: now also U201.TXD; no longer U2.TXD
- net GPS_VBKP: now also C1.C1, C207.C1, R205.1, U201.V_BKP; no longer C14.C1, R9.1, U2.V_BKP
- net I2C0_SCL: now also R103.1, U201.SCL; no longer R3.1, U2.SCL
- net I2C0_SDA: now also R102.1, U201.SDA; no longer R2.1, U2.SDA
- net MCU_LED: now also R101.2; no longer R1.2
- net MCU_SWCLK: now also TC101-4(TCK/SWCLK).S, U101.PF0; no longer TC1-4(TCK/SWCLK).S, U1.PF0
- net MCU_SWDIO: now also TC101-2(TMS/SWDIO).S, U101.PF1; no longer TC1-2(TMS/SWDIO).S, U1.PF1
- net MCU_SWO: now also TC101-6(TDO/SWO).S, U101.PF2; no longer TC1-6(TDO/SWO).S, U1.PF2
- net N$1: now also C501.C1, L505.2; no longer C57.C1, L6.2
- net N$10: now also C514.C2; no longer C70.C2
- net N$100: now also R423.2; no longer R37.2
- net N$101: now also R424.2; no longer R38.2
- net N$103: now also C407.C1, FB402.2; no longer C35.C1, FB4.2
- net N$104: now also C428.C1, FB404.2; no longer C56.C1, FB6.2
- net N$105: now also C606.C1; no longer C94.C1
- net N$11: now also D201.C, R205.2; no longer D2.C, R9.2
- net N$12: now also C205.C1, U201.RF_IN; no longer C12.C1, U2.RF_IN
- net N$13: now also C205.C2, RFCON201.SIGNAL; no longer C12.C2, RFCON1.SIGNAL
- net N$14: now also R203.1, R204.2; no longer R7.1, R8.2
- net N$144: now also D101.A, D2.A, R101.1; no longer D1.A, R1.1
- net N$149: now also D1.A, D601.A, R611.1; no longer D3.A, R50.1
- net N$15: now also R418.2; no longer R32.2
- net N$16: now also C401.C2, C403.C1, R401.1, R402.2; no longer C29.C2, C31.C1, R15.1, R16.2
- net N$17: now also C415.C1, C418.C1, R407.2; no longer C43.C1, C46.C1, R21.2
- net N$18: now also R416.2; no longer R30.2
- net N$2: now also C505.C1, L513.2; no longer C61.C1, L14.2
- net N$20: now also R415.2; no longer R29.2
- net N$21: now also R414.2; no longer R28.2
- net N$22: now also R413.2; no longer R27.2
- net N$23: now also R412.2; no longer R26.2
- net N$24: now also R411.2; no longer R25.2
- net N$25: now also R410.2; no longer R24.2
- net N$26: now also C622.C1; no longer C110.C1
- net N$27: now also C307.C1, FB302.2; no longer C20.C1, FB2.2
- net N$28: now also C609.C1; no longer C97.C1
- net N$3: now also C509.C1, L521.2; no longer C65.C1, L22.2
- net N$30: now also C422.C1; no longer C50.C1
- net N$33: now also L518.2, L522.1, L526.1; no longer L19.2, L23.1, L27.1
- net N$34: now also C502.C1, L506.2; no longer C58.C1, L7.2
- net N$35: now also C506.C1, L514.2; no longer C62.C1, L15.2
- net N$36: now also C510.C1, L522.2; no longer C66.C1, L23.2
- net N$37: now also C305.C1, C306.C1, U301.VOUT; no longer C19.C1, U3.VOUT
- net N$38: now also C514.C1, L526.2; no longer C70.C1, L27.2
- net N$39: now also L501.2, L505.1, L509.1; no longer L10.1, L2.2, L6.1
- net N$4: now also C513.C1, L525.2; no longer C69.C1, L26.2
- net N$40: now also L509.2, L513.1, L517.1; no longer L10.2, L14.1, L18.1
- net N$41: now also C513.C2; no longer C69.C2
- net N$42: now also L517.2, L521.1, L525.1; no longer L18.2, L22.1, L26.1
- net N$43: now also L503.2, L507.1, L511.1; no longer L12.1, L4.2, L8.1
- net N$44: now also L511.2, L515.1, L519.1; no longer L12.2, L16.1, L20.1
- net N$45: now also C515.C2; no longer C71.C2
- net N$46: now also L519.2, L523.1, L527.1; no longer L20.2, L24.1, L28.1
- net N$47: now also C503.C1, L507.2; no longer C59.C1, L8.2
- net N$48: now also C507.C1, L515.2; no longer C63.C1, L16.2
- net N$49: now also C511.C1, L523.2; no longer C67.C1, L24.2
- net N$5: now also L502.2, L506.1, L510.1; no longer L11.1, L3.2, L7.1
- net N$50: now also C515.C1, L527.2; no longer C71.C1, L28.2
- net N$51: now also L504.2, L508.1, L512.1; no longer L13.1, L5.2, L9.1
- net N$52: now also L512.2, L516.1, L520.1; no longer L13.2, L17.1, L21.1
- net N$53: now also C516.C2; no longer C72.C2
- net N$54: now also L520.2, L524.1, L528.1; no longer L21.2, L25.1, L29.1
- net N$55: now also C504.C1, L508.2; no longer C60.C1, L9.2
- net N$56: now also C508.C1, L516.2; no longer C64.C1, L17.2
- net N$57: now also C512.C1, L524.2; no longer C68.C1, L25.2
- net N$58: now also C516.C1, L528.2; no longer C72.C1, L29.2
- net N$59: now also L529.2, L533.1, L537.1; no longer L30.2, L34.1, L38.1
- net N$6: now also L510.2, L514.1, L518.1; no longer L11.2, L15.1, L19.1
- net N$60: now also L537.2, L541.1, L545.1; no longer L38.2, L42.1, L46.1
- net N$61: now also C529.C2; no longer C85.C2
- net N$62: now also L545.2, L549.1, L553.1; no longer L46.2, L50.1, L54.1
- net N$63: now also C517.C1, L533.2; no longer C73.C1, L34.2
- net N$64: now also C521.C1, L541.2; no longer C77.C1, L42.2
- net N$65: now also C525.C1, L549.2; no longer C81.C1, L50.2
- net N$66: now also C529.C1, L553.2; no longer C85.C1, L54.2
- net N$67: now also L530.2, L534.1, L538.1; no longer L31.2, L35.1, L39.1
- net N$68: now also L538.2, L542.1, L546.1; no longer L39.2, L43.1, L47.1
- net N$69: now also C530.C2; no longer C86.C2
- net N$7: now also C309.C1, U303.1.+IN; no longer C22.C1, U5.1.+IN
- net N$70: now also L546.2, L550.1, L554.1; no longer L47.2, L51.1, L55.1
- net N$71: now also C518.C1, L534.2; no longer C74.C1, L35.2
- net N$72: now also C522.C1, L542.2; no longer C78.C1, L43.2
- net N$73: now also C526.C1, L550.2; no longer C82.C1, L51.2
- net N$74: now also C530.C1, L554.2; no longer C86.C1, L55.2
- net N$75: now also L531.2, L535.1, L539.1; no longer L32.2, L36.1, L40.1
- net N$76: now also L539.2, L543.1, L547.1; no longer L40.2, L44.1, L48.1
- net N$77: now also C531.C2; no longer C87.C2
- net N$78: now also L547.2, L551.1, L555.1; no longer L48.2, L52.1, L56.1
- net N$79: now also C519.C1, L535.2; no longer C75.C1, L36.2
- net N$80: now also C523.C1, L543.2; no longer C79.C1, L44.2
- net N$81: now also C527.C1, L551.2; no longer C83.C1, L52.2
- net N$82: now also C531.C1, L555.2; no longer C87.C1, L56.2
- net N$91: now also C418.C2; no longer C46.C2
- net N$93: now also C413.C2, C421.C1, R408.1, R409.2; no longer C41.C2, C49.C1, R22.1, R23.2
- net N$94: now also C402.C1, R402.1; no longer C30.C1, R16.1
- net N$95: now also C417.C1, R409.1; no longer C45.C1, R23.1
- net N$96: now also R419.2; no longer R33.2
- net N$97: now also R420.2; no longer R34.2
- net N$98: now also R421.2; no longer R35.2
- net N$99: now also R422.2; no longer R36.2
- net OCXO_CLK: now also R302.2, U2.1.A, U304.CLK; no longer C41.C1, R14.1, R22.2
- net OCXO_EN: now also R603.2; no longer R42.2
- net OCXO_VCONT: now also C311.C1, C314.C1, R301.2, U303.1.-IN, U303.1.OUT; no longer C27.C1, C28.C1, R12.1, R13.2, U5.2.OUT
- net PLL_IN0_N: now also C404.C1; no longer C32.C1
- net PLL_IN0_P: now also C403.C2; no longer C31.C2
- net PLL_IN1_N: now also C425.C1; no longer C53.C1
- net PLL_IN1_P: now also C421.C2; no longer C49.C2
- net PLL_OUT0: now also L501.1, R410.1; no longer L2.1, R24.1
- net PLL_OUT1: now also L502.1, R411.1; no longer L3.1, R25.1
- net PLL_OUT2: now also L503.1, R412.1; no longer L4.1, R26.1
- net PLL_OUT3: now also L504.1, R413.1; no longer L5.1, R27.1
- net PLL_OUT4: now also L529.1, R414.1; no longer L30.1, R28.1
- net PLL_OUT5: now also L530.1, R415.1; no longer L31.1, R29.1
- net PLL_OUT6: now also L531.1, R416.1; no longer L32.1, R30.1
- net VIN: now also R601.2, R612.2; no longer R40.2, R51.2
- net VIN_VSENSE: now also C629.C1, R612.1, R613.2; no longer C117.C1, R51.1, R52.2

Commit message: Work on GPSDO
Signed-off-by: João Silva <jgc3silva@gmail.com>
Parts:
- removed C401, C413: 6pF, Capacitor:CAPACITOR-0402
- removed C402, C403, C404, C417, C418, C421, C422, C425, C529, C530, C531, C626, C628: 100nF, Capacitor:CAPACITOR-0402
- removed C406, C407, C408, C409, C410, C412, C414, C419, C420, C423, C424, C426, C427, C428: 1uF, Capacitor:CAPACITOR-0402
- removed C411, C416, C627: 10uF, Capacitor:CAPACITOR-0603
- removed C415: 10pF, Capacitor:CAPACITOR-0402
- removed C517, C518, C519: 270pF, Capacitor:CAPACITOR-0402
- removed C521, C522, C523, C525, C526, C527: 220pF, Capacitor:CAPACITOR-0402
- removed C625: 100uF, Capacitor:CAPACITOR-1206
- removed C629: 470pF, Capacitor:CAPACITOR-0402
- removed C631: 10uF, Capacitor:CAPACITOR-1206
- removed D101: LED0603, LED:LED0603
- removed FB402, FB403, FB404: 1uH, Inductor:FERRITE-0603
- removed L529, L530, L531: 560nH, Inductor:INDUCTOR-0402
- removed L533, L534, L535: 68nH, Inductor:INDUCTOR-0402
- removed L537, L538, L539: 1uH, Inductor:INDUCTOR-0402
- removed L541, L542, L543: 330nH, Inductor:INDUCTOR-0402
- removed L545, L546, L547: 820nH, Inductor:INDUCTOR-0402
- removed L549, L550, L551: 220nH, Inductor:INDUCTOR-0402
- removed L553, L554, L555: 470nH, Inductor:INDUCTOR-0402
- removed R202, R302: 49.9 Ohms, Resistor:RESISTOR-0603
- removed R403, R404, R405, R406, R407: 10K Ohms, Resistor:RESISTOR-0402
- removed R408: 470 Ohms, Resistor:RESISTOR-0402
- removed R409: 865 Ohms, Resistor:RESISTOR-0402
- removed R410, R411, R412, R413, R414, R415, R416, R418, R419, R420, R421, R422, R423, R424: 28 Ohms, Resistor:RESISTOR-0402
- removed RFCON505, RFCON506, RFCON507, RFCON509, RFCON510, RFCON511, RFCON512, RFCON513, RFCON514, RFCON515: RFCON-U.FL, RF Connector:RFCON-U.FL
- removed U101: EFM32GG11B120F2048GM64, EFM32:EFM32GG11B120F2048GM64
- removed U201: MAX-M8Q, U-Blox:MAX-M8Q
- removed U401: DSB321SDA, Crystal:DSB321SDA
- removed U402: SI5347A, Silicon Labs:SI5347A
- added C12, C28, C38: 10uF, Capacitor:CAPACITOR-0603
- added C29, C30, C31, C32, C33, C34, C36, C39, C41, C43, C44, C6, C73, C74, C75, C76, C77: 1uF, Capacitor:CAPACITOR-0402
- added C35: 10pF, Capacitor:CAPACITOR-0402
- added C37, C4, C40, C5, C67, C68, C69, C70, C71, C72: 100nF, Capacitor:CAPACITOR-0402
- added C42, C45: 220nF, Capacitor:CAPACITOR-0402
- added C46, C47: 3.9nF, Capacitor:CAPACITOR-0402
- added C52: 270pF, Capacitor:CAPACITOR-0402
- added C57, C62: 220pF, Capacitor:CAPACITOR-0402
- added CON1: 3P-SH-SIDE, JST:3P-SH-SIDE
- added CON2: 4P-SH-TOP, JST:4P-SH-TOP
- added D10: LEDTH3MM, LED:LEDTH3MM
- added D4, D5, D6, D7, D8: BAV99, Generic Diode:BAV99
- added FB3: 10uH, Inductor:FERRITE-0603
- added FB4, FB5, FB6: 1uH, Inductor:FERRITE-0603
- added L11: 68nH, Inductor:INDUCTOR-0402
- added L16: 1uH, Inductor:INDUCTOR-0402
- added L21: 330nH, Inductor:INDUCTOR-0402
- added L26: 820nH, Inductor:INDUCTOR-0402
- added L31: 220nH, Inductor:INDUCTOR-0402
- added L36: 470nH, Inductor:INDUCTOR-0402
- added L6: 560nH, Inductor:INDUCTOR-0402
- added R1, R5: 4.7K Ohms, Resistor:RESISTOR-0402
- added R14, R15, R16, R17, R23, R24, R25: 10K Ohms, Resistor:RESISTOR-0402
- added R2, R27, R29, R3, R31, R33, R35: 100 Ohms, Resistor:RESISTOR-0402
- added R20: 470 Ohms, Resistor:RESISTOR-0402
- added R21: 865 Ohms, Resistor:RESISTOR-0402
- added R22, R41, R42, R43, R44, R45: 0 Ohms, Resistor:RESISTOR-0402
- added R26, R28, R30, R32, R34: 49.9 Ohms, Resistor:RESISTOR-0402
- added R36, R37, R38, R39, R40: 10K Ohms, Potentiometer:POTENTIOMETER-SMD-3X3
- added RFCON10, RFCON11, RFCON6, RFCON7, RFCON8, RFCON9: RFCON-U.FL, RF Connector:RFCON-U.FL
- added U10, U11, U12, U13, U9: 74LVC1G17, Logic:74LVC1G17
- added U7: DSB321SDA, Crystal:DSB321SDA
- added U8: AD9544, Analog Devices:AD9544
- C1: value 10uF -> 100nF; device Capacitor:CAPACITOR-0603 -> Capacitor:CAPACITOR-0402
- C101: value 100nF -> 100uF; device Capacitor:CAPACITOR-0402 -> Capacitor:CAPACITOR-1206
- C103: value 100nF -> 10uF; device Capacitor:CAPACITOR-0402 -> Capacitor:CAPACITOR-0603
- C105: value 100nF -> 470pF
- C107: value 1uF -> 10uF; device Capacitor:CAPACITOR-0402 -> Capacitor:CAPACITOR-1206; VOLTAGE (none) -> 50V
- D1: value LEDTH3MM -> LED0603; device LED:LEDTH3MM -> LED:LED0603; COLOR GREEN -> BLUE
- U1: value 74LVC1G17 -> EFM32GG11B120F2048GM64; device Logic:74LVC1G17 -> EFM32:EFM32GG11B120F2048GM64
- U2: value 74LVC1G17 -> MAX-M8Q; device Logic:74LVC1G17 -> U-Blox:MAX-M8Q
- renumbered BAT201 to BAT1, C201 to C7, C202 to C8, C203 to C9, C204 to C10, C205 to C11, C206 to C13, C207 to C14, C302 to C15, C303 to C16, C304 to C17, C305 to C18, C306 to C19, C307 to C20, C308 to C21, C309 to C22, C310 to C23, C311 to C24, C312 to C25, C313 to C26, C314 to C27, C501 to C48, C502 to C49, C503 to C50, C504 to C51, C505 to C53, C506 to C54, C507 to C55, C508 to C56, C509 to C58, C510 to C59, C511 to C60, C512 to C61, C513 to C63, C514 to C64, C515 to C65, C516 to C66, C601 to C78, C602 to C79, C603 to C80, C604 to C81, C605 to C82, C606 to C83, C607 to C84, C608 to C85, C609 to C86, C610 to C87, C611 to C88, C612 to C89, C613 to C90, C614 to C91, C615 to C92, C616 to C93, C617 to C94, C618 to C95, C619 to C96, C620 to C97, C621 to C98, C622 to C99, C624 to C100, C630 to C106, CON201 to CON3, CON601 to CON4, D201 to D3, D601 to D9, D602 to D11, F601 to F1, FB301 to FB1, FB302 to FB2, J601 to J1, L201 to L1, L501 to L2, L502 to L3, L503 to L4, L504 to L5, L505 to L7, L506 to L8, L507 to L9, L508 to L10, L509 to L12, L510 to L13, L511 to L14, L512 to L15, L513 to L17, L514 to L18, L515 to L19, L516 to L20, L517 to L22, L518 to L23, L519 to L24, L520 to L25, L521 to L27, L522 to L28, L523 to L29, L524 to L30, L525 to L32, L526 to L33, L527 to L34, L528 to L35, L601 to L37, L602 to L38, LOGO101 to LOGO1, R101 to R4, R102 to R6, R103 to R8, R104 to R7, R201 to R9, R203 to R10, R204 to R11, R205 to R12, R301 to R13, R401 to R18, R402 to R19, R601 to R46, R602 to R47, R603 to R48, R604 to R49, R605 to R50, R606 to R51, R607 to R52, R608 to R53, R609 to R54, R610 to R55, R611 to R56, R612 to R57, R613 to R58, R614 to R59, R615 to R60, RFCON201 to RFCON1, RFCON501 to RFCON2, RFCON502 to RFCON3, RFCON503 to RFCON4, RFCON504 to RFCON5, TC101 to TC1, U301 to U3, U302 to U4, U303 to U5, U304 to U6, U601 to U14, U602 to U15, U603 to U16, U604 to U17, U605 to U18
Connections:
- net 5V0_ANA_OCXO_FILT renamed 5V0_ANA_OCXO_CLEAN_FILT
- removed net !PLL_LOLA: U402.!LOL_A
- removed net !PLL_LOLB: U402.!LOL_B
- removed net !PLL_LOLC: U402.!LOL_C
- removed net !PLL_LOLD: U402.!LOL_D
- removed net !PLL_OE0: R405.1, U402.!OE0
- removed net !PLL_OE1: R406.1, U402.!OE1
- removed net !PLL_OUT0: R418.1, RFCON509.SIGNAL
- removed net !PLL_OUT1: R419.1, RFCON512.SIGNAL
- removed net !PLL_OUT2: R420.1, RFCON514.SIGNAL
- removed net !PLL_OUT3: R421.1, RFCON510.SIGNAL
- removed net !PLL_OUT4: R422.1, RFCON513.SIGNAL
- removed net !PLL_OUT5: R423.1, RFCON515.SIGNAL
- removed net !PLL_OUT6: R424.1, RFCON511.SIGNAL
- removed net !PLL_XTAL_LOS: U402.!LOS_XAXB
- removed net 3V3_ANA_PLL_CLEAN: C406.C1, C408.C1, C409.C1, C410.C1, C412.C1, C414.C1, C420.C1, C424.C1, C427.C1, C627.C1, C628.C1, FB402.1, U18.SENSE, U18.VOUT, U402.VDDA, U402.VDDO0, U402.VDDO1, U402.VDDO2, U402.VDDO3, U402.VDDO4, U402.VDDO5, U402.VDDO6, U402.VDDO7
- removed net GPS_BIAS_EXT: R11.1
- removed net GPS_TIMEPULSE_BUF: U1.1.Y
- removed net GPS_TIMEPULSE_KZ: C401.C1, R18.2, R202.1
- removed net N$100: R423.2, U402.!OUT5
- removed net N$101: R424.2, U402.!OUT6
- removed net N$104: C428.C1, FB404.2, U402.VDDS
- removed net N$15: R418.2, U402.!OUT0
- removed net N$76: L539.2, L543.1, L547.1
- removed net N$77: C531.C2, RFCON507.SIGNAL
- removed net N$78: L547.2, L551.1, L555.1
- removed net N$79: C519.C1, L535.2
- removed net N$80: C523.C1, L543.2
- removed net N$81: C527.C1, L551.2
- removed net N$82: C531.C1, L555.2
- removed net N$93: C413.C2, C421.C1, R408.1, R409.2
- removed net N$94: C402.C1, R19.1
- removed net N$95: C417.C1, R409.1
- removed net N$96: R419.2, U402.!OUT1
- removed net N$97: R420.2, U402.!OUT2
- removed net N$98: R421.2, U402.!OUT3
- removed net N$99: R422.2, U402.!OUT4
- removed net OCXO_CLK_BUF: U2.1.Y
- removed net OCXO_CLK_KZ: C413.C1, R302.1, R408.2
- removed net PLL_FDEC: U402.FDEC
- removed net PLL_FINC: U402.FINC
- removed net PLL_IN0_N: C404.C1, U402.!IN0
- removed net PLL_IN0_P: C403.C2, U402.IN0
- removed net PLL_IN1_N: C425.C1, U402.!IN1
- removed net PLL_IN1_P: C421.C2, U402.IN1
- removed net PLL_OUT0: L2.1, R410.1
- removed net PLL_OUT1: L3.1, R411.1
- removed net PLL_OUT2: L4.1, R412.1
- removed net PLL_OUT3: L5.1, R413.1
- removed net PLL_OUT4: L529.1, R414.1
- removed net PLL_OUT5: L530.1, R415.1
- removed net PLL_OUT6: L531.1, R416.1
- removed net PLL_SEL0: U402.DSPLL_SEL0
- removed net PLL_SEL1: U402.DSPLL_SEL1
- new net !CLK0: L2.1, R26.2, U8.!OUT0A
- new net !CLK1: L3.1, R28.2, U8.!OUT0B
- new net !CLK2: L4.1, R30.2, U8.!OUT0C
- new net !CLK3: L5.1, R32.2, U8.!OUT1B
- new net !CLK4: L6.1, R34.2, U8.!OUT1A
- new net 3V3_ANA_CLEAN: C103.C1, C104.C1, C73.C1, C74.C1, C75.C1, C76.C1, C77.C1, R36.CCW, R37.CCW, R38.CCW, R39.CCW, R40.CCW, U10.PWR.VCC, U11.PWR.VCC, U12.PWR.VCC, U13.PWR.VCC, U18.SENSE, U18.VOUT, U9.PWR.VCC
- new net 3V3_PLL_FILT: C44.C1, FB6.2, U8.VDDIOA, U8.VDDIOB
- new net CLK0: C68.C1, R27.2, U8.OUT0A
- new net CLK1: C69.C1, R29.2, U8.OUT0B
- new net CLK2: C70.C1, R31.2, U8.OUT0C
- new net CLK3: C71.C1, R33.2, U8.OUT1B
- new net CLK4: C72.C1, R35.2, U8.OUT1A
- new net I2C1_SCL: R3.2, R8.1
- new net I2C1_SDA: R2.2, R6.1
- new net N$19: CON1-1.S, R2.1
- new net N$29: R44.2, U12.1.Y
- new net N$32: C71.C2, R39.WIPER, U12.1.A
- new net N$8: R45.1, RFCON11.SIGNAL
- new net N$9: CON1-2.S, R3.1
- new net PLL_M3: R14.2, U8.M3
- new net PLL_M4: R15.1, U8.M4
- new net PLL_M5: R16.2, U8.M5/SDO
- new net PLL_M6: R17.2, U8.M6/!CS
- new net PLL_REFA: R20.1, R21.2, U8.REFA
- new net PLL_REFB: R18.1, R19.2, U8.REFB
- net !GPS_RESET: now also U2.!RESET; no longer U201.!RESET
- net !MCU_RESET: now also U1.!RESET; no longer U101.!RESET
- net !PLL_IRQ: now also R25.1, U8.M0; no longer R404.1, U402.!INTR
- net !PLL_RESET: now also R23.1, U8.!RESET; no longer R403.1, U402.!RST
- net 1V8_PLL_CLEAN: now also C28.C1, FB3.1, FB4.1, FB5.1; no longer C411.C1, FB403.1
- net 1V8_PLL_CLEAN_FILT: now also C30.C1, C31.C1, C32.C1, C33.C1, C34.C1, C36.C1, C39.C1, C41.C1, C43.C1, FB4.2, FB5.2, U8.VDD; no longer C419.C1, C423.C1, C426.C1, FB403.2, U402.VDD
- net 3V3: now also C1.C1, C38.C1, C4.C1, C5.C1, CON2-1.S, FB6.1, R1.2, R15.2, R23.2, R25.2, R5.2, U1.AVDD@0, U1.AVDD@1, U1.DVDD, U1.IOVDD0@0, U1.IOVDD0@1, U1.IOVDD0@2, U2.VCC, U2.VCC_IO; no longer C101.C1, C102.C1, C103.C1, C104.C1, C105.C1, C416.C1, FB404.1, R403.2, R404.2, R405.2, R406.2, U1.PWR.VCC, U101.AVDD@0, U101.AVDD@1, U101.DVDD, U101.IOVDD0@0, U101.IOVDD0@1, U101.IOVDD0@2, U2.PWR.VCC, U201.VCC, U201.VCC_IO, U402.A0/!CS, U402.A1/SDO
- net 5V0: now also C101.C1, C102.C1, R11.1; no longer C625.C1, C626.C1
- net GND: now also C12.C2, C28.C2, C29.C2, C30.C2, C31.C2, C32.C2, C33.C2, C34.C2, C35.C2, C36.C2, C38.C2, C39.C2, C4.C2, C40.C2, C41.C2, C42.C2, C43.C2, C44.C2, C45.C2, C5.C2, C52.C2, C57.C2, C6.C2, C62.C2, C73.C2, C74.C2, C75.C2, C76.C2, C77.C2, CON1-3.S, CON2-4.S, D10.C, D4.A, D4.C, D5.A, D5.C, D6.A, D6.C, D7.A, D7.C, D8.A, D8.C, R14.1, R16.1, R17.1, R19.1, R21.1, R24.1, R26.1, R27.1, R28.1, R29.1, R30.1, R31.1, R32.1, R33.1, R34.1, R35.1, R36.CW, R37.CW, R38.CW, R39.CW, R40.CW, RFCON10.GND, RFCON11.GND, RFCON6.GND, RFCON7.GND, RFCON8.GND, RFCON9.GND, U1.VSS@0, U10.PWR.GND, U11.PWR.GND, U12.PWR.GND, U13.PWR.GND, U2.GND@0, U2.GND@1, U2.GND@2, U7.GND, U8.GND, U9.PWR.GND; no longer C402.C2, C404.C2, C406.C2, C407.C2, C408.C2, C409.C2, C410.C2, C411.C2, C412.C2, C414.C2, C415.C2, C416.C2, C417.C2, C419.C2, C420.C2, C422.C2, C423.C2, C424.C2, C425.C2, C426.C2, C427.C2, C428.C2, C517.C2, C518.C2, C519.C2, C521.C2, C522.C2, C523.C2, C525.C2, C526.C2, C527.C2, C625.C2, C626.C2, C627.C2, C628.C2, C629.C2, C631.C2, D101.C, R407.1, RFCON505.GND, RFCON506.GND, RFCON507.GND, RFCON509.GND, RFCON510.GND, RFCON511.GND, RFCON512.GND, RFCON513.GND, RFCON514.GND, RFCON515.GND, U1.PWR.GND, U101.VSS@0, U2.PWR.GND, U201.GND@0, U201.GND@1, U201.GND@2, U401.GND, U402.GND
- net GPS_BIAS_INT: now also U2.VCC_RF; no longer U201.VCC_RF
- net GPS_RXD: now also U2.RXD; no longer U201.RXD
- net GPS_TIMEPULSE: now also R18.2, U2.TIMEPULSE; no longer R202.2, U1.1.A, U201.TIMEPULSE
- net GPS_TXD/TXREADY: now also U2.TXD; no longer U201.TXD
- net GPS_VBKP: now also C12.C1, U2.V_BKP; no longer C1.C1, U201.V_BKP
- net I2C0_SCL: now also CON2-3.S, R5.1, U2.SCL, U8.SCL/SCLK; no longer R8.1, U201.SCL, U402.SCLK
- net I2C0_SDA: now also CON2-2.S, R1.1, U2.SDA, U8.SDA/SDIO; no longer R6.1, U201.SDA, U402.SDA/SDIO
- net MCU_LED: now also U1.PB11
- net MCU_SWCLK: now also U1.PF0; no longer U101.PF0
- net MCU_SWDIO: now also U1.PF1; no longer U101.PF1
- net MCU_SWO: now also U1.PF2; no longer U101.PF2
- net MCU_VCORE: now also C6.C1, U1.DECOUPLE; no longer C107.C1, U101.DECOUPLE
- net N$10: now also D5.MID
- net N$103: now also C29.C1, FB3.2, U7.VDD; no longer C407.C1, FB402.2, U401.VDD
- net N$12: now also U2.RF_IN; no longer U201.RF_IN
- net N$144: now also D1.A; no longer D101.A
- net N$149: now also D10.A; no longer D1.A
- net N$16: now also C72.C2, R40.WIPER, U13.1.A; no longer C401.C2, C403.C1, R18.1, R19.2
- net N$17: now also C35.C1, C37.C1, R22.1, R24.2; no longer C415.C1, C418.C1, R407.2, U401.CLK
- net N$18: now also R22.2, U7.CLK; no longer R416.2, U402.OUT6
- net N$20: now also C45.C1, C47.C1, U8.LDO1; no longer R415.2, U402.OUT5
- net N$21: now also C42.C1, C46.C1, U8.LDO0; no longer R414.2, U402.OUT4
- net N$22: now also C47.C2, U8.LF1; no longer R413.2, U402.OUT3
- net N$23: now also C46.C2, U8.LF0; no longer R412.2, U402.OUT2
- net N$24: now also R45.2, U13.1.Y; no longer R411.2, U402.OUT1
- net N$25: now also R44.1, RFCON10.SIGNAL; no longer R410.2, U402.OUT0
- net N$30: now also C40.C1, U8.XOB; no longer C422.C1, U402.XB
- net N$41: now also D4.MID
- net N$45: now also D6.MID
- net N$53: now also D7.MID
- net N$59: now also L11.1, L16.1, L6.2; no longer L529.2, L533.1, L537.1
- net N$60: now also L16.2, L21.1, L26.1; no longer L537.2, L541.1, L545.1
- net N$61: now also C67.C2, D8.MID, RFCON6.SIGNAL; no longer C529.C2, RFCON505.SIGNAL
- net N$62: now also L26.2, L31.1, L36.1; no longer L545.2, L549.1, L553.1
- net N$63: now also C52.C1, L11.2; no longer C517.C1, L533.2
- net N$64: now also C57.C1, L21.2; no longer C521.C1, L541.2
- net N$65: now also C62.C1, L31.2; no longer C525.C1, L549.2
- net N$66: now also C67.C1, L36.2; no longer C529.C1, L553.2
- net N$67: now also R43.1, RFCON9.SIGNAL; no longer L530.2, L534.1, L538.1
- net N$68: now also R43.2, U11.1.Y; no longer L538.2, L542.1, L546.1
- net N$69: now also C70.C2, R38.WIPER, U11.1.A; no longer C530.C2, RFCON506.SIGNAL
- net N$70: now also R42.1, RFCON8.SIGNAL; no longer L546.2, L550.1, L554.1
- net N$71: now also R42.2, U10.1.Y; no longer C518.C1, L534.2
- net N$72: now also C69.C2, R37.WIPER, U10.1.A; no longer C522.C1, L542.2
- net N$73: now also R41.1, RFCON7.SIGNAL; no longer C526.C1, L550.2
- net N$74: now also R41.2, U9.1.Y; no longer C530.C1, L554.2
- net N$75: now also C68.C2, R36.WIPER, U9.1.A; no longer L531.2, L535.1, L539.1
- net N$91: now also C37.C2, U8.XOA; no longer C418.C2, U402.XA
- net OCXO_CLK: now also R20.2; no longer R302.2, U2.1.A
- net VIN: now also C107.C1; no longer C631.C1
- net VIN_VSENSE: now also C105.C1; no longer C629.C1
Other:
- note added: "Do not load from EEPROM"
- note added: "I2C Address 0x48"
- note added: "Select I2C Interface"
- note removed: "Po = +10 dBm"

Commit message: Work on GPSDO
Signed-off-by: João Silva <jgc3silva@gmail.com>
Parts:
- added C108, C109: 10uF, Capacitor:CAPACITOR-0603
- added C110, C111: 100nF, Capacitor:CAPACITOR-0402
- added U19, U20: 74LVC1G17, Logic:74LVC1G17
Connections:
- removed net I2C1_SCL: R3.2, R8.1
- removed net I2C1_SDA: R2.2, R6.1
- new net GPS_TIMEPULSE_BUF: U19.1.Y
- new net I2C2_SCL: R3.2, R8.1, U1.PF5
- new net I2C2_SDA: R2.2, R6.1, U1.PF4
- new net OCXO_CLK_BUF: U20.1.Y
- net !DAC_CS: now also U1.PE13
- net !PLL_IRQ: now also U1.PC13
- net !PLL_RESET: now also U1.PC12
- net 3V3: now also C109.C1, C110.C1, C111.C1, U19.PWR.VCC, U20.PWR.VCC
- net 3V3_PGOOD: no longer U18.EN
- net 5V0: now also C108.C1
- net 5V0_PGOOD: now also U18.EN
- net 5V0_VSENSE: now also U1.PD6
- net DAC_DIN: now also U1.PE10
- net DAC_SCLK: now also U1.PE12
- net GND: now also C108.C2, C109.C2, C110.C2, C111.C2, U19.PWR.GND, U20.PWR.GND
- net GPS_TIMEPULSE: now also U19.1.A
- net I2C0_SCL: now also U1.PC15
- net I2C0_SDA: now also U1.PC14
- net OCXO_CLK: now also U20.1.A
- net OCXO_EN: now also U1.PE11
- net VIN_VSENSE: now also U1.PD1
