File: pcb/gpsdo/qo-100-gpsdo.sch (EAGLE design)
At the start: 266 parts, among them CON1 3P-SH-SIDE, CON2 4P-SH-TOP, CON3 3P-SH-TOP, CON4 2EDG-2P-5MM, J1 DCJACK, U1 EFM32GG11B120F2048GM64, U10 74LVC1G17, U11 74LVC1G17, U12 74LVC1G17, U13 74LVC1G17, U14 ADM7171ACPZ-1.8, U15 ADM7171ACPZ-5.0, U16 MIC23155, U17 LT8636, U18 ADM7171ACPZ-3.3, U19 74LVC1G17, U2 MAX-M8Q, U20 74LVC1G17, U3 MCP1501-40, U4 AD5541ACPZ, U5 MCP6V31, U6 OSC5A2B02, U7 DSB321SDA, U8 AD9544, U9 74LVC1G17

Commit message: Generate production files for GPSDO
Signed-off-by: João Silva <jgc3silva@gmail.com>
Parts:
- added C112, C114: 100nF, Capacitor:CAPACITOR-0402
- added C113: 10uF, Capacitor:CAPACITOR-0603
- added C115, C116: 470pF, Capacitor:CAPACITOR-0402
- added C117: 10uF, Capacitor:CAPACITOR-1206
- C10, C102, C20: value 100nF -> 10uF; device Capacitor:CAPACITOR-0402 -> Capacitor:CAPACITOR-0603
- C100: value 100uF -> 10uF; device Capacitor:CAPACITOR-1206 -> Capacitor:CAPACITOR-0603
- C101, C25, C7: value 100uF -> 100nF; device Capacitor:CAPACITOR-1206 -> Capacitor:CAPACITOR-0402
- C103, C12, C18, C90: value 10uF -> 100nF; device Capacitor:CAPACITOR-0603 -> Capacitor:CAPACITOR-0402
- C105: value 470pF -> 10pF
- C106: value 470pF -> 100nF
- C107: value 10uF -> 100nF; device Capacitor:CAPACITOR-1206 -> Capacitor:CAPACITOR-0402; VOLTAGE 50V -> (none)
- C108: value 10uF -> 100uF; device Capacitor:CAPACITOR-0603 -> Capacitor:CAPACITOR-1206
- C109: value 10uF -> 10nF; device Capacitor:CAPACITOR-0603 -> Capacitor:CAPACITOR-0402
- C11: value 47pF -> 100uF; device Capacitor:CAPACITOR-0402 -> Capacitor:CAPACITOR-1206
- C110, C111: value 100nF -> 100uF; device Capacitor:CAPACITOR-0402 -> Capacitor:CAPACITOR-1206
- C15: value 10uF -> 47pF; device Capacitor:CAPACITOR-0603 -> Capacitor:CAPACITOR-0402
- C16, C17, C23, C33, C43: value 1uF -> 10uF; device Capacitor:CAPACITOR-0402 -> Capacitor:CAPACITOR-0603
- C22, C26, C37, C78, C79, C8: value 100nF -> 1uF
- C28, C38: value 10uF -> 1uF; device Capacitor:CAPACITOR-0603 -> Capacitor:CAPACITOR-0402
- C29, C31, C32, C6, C73, C74, C75, C76, C77, C88: value 1uF -> 100nF
- C30: value 1uF -> 100uF; device Capacitor:CAPACITOR-0402 -> Capacitor:CAPACITOR-1206
- C35: value 10pF -> 1uF
- C40: value 100nF -> 10pF
- C42, C45: value 220nF -> 100nF
- C46: value 3.9nF -> 1uF
- C47: value 3.9nF -> 220nF
- C48, C49: value 270pF -> 1uF
- C50: value 270pF -> 220nF
- C51, C52: value 270pF -> 3.9nF
- C53, C54: value 220pF -> 270pF
- C55, C56: value 220pF -> 100pF
- C57, C60, C61: value 220pF -> 68pF
- C58, C59: value 220pF -> 180pF
- C62: value 220pF -> 47pF
- C63, C64: value 100nF -> 180pF
- C65, C66: value 100nF -> 68pF
- C67: value 100nF -> 47pF
- C81: value 4.7uF -> 100nF; device Capacitor:CAPACITOR-0603 -> Capacitor:CAPACITOR-0402
- C82: value 4.7uF -> 100nF; device Capacitor:CAPACITOR-0603 -> Capacitor:CAPACITOR-0402; VOLTAGE 35V -> (none)
- C83, C89: value 10nF -> 100nF
- C84: value 1uF -> 100nF; device Capacitor:CAPACITOR-0603 -> Capacitor:CAPACITOR-0402; VOLTAGE 50V -> (none)
- C85: device Capacitor:CAPACITOR-0603 -> Capacitor:CAPACITOR-0402; VOLTAGE 50V -> (none)
- C86: value 10nF -> 1uF
- C87: value 470pF -> 1uF
- C91: value 100nF -> 4.7uF; device Capacitor:CAPACITOR-0402 -> Capacitor:CAPACITOR-0603
- C92: value 10uF -> 4.7uF; VOLTAGE (none) -> 35V
- C93, C96: value 100nF -> 10nF
- C94: value 100nF -> 1uF; device Capacitor:CAPACITOR-0402 -> Capacitor:CAPACITOR-0603; VOLTAGE (none) -> 50V
- C95: value 10pF -> 1uF; device Capacitor:CAPACITOR-0402 -> Capacitor:CAPACITOR-0603; VOLTAGE (none) -> 50V
- C97: value 100nF -> 470pF
- C98: value 100uF -> 1uF; device Capacitor:CAPACITOR-1206 -> Capacitor:CAPACITOR-0402
- L10, L9: value 68nH -> 33nH
- L11: value 68nH -> 22nH
- L12, L13: value 1uH -> 820nH
- L14, L15: value 1uH -> 270nH
- L16: value 1uH -> 180nH
- L17, L18: value 330nH -> 470nH
- L19, L20: value 330nH -> 180nH
- L21: value 330nH -> 120nH
- L22, L23: value 820nH -> 680nH
- L24, L25: value 820nH -> 270nH
- L26: value 820nH -> 180nH
- L27, L28: value 220nH -> 330nH
- L29, L30: value 220nH -> 120nH
- L31: value 220nH -> 82nH
- L32, L33: value 470nH -> 390nH
- L34, L35: value 470nH -> 150nH
- L36: value 470nH -> 100nH
- L4, L5: value 560nH -> 220nH
- L6: value 560nH -> 150nH
- L7, L8: value 68nH -> 82nH
- R18: value 267 Ohms -> 280 Ohms
- R19: value 865 Ohms -> 330 Ohms
- R20: value 470 Ohms -> 510 Ohms
- R21: value 865 Ohms -> 270 Ohms
- R36, R37, R38, R39, R40: value 10K Ohms -> 100K Ohms
- U1: value EFM32GG11B120F2048GM64 -> EFM32GG11B420F2048GM64; device EFM32:EFM32GG11B120F2048GM64 -> EFM32:EFM32GG11B420F2048GM64
- U10: value 74LVC1G17 -> AD9544; device Logic:74LVC1G17 -> Analog Devices:AD9544
- U14: value ADM7171ACPZ-1.8 -> 74LVC1G17; device Analog Devices:ADM7171ACPZ-1.8 -> Logic:74LVC1G17
- U15: value ADM7171ACPZ-5.0 -> 74LVC1G17; device Analog Devices:ADM7171ACPZ-5.0 -> Logic:74LVC1G17
- U16: value MIC23155 -> ADM7171ACPZ-1.8; device Microchip:MIC23155 -> Analog Devices:ADM7171ACPZ-1.8
- U17: value LT8636 -> ADM7171ACPZ-5.0; device Analog Devices:LT8636 -> Analog Devices:ADM7171ACPZ-5.0
- U18: value ADM7171ACPZ-3.3 -> MIC23155; device Analog Devices:ADM7171ACPZ-3.3 -> Microchip:MIC23155
- U19: value 74LVC1G17 -> LT8636; device Logic:74LVC1G17 -> Analog Devices:LT8636
- U2: value MAX-M8Q -> 74LVC1G17; device U-Blox:MAX-M8Q -> Logic:74LVC1G17
- U20: value 74LVC1G17 -> ADM7171ACPZ-3.3; device Logic:74LVC1G17 -> Analog Devices:ADM7171ACPZ-3.3
- U3: value MCP1501-40 -> 74LVC1G17; device Microchip:MCP1501-40 -> Logic:74LVC1G17
- U4: value AD5541ACPZ -> MAX-M8Q; device Analog Devices:AD5541ACPZ -> U-Blox:MAX-M8Q
- U5: value MCP6V31 -> MCP1501-40; device Microchip:MCP6V31 -> Microchip:MCP1501-40
- U6: value OSC5A2B02 -> AD5541ACPZ; device Crystal:OSC5A2B02 -> Analog Devices:AD5541ACPZ
- U7: value DSB321SDA -> MCP6V31; device Crystal:DSB321SDA -> Microchip:MCP6V31
- U8: value AD9544 -> OSC5A2B02; device Analog Devices:AD9544 -> Crystal:OSC5A2B02
- U9: value 74LVC1G17 -> DSB321SDA; device Logic:74LVC1G17 -> Crystal:DSB321SDA
Connections:
- net !CLK0: now also U10.!OUT0A; no longer U8.!OUT0A
- net !CLK1: now also U10.!OUT0B; no longer U8.!OUT0B
- net !CLK2: now also U10.!OUT0C; no longer U8.!OUT0C
- net !CLK3: now also U10.!OUT1B; no longer U8.!OUT1B
- net !CLK4: now also U10.!OUT1A; no longer U8.!OUT1A
- net !DAC_CS: now also U6.!CS; no longer U4.!CS
- net !GPS_RESET: now also U1.PA2, U4.!RESET; no longer U2.!RESET
- net !PLL_IRQ: now also U1.PF11, U10.M0; no longer U1.PC13, U8.M0
- net !PLL_RESET: now also U1.PF10, U10.!RESET; no longer U1.PC12, U8.!RESET
- net 1V8_PLL_CLEAN: now also C100.C1, C101.C1, C33.C1, U16.SENSE, U16.VOUT; no longer C28.C1, C90.C1, C91.C1, U14.SENSE, U14.VOUT
- net 1V8_PLL_CLEAN_FILT: now also C35.C1, C37.C1, C38.C1, C44.C1, C46.C1, C48.C1, U10.VDD; no longer C30.C1, C31.C1, C32.C1, C33.C1, C34.C1, C43.C1, U8.VDD
- net 3V3: now also C10.C1, C107.C1, C108.C1, C11.C1, C12.C1, C18.C1, C22.C1, C43.C1, C6.C1, C89.C1, U1.VREGI, U1.VREGO, U16.VIN, U18.SNS, U2.PWR.VCC, U3.PWR.VCC, U4.VCC, U4.VCC_IO; no longer C109.C1, C110.C1, C111.C1, C17.C1, C38.C1, C79.C1, C8.C1, C97.C1, C98.C1, U14.VIN, U16.SNS, U19.PWR.VCC, U2.VCC, U2.VCC_IO, U20.PWR.VCC
- net 3V3_ANA_CLEAN: now also C113.C1, C114.C1, C78.C1, C79.C1, C80.C1, C81.C1, C82.C1, C83.C1, C84.C1, C85.C1, C86.C1, C87.C1, U14.PWR.VCC, U15.PWR.VCC, U20.SENSE, U20.VOUT; no longer C103.C1, C104.C1, C73.C1, C74.C1, C75.C1, C76.C1, C77.C1, U10.PWR.VCC, U18.SENSE, U18.VOUT, U9.PWR.VCC
- net 3V3_FB: now also U18.FB; no longer U16.FB
- net 3V3_PGOOD: now also U1.PB3, U16.EN, U18.PG; no longer U14.EN, U16.PG
- net 3V3_PLL_FILT: now also C49.C1, U10.VDDIOA, U10.VDDIOB; no longer C44.C1, U8.VDDIOA, U8.VDDIOB
- net 3V3_SS: now also C97.C1, U18.SS; no longer C87.C1, U16.SS
- net 3V3_SW: now also U18.SW; no longer U16.SW
- net 5V0: now also C105.C1, C106.C1, C110.C1, C111.C1, C112.C1, C16.C1, C88.C1, C90.C1, C91.C1, U17.VIN, U18.VIN@0, U18.VIN@1, U19.BIAS, U20.VIN; no longer C100.C1, C101.C1, C102.C1, C108.C1, C78.C1, C80.C1, C81.C1, C95.C1, C96.C1, U15.VIN, U16.VIN@0, U16.VIN@1, U17.BIAS, U18.VIN
- net 5V0_ANA_OCXO_CLEAN: now also C102.C1, C103.C1, C20.C1, C30.C1, C31.C1, U17.SENSE, U17.VOUT, U8.VDD; no longer C15.C1, C25.C1, C26.C1, C92.C1, C93.C1, U15.SENSE, U15.VOUT, U6.VDD
- net 5V0_ANA_OCXO_CLEAN_FILT: now also C26.C1, C28.C1, U5.!SHDN, U5.VDD, U6.VDD, U7.PWR.V+; no longer C16.C1, C23.C1, U3.!SHDN, U3.VDD, U4.VDD, U5.PWR.V+
- net 5V0_BST: now also C104.C2, U19.BST; no longer C94.C2, U17.BST
- net 5V0_EN: now also U19.EN/UV; no longer U17.EN/UV
- net 5V0_FB: now also C105.C2, U19.FB; no longer C95.C2, U17.FB
- net 5V0_INTVCC: now also C98.C1, U19.INTVCC, U19.SYNC/MODE; no longer C88.C1, U17.INTVCC, U17.SYNC/MODE
- net 5V0_PGOOD: now also U1.PB4, U19.PG, U20.EN; no longer U16.EN, U17.PG
- net 5V0_RT: now also U19.RT; no longer U17.RT
- net 5V0_SS: now also C99.C1, U19.TR/SS; no longer C89.C1, U17.TR/SS
- net 5V0_SW: now also C104.C1, U19.SW; no longer C94.C1, U17.SW
- net 5V0_VSENSE: now also C116.C1; no longer C106.C1
- net CLK0: now also C73.C1, U10.OUT0A; no longer C68.C1, U8.OUT0A
- net CLK1: now also C74.C1, U10.OUT0B; no longer C69.C1, U8.OUT0B
- net CLK2: now also C75.C1, U10.OUT0C; no longer C70.C1, U8.OUT0C
- net CLK3: now also C76.C1, U10.OUT1B; no longer C71.C1, U8.OUT1B
- net CLK4: now also C77.C1, U10.OUT1A; no longer C72.C1, U8.OUT1A
- net DAC_DIN: now also U6.DIN; no longer U4.DIN
- net DAC_SCLK: now also U6.SCLK; no longer U4.SCLK
- net GND: now also C11.C2, C112.C2, C113.C2, C114.C2, C115.C2, C116.C2, C117.C2, C37.C2, C46.C2, C47.C2, C63.C2, C64.C2, C65.C2, C66.C2, C67.C2, C94.C2, C95.C2, U10.GND, U14.PWR.GND, U15.PWR.GND, U16.GND, U18.AGND, U18.PGND@0, U18.PGND@1, U19.GND, U2.PWR.GND, U20.GND, U3.PWR.GND, U4.GND@0, U4.GND@1, U4.GND@2, U5.GND@0, U5.GND@1, U5.GND@2, U6.!LDAC, U6.AGND, U6.DGND, U7.PWR.V-, U9.GND; no longer C104.C2, C105.C2, C15.C2, C42.C2, C51.C2, C52.C2, C73.C2, C74.C2, C75.C2, C76.C2, C77.C2, U10.PWR.GND, U14.GND, U15.GND, U16.AGND, U16.PGND@0, U16.PGND@1, U18.GND, U19.PWR.GND, U2.GND@0, U2.GND@1, U2.GND@2, U20.PWR.GND, U3.GND@0, U3.GND@1, U3.GND@2, U4.!LDAC, U4.AGND, U4.DGND, U5.PWR.V-, U6.GND, U7.GND, U9.PWR.GND
- net GPS_BIAS_INT: now also C14.C1, U4.VCC_RF; no longer C10.C1, U2.VCC_RF
- net GPS_RXD: now also U1.PA0, U4.RXD; no longer U2.RXD
- net GPS_TIMEPULSE: now also U3.1.A, U4.TIMEPULSE; no longer U19.1.A, U2.TIMEPULSE
- net GPS_TIMEPULSE_BUF: now also U1.PE15, U3.1.Y; no longer U19.1.Y
- net GPS_TXD/TXREADY: now also U1.PA1, U4.TXD; no longer U2.TXD
- net GPS_VBKP: now also C17.C1, C19.C1, U4.V_BKP; no longer C12.C1, C14.C1, U2.V_BKP
- net I2C0_SCL: now also U1.PE5, U10.SCL/SCLK, U4.SCL; no longer U1.PC15, U2.SCL, U8.SCL/SCLK
- net I2C0_SDA: now also U1.PE4, U10.SDA/SDIO, U4.SDA; no longer U1.PC14, U2.SDA, U8.SDA/SDIO
- net I2C2_SDA: now also U1.PE8; no longer U1.PF4
- net MCU_VCORE: now also C8.C1; no longer C6.C1
- net N$1: now also C53.C1; no longer C48.C1
- net N$10: now also C69.C2; no longer C64.C2
- net N$103: now also C34.C1, U9.VDD; no longer C29.C1, U7.VDD
- net N$105: now also C93.C1, U16.SS; no longer C83.C1, U14.SS
- net N$12: now also C15.C1, U4.RF_IN; no longer C11.C1, U2.RF_IN
- net N$13: now also C15.C2; no longer C11.C2
- net N$16: now also C77.C2, U15.1.A; no longer C72.C2, U13.1.A
- net N$17: now also C40.C1, C42.C1; no longer C35.C1, C37.C1
- net N$18: now also U9.CLK; no longer U7.CLK
- net N$2: now also C58.C1; no longer C53.C1
- net N$20: now also C50.C1, C52.C1, U10.LDO1; no longer C45.C1, C47.C1, U8.LDO1
- net N$21: now also C47.C1, C51.C1, U10.LDO0; no longer C42.C1, C46.C1, U8.LDO0
- net N$22: now also C52.C2, U10.LF1; no longer C47.C2, U8.LF1
- net N$23: now also C51.C2, U10.LF0; no longer C46.C2, U8.LF0
- net N$24: now also U15.1.Y; no longer U13.1.Y
- net N$26: now also C109.C1, U20.SS; no longer C99.C1, U18.SS
- net N$27: now also C25.C1, U6.VLOGIC; no longer C20.C1, U4.VLOGIC
- net N$28: now also C96.C1, U17.SS; no longer C86.C1, U15.SS
- net N$29: now also U14.1.Y; no longer U12.1.Y
- net N$3: now also C63.C1; no longer C58.C1
- net N$30: now also C45.C1, U10.XOB; no longer C40.C1, U8.XOB
- net N$32: now also C76.C2, U14.1.A; no longer C71.C2, U12.1.A
- net N$34: now also C54.C1; no longer C49.C1
- net N$35: now also C59.C1; no longer C54.C1
- net N$36: now also C64.C1; no longer C59.C1
- net N$37: now also C23.C1, C24.C1, U5.VOUT, U6.REF; no longer C18.C1, C19.C1, U3.VOUT, U4.REF
- net N$38: now also C69.C1; no longer C64.C1
- net N$4: now also C68.C1; no longer C63.C1
- net N$41: now also C68.C2; no longer C63.C2
- net N$45: now also C70.C2; no longer C65.C2
- net N$47: now also C55.C1; no longer C50.C1
- net N$48: now also C60.C1; no longer C55.C1
- net N$49: now also C65.C1; no longer C60.C1
- net N$50: now also C70.C1; no longer C65.C1
- net N$53: now also C71.C2; no longer C66.C2
- net N$55: now also C56.C1; no longer C51.C1
- net N$56: now also C61.C1; no longer C56.C1
- net N$57: now also C66.C1; no longer C61.C1
- net N$58: now also C71.C1; no longer C66.C1
- net N$61: now also C72.C2; no longer C67.C2
- net N$63: now also C57.C1; no longer C52.C1
- net N$64: now also C62.C1; no longer C57.C1
- net N$65: now also C67.C1; no longer C62.C1
- net N$66: now also C72.C1; no longer C67.C1
- net N$68: now also U13.1.Y; no longer U11.1.Y
- net N$69: now also C75.C2, U13.1.A; no longer C70.C2, U11.1.A
- net N$7: now also C27.C1, U6.VOUT, U7.1.+IN; no longer C22.C1, U4.VOUT, U5.1.+IN
- net N$71: now also U12.1.Y; no longer U10.1.Y
- net N$72: now also C74.C2, U12.1.A; no longer C69.C2, U10.1.A
- net N$74: now also U11.1.Y; no longer U9.1.Y
- net N$75: now also C73.C2, U11.1.A; no longer C68.C2, U9.1.A
- net N$91: now also C42.C2, U10.XOA; no longer C37.C2, U8.XOA
- net OCXO_CLK: now also U2.1.A, U8.CLK; no longer U20.1.A, U6.CLK
- net OCXO_CLK_BUF: now also U1.PE9, U2.1.Y; no longer U20.1.Y
- net OCXO_EN: now also U17.EN; no longer U15.EN
- net OCXO_VCONT: now also C29.C1, C32.C1, U7.1.-IN, U7.1.OUT, U8.VCONT; no longer C24.C1, C27.C1, U5.1.-IN, U5.1.OUT, U6.VCONT
- net PLL_M3: now also U10.M3; no longer U8.M3
- net PLL_M4: now also U10.M4; no longer U8.M4
- net PLL_M5: now also U10.M5/SDO; no longer U8.M5/SDO
- net PLL_M6: now also U10.M6/!CS; no longer U8.M6/!CS
- net PLL_REFA: now also U10.REFA; no longer U8.REFA
- net PLL_REFB: now also U10.REFB; no longer U8.REFB
- net VIN: now also C117.C1, C92.C1, C94.C1, C95.C1, U19.VIN; no longer C107.C1, C82.C1, C84.C1, C85.C1, U17.VIN
- net VIN_VSENSE: now also C115.C1; no longer C105.C1
Other:
- note added: "7th order Eliptic LPF Fc = 15 MHz"
- note added: "7th order Eliptic LPF Fc = 40 MHz"
- note added: "7th order Eliptic LPF Fc = 60 MHz"
- note added: "Analog Rail Output stages"
- note removed: "5th order Eliptic LPF Fc = 13 MHz"
- note removed: "Analog Rail PLL, Clock outputs"
- moved on the sheet: C100, C101, C102, C103, C104, C105, C106, C107, C11, C12, C13, C14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

Commit message: Rework GPSDO to fit a BGA MCU instead of a QFN since it is unobtanium
Signed-off-by: João Silva <jgc3silva@gmail.com>
Parts:
- C1: value 100nF -> 10uF; device Capacitor:CAPACITOR-0402 -> Capacitor:CAPACITOR-0603
- U1: value EFM32GG11B420F2048GM64 -> EFM32GG11B420F2048GL112; device EFM32:EFM32GG11B420F2048GM64 -> EFM32:EFM32GG11B420F2048GL112
Connections:
- removed net I2C0_SCL: CON2-3.S, R5.1, U1.PE5, U10.SCL/SCLK, U4.SCL
- removed net I2C0_SDA: CON2-2.S, R1.1, U1.PE4, U10.SDA/SDIO, U4.SDA
- new net I2C1_SCL: R3.2, R8.1, U1.PB12
- new net I2C1_SDA: R2.2, R6.1, U1.PB11
- net !PLL_IRQ: now also U1.PD10; no longer U1.PF11
- net !PLL_RESET: now also U1.PF7; no longer U1.PF10
- net 3V3: now also U1.AVDD@2, U1.IOVDD0@3, U1.IOVDD1, U1.IOVDD2
- net 3V3_PGOOD: now also U1.PA6; no longer U1.PB3
- net 5V0_PGOOD: no longer U1.PB4
- net GND: now also U1.VSS@1, U1.VSS@2, U1.VSS@3, U1.VSS@4, U1.VSS@5, U1.VSS@6, U1.VSS@7, U1.VSS@8, U1.VSS@9
- net I2C2_SCL: now also CON2-3.S, R5.1, U10.SCL/SCLK, U4.SCL; no longer R3.2, R8.1
- net I2C2_SDA: now also CON2-2.S, R1.1, U10.SDA/SDIO, U4.SDA; no longer R2.2, R6.1
- net MCU_LED: now also U1.PB13; no longer U1.PB11
- net OCXO_CLK_BUF: now also U1.PF12; no longer U1.PE9
- net VIN_VSENSE: now also U1.PD4; no longer U1.PD1
