File: pcb/gpsdo/qo-100-gpsdo.brd (EAGLE design)
At the start: 50 x 50 mm, 222 parts, among them CON1 3P-SH-TOP, J1 DCJACK, U1 ICE40HX8K-SG32, U10 74LVC1G17, U11 74LVC1G17, U12 74LVC1G17, U13 74LVC1G17, U14 74LVC1G17, U15 74LVC1G17, U16 74LVC1G17, U17 74LVC1G17, U18 74LVC1G17, U19 MIC23159, U2 MCP1700-330, U20 ADP150UJZ-3.3, U21 ADP3334, U22 LT8636, U23 EFM32GG12B810F1024GM64, U3 NEO-7M, U4 MCP1501-40, U5 AD5541ACPZ, U6 MCP6V32-E/MNY, U7 OSC5A2B02, U8 74LVC1G17, U9 SI5351C-B-GM

Commit message: Work on GPSDO
Signed-off-by: João Silva <jgc3silva@gmail.com>
Parts:
- removed D5: SMAJ24A, TVS:DO214AC
- removed D6: LED0603, LED:0603
- removed U14, U15, U16, U17, U18: 74LVC1G17, Logic:SC70-5
- removed U19: MIC23159, Microchip:VQFN20
- removed U20: ADP150UJZ-3.3, Analog Devices:SOT23-5
- removed U21: ADP3334, Analog Devices:LFCSP8_3X3
- removed U22: LT8636, Analog Devices:QFN20_ASYM_CORNER
- removed U23: EFM32GG12B810F1024GM64, EFM32:QFN64
- removed USB1: USB-C-16P-SMD-FLAT-SIDE-TYPE-2, USB Connector:USB-C-16P-SMD-FLAT-SIDE-TYPE-2
- added C103, C114: 10uF, Capacitor:CAP0603
- added C104, C105, C106, C107, C115, C116: 100nF, Capacitor:CAP0603
- added C108: 10pF, Capacitor:CAP0603
- added C109, C111, C112, C113: 100uF, Capacitor:CAP1206
- added C110: 10nF, Capacitor:CAP0603
- added C117, C118: 470pF, Capacitor:CAP0603
- added C119: 10uF, Capacitor:CAP1206
- added CON2: 2EDG-2P-5MM, Generic Connector:2EDG-2P-5MM
- added FB1, FB2, FB3, FB4, FB5, FB6: 1uH, Inductor:IND0805
- added L32, L33: 560nH, Inductor:IND0603
- added L34, L35, L36, L37: 68nH, Inductor:IND0603
- added L38, L39, L40, L41: 1uH, Inductor:IND0603
- added L42, L43, L44, L45: 330nH, Inductor:IND0603
- added L46, L47, L48, L49: 820nH, Inductor:IND0603
- added L50, L51, L52, L53: 220nH, Inductor:IND0603
- added L54, L55, L56, L57: 470nH, Inductor:IND0603
- added L58: 2.2uH, Inductor:IND3515
- added L59: 4.7uH, Inductor:IND0404
- added R45: 41.2K Ohms, Resistor:RES0603
- added R46: 309K Ohms, Resistor:RES0603
- added R47: 71.5K Ohms, Resistor:RES0603
- added R48: 1M Ohms, Resistor:RES0603
- added R49: 226K Ohms, Resistor:RES0603
- added R50: 510 Ohms, Resistor:RES0603
- added R51, R53: 100K Ohms, Resistor:RES0603
- added R52: 10K Ohms, Resistor:RES0603
- added R54: 75K Ohms, Resistor:RES0603
- added RFCON11, RFCON12, RFCON13, RFCON14, RFCON15, RFCON16: RFCON-U.FL, RF Connector:U.FL
- added TC1: TC2050-IDC, TagConnect:TC2050-IDC
- C1, C87: value 100uF -> 100nF; device Capacitor:CAP1206 -> Capacitor:CAP0603
- C100: value 1uF -> 10uF
- C101: value 100nF -> 10nF
- C102: value 10uF -> 100nF; device Capacitor:CAP1206 -> Capacitor:CAP0603
- C11, C3, C4, C85, C90, C91: value 1uF -> 100nF
- C12: value 10uF -> 47pF
- C16: value 100uF -> 10uF; device Capacitor:CAP1206 -> Capacitor:CAP0603
- C17, C18, C21, C23, C37, C42, C47, C48, C51, C55, C7: value 100nF -> 1uF
- C19: value 100nF -> 10uF
- C25, C8: value 100nF -> 100uF; device Capacitor:CAP0603 -> Capacitor:CAP1206
- C28, C30, C31: value 470pF -> 100nF
- C29: value 470pF -> 6pF
- C33: value 560pF -> 10uF
- C34, C35, C36, C54: value 560pF -> 1uF
- C38, C40, C56: value 510pF -> 1uF
- C39: value 510pF -> 10uF
- C41: value 510pF -> 6pF
- C43: value 200pF -> 10pF
- C44: value 200pF -> 10uF
- C45, C46, C71, C72: value 200pF -> 100nF
- C52: value 470pF -> 1uF
- C57, C73, C74: value 200pF -> 270pF
- C58, C75, C76: value 100nF -> 270pF
- C59, C60: value 470pF -> 270pF
- C61, C62, C83, C84: value 470pF -> 220pF
- C63, C64, C65, C66: value 560pF -> 220pF
- C67, C68: value 510pF -> 220pF
- C69, C70: value 510pF -> 100nF
- C77, C78, C79, C81: value 100nF -> 220pF
- C80: value 4.7uF -> 220pF
- C82: value 100uF -> 220pF; device Capacitor:CAP1206 -> Capacitor:CAP0603
- C89: value 4.7uF -> 100nF
- C92: value 470pF -> 4.7uF
- C93: value 1uF -> 4.7uF
- C94: value 4.7uF -> 10nF
- C95: value 10nF -> 1uF
- C97: value 100uF -> 10nF; device Capacitor:CAP1206 -> Capacitor:CAP0603
- C98: value 100nF -> 470pF
- C99: value 10pF -> 1uF
- D1: value SP0503BAHT -> LED0603; device TVS:SOT143 -> LED:0603
- D2: value LED0603 -> B0530W; device LED:0603 -> Generic Diode:SOD-123
- D3: value B0530W -> LED0603; device Generic Diode:SOD-123 -> LED:0603
- D4: value LED0603 -> SMAJ24A; device LED:0603 -> TVS:DO214AC
- L1: value (none) -> 27nH
- L10, L11, L12, L13: value 1.1uH -> 1uH
- L14, L15, L17: value 1.3uH -> 330nH
- L16: value 1.1uH -> 330nH
- L18, L19, L20, L21: value 1.3uH -> 820nH
- L2, L3, L4, L5: value 1.3uH -> 560nH
- L22, L23, L24: value 1.3uH -> 220nH
- L25: value 1.1uH -> 220nH
- L26, L27, L28: value 1.1uH -> 470nH
- L29: value 2.2uH -> 470nH; device Inductor:IND0805 -> Inductor:IND0603
- L30: value 2.2uH -> 560nH; device Inductor:IND2520 -> Inductor:IND0603
- L31: value 4.7uH -> 560nH; device Inductor:IND0606 -> Inductor:IND0603
- L6, L7, L8, L9: value 1.3uH -> 68nH
- R1: value 5.1K Ohms -> 330 Ohms
- R11, R12: value 10K Ohms -> 2K Ohms
- R13: value 0 Ohms -> 470 Ohms
- R14: value 0 Ohms -> 49.9 Ohms
- R15: value 0 Ohms -> 267 Ohms
- R16: value 0 Ohms -> 865 Ohms
- R17, R18, R19, R20: value 0 Ohms -> 10K Ohms
- R2: value 5.1K Ohms -> 4.7K Ohms
- R21: value 100 Ohms -> 10K Ohms
- R22: value 100 Ohms -> 470 Ohms
- R23: value 100 Ohms -> 865 Ohms
- R24, R25, R26, R27, R28, R29: value 100 Ohms -> 28 Ohms
- R3: value 27 Ohms -> 4.7K Ohms
- R30: value 274K Ohms -> 28 Ohms
- R31: value 294K Ohms -> 28 Ohms
- R32, R33, R37: value 100K Ohms -> 28 Ohms
- R34: value 309K Ohms -> 28 Ohms
- R35: value 71.5K Ohms -> 28 Ohms
- R36: value 330 Ohms -> 28 Ohms
- R38: value 210K Ohms -> 28 Ohms
- R39: value 64.9K Ohms -> 28 Ohms
- R4: value 27 Ohms -> 10K Ohms
- R40: value 41.2K Ohms -> 75K Ohms
- R41: value 1M Ohms -> 10K Ohms
- R42: value 226K Ohms -> 10K Ohms
- R43, R5: value 510 Ohms -> 10K Ohms
- R6: value 10K Ohms -> 49.9 Ohms; device Resistor:RES0603 -> Resistor:RES1206
- R7: value 1K Ohms -> DNP; device Resistor:RES0603 -> Resistor:RES1206
- R8: value DNP -> 100 Ohms
- R9: value 100 Ohms -> 1K Ohms; device Resistor:RES1206 -> Resistor:RES0603
- U1: value ICE40HX8K-SG32 -> EFM32GG11B120F2048GM64; device Lattice:QFN32 -> EFM32:QFN64
- U10: value 74LVC1G17 -> ADM7171ACPZ-5.0; device Logic:SC70-5 -> Analog Devices:LFCSP8_3X3
- U11: value 74LVC1G17 -> MIC23155; device Logic:SC70-5 -> Microchip:DFN10
- U12: value 74LVC1G17 -> LT8636; device Logic:SC70-5 -> Analog Devices:QFN20_ASYM_3X4_CORNER
- U13: value 74LVC1G17 -> ADM7171ACPZ-3.3; device Logic:SC70-5 -> Analog Devices:LFCSP8_3X3
- U2: value MCP1700-330 -> MAX-M8Q; device Microchip:SOT23 -> U-Blox:MAX-M8
- U3: value NEO-7M -> MCP1501-40; device U-Blox:NEO-6/7 -> Microchip:SOT23-6
- U4: value MCP1501-40 -> AD5541ACPZ; device Microchip:SOT23-6 -> Analog Devices:DFN10
- U5: value AD5541ACPZ -> MCP6V32-E/MNY; device Analog Devices:DFN10 -> Microchip:TDFN8
- U6: value MCP6V32-E/MNY -> OSC5A2B02; device Microchip:TDFN8 -> Crystal:OSC5A2B02
- U7: value OSC5A2B02 -> DSB321SDA; device Crystal:OSC5A2B02 -> Crystal:TCXO-3225
- U8: value 74LVC1G17 -> SI5347A; device Logic:SC70-5 -> Silicon Labs:QFN64-L-PAD
- U9: value SI5351C-B-GM -> ADM7171ACPZ-1.8; device Silicon Labs:QFN20 -> Analog Devices:LFCSP8_3X3
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Connections:
- removed net !5V0_PA_BIAS_EN: R37.1, U21.6
- removed net 1V2: C81.1, C82.1, L29.1, R30.2, U19.17
- removed net 1V2_FB: R30.1, R31.2, U19.16
- removed net 1V2_PGOOD: R32.1, U19.15
- removed net 1V2_SOFTSTART: C83.1, U19.14
- removed net 3V3_ANA_SYNTH_CLEAN: C21.1, C22.1, C23.1, C24.1, U8.5, U9.10, U9.11, U9.14, U9.18
- removed net 3V3_ANA_TXPLL_CLEAN: C90.1, U20.5
- removed net 3V3_FB: R34.1, R35.2, U19.11
- removed net 3V3_SOFTSTART: C84.1, U19.13
- removed net 3V6_ANA: C85.1, U20.1, U20.3
- removed net 5V0_ANA_COMP_CLEAN: C10.1, C11.1, C13.1, U4.4, U4.6, U5.1, U6.8
- removed net 5V0_ANA_OUT_CLEAN: C25.1, C26.1, C27.1, C32.1, C37.1, C42.1, C47.1, C53.1, C55.1, U10.5, U11.5, U12.5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
- removed net 5V0_ANA_PA_CLEAN: C92.1, R38.2, U21.1, U21.2
- removed net GPS_PROG_RXD: CON1.2, U3.17
- removed net GPS_PROG_TXD: CON1.1, U3.16
- removed net GPS_TXD: U3.20
- removed net GPS_USB_D+: R3.1, U3.6
- removed net GPS_USB_D-: R4.1, U3.5
- removed net GPS_VDD_USB: C4.1, R7.2, U2.2, U3.7
- removed net I2S_BRG_VBUS: C3.1, D1.2, R5.2, U2.3, USB1.A4/B9, USB1.B4/A9
- removed net N$147: D2.A, R5.1
- removed net N$148: D4.A, R36.1
- removed net OCXO_CLK_SQ_UNBUF: U14.2, U7.1, U8.2
- removed net SYNTH_CLK0: R13.1, U10.2
- removed net SYNTH_CLK1: R17.1, U11.2
- removed net SYNTH_CLK2: R14.1, U12.2
- removed net SYNTH_CLK3: R18.1, U13.2
- removed net SYNTH_CLK4: R15.1, U15.2
- removed net SYNTH_CLK5: R19.1, U16.2
- removed net SYNTH_CLK6: R16.1, U17.2
- removed net SYNTH_CLK7: R20.1, U18.2
- removed net VCC: U1.25
- removed net VCCIO0: U1.28
- removed net VCCIO1: U1.17
- removed net VCCIO2: U1.9
- removed net VCCIO3: U1.4
- removed net VCC_SPI: U1.16
- removed net VPP_2V5: U1.24
- new net !DAC_CS: U4.5
- new net !MCU_RESET: R4.1, TC1.10, U1.20
- new net !PLL_IRQ: R18.1, U8.12
- new net !PLL_LOLA: U8.3
- new net !PLL_LOLB: U8.4
- new net !PLL_LOLC: U8.5
- new net !PLL_LOLD: U8.47
- new net !PLL_OE0: R19.1, U8.11
- new net !PLL_OE1: R20.1, U8.41
- new net !PLL_OUT0: R32.1, RFCON10.P$3
- new net !PLL_OUT1: R33.1, RFCON13.P$3
- new net !PLL_OUT2: R34.1, RFCON15.P$3
- new net !PLL_OUT3: R35.1, RFCON11.P$3
- new net !PLL_OUT4: R36.1, RFCON14.P$3
- new net !PLL_OUT5: R37.1, RFCON16.P$3
- new net !PLL_OUT6: R38.1, RFCON12.P$3
- new net !PLL_OUT7: R39.1
- new net !PLL_RESET: R17.1, U8.6
- new net !PLL_XTAL_LOS: U8.25
- new net 1V8_PLL_CLEAN: C100.1, C102.1, C39.1, FB5.1, U9.1, U9.2, U9.3
- new net 2V5_FB1: R46.1, R47.2, U11.4
- new net 2V5_SS1: C98.1, U11.6
- new net 2V5_SW1: L58.1, U11.1
- new net 3V3_ANA_MPLL_FILT: C34.1, C36.1, C37.1, C38.1, C40.1, C42.1, C48.1, C52.1, C55.1, FB3.2, U8.13, U8.22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
- new net 3V3_ANA_MPLL_FILT1: C47.1, C51.1, C54.1, FB5.2, U8.32, U8.46, U8.60
- new net 3V3_ANA_PLL_CLEAN: C114.1, C116.1, C33.1, FB3.1, FB4.1, U13.1, U13.2, U13.3
- new net 5V0_EN: R40.1, R41.2, U12.14
- new net 5V0_PGOOD: R44.1, U11.2, U12.1
- new net 5V0_VSENSE: C118.1, R53.1, R54.2
- new net DAC_DIN: U4.7
- new net DAC_SCLK: U4.6
- new net GPS_TXD/TXREADY: CON1.1, U2.2
- new net I2C0_SCL: R3.1, U2.17, U8.16
- new net I2C0_SDA: R2.1, U2.16, U8.18
- new net MCU_LED: R1.2
- new net MCU_SWCLK: TC1.4, U1.49
- new net MCU_SWDIO: TC1.2, U1.50
- new net MCU_SWO: TC1.6, U1.51
- new net N$100: R37.2, U8.50
- new net N$101: R38.2, U8.53
- new net N$102: R39.2, U8.58
- new net N$103: C35.1, FB4.2, U7.4
- new net N$104: C56.1, FB6.2, U8.40
- new net N$105: C94.1, U9.4
- new net N$144: D1.A, R1.1
- new net N$33: L19.2, L23.1, L27.1
- new net N$34: C58.1, L7.2
- new net N$35: C62.1, L15.2
- new net N$36: C66.1, L23.2
- new net N$85: C88.2, RFCON9.P$3
- new net N$86: L49.2, L53.1, L57.1
- new net N$87: C76.1, L37.2
- new net N$88: C80.1, L45.2
- new net N$89: C84.1, L53.2
- new net N$90: C88.1, L57.2
- new net N$91: C46.2, U8.8
- new net N$92: R6.1, U2.4
- new net N$93: C41.2, C49.1, R22.1, R23.2
- new net N$94: C30.1, R16.1
- new net N$95: C45.1, R23.1
- new net N$96: R33.2, U8.30
- new net N$97: R34.2, U8.34
- new net N$98: R35.2, U8.37
- new net N$99: R36.2, U8.44
- new net OCXO_CLK: C41.1, R14.1, R22.2
- new net OCXO_EN: R42.2, U10.5
- new net PLL_FDEC: U8.42
- new net PLL_FINC: U8.48
- new net PLL_IN0_N: C32.1, U8.64
- new net PLL_IN0_P: C31.2, U8.63
- new net PLL_IN1_N: C53.1, U8.2
- new net PLL_IN1_P: C49.2, U8.1
- new net PLL_OUT0: L2.1, R24.1
- new net PLL_OUT1: L3.1, R25.1
- new net PLL_OUT2: L4.1, R26.1
- new net PLL_OUT3: L5.1, R27.1
- new net PLL_OUT4: L30.1, R28.1
- new net PLL_OUT5: L31.1, R29.1
- new net PLL_OUT6: L32.1, R30.1
- new net PLL_OUT7: L33.1, R31.1
- new net PLL_SEL0: U8.26
- new net PLL_SEL1: U8.27
- new net SMC_VCORE: C7.1, U1.40
- new net VIN_VSENSE: C117.1, R51.1, R52.2
- net !GPS_RESET: now also R5.1, U2.9; no longer R6.1, U3.8
- net 3V3: now also C10.1, C106.1, C109.1, C111.1, C13.1, C15.1, C18.1, C3.1, C4.1, C44.1, C5.1, C6.1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; no longer C20.1, C7.1, C86.1, C87.1, D3.A, L30.2, R32.2, R33.2, R34.2, R36.2, R37.2, R6.2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
- net 3V3_PGOOD: now also R43.1, U11.5, U13.5, U9.5; no longer R33.1, U19.12
- net 5V0: now also C105.1, C108.1, C112.1, C113.1, C115.1, C92.1, L59.2, R44.2, R48.2, R50.2, R53.2, U10.7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; no longer C101.1, C79.1, C80.1, C88.1, C97.1, C99.1, L31.2, R41.2, R43.2, U19.1, U19.18, U19.20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
- net 5V0_ANA_OCXO_CLEAN: now also C103.1, C104.1, C21.1, C23.1, C25.1, C26.1, FB1.1, FB1.2, U10.1, U10.2, U10.3, U3.4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; no longer U7.5
- net 5V0_BST: now also C107.2, U12.7; no longer C98.2, U22.7
- net 5V0_FB: now also C108.2, R48.1, R49.2, U12.19, U12.20; no longer C99.2, R41.1, R42.2, U22.19, U22.20
- net 5V0_INTVCC: now also C99.1, U12.15, U12.3; no longer C96.1, U22.15, U22.3
- net 5V0_RT: now also R45.2, U12.17; no longer R40.2, U22.17
- net 5V0_SS: now also C101.1, U12.18; no longer C95.1, U22.18
- net 5V0_SW: now also C107.1, L59.1, U12.10, U12.8, U12.9; no longer C98.1, L31.1, U22.10, U22.8, U22.9
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Other:
- board size 50 x 50 mm -> 100 x 75 mm

Commit message: Work on GPSDO
Signed-off-by: João Silva <jgc3silva@gmail.com>
Parts:
- removed BAT1: CR2032, Battery:CR2032
- removed C10, C106, C11, C115, C116, C13, C14, C15, C20, C22, C24, C26, C27, C28, C30, C31, C32, C4, C45, C46, C49, C5, C50, C53, C6, C69, C70, C71, C72, C85, C86, C87, C88, C89, C9, C90, C91: 100nF, Capacitor:CAP0603
- removed C100, C114, C16, C19, C33, C39, C44: 10uF, Capacitor:CAP0603
- removed C108, C43: 10pF, Capacitor:CAP0603
- removed C109, C111, C112, C113, C25, C8: 100uF, Capacitor:CAP1206
- removed C110, C94, C97: 10nF, Capacitor:CAP0603
- removed C117, C118, C98: 470pF, Capacitor:CAP0603
- removed C119: 10uF, Capacitor:CAP1206
- removed C12: 47pF, Capacitor:CAP0603
- removed C17, C18, C21, C23, C34, C35, C36, C37, C38, C40, C42, C47, C48, C51, C52, C54, C55, C56, C7, C95, C96, C99: 1uF, Capacitor:CAP0603
- removed C29, C41: 6pF, Capacitor:CAP0603
- removed C57, C58, C59, C60, C73, C74, C75, C76: 270pF, Capacitor:CAP0603
- removed C61, C62, C63, C64, C65, C66, C67, C68, C77, C78, C79, C80, C81, C82, C83, C84: 220pF, Capacitor:CAP0603
- removed C92, C93: 4.7uF, Capacitor:CAP0603
- removed CON1: 3P-SH-TOP, JST:SH-03-TOP
- removed CON2: 2EDG-2P-5MM, Generic Connector:2EDG-2P-5MM
- removed D3: LED0603, LED:0603
- removed D4: SMAJ24A, TVS:DO214AC
- removed F1: 2.6A Hold, PTC Fuses:1206
- removed FB1, FB2, FB3, FB4, FB5, FB6: 1uH, Inductor:IND0805
- removed J1: DCJACK, Barrel Jack:DC-050
- removed L1: 27nH, Inductor:IND0805
- removed L10, L11, L12, L13, L38, L39, L40, L41: 1uH, Inductor:IND0603
- removed L14, L15, L16, L17, L42, L43, L44, L45: 330nH, Inductor:IND0603
- removed L18, L19, L20, L21, L46, L47, L48, L49: 820nH, Inductor:IND0603
- removed L2, L3, L30, L31, L32, L33, L4, L5: 560nH, Inductor:IND0603
- removed L22, L23, L24, L25, L50, L51, L52, L53: 220nH, Inductor:IND0603
- removed L26, L27, L28, L29, L54, L55, L56, L57: 470nH, Inductor:IND0603
- removed L34, L35, L36, L37, L6, L7, L8, L9: 68nH, Inductor:IND0603
- removed L58: 2.2uH, Inductor:IND3515
- removed L59: 4.7uH, Inductor:IND0404
- removed LOGO1: JS-5MM, Silkscreen:JS_5MM
- removed R1: 330 Ohms, Resistor:RES0603
- removed R10, R9: 1K Ohms, Resistor:RES0603
- removed R11, R12: 2K Ohms, Resistor:RES0603
- removed R13, R22: 470 Ohms, Resistor:RES0603
- removed R14: 49.9 Ohms, Resistor:RES0603
- removed R15: 267 Ohms, Resistor:RES0603
- removed R16, R23: 865 Ohms, Resistor:RES0603
- removed R17, R18, R19, R20, R21, R4, R41, R42, R43, R44, R5, R52: 10K Ohms, Resistor:RES0603
- removed R2, R3: 4.7K Ohms, Resistor:RES0603
- removed R24, R25, R26, R27, R28, R29, R30, R31, R32, R33, R34, R35, R36, R37, R38, R39: 28 Ohms, Resistor:RES0603
- removed R40, R54: 75K Ohms, Resistor:RES0603
- removed R45: 41.2K Ohms, Resistor:RES0603
- removed R46: 309K Ohms, Resistor:RES0603
- removed R47: 71.5K Ohms, Resistor:RES0603
- removed R48: 1M Ohms, Resistor:RES0603
- removed R49: 226K Ohms, Resistor:RES0603
- removed R50: 510 Ohms, Resistor:RES0603
- removed R51, R53: 100K Ohms, Resistor:RES0603
- removed R6: 49.9 Ohms, Resistor:RES1206
- removed R7: DNP, Resistor:RES1206
- removed R8: 100 Ohms, Resistor:RES1206
- removed RFCON1, RFCON10, RFCON11, RFCON12, RFCON13, RFCON14, RFCON15, RFCON16, RFCON2, RFCON3, RFCON4, RFCON5, RFCON6, RFCON7, RFCON8, RFCON9: RFCON-U.FL, RF Connector:U.FL
- removed TC1: TC2050-IDC, TagConnect:TC2050-IDC
- removed U10: ADM7171ACPZ-5.0, Analog Devices:LFCSP8_3X3
- removed U11: MIC23155, Microchip:DFN10
- removed U12: LT8636, Analog Devices:QFN20_ASYM_3X4_CORNER
- removed U13: ADM7171ACPZ-3.3, Analog Devices:LFCSP8_3X3
- removed U3: MCP1501-40, Microchip:SOT23-6
- removed U4: AD5541ACPZ, Analog Devices:DFN10
- removed U5: MCP6V32-E/MNY, Microchip:TDFN8
- removed U6: OSC5A2B02, Crystal:OSC5A2B02
- removed U7: DSB321SDA, Crystal:TCXO-3225
- removed U8: SI5347A, Silicon Labs:QFN64-L-PAD
- removed U9: ADM7171ACPZ-1.8, Analog Devices:LFCSP8_3X3
- added BAT201: CR2032, Battery:CR2032
- added C201, C312, C621, C624, C625: 100uF, Capacitor:CAP1206
- added C202, C203, C204, C206, C207, C306, C307, C309, C311, C313, C314, C402, C403, C404, C417, C418, C421, C422, C425, C513, C514, C515, C516, C529, C530, C531, C601, C602, C603, C614, C616, C617, C619, C620, C626, C628: 100nF, Capacitor:CAP0402
- added C205: 47pF, Capacitor:CAP0402
- added C302, C305, C411, C416, C613, C615, C627: 10uF, Capacitor:CAP0603
- added C303, C304, C308, C310, C406, C407, C408, C409, C410, C412, C414, C419, C420, C423, C424, C426, C427, C428, C611: 1uF, Capacitor:CAP0402
- added C401, C413: 6pF, Capacitor:CAP0402
- added C415, C618: 10pF, Capacitor:CAP0402
- added C501, C502, C503, C504, C517, C518, C519: 270pF, Capacitor:CAP0402
- added C505, C506, C507, C508, C509, C510, C511, C512, C521, C522, C523, C525, C526, C527: 220pF, Capacitor:CAP0402
- added C604, C605: 4.7uF, Capacitor:CAP0603
- added C606, C609, C612, C622: 10nF, Capacitor:CAP0402
- added C607, C608: 1uF, Capacitor:CAP0603
- added C610, C629, C630: 470pF, Capacitor:CAP0402
- added C631: 10uF, Capacitor:CAP1206
- added CON201: 3P-SH-TOP, JST:SH-03-TOP
- added CON601: 2EDG-2P-5MM, Generic Connector:2EDG-2P-5MM
- added D101, D601: LED0603, LED:0603
- added D201: B0530W, Generic Diode:SOD-123
- added D602: SMAJ24A, TVS:DO214AC
- added F601: 2.6A Hold, PTC Fuses:1206
- added FB301, FB302, FB402, FB403, FB404: 1uH, Inductor:IND0603
- added J601: DCJACK, Barrel Jack:DC-050
- added L201: 27nH, Inductor:IND0805
- added L501, L502, L503, L504, L529, L530, L531: 560nH, Inductor:IND0402
- added L505, L506, L507, L508, L533, L534, L535: 68nH, Inductor:IND0402
- added L509, L510, L511, L512, L537, L538, L539: 1uH, Inductor:IND0402
- added L513, L514, L515, L516, L541, L542, L543: 330nH, Inductor:IND0402
- added L517, L518, L519, L520, L545, L546, L547: 820nH, Inductor:IND0402
- added L521, L522, L523, L524, L549, L550, L551: 220nH, Inductor:IND0402
- added L525, L526, L527, L528, L553, L554, L555: 470nH, Inductor:IND0402
- added L601: 2.2uH, Inductor:IND3515
- added L602: 4.7uH, Inductor:IND0404
- added LOGO101: JS-5MM, Silkscreen:JS_5MM
- added R101: 330 Ohms, Resistor:RES0402
- added R102, R103: 4.7K Ohms, Resistor:RES0402
- added R104, R201, R403, R404, R405, R406, R407, R602, R603, R604, R605, R613: 10K Ohms, Resistor:RES0402
- added R202, R302: 49.9 Ohms, Resistor:RES0603
- added R203: 10 Ohms, Resistor:RES0603
- added R204: DNP, Resistor:RES0603
- added R205: 1K Ohms, Resistor:RES0402
- added R301, R408: 470 Ohms, Resistor:RES0402
- added R401: 267 Ohms, Resistor:RES0402
- added R402, R409: 865 Ohms, Resistor:RES0402
- added R410, R411, R412, R413, R414, R415, R416, R418, R419, R420, R421, R422, R423, R424: 28 Ohms, Resistor:RES0402
- added R601, R615: 75K Ohms, Resistor:RES0402
- added R606: 41.2K Ohms, Resistor:RES0402
- added R607: 309K Ohms, Resistor:RES0402
- added R608: 71.5K Ohms, Resistor:RES0402
- added R609: 1M Ohms, Resistor:RES0402
- added R610: 226K Ohms, Resistor:RES0402
- added R611: 510 Ohms, Resistor:RES0402
- added R612, R614: 100K Ohms, Resistor:RES0402
- added RFCON201: RFCON-SMA-EDGE, RF Connector:SMA-EDGE
- added RFCON501, RFCON502, RFCON503, RFCON504, RFCON505, RFCON506, RFCON507, RFCON509, RFCON510, RFCON511, RFCON512, RFCON513, RFCON514, RFCON515: RFCON-U.FL, RF Connector:U.FL
- added TC101: TC2050-IDC, TagConnect:TC2050-IDC
- added U101: EFM32GG11B120F2048GM64, EFM32:QFN64
- added U201: MAX-M8Q, U-Blox:MAX-M8
- added U301: MCP1501-40, Microchip:SOT23-6
- added U302: AD5541ACPZ, Analog Devices:DFN10
- added U303: MCP6V31, Microchip:SOT23-5
- added U304: OSC5A2B02, Crystal:OSC5A2B02
- added U401: DSB321SDA, Crystal:TCXO-3225
- added U402: SI5347A, Silicon Labs:QFN64-L-PAD
- added U601: ADM7171ACPZ-1.8, Analog Devices:LFCSP8_3X3
- added U602: ADM7171ACPZ-5.0, Analog Devices:LFCSP8_3X3
- added U603: MIC23155, Microchip:DFN10
- added U604: LT8636, Analog Devices:QFN20_ASYM_3X4_CORNER
- added U605: ADM7171ACPZ-3.3, Analog Devices:LFCSP8_3X3
- C1: value 100nF -> 10uF
- C101: value 10nF -> 100nF; device Capacitor:CAP0603 -> Capacitor:CAP0402
- C102, C104, C105, C2, C3: device Capacitor:CAP0603 -> Capacitor:CAP0402
- C103: value 10uF -> 100nF; device Capacitor:CAP0603 -> Capacitor:CAP0402
- C107: value 100nF -> 1uF; device Capacitor:CAP0603 -> Capacitor:CAP0402
- D1: value LED0603 -> LEDTH3MM; device LED:0603 -> LED:LED_3MM
- D2: value B0530W -> LEDTH3MM; device Generic Diode:SOD-123 -> LED:LED_3MM
- U1: value EFM32GG11B120F2048GM64 -> 74LVC1G17; device EFM32:QFN64 -> Logic:SC70-5
- U2: value MAX-M8Q -> 74LVC1G17; device U-Blox:MAX-M8 -> Logic:SC70-5
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Connections:
- removed net !PLL_OUT7: R39.1
- removed net 2V5_FB1: R46.1, R47.2, U11.4
- removed net 2V5_SS1: C98.1, U11.6
- removed net 2V5_SW1: L58.1, U11.1
- removed net 3V3_ANA_MPLL_FILT: C34.1, C36.1, C37.1, C38.1, C40.1, C42.1, C48.1, C52.1, C55.1, FB3.2, U8.13, U8.22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
- removed net 3V3_ANA_MPLL_FILT1: C47.1, C51.1, C54.1, FB5.2, U8.32, U8.46, U8.60
- removed net N$102: R39.2, U8.58
- removed net N$19: R31.2, U8.59
- removed net N$29: R14.2, U6.1
- removed net N$32: R10.1, U5.5
- removed net N$8: C24.1, R10.2, U5.1, U5.2
- removed net N$83: L33.2, L37.1, L41.1
- removed net N$84: L41.2, L45.1, L49.1
- removed net N$85: C88.2, RFCON9.P$3
- removed net N$86: L49.2, L53.1, L57.1
- removed net N$87: C76.1, L37.2
- removed net N$88: C80.1, L45.2
- removed net N$89: C84.1, L53.2
- removed net N$9: R11.2, R12.2, U5.6
- removed net N$90: C88.1, L57.2
- removed net N$92: R6.1, U2.4
- removed net PLL_OUT7: L33.1, R31.1
- removed net SMC_VCORE: C7.1, U1.40
- new net 1V8_PLL_CLEAN_FILT: C419.1, C423.1, C426.1, FB403.2, U402.32, U402.46, U402.60
- new net 3V3_FB: R607.1, R608.2, U603.4
- new net 3V3_SS: C610.1, U603.6
- new net 3V3_SW: L601.1, U603.1
- new net 5V0_ANA_OCXO_FILT: C303.1, C308.1, C310.1, FB301.2, U301.4, U301.6, U302.1, U303.5
- new net GPS_TIMEPULSE_BUF: U1.4
- new net GPS_TIMEPULSE_KZ: C401.1, R202.1, R401.2
- new net MCU_VCORE: C107.1, U101.40
- new net OCXO_CLK_BUF: U2.4
- new net OCXO_CLK_KZ: C413.1, R302.1, R408.2
- net !DAC_CS: now also U302.5; no longer U4.5
- net !GPS_RESET: now also R201.1, U201.9; no longer R5.1, U2.9
- net !MCU_RESET: now also R104.1, TC101.10, U101.20; no longer R4.1, TC1.10, U1.20
- net !PLL_IRQ: now also R404.1, U402.12; no longer R18.1, U8.12
- net !PLL_LOLA: now also U402.3; no longer U8.3
- net !PLL_LOLB: now also U402.4; no longer U8.4
- net !PLL_LOLC: now also U402.5; no longer U8.5
- net !PLL_LOLD: now also U402.47; no longer U8.47
- net !PLL_OE0: now also R405.1, U402.11; no longer R19.1, U8.11
- net !PLL_OE1: now also R406.1, U402.41; no longer R20.1, U8.41
- net !PLL_OUT0: now also R418.1, RFCON509.P$3; no longer R32.1, RFCON10.P$3
- net !PLL_OUT1: now also R419.1, RFCON512.P$3; no longer R33.1, RFCON13.P$3
- net !PLL_OUT2: now also R420.1, RFCON514.P$3; no longer R34.1, RFCON15.P$3
- net !PLL_OUT3: now also R421.1, RFCON510.P$3; no longer R35.1, RFCON11.P$3
- net !PLL_OUT4: now also R422.1, RFCON513.P$3; no longer R36.1, RFCON14.P$3
- net !PLL_OUT5: now also R423.1, RFCON515.P$3; no longer R37.1, RFCON16.P$3
- net !PLL_OUT6: now also R424.1, RFCON511.P$3; no longer R38.1, RFCON12.P$3
- net !PLL_RESET: now also R403.1, U402.6; no longer R17.1, U8.6
- net !PLL_XTAL_LOS: now also U402.25; no longer U8.25
- net 1V8_PLL_CLEAN: now also C411.1, C613.1, C614.1, FB403.1, U601.1, U601.2, U601.3; no longer C100.1, C102.1, C39.1, FB5.1, U9.1, U9.2, U9.3
- net 3V3: now also C101.1, C102.1, C103.1, C104.1, C105.1, C201.1, C202.1, C203.1, C206.1, C304.1, C416.1, C602.1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; no longer C1.1, C10.1, C106.1, C109.1, C111.1, C13.1, C15.1, C18.1, C4.1, C44.1, C5.1, C6.1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
- net 3V3_ANA_PLL_CLEAN: now also C406.1, C408.1, C409.1, C410.1, C412.1, C414.1, C420.1, C424.1, C427.1, C627.1, C628.1, FB402.1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; no longer C114.1, C116.1, C33.1, FB3.1, FB4.1, U13.1, U13.2, U13.3
- net 3V3_PGOOD: now also R604.1, U601.5, U603.5, U605.5; no longer R43.1, U11.5, U13.5, U9.5
- net 5V0: now also C601.1, C603.1, C604.1, C618.1, C619.1, C624.1, C625.1, C626.1, L602.2, R605.2, R609.2, R611.2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; no longer C105.1, C108.1, C112.1, C113.1, C115.1, C89.1, C91.1, C92.1, L59.2, R44.2, R48.2, R50.2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
Routing:
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- added copper zone on layer 1, net GND
- added copper zone on layer 15, net GND
- added copper zone on layer 16, net GND
- added copper zone on layer 2, net GND
Other:
- board size 100 x 75 mm -> 100 x 69.5 mm
- board text added: "0"
- board text added: "1"
- board text added: "2"
- board text added: "3"
- board text added: "4"
- board text added: "5"
- board text added: "6"
- board text added: "Bkp. Bat. Charge"
- board text added: "GPS Ant"
- board text added: "IcyRadio GPSDO v1 Jul 2021"
- board text added: "Sine"
- board text added: "Square"

Commit message: Work on GPSDO
Signed-off-by: João Silva <jgc3silva@gmail.com>
Parts:
- removed C201, C624, C625: 100uF, Capacitor:CAP1206
- removed C204, C313, C314, C402, C403, C404, C417, C421, C422, C425, C513, C514, C515, C516, C529, C530, C531, C602, C614, C616, C617, C619, C626, C628: 100nF, Capacitor:CAP0402
- removed C302, C411, C416, C613, C615, C627: 10uF, Capacitor:CAP0603
- removed C303, C310, C406, C407, C408, C409, C410, C412, C414, C419, C420, C423, C424, C426, C427, C428: 1uF, Capacitor:CAP0402
- removed C401, C413: 6pF, Capacitor:CAP0402
- removed C501, C502, C503, C504, C517, C518, C519: 270pF, Capacitor:CAP0402
- removed C505, C506, C507, C508, C509, C510, C511, C512, C521, C522, C523, C525, C526, C527: 220pF, Capacitor:CAP0402
- removed C604, C605: 4.7uF, Capacitor:CAP0603
- removed C606, C609, C622: 10nF, Capacitor:CAP0402
- removed C607: 1uF, Capacitor:CAP0603
- removed C629: 470pF, Capacitor:CAP0402
- removed C631: 10uF, Capacitor:CAP1206
- removed D101: LED0603, LED:0603
- removed FB402, FB403, FB404: 1uH, Inductor:IND0603
- removed L501, L502, L503, L504, L529, L530, L531: 560nH, Inductor:IND0402
- removed L505, L506, L507, L508, L533, L534, L535: 68nH, Inductor:IND0402
- removed L509, L510, L511, L512, L537, L538, L539: 1uH, Inductor:IND0402
- removed L513, L514, L515, L516, L541, L542, L543: 330nH, Inductor:IND0402
- removed L517, L518, L519, L520, L545, L546, L547: 820nH, Inductor:IND0402
- removed L521, L522, L523, L524, L549, L550, L551: 220nH, Inductor:IND0402
- removed L525, L526, L527, L528, L553, L554, L555: 470nH, Inductor:IND0402
- removed LOGO101: JS-5MM, Silkscreen:JS_5MM
- removed R101: 330 Ohms, Resistor:RES0402
- removed R102, R103: 4.7K Ohms, Resistor:RES0402
- removed R104, R405, R406, R605, R613: 10K Ohms, Resistor:RES0402
- removed R202, R302: 49.9 Ohms, Resistor:RES0603
- removed R301, R408: 470 Ohms, Resistor:RES0402
- removed R401: 267 Ohms, Resistor:RES0402
- removed R402, R409: 865 Ohms, Resistor:RES0402
- removed R410, R411, R412, R413, R414, R415, R416, R418, R419, R420, R421, R422, R423, R424: 28 Ohms, Resistor:RES0402
- removed R612: 100K Ohms, Resistor:RES0402
- removed R615: 75K Ohms, Resistor:RES0402
- removed RFCON501, RFCON502, RFCON503, RFCON504, RFCON505, RFCON506, RFCON507, RFCON512, RFCON513, RFCON514, RFCON515: RFCON-U.FL, RF Connector:U.FL
- removed TC101: TC2050-IDC, TagConnect:TC2050-IDC
- removed U101: EFM32GG11B120F2048GM64, EFM32:QFN64
- removed U201: MAX-M8Q, U-Blox:MAX-M8
- removed U401: DSB321SDA, Crystal:TCXO-3225
- removed U402: SI5347A, Silicon Labs:QFN64-L-PAD
- removed U605: ADM7171ACPZ-3.3, Analog Devices:LFCSP8_3X3
- added C10, C26, C27, C4, C40, C5, C63, C64, C65, C66, C67, C68, C69, C70, C71, C72, C79, C91, C93, C94, C96: 100nF, Capacitor:CAP0402
- added C100, C7: 100uF, Capacitor:CAP1206
- added C12, C15, C28, C38, C90, C92: 10uF, Capacitor:CAP0603
- added C16, C23, C29, C30, C31, C32, C33, C34, C36, C39, C41, C43, C44, C6, C73, C74, C75, C76, C77: 1uF, Capacitor:CAP0402
- added C42, C45: 220nF, Capacitor:CAP0402
- added C46, C47: 3.9nF, Capacitor:CAP0402
- added C48, C49, C50, C51, C52: 270pF, Capacitor:CAP0402
- added C53, C54, C55, C56, C57, C58, C59, C60, C61, C62: 220pF, Capacitor:CAP0402
- added C81, C82: 4.7uF, Capacitor:CAP0603
- added C83, C86, C99: 10nF, Capacitor:CAP0402
- added C84: 1uF, Capacitor:CAP0603
- added CON1: 3P-SH-SIDE, JST:SH-03-SIDE
- added CON2: 4P-SH-TOP, JST:SH-04-TOP
- added D10: LEDTH3MM, LED:LED_3MM
- added D4, D5, D6, D7, D8: BAV99, Generic Diode:SOT23
- added FB3: 10uH, Inductor:IND0603
- added FB4, FB5, FB6: 1uH, Inductor:IND0603
- added L10, L11, L7, L8, L9: 68nH, Inductor:IND0402
- added L12, L13, L14, L15, L16: 1uH, Inductor:IND0402
- added L17, L18, L19, L20, L21: 330nH, Inductor:IND0402
- added L2, L3, L4, L5, L6: 560nH, Inductor:IND0402
- added L22, L23, L24, L25, L26: 820nH, Inductor:IND0402
- added L27, L28, L29, L30, L31: 220nH, Inductor:IND0402
- added L32, L33, L34, L35, L36: 470nH, Inductor:IND0402
- added LOGO1: JS-5MM, Silkscreen:JS_5MM
- added R1, R5, R6, R8: 4.7K Ohms, Resistor:RES0402
- added R13, R20: 470 Ohms, Resistor:RES0402
- added R14, R15, R16, R17, R50, R58, R7: 10K Ohms, Resistor:RES0402
- added R18: 267 Ohms, Resistor:RES0402
- added R19, R21: 865 Ohms, Resistor:RES0402
- added R2, R27, R29, R3, R31, R33, R35: 100 Ohms, Resistor:RES0402
- added R22, R41, R42, R43, R44, R45: 0 Ohms, Resistor:RES0402
- added R26, R28, R30, R32, R34: 49.9 Ohms, Resistor:RES0402
- added R36, R37, R38, R39, R40: 10K Ohms, Potentiometer:POT3MM
- added R4: 330 Ohms, Resistor:RES0402
- added R57: 100K Ohms, Resistor:RES0402
- added R60: 75K Ohms, Resistor:RES0402
- added RFCON10, RFCON2, RFCON3, RFCON4, RFCON5, RFCON6, RFCON8: RFCON-U.FL, RF Connector:U.FL
- added TC1: TC2050-IDC, TagConnect:TC2050-IDC
- added U10, U11, U12, U13, U9: 74LVC1G17, Logic:SC70-5
- added U18: ADM7171ACPZ-3.3, Analog Devices:LFCSP8_3X3
- added U7: DSB321SDA, Crystal:TCXO-3225
- added U8: AD9544, Analog Devices:QFN48_2
- C1: value 10uF -> 100nF; device Capacitor:CAP0603 -> Capacitor:CAP0402
- C101: value 100nF -> 100uF; device Capacitor:CAP0402 -> Capacitor:CAP1206
- C103: value 100nF -> 10uF; device Capacitor:CAP0402 -> Capacitor:CAP0603
- C105: value 100nF -> 470pF
- C107: value 1uF -> 10uF; device Capacitor:CAP0402 -> Capacitor:CAP1206
- D1: value LEDTH3MM -> LED0603; device LED:LED_3MM -> LED:0603
- U1: value 74LVC1G17 -> EFM32GG11B120F2048GM64; device Logic:SC70-5 -> EFM32:QFN64
- U2: value 74LVC1G17 -> MAX-M8Q; device Logic:SC70-5 -> U-Blox:MAX-M8
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- renumbered BAT201 to BAT1, C202 to C8, C203 to C9, C205 to C11, C206 to C13, C207 to C14, C304 to C17, C305 to C18, C306 to C19, C307 to C20, C308 to C21, C309 to C22, C311 to C24, C312 to C25, C415 to C35, C418 to C37, C601 to C78, C603 to C80, C608 to C85, C610 to C87, C611 to C88, C612 to C89, C618 to C95, C620 to C97, C621 to C98, C630 to C106, CON201 to CON3, CON601 to CON4, D201 to D3, D601 to D9, D602 to D11, F601 to F1, FB301 to FB1, FB302 to FB2, J601 to J1, L201 to L1, L601 to L37, L602 to L38, R201 to R9, R203 to R10, R204 to R11, R205 to R12, R403 to R23, R404 to R25, R407 to R24, R601 to R46, R602 to R47, R603 to R48, R604 to R49, R606 to R51, R607 to R52, R608 to R53, R609 to R54, R610 to R55, R611 to R56, R614 to R59, RFCON201 to RFCON1, RFCON509 to RFCON7, RFCON510 to RFCON9, RFCON511 to RFCON11, U301 to U3, U302 to U4, U303 to U5, U304 to U6, U601 to U14, U602 to U15, U603 to U16, U604 to U17
Connections:
- removed net !PLL_LOLA: U402.3
- removed net !PLL_LOLB: U402.4
- removed net !PLL_LOLC: U402.5
- removed net !PLL_LOLD: U402.47
- removed net !PLL_OE0: R405.1, U402.11
- removed net !PLL_OE1: R406.1, U402.41
- removed net !PLL_OUT0: R418.1, RFCON7.P$3
- removed net !PLL_OUT1: R419.1, RFCON512.P$3
- removed net !PLL_OUT2: R420.1, RFCON514.P$3
- removed net !PLL_OUT3: R421.1, RFCON9.P$3
- removed net !PLL_OUT4: R422.1, RFCON513.P$3
- removed net !PLL_OUT5: R423.1, RFCON515.P$3
- removed net !PLL_OUT6: R424.1, RFCON11.P$3
- removed net !PLL_XTAL_LOS: U402.25
- removed net 3V3_ANA_PLL_CLEAN: C406.1, C408.1, C409.1, C410.1, C412.1, C414.1, C420.1, C424.1, C427.1, C627.1, C628.1, FB402.1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
- removed net 5V0_ANA_OCXO_FILT: C21.1, C303.1, C310.1, FB1.2, U3.4, U3.6, U4.1, U5.5
- removed net GPS_BIAS_EXT: R11.1
- removed net GPS_TIMEPULSE_BUF: U1.4
- removed net GPS_TIMEPULSE_KZ: C401.1, R202.1, R401.2
- removed net N$100: R423.2, U402.50
- removed net N$101: R424.2, U402.53
- removed net N$104: C428.1, FB404.2, U402.40
- removed net N$15: R418.2, U402.23
- removed net N$76: L539.2, L543.1, L547.1
- removed net N$77: C531.2, RFCON507.P$3
- removed net N$78: L547.2, L551.1, L555.1
- removed net N$79: C519.1, L535.2
- removed net N$80: C523.1, L543.2
- removed net N$81: C527.1, L551.2
- removed net N$82: C531.1, L555.2
- removed net N$93: C413.2, C421.1, R408.1, R409.2
- removed net N$94: C402.1, R402.1
- removed net N$95: C417.1, R409.1
- removed net N$96: R419.2, U402.30
- removed net N$97: R420.2, U402.34
- removed net N$98: R421.2, U402.37
- removed net N$99: R422.2, U402.44
- removed net OCXO_CLK_BUF: U2.4
- removed net OCXO_CLK_KZ: C413.1, R302.1, R408.2
- removed net PLL_FDEC: U402.42
- removed net PLL_FINC: U402.48
- removed net PLL_IN0_N: C404.1, U402.64
- removed net PLL_IN0_P: C403.2, U402.63
- removed net PLL_IN1_N: C425.1, U402.2
- removed net PLL_IN1_P: C421.2, U402.1
- removed net PLL_OUT0: L501.1, R410.1
- removed net PLL_OUT1: L502.1, R411.1
- removed net PLL_OUT2: L503.1, R412.1
- removed net PLL_OUT3: L504.1, R413.1
- removed net PLL_OUT4: L529.1, R414.1
- removed net PLL_OUT5: L530.1, R415.1
- removed net PLL_OUT6: L531.1, R416.1
- removed net PLL_SEL0: U402.26
- removed net PLL_SEL1: U402.27
- new net !CLK0: L2.1, R26.2, U8.12
- new net !CLK1: L3.1, R28.2, U8.15
- new net !CLK2: L4.1, R30.2, U8.18
- new net !CLK3: L5.1, R32.2, U8.23
- new net !CLK4: L6.1, R34.2, U8.26
- new net 3V3_ANA_CLEAN: C103.1, C104.1, C73.1, C74.1, C75.1, C76.1, C77.1, R36.1, R37.1, R38.1, R39.1, R40.1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
- new net 3V3_PLL_FILT: C44.1, FB6.2, U8.3, U8.34
- new net 5V0_ANA_OCXO_CLEAN_FILT: C16.1, C21.1, C23.1, FB1.2, U3.4, U3.6, U4.1, U5.5
- new net CLK0: C68.1, R27.2, U8.11
- new net CLK1: C69.1, R29.2, U8.14
- new net CLK2: C70.1, R31.2, U8.17
- new net CLK3: C71.1, R33.2, U8.22
- new net CLK4: C72.1, R35.2, U8.25
- new net I2C1_SCL: R3.2, R8.1
- new net I2C1_SDA: R2.2, R6.1
- new net N$19: CON1.1, R2.1
- new net N$29: R44.2, U12.4
- new net N$32: C71.2, R39.2, U12.2
- new net N$8: R45.1, RFCON11.P$3
- new net N$9: CON1.2, R3.1
- new net PLL_M3: R14.2, U8.36
- new net PLL_M4: R15.1, U8.37
- new net PLL_M5: R16.2, U8.1
- new net PLL_M6: R17.2, U8.5
- new net PLL_REFA: R20.1, R21.2, U8.47
- new net PLL_REFB: R18.1, R19.2, U8.38
- net !GPS_RESET: now also U2.9; no longer U201.9
- net !MCU_RESET: now also R7.1, TC1.10, U1.20; no longer R104.1, TC101.10, U101.20
- net !PLL_IRQ: now also U8.32; no longer U402.12
- net !PLL_RESET: now also U8.48; no longer U402.6
- net 1V8_PLL_CLEAN: now also C28.1, C90.1, C91.1, FB3.1, FB4.1, FB5.1; no longer C411.1, C613.1, C614.1, FB403.1
- net 1V8_PLL_CLEAN_FILT: now also C30.1, C31.1, C32.1, C33.1, C34.1, C36.1, C39.1, C41.1, C43.1, FB4.2, FB5.2, U8.10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; no longer C419.1, C423.1, C426.1, FB403.2, U402.32, U402.46, U402.60
- net 3V3: now also C1.1, C38.1, C4.1, C5.1, C7.1, C79.1, CON2.1, FB6.1, R1.2, R15.2, R5.2, R6.2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; no longer C101.1, C102.1, C103.1, C104.1, C105.1, C201.1, C416.1, C602.1, FB404.1, R102.2, R103.2, R104.2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
- net 3V3_PGOOD: now also U18.5; no longer U605.5
- net 5V0: now also C100.1, C101.1, C102.1, C81.1, C96.1, R11.1, R50.2, U18.7, U18.8; no longer C604.1, C619.1, C624.1, C625.1, C626.1, R605.2, U605.7, U605.8
- net 5V0_ANA_OCXO_CLEAN: now also C15.1, C26.1, C92.1, C93.1; no longer C302.1, C313.1, C615.1, C616.1
- net 5V0_BST: now also C94.2; no longer C617.2
- net 5V0_PGOOD: now also R50.1; no longer R605.1
- net 5V0_SW: now also C94.1; no longer C617.1
- net 5V0_VSENSE: now also R60.2; no longer R615.2
- net GND: now also C10.2, C100.2, C12.2, C15.2, C16.2, C23.2, C26.2, C27.2, C28.2, C29.2, C30.2, C31.2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; no longer C201.2, C204.2, C302.2, C303.2, C310.2, C313.2, C314.2, C402.2, C404.2, C406.2, C407.2, C408.2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
- net GPS_BIAS_INT: now also C10.1, U2.14; no longer C204.1, U201.14
- net GPS_RXD: now also U2.3; no longer U201.3
- net GPS_TIMEPULSE: now also R18.2, U2.4; no longer R202.2, U1.2, U201.4
- net GPS_TXD/TXREADY: now also U2.2; no longer U201.2
- net GPS_VBKP: now also C12.1, U2.6; no longer C1.1, U201.6
- net I2C0_SCL: now also CON2.3, R5.1, U2.17, U8.2; no longer R103.1, U201.17, U402.16
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Routing:
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- added copper zone on layer 1, net 1V8_PLL_CLEAN
- added copper zone on layer 15, net 1V8_PLL_CLEAN
- added copper zone on layer 1, net 1V8_PLL_CLEAN_FILT
- added copper zone on layer 15, net 1V8_PLL_CLEAN_FILT
- added copper zone on layer 1, net 3V3
- added copper zone on layer 15, net 3V3
- added copper zone on layer 1, net 3V3_ANA_CLEAN
- added copper zone on layer 15, net 3V3_ANA_CLEAN
- added copper zone on layer 1, net 3V3_SW
- added copper zone on layer 1, net 5V0
- added copper zone on layer 1, net 5V0_ANA_OCXO_CLEAN
- added copper zone on layer 15, net 5V0_ANA_OCXO_CLEAN
- added copper zone on layer 1, net 5V0_ANA_OCXO_CLEAN_FILT
- added copper zone on layer 15, net 5V0_ANA_OCXO_CLEAN_FILT
- added copper zone on layer 1, net 5V0_SW
- added copper zone on layer 1, net VIN
- added copper zone on layer 15, net VIN
Other:
- outline, holes or cut-outs redrawn
- board text added: "IcyRadio GPSDO v1 Aug 2021"
- board text removed: "5"
- board text removed: "6"
- board text removed: "IcyRadio GPSDO v1 Jul 2021"

Commit message: Work on GPSDO
Signed-off-by: João Silva <jgc3silva@gmail.com>
Parts:
- added C108, C109: 10uF, Capacitor:CAP0603
- added C110, C111: 100nF, Capacitor:CAP0402
- added U19, U20: 74LVC1G17, Logic:SC70-5
- moved R25 47.0 mm to (15.3, 5.25), turned to 270 degrees
- moved R23 46.2 mm to (14.3, 5.25), turned to 270 degrees
- moved R5 35.5 mm to (17.3, 5.25), turned to 270 degrees
- moved R1 34.8 mm to (16.3, 5.25), turned to 270 degrees
- moved C106 31.2 mm to (9.50, 5.25), turned to 270 degrees
- moved R48 29.8 mm to (19.8, 13.5)
- moved C105 28.0 mm to (5.95, 9.50), turned to 270 degrees
- moved R59 6.60 mm to (15.9, 19.8)
- moved R60 3.60 mm to (17.4, 19.2), turned to 180 degrees
- moved C7 2.38 mm to (29.1, 48.7)
- moved TC1 0.50 mm to (31.3, 6.65)
- moved C12 0.11 mm to (30.2, 54.9)
- moved C14 0.10 mm to (28.2, 54.4)
Connections:
- removed net I2C1_SCL: R3.2, R8.1
- removed net I2C1_SDA: R2.2, R6.1
- new net GPS_TIMEPULSE_BUF: U19.4
- new net I2C2_SCL: R3.2, R8.1, U1.54
- new net I2C2_SDA: R2.2, R6.1, U1.53
- new net OCXO_CLK_BUF: U20.4
- net !DAC_CS: now also U1.61
- net !PLL_IRQ: now also U1.46
- net !PLL_RESET: now also U1.45
- net 3V3: now also C109.1, C110.1, C111.1, U19.5, U20.5
- net 3V3_PGOOD: no longer U18.5
- net 5V0: now also C108.1
- net 5V0_PGOOD: now also U18.5
- net 5V0_VSENSE: now also U1.34
- net DAC_DIN: now also U1.58
- net DAC_SCLK: now also U1.60
- net GND: now also C108.2, C109.2, C110.2, C111.2, U19.3, U20.3
- net GPS_TIMEPULSE: now also U19.2
- net I2C0_SCL: now also U1.48
- net I2C0_SDA: now also U1.47
- net OCXO_CLK: now also U20.2
- net OCXO_EN: now also U1.59
- net VIN_VSENSE: now also U1.29
Routing:
- net I2C0_SCL: track 0.76 -> 121.8 mm, vias 1 -> 5
- net I2C0_SDA: track 2.13 -> 122.7 mm, vias 1 -> 3
- net !PLL_IRQ: track 0.00 -> 56.4 mm, vias 0 -> 3
- net !PLL_RESET: track 0.00 -> 48.3 mm, vias 0 -> 1
- net 3V3_PGOOD: track 0.00 -> 47.2 mm, vias 0 -> 7
- net !GPS_RESET: track 5.25 -> 51.4 mm, vias 2 -> 3
- net 3V3: track 77.4 -> 120.3 mm, vias 53 -> 55
- net 5V0_PGOOD: track 2.94 -> 43.2 mm, vias 1 -> 7
- net GPS_TIMEPULSE_BUF: track 0.00 -> 40.1 mm, vias 0 -> 1
- net GPS_RXD: track 20.2 -> 58.6 mm
- net GPS_TXD/TXREADY: track 20.4 -> 58.4 mm, vias 2 -> 3
- net OCXO_CLK_BUF: track 0.00 -> 36.9 mm, vias 0 -> 1
- net !MCU_RESET: track 2.05 -> 37.9 mm, vias 0 -> 2
- net VIN_VSENSE: track 0.00 -> 29.8 mm, vias 0 -> 2
- net !DAC_CS: track 0.00 -> 21.9 mm, vias 0 -> 1
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