File: pcb/i2c-buffer/qo-100-i2c-buffer.brd (EAGLE design)
At the start: 30 x 60 mm, 37 parts, among them CON1 3P-SH-SIDE, CON2 3P-SH-SIDE, CON3 3P-SH-SIDE, CON4 3P-SH-SIDE, CON5 4P-SH-SIDE, U1 LTC4313-1, U2 LTC4313-1, U3 LTC4313-1, U4 LTC4313-1

Commit message: Update I2C Buffer
Signed-off-by: João Silva <jgc3silva@gmail.com>
Parts:
- added C10, C11, C12, C8, C9: 100nF, Capacitor:CAP0402
- added C13, C14: 10uF, Capacitor:CAP0603
- added C15: 1uF, Capacitor:CAP0402
- added D10, D6, D7, D8, D9: LED0603, LED:0603
- added R16, R17, R18, R19, R20: 10K Ohms, Resistor:RES0402
- added R21, R22, R23, R24, R25: 1K Ohms, Resistor:RES0402
- added SJ1, SJ2, SJ3, SJ4: SJCS, Solder Jumper:SJC_S
- added TC1: TC2050-IDC-NL, TagConnect:TC2050-IDC-NL
- added U5: LTC4313-1, Analog Devices:DFN8
- added U6, U7, U8, U9: MIC2019, Microchip:SOT23-6
- C1, C2, C3: device Capacitor:CAP0603 -> Capacitor:CAP0402
- C4: value 100nF -> 1uF; device Capacitor:CAP0603 -> Capacitor:CAP0402
- C5, C6: value 10uF -> 100nF; device Capacitor:CAP0603 -> Capacitor:CAP0402
- C7: value 1uF -> 100nF; device Capacitor:CAP0603 -> Capacitor:CAP0402
- CON1: value 3P-SH-SIDE -> 4P-SH-SIDE; device JST:SH-03-SIDE -> JST:SH-04-SIDE
- CON5: value 4P-SH-SIDE -> 3P-SH-SIDE; device JST:SH-04-SIDE -> JST:SH-03-SIDE
- R1, R13, R14, R15: value 1K Ohms -> 10K Ohms; device Resistor:RES0603 -> Resistor:RES0402
- R10, R11, R12, R2, R3, R5, R6, R7, R8, R9: device Resistor:RES0603 -> Resistor:RES0402
- R4: value 1K Ohms -> 330 Ohms; device Resistor:RES0603 -> Resistor:RES0402
- U1: value LTC4313-1 -> EFM32TG11B120F128GM32; device Analog Devices:DFN8 -> EFM32:QFN32_0.5P_TG
- moved D1 39.8 mm to (8.60, 48.1), turned to 180 degrees
- moved R1 35.8 mm to (13.3, 47.8), turned to 270 degrees
- moved C1 33.5 mm to (11.3, 38.3), turned to 0 degrees
- moved U1 31.3 mm to (6.40, 38.9), turned to 0 degrees
- moved C5 30.6 mm to (12.8, 5.90), turned to 270 degrees
- moved CON1 29.8 mm to (2.00, 25.0), turned to 270 degrees
- moved CON5 27.9 mm to (28.0, 40.0), turned to 90 degrees
- moved C2 27.6 mm to (1.95, 39.6), turned to 90 degrees
- moved R13 26.1 mm to (23.0, 8.40), turned to 270 degrees
- moved R14 25.9 mm to (23.0, 18.4), turned to 270 degrees
- moved D4 24.6 mm to (13.7, 23.4)
- moved D3 21.6 mm to (13.7, 13.4)
- moved CON4 19.5 mm to (28.0, 30.0)
- moved U4 19.5 mm to (19.5, 30.0)
- moved C6 19.2 mm to (12.8, 15.9), turned to 270 degrees
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Connections:
- removed net I2C_READY1: D1.A, R1.1, U1.5
- removed net I2C_READY2: D2.A, R2.1, U2.5
- removed net I2C_READY3: D3.A, R3.1, U3.5
- removed net I2C_READY4: D4.A, R4.1, U4.5
- new net !RESET: R1.1, TC1.10, U1.9
- new net I2C_BIAS_EN1: D2.A, R5.1, U1.31, U2.5, U6.3
- new net I2C_BIAS_EN2: D3.A, R6.1, U1.2, U3.5, U7.3
- new net I2C_BIAS_EN3: D4.A, R7.1, U1.12, U4.5, U8.3
- new net I2C_BIAS_EN4: D5.A, R8.1, U1.17, U5.5, U9.3
- new net I2C_BUF_EN1: R21.2, U1.1, U2.1
- new net I2C_BUF_EN2: R22.2, U1.10, U3.1
- new net I2C_BUF_EN3: R23.2, U1.16, U4.1
- new net I2C_BUF_EN4: R24.2, U1.22, U5.1
- new net I2C_SCL_BUF_SENSE1: SJ1.2, U1.8
- new net I2C_SCL_BUF_SENSE2: SJ2.2, U1.7
- new net I2C_SCL_BUF_SENSE3: SJ3.2, U1.24
- new net I2C_SCL_BUF_SENSE4: SJ4.2, U1.23
- new net I2C_VBIAS1: C9.1, R13.2, R17.2, U1.32, U6.6
- new net I2C_VBIAS2: C10.1, R14.2, R18.2, U1.3, U7.6
- new net I2C_VBIAS3: C11.1, R15.2, R19.2, U1.13, U8.6
- new net I2C_VBIAS4: C12.1, R16.2, R20.2, U1.18, U9.6
- new net LED: R4.2, U1.29
- new net N$14: C4.1, U1.21
- new net N$15: D1.A, R4.1
- new net N$2: R9.2, U6.5
- new net N$3: R10.2, U7.5
- new net N$4: R11.2, U8.5
- new net N$5: R12.2, U9.5
- new net N$6: D6.A, R21.1
- new net N$7: D7.A, R22.1
- new net N$8: D8.A, R23.1
- new net N$9: D9.A, R24.1
- new net SWCLK: TC1.4, U1.25
- new net SWDIO: TC1.2, U1.26
- new net SWO: TC1.6, U1.27
- net 3V3: now also C13.1, C14.1, C15.1, C8.1, CON1.1, R25.2, TC1.1, U1.11, U1.14, U1.15, U1.20, U1.28, U1.4, U5.8, U6.1, U7.1, U8.1, U9.1; no longer C4.1, CON5.1, R10.2, R11.2, R12.2, R13.2, R14.2, R15.2, R4.2, R9.2, U1.1, U1.8, U2.1, U3.1, U4.1
- net GND: now also C10.2, C11.2, C12.2, C13.2, C14.2, C15.2, C8.2, C9.2, CON1.4, CON5.3, D10.C, D6.C, D7.C, D8.C, D9.C, R10.1, R11.1, R12.1, R9.1, TC1.3, U1.33, U5.4, U5.9, U6.2, U7.2, U8.2, U9.2; no longer CON1.3, CON5.4, U1.4, U1.9
- net I2C_SCL: now also CON1.3, R3.1, U1.6, U5.3; no longer CON5.3, R15.1, U1.3
- net I2C_SCL_BUF1: now also CON2.2, R17.1, SJ1.1, U2.2; no longer CON1.2, R9.1, U1.2
- net I2C_SCL_BUF2: now also CON3.2, R18.1, SJ2.1, U3.2; no longer CON2.2, R10.1, U2.2
- net I2C_SCL_BUF3: now also CON4.2, R19.1, SJ3.1, U4.2; no longer CON3.2, R11.1, U3.2
- net I2C_SCL_BUF4: now also CON5.2, R20.1, SJ4.1, U5.2; no longer CON4.2, R12.1, U4.2
- net I2C_SDA: now also CON1.2, R2.1, U1.5, U5.6; no longer CON5.2, R13.1, U1.6
- net I2C_SDA_BUF1: now also CON2.1, R13.1, U2.7; no longer CON1.1, R5.1, U1.7
- net I2C_SDA_BUF2: now also CON3.1, R14.1, U3.7; no longer CON2.1, R6.1, U2.7
- net I2C_SDA_BUF3: now also CON4.1, R15.1, U4.7; no longer CON3.1, R7.1, U3.7
- net I2C_SDA_BUF4: now also CON5.1, R16.1, U5.7; no longer CON4.1, R8.1, U4.7
- net N$1: now also D10.A, R25.1; no longer D5.A, R14.1
Routing:
- net 3V3: track 143.7 -> 35.1 mm, vias 7 -> 24
- net I2C_VBIAS1: track 0.00 -> 57.8 mm, vias 0 -> 4
- net I2C_BIAS_EN1: track 0.00 -> 55.7 mm, vias 0 -> 2
- net I2C_VBIAS2: track 0.00 -> 49.1 mm, vias 0 -> 4
- net I2C_SCL_BUF_SENSE2: track 0.00 -> 48.9 mm, vias 0 -> 5
- net I2C_BUF_EN1: track 0.00 -> 47.6 mm, vias 0 -> 3
- net I2C_SCL_BUF_SENSE1: track 0.00 -> 46.9 mm, vias 0 -> 5
- net I2C_BIAS_EN2: track 0.00 -> 45.8 mm, vias 0 -> 2
- net I2C_SCL_BUF_SENSE3: track 0.00 -> 33.5 mm, vias 0 -> 1
- net I2C_VBIAS3: track 0.00 -> 29.3 mm, vias 0 -> 4
- net !RESET: track 0.00 -> 27.6 mm, vias 0 -> 4
- net I2C_BUF_EN2: track 0.00 -> 27.5 mm, vias 0 -> 3
- net I2C_BIAS_EN3: track 0.00 -> 25.6 mm, vias 0 -> 2
- net I2C_SCL_BUF_SENSE4: track 0.00 -> 22.4 mm, vias 0 -> 1
- net I2C_VBIAS4: track 0.00 -> 21.6 mm, vias 0 -> 4
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- added copper zone on layer 15, net 3V3
- added copper zone on layer 15, net GND
- added copper zone on layer 2, net GND
Other:
- board size 30 x 60 mm -> 30 x 50 mm
- board text added: "IcyRadio I2C Buffer v2 Jul 2022"
- board text removed: "IcyRadio I2C Buffer Mar 2021"
