File: pcb/i2c-buffer/qo-100-i2c-buffer.sch (EAGLE design)
At the start: 37 parts, among them CON1 3P-SH-SIDE, CON2 3P-SH-SIDE, CON3 3P-SH-SIDE, CON4 3P-SH-SIDE, CON5 4P-SH-SIDE, U1 LTC4313-1, U2 LTC4313-1, U3 LTC4313-1, U4 LTC4313-1

Commit message: Update I2C Buffer
Signed-off-by: João Silva <jgc3silva@gmail.com>
Parts:
- added C10, C11, C12, C8, C9: 100nF, Capacitor:CAPACITOR-0402
- added C13, C14: 10uF, Capacitor:CAPACITOR-0603
- added C15: 1uF, Capacitor:CAPACITOR-0402
- added D10, D6, D7, D8, D9: LED0603, LED:LED0603
- added R16, R17, R18, R19, R20: 10K Ohms, Resistor:RESISTOR-0402
- added R21, R22, R23, R24, R25: 1K Ohms, Resistor:RESISTOR-0402
- added SJ1, SJ2, SJ3, SJ4: SJCS, Solder Jumper:SJCS
- added TC1: TC2050-IDC-NL, TagConnect:TC2050-IDC-NL
- added U5: LTC4313-1, Analog Devices:LTC4313-1
- added U6, U7, U8, U9: MIC2019, Microchip:MIC2019
- C1, C2, C3: device Capacitor:CAPACITOR-0603 -> Capacitor:CAPACITOR-0402
- C4: value 100nF -> 1uF; device Capacitor:CAPACITOR-0603 -> Capacitor:CAPACITOR-0402
- C5, C6: value 10uF -> 100nF; device Capacitor:CAPACITOR-0603 -> Capacitor:CAPACITOR-0402
- C7: value 1uF -> 100nF; device Capacitor:CAPACITOR-0603 -> Capacitor:CAPACITOR-0402
- CON1: value 3P-SH-SIDE -> 4P-SH-SIDE; device JST:3P-SH-SIDE -> JST:4P-SH-SIDE
- CON5: value 4P-SH-SIDE -> 3P-SH-SIDE; device JST:4P-SH-SIDE -> JST:3P-SH-SIDE
- D1: COLOR GREEN -> BLUE
- D5: COLOR RED -> GREEN
- R1, R13, R14, R15: value 1K Ohms -> 10K Ohms; device Resistor:RESISTOR-0603 -> Resistor:RESISTOR-0402
- R10, R11, R12, R2, R3, R5, R6, R7, R8, R9: device Resistor:RESISTOR-0603 -> Resistor:RESISTOR-0402
- R4: value 1K Ohms -> 330 Ohms; device Resistor:RESISTOR-0603 -> Resistor:RESISTOR-0402
- U1: value LTC4313-1 -> EFM32TG11B120F128GM32; device Analog Devices:LTC4313-1 -> EFM32:EFM32TG11B120F128GM32
Connections:
- removed net I2C_READY1: D1.A, R1.1, U1.READY
- removed net I2C_READY2: D2.A, R2.1, U2.READY
- removed net I2C_READY3: D3.A, R3.1, U3.READY
- removed net I2C_READY4: D4.A, R4.1, U4.READY
- new net !RESET: R1.1, TC1-10(!RESET!).S, U1.!RESET
- new net I2C_BIAS_EN1: D2.A, R5.1, U1.PE12, U2.READY, U6.EN
- new net I2C_BIAS_EN2: D3.A, R6.1, U1.PA1, U3.READY, U7.EN
- new net I2C_BIAS_EN3: D4.A, R7.1, U1.PB13, U4.READY, U8.EN
- new net I2C_BIAS_EN4: D5.A, R8.1, U1.PD5, U5.READY, U9.EN
- new net I2C_BUF_EN1: R21.2, U1.PA0, U2.ENABLE
- new net I2C_BUF_EN2: R22.2, U1.PB11, U3.ENABLE
- new net I2C_BUF_EN3: R23.2, U1.PD4, U4.ENABLE
- new net I2C_BUF_EN4: R24.2, U1.PC13, U5.ENABLE
- new net I2C_SCL_BUF_SENSE1: SJ1.2, U1.PB8
- new net I2C_SCL_BUF_SENSE2: SJ2.2, U1.PB7
- new net I2C_SCL_BUF_SENSE3: SJ3.2, U1.PC15
- new net I2C_SCL_BUF_SENSE4: SJ4.2, U1.PC14
- new net I2C_VBIAS1: C9.C1, R13.2, R17.2, U1.PE13, U6.VOUT
- new net I2C_VBIAS2: C10.C1, R14.2, R18.2, U1.PA2, U7.VOUT
- new net I2C_VBIAS3: C11.C1, R15.2, R19.2, U1.PB14, U8.VOUT
- new net I2C_VBIAS4: C12.C1, R16.2, R20.2, U1.PD6, U9.VOUT
- new net LED: R4.2, U1.PE10
- new net N$14: C4.C1, U1.DECOUPLE
- new net N$15: D1.A, R4.1
- new net N$2: R9.2, U6.ILIMIT
- new net N$3: R10.2, U7.ILIMIT
- new net N$4: R11.2, U8.ILIMIT
- new net N$5: R12.2, U9.ILIMIT
- new net N$6: D6.A, R21.1
- new net N$7: D7.A, R22.1
- new net N$8: D8.A, R23.1
- new net N$9: D9.A, R24.1
- new net SWCLK: TC1-4(TCK/SWCLK).S, U1.PF0
- new net SWDIO: TC1-2(TMS/SWDIO).S, U1.PF1
- new net SWO: TC1-6(TDO/SWO).S, U1.PF2
- net 3V3: now also C13.C1, C14.C1, C15.C1, C8.C1, CON1-1.S, R25.2, TC1-1(VTARGET).S, U1.AVDD@0, U1.AVDD@1, U1.DVDD, U1.IOVDD0@0, U1.IOVDD0@1, U1.IOVDD0@2, U5.VCC, U6.VIN, U7.VIN, U8.VIN, U9.VIN; no longer C4.C1, CON5-1.S, R10.2, R11.2, R12.2, R13.2, R14.2, R15.2, R4.2, R9.2, U1.ENABLE, U1.VCC, U2.ENABLE, U3.ENABLE, U4.ENABLE
- net GND: now also C10.C2, C11.C2, C12.C2, C13.C2, C14.C2, C15.C2, C8.C2, C9.C2, CON1-4.S, CON5-3.S, D10.C, D6.C, D7.C, D8.C, D9.C, R10.1, R11.1, R12.1, R9.1, TC1-3(GND).S, U1.VSS@0, U5.GND, U6.GND, U7.GND, U8.GND, U9.GND; no longer CON1-3.S, CON5-4.S, U1.GND
- net I2C_SCL: now also CON1-3.S, R3.1, U1.PC1, U5.SCLIN; no longer CON5-3.S, R15.1, U1.SCLIN
- net I2C_SCL_BUF1: now also CON2-2.S, R17.1, SJ1.1, U2.SCLOUT; no longer CON1-2.S, R9.1, U1.SCLOUT
- net I2C_SCL_BUF2: now also CON3-2.S, R18.1, SJ2.1, U3.SCLOUT; no longer CON2-2.S, R10.1, U2.SCLOUT
- net I2C_SCL_BUF3: now also CON4-2.S, R19.1, SJ3.1, U4.SCLOUT; no longer CON3-2.S, R11.1, U3.SCLOUT
- net I2C_SCL_BUF4: now also CON5-2.S, R20.1, SJ4.1, U5.SCLOUT; no longer CON4-2.S, R12.1, U4.SCLOUT
- net I2C_SDA: now also CON1-2.S, R2.1, U1.PC0, U5.SDAIN; no longer CON5-2.S, R13.1, U1.SDAIN
- net I2C_SDA_BUF1: now also CON2-1.S, R13.1, U2.SDAOUT; no longer CON1-1.S, R5.1, U1.SDAOUT
- net I2C_SDA_BUF2: now also CON3-1.S, R14.1, U3.SDAOUT; no longer CON2-1.S, R6.1, U2.SDAOUT
- net I2C_SDA_BUF3: now also CON4-1.S, R15.1, U4.SDAOUT; no longer CON3-1.S, R7.1, U3.SDAOUT
- net I2C_SDA_BUF4: now also CON5-1.S, R16.1, U5.SDAOUT; no longer CON4-1.S, R8.1, U4.SDAOUT
- net N$1: now also D10.A, R25.1; no longer D5.A, R14.1
Other:
- note removed: "To enable automatic bus disconnection on loss of power do not place pullup resistors"
